Commit message: WIP: trying to get GZ sim working

File: description/ros2_control.xacro (robot description, xacro)
@@ -19,6 +19,10 @@
                     <param name="max">10</param>
                 </command_interface>
-                <state_interface name="velocity"/>
-                <state_interface name="position"/>
+                <state_interface name="velocity">
+                    <param name="initial_value">0.0</param>
+                </state_interface>
+                <state_interface name="position">
+                    <param name="initial_value">0.0</param>
+                </state_interface>
             </joint>
             <joint name="right_wheel_joint">
@@ -27,13 +31,21 @@
                     <param name="max">10</param>
                 </command_interface>
-                <state_interface name="velocity"/>
-                <state_interface name="position"/>
+                <state_interface name="velocity">
+                    <param name="initial_value">0.0</param>
+                </state_interface>
+                <state_interface name="position">
+                    <param name="initial_value">0.0</param>
+                </state_interface>
             </joint>
         </ros2_control>
     </xacro:unless>
     <xacro:if value="$(arg sim_mode)">
-        <ros2_control name="GazeboSystem" type="system">
+        <ros2_control name="IgnitionSystem" type="system">
+            <!-- hardware>
+                <plugin>ign_ros2_control/IgnitionSystem</plugin>
+            </hardware -->
             <hardware>
-                <plugin>gazebo_ros2_control/GazeboSystem</plugin>
+                <plugin>mock_components/GenericSystem</plugin>
+                <param name="calculate_dynamics">true</param>
             </hardware>
             <joint name="left_wheel_joint">
@@ -42,6 +54,10 @@
                     <param name="max">10</param>
                 </command_interface>
-                <state_interface name="velocity"/>
-                <state_interface name="position"/>
+                <state_interface name="velocity">
+                    <param name="initial_value">0.0</param>
+                </state_interface>
+                <state_interface name="position">
+                    <param name="initial_value">0.0</param>
+                </state_interface>
             </joint>
             <joint name="right_wheel_joint">
@@ -50,14 +66,58 @@
                     <param name="max">10</param>
                 </command_interface>
-                <state_interface name="velocity"/>
-                <state_interface name="position"/>
+                <state_interface name="velocity">
+                    <param name="initial_value">0.0</param>
+                </state_interface>
+                <state_interface name="position">
+                    <param name="initial_value">0.0</param>
+                </state_interface>
             </joint>
         </ros2_control>
+        <!-- ros2_control name="GazeboSystem" type="system">
+            <hardware -->
+               <!-- plugin>mock_components/GenericSystem</plugin -->
+               <!-- plugin>fake_robot/FakeRobot</plugin -->
+               <!-- plugin>diffdrive_arduino/DiffDriveArduino</plugin -->
+        <!--    <plugin>gazebo_ros2_control/GazeboSystem</plugin>
+            </hardware>
+            <joint name="left_wheel_joint">
+                <command_interface name="velocity">
+                    <param name="min">-10</param>
+                    <param name="max">10</param>
+                </command_interface>
+                <state_interface name="velocity">
+                    <param name="initial_value">0.0</param>
+                </state_interface>
+                <state_interface name="position">
+                    <param name="initial_value">0.0</param>
+                </state_interface>
+            </joint>
+            <joint name="right_wheel_joint">
+                <command_interface name="velocity">
+                    <param name="min">-10</param>
+                    <param name="max">10</param>
+                </command_interface>
+                <state_interface name="velocity">
+                    <param name="initial_value">0.0</param>
+                </state_interface>
+                <state_interface name="position">
+                    <param name="initial_value">0.0</param>
+                </state_interface>
+            </joint>
+        </ros2_control -->
     </xacro:if>
     <gazebo>
+        <plugin filename="libgz_ros2_control-system.so" name="gz_ros2_control::GazeboSimROS2ControlPlugin">
+            <robot_param>robot_description</robot_param>
+            <robot_param_node>robot_state_publisher</robot_param_node>
+            <parameters>$(find articubot_one)/config/my_controllers.yaml</parameters>
+            <parameters>$(find articubot_one)/config/gaz_ros2_ctl_use_sim.yaml</parameters>
+        </plugin>
+    </gazebo>
+    <!-- gazebo>
         <plugin name="gazebo_ros2_control" filename="libgazebo_ros2_control.so">
             <parameters>$(find articubot_one)/config/my_controllers.yaml</parameters>
             <parameters>$(find articubot_one)/config/gaz_ros2_ctl_use_sim.yaml</parameters>
         </plugin>
-    </gazebo>
+    </gazebo -->
 </robot>

Commit message: Cleaned up launch and ros2_control.xacro files

File: description/ros2_control.xacro (robot description, xacro)
@@ -1,8 +1,8 @@
 <?xml version="1.0"?>
 <robot xmlns:xacro="http://www.ros.org/wiki/xacro">
-    <xacro:unless value="$(arg sim_mode)">
-        <ros2_control name="RealRobot" type="system">
-            <hardware>
-				<!-- Values corrected for Dragger robot -->
+    <ros2_control name="DraggerRobot" type="system">
+        <hardware>
+            <xacro:unless value="$(arg sim_mode)">
+                <!-- Values corrected for Dragger robot -->
                 <plugin>diffdrive_arduino/DiffDriveArduino</plugin>
                 <param name="left_wheel_name">left_wheel_joint</param>
@@ -13,114 +13,45 @@
                 <param name="timeout">1000</param>
                 <param name="enc_counts_per_rev">13730</param>
-            </hardware>
-            <joint name="left_wheel_joint">
-                <command_interface name="velocity">
-                    <param name="min">-10</param>
-                    <param name="max">10</param>
-                </command_interface>
-                <state_interface name="velocity">
-                    <param name="initial_value">0.0</param>
-                </state_interface>
-                <state_interface name="position">
-                    <param name="initial_value">0.0</param>
-                </state_interface>
-            </joint>
-            <joint name="right_wheel_joint">
-                <command_interface name="velocity">
-                    <param name="min">-10</param>
-                    <param name="max">10</param>
-                </command_interface>
-                <state_interface name="velocity">
-                    <param name="initial_value">0.0</param>
-                </state_interface>
-                <state_interface name="position">
-                    <param name="initial_value">0.0</param>
-                </state_interface>
-            </joint>
-        </ros2_control>
-    </xacro:unless>
-    <xacro:if value="$(arg sim_mode)">
-        <ros2_control name="RobotSystem" type="system">
-            <hardware>
+            </xacro:unless>
+            <xacro:if value="$(arg sim_mode)">
                 <plugin>ign_ros2_control/IgnitionSystem</plugin>
                 <!-- plugin>gz_ros2_control/GazeboSimSystem</plugin -->
-            </hardware>
-            <!-- hardware>
-                <plugin>mock_components/GenericSystem</plugin>
-                <param name="calculate_dynamics">true</param>
-            </hardware -->
-            <joint name="left_wheel_joint">
-                <command_interface name="velocity">
-                    <param name="min">-10</param>
-                    <param name="max">10</param>
-                </command_interface>
-                <state_interface name="velocity">
-                    <param name="initial_value">0.0</param>
-                </state_interface>
-                <state_interface name="position">
-                    <param name="initial_value">0.0</param>
-                </state_interface>
-            </joint>
-            <joint name="right_wheel_joint">
-                <command_interface name="velocity">
-                    <param name="min">-10</param>
-                    <param name="max">10</param>
-                </command_interface>
-                <state_interface name="velocity">
-                    <param name="initial_value">0.0</param>
-                </state_interface>
-                <state_interface name="position">
-                    <param name="initial_value">0.0</param>
-                </state_interface>
-            </joint>
-        </ros2_control>
-        <!-- ros2_control name="GazeboSystem" type="system">
-            <hardware -->
-               <!-- plugin>mock_components/GenericSystem</plugin -->
-               <!-- plugin>fake_robot/FakeRobot</plugin -->
-               <!-- plugin>diffdrive_arduino/DiffDriveArduino</plugin -->
-        <!--    <plugin>gazebo_ros2_control/GazeboSystem</plugin>
-            </hardware>
-            <joint name="left_wheel_joint">
-                <command_interface name="velocity">
-                    <param name="min">-10</param>
-                    <param name="max">10</param>
-                </command_interface>
-                <state_interface name="velocity">
-                    <param name="initial_value">0.0</param>
-                </state_interface>
-                <state_interface name="position">
-                    <param name="initial_value">0.0</param>
-                </state_interface>
-            </joint>
-            <joint name="right_wheel_joint">
-                <command_interface name="velocity">
-                    <param name="min">-10</param>
-                    <param name="max">10</param>
-                </command_interface>
-                <state_interface name="velocity">
-                    <param name="initial_value">0.0</param>
-                </state_interface>
-                <state_interface name="position">
-                    <param name="initial_value">0.0</param>
-                </state_interface>
-            </joint>
-        </ros2_control -->
-    </xacro:if>
+            </xacro:if>
+        </hardware>
+        <joint name="left_wheel_joint">
+            <command_interface name="velocity">
+                <param name="min">-10</param>
+                <param name="max">10</param>
+            </command_interface>
+            <state_interface name="velocity">
+                <param name="initial_value">0.0</param>
+            </state_interface>
+            <state_interface name="position">
+                <param name="initial_value">0.0</param>
+            </state_interface>
+        </joint>
+        <joint name="right_wheel_joint">
+            <command_interface name="velocity">
+                <param name="min">-10</param>
+                <param name="max">10</param>
+            </command_interface>
+            <state_interface name="velocity">
+                <param name="initial_value">0.0</param>
+            </state_interface>
+            <state_interface name="position">
+                <param name="initial_value">0.0</param>
+            </state_interface>
+        </joint>
+    </ros2_control>
     <gazebo>
-        <!-- library: /opt/ros/humble/lib/libign_ros2_control-system.so -->
+        <!-- library: /opt/ros/humble/lib/libign_ros2_control-system.so - GZ Fortress on ROS Humble -->
         <plugin filename="libign_ros2_control-system.so" name="ign_ros2_control::IgnitionROS2ControlPlugin">
         <!-- plugin filename="gz_ros2_control-system" name="gz_ros2_control::GazeboSimROS2ControlPlugin" -->
+            <!-- the following are just default parameters anyway. Skip them unless you want to reaasign them:
             <robot_param>robot_description</robot_param>
-            <robot_param_node>robot_state_publisher</robot_param_node>
+            <robot_param_node>robot_state_publisher</robot_param_node> -->
             <parameters>$(find articubot_one)/config/gaz_ros2_ctl_use_sim.yaml</parameters>
             <parameters>$(find articubot_one)/config/my_controllers.yaml</parameters>
         </plugin>
     </gazebo>
-    <!-- gazebo>
-        <plugin name="gazebo_ros2_control" filename="libgazebo_ros2_control.so">
-            <parameters>$(find articubot_one)/config/my_controllers.yaml</parameters>
-            <parameters>$(find articubot_one)/config/gaz_ros2_ctl_use_sim.yaml</parameters>
-        </plugin>
-    </gazebo -->
 </robot>

Commit message: Better cooperation between joint_state_broadcaster and Rviz

File: description/ros2_control.xacro (robot description, xacro)
@@ -29,7 +29,7 @@
                 <param name="initial_value">0.0</param>
             </state_interface>
-            <state_interface name="effort">
+            <!-- state_interface name="effort">
                 <param name="initial_value">0.0</param>
-            </state_interface>
+            </state_interface -->
         </joint>
         <joint name="right_wheel_joint">
@@ -44,8 +44,27 @@
                 <param name="initial_value">0.0</param>
             </state_interface>
-            <state_interface name="effort">
+            <!-- state_interface name="effort">
                 <param name="initial_value">0.0</param>
-            </state_interface>
+            </state_interface -->
         </joint>
+        <xacro:if value="$(arg sim_mode)">
+            <!-- we need this for Rviz to reflect rotations of joints published by broad_cont in Gazebo -->
+            <joint name="left_caster_wheel_joint">
+                <state_interface name="velocity">
+                    <param name="initial_value">0.0</param>
+                </state_interface>
+                <state_interface name="position">
+                    <param name="initial_value">0.0</param>
+                </state_interface>
+            </joint>
+            <joint name="right_caster_wheel_joint">
+                <state_interface name="velocity">
+                    <param name="initial_value">0.0</param>
+                </state_interface>
+                <state_interface name="position">
+                    <param name="initial_value">0.0</param>
+                </state_interface>
+            </joint>
+        </xacro:if>
     </ros2_control>
     <gazebo>
