Commit message: Wheel markers and fresh URDF rendering

File: description/robot.urdf (robot description, URDF)
Before this commit: robot robot, 12 links, 11 joints
Links:
- link left_wheel: geometry collision sphere radius=0.192; visual box size=0.038400000000000004 0.0576 0.099
- link right_wheel: geometry collision sphere radius=0.192; visual box size=0.038400000000000004 0.0576 0.099

File: description/robot_core.xacro (robot description, xacro)
@@ -96,22 +96,17 @@
             <material name="port_red"/>
         </visual>
+        <visual name="left_wheel_axis_visual">
+            <geometry>
+                <cylinder radius="${wheel_radius*0.1}" length="${wheel_thickness*1.1}"/>
+            </geometry>
+            <material name="blue"/>
+        </visual>
         <visual name="left_wheel_marker_visual">
-            <geometry>
-                <box size="${wheel_radius*0.5} ${wheel_radius*0.5} ${wheel_thickness*1.1}"/>
-            </geometry>
-            <material name="blue"/>
-        </visual>
-        <!-- visual name="left_wheel_marker_visual">
-            <pose>0.17 0 0 0 0 0</pose>
-            <geometry>
-                <box size=".10 .01 .21"/>
-            </geometry>
-            <material>
-                <ambient>1.0 0.2 0.2 1</ambient>
-                <diffuse>1.0 0.1 0.1 1</diffuse>
-                <specular>0 0 0 0</specular>
-                <emissive>0 0 0 1</emissive>
-            </material>
-        </visual -->
+            <origin xyz="0 ${wheel_radius*0.7} 0" rpy="0 0 0" />
+            <geometry>
+                <box size="${wheel_radius*0.2} ${wheel_radius*0.3} ${wheel_thickness*1.1}"/>
+            </geometry>
+            <material name="blue"/>
+        </visual>
         <collision>
             <geometry>
@@ -131,5 +126,5 @@
     </joint>
     <link name="right_wheel">
-        <visual>
+        <visual name="right_wheel_visual">
             <geometry>
                 <cylinder radius="${wheel_radius}" length="${wheel_thickness}"/>
@@ -137,7 +132,14 @@
             <material name="starboard_green"/>
         </visual>
+        <visual name="right_wheel_axis_visual">
+            <geometry>
+                <cylinder radius="${wheel_radius*0.1}" length="${wheel_thickness*1.1}"/>
+            </geometry>
+            <material name="blue"/>
+        </visual>
         <visual name="right_wheel_marker_visual">
-            <geometry>
-                <box size="${wheel_radius*0.5} ${wheel_radius*0.5} ${wheel_thickness*1.1}"/>
+            <origin xyz="0 ${-wheel_radius*0.7} 0" rpy="0 0 0" />
+            <geometry>
+                <box size="${wheel_radius*0.2} ${wheel_radius*0.3} ${wheel_thickness*1.1}"/>
             </geometry>
             <material name="blue"/>
@@ -160,5 +162,5 @@
     </joint>
     <link name="left_caster_wheel">
-        <visual>
+        <visual name="left_caster_visual">
             <geometry>
                <cylinder radius="${caster_wheel_radius}" length="${caster_wheel_thickness}"/>
@@ -188,5 +190,5 @@
     </joint>
     <link name="right_caster_wheel">
-        <visual>
+        <visual name="right_caster_visual">
             <geometry>
                <cylinder radius="${caster_wheel_radius}" length="${caster_wheel_thickness}"/>
@@ -194,5 +196,5 @@
             <material name="starboard_green"/>
         </visual>
-        <visual name="left_caster_marker_visual">
+        <visual name="right_caster_marker_visual">
             <geometry>
                 <box size="${caster_wheel_radius*0.5} ${caster_wheel_radius*0.5} ${caster_wheel_thickness*1.1}"/>
@@ -210,10 +212,4 @@
     </link>
     <!-- gazebo reference="right_caster_wheel">
-        <material>Gazebo/Green</material>
-        <mu1 value="0.001"/>
-        <mu2 value="0.001"/>
-    </gazebo>
-    <gazebo reference="left_caster_wheel">
-        <material>Gazebo/Red</material>
         <material>
             <ambient>1.0 0.2 0.2 1</ambient>
@@ -222,10 +218,4 @@
         <mu1 value="0.001"/>
         <mu2 value="0.001"/>
-    </gazebo>
-    <gazebo reference="left_wheel">
-        <material>Gazebo/Red</material>
-    </gazebo>
-    <gazebo reference="right_wheel">
-        <material>Gazebo/Green</material>
     </gazebo -->
 </robot>

Commit message: fresh rendition of robot.urdf

File: description/robot.urdf (robot description, URDF)
Before this commit: robot robot, 12 links, 11 joints
Links:
- link base_footprint: geometry visual box size=0.9 0.4 0.02
- link base_link: geometry visual sphere radius=0.03
- link chassis_link: geometry collision box size=0.9 0.4 0.5; visual box size=0.405 0.38 0.25
- link imu_link: geometry visual box size=0.1 0.1 0.1
- link laser_link: geometry collision cylinder length=0.04 radius=0.05; visual cylinder length=0.04 radius=0.05
- link left_caster_wheel: geometry collision cylinder length=0.05 radius=0.12; visual box size=0.06 0.06 0.05500000000000001
- link left_wheel: geometry collision cylinder length=0.09 radius=0.192; visual box size=0.038400000000000004 0.0576 0.099
- link right_caster_wheel: geometry collision cylinder length=0.05 radius=0.12; visual box size=0.06 0.06 0.05500000000000001
- link right_wheel: geometry collision cylinder length=0.09 radius=0.192; visual box size=0.038400000000000004 0.0576 0.099
Joints:
- joint camera_joint: origin xyz=0.2 0 0.55 rpy=0 0.18 0 -> xyz=0.41000000000000003 0 0.55 rpy=0 0.18 0; parent base_link -> chassis_link
- joint camera_optical_joint: origin xyz=0 0 0 rpy=-1.5707963267948966 0 -1.5707963267948966 -> xyz=0 0 0 rpy=0 0 0
- joint chassis_joint: origin xyz=-0.7 0 -0.01 -> xyz=-0.248 0 -0.01
- joint gps_joint: origin xyz=-0.1 0 0.65 rpy=0 0 3.1459 -> xyz=0.05 0 0.65 rpy=0 0 3.1459; parent base_link -> chassis_link
- joint imu_joint: origin xyz=0 0 0.01 -> xyz=0.248 0 0.04 rpy=0 0 0; parent base_link -> chassis_link
- joint laser_joint: origin xyz=-0.01 0 0.57 rpy=0 0 3.1459 -> xyz=0.275 0 0.57 rpy=0 0 3.1459; parent base_link -> chassis_link
- joint left_caster_wheel_joint: origin xyz=0.1 0.28 -0.062 rpy=1.5707963267948966 0 0 -> xyz=-0.32 0.27 -0.062 rpy=1.5707963267948966 0 0
- joint left_wheel_joint: origin xyz=0 0.29 0 rpy=-1.5707963267948966 0 0 -> xyz=0.248 0.29 0 rpy=-1.5707963267948966 0 0; parent base_link -> chassis_link
- joint right_caster_wheel_joint: origin xyz=0.1 -0.28 -0.062 rpy=1.5707963267948966 0 0 -> xyz=-0.32 -0.27 -0.062 rpy=1.5707963267948966 0 0
- joint right_wheel_joint: origin xyz=0 -0.29 0 rpy=1.5707963267948966 0 0 -> xyz=0.248 -0.29 0 rpy=1.5707963267948966 0 0; parent base_link -> chassis_link

Commit message: Gave up renaming /diff_cont/odom from params

File: description/robot.urdf (robot description, URDF)
Before this commit: robot robot, 12 links, 11 joints
Links:
- removed link laser_link
- added link laser_frame, mass 0.1; collision cylinder length=0.04 radius=0.05; visual cylinder length=0.04 radius=0.05
- link chassis_link: geometry collision box size=0.9 0.4 0.5; visual box size=0.405 0.38 0.25
- link left_wheel: geometry collision cylinder length=0.09 radius=0.177; visual box size=0.0354 0.053099999999999994 0.099
- link right_wheel: geometry collision cylinder length=0.09 radius=0.177; visual box size=0.0354 0.053099999999999994 0.099
Joints:
- joint base_joint: origin xyz=0 0 0.192 rpy=0 0 0 -> xyz=0 0 0.177 rpy=0 0 0
- joint chassis_joint: origin xyz=-0.248 0 -0.01 -> xyz=-0.263 0 -0.01
- joint imu_joint: origin xyz=0.248 0 0.04 rpy=0 0 0 -> xyz=0.263 0 0.04 rpy=0 0 0
- joint laser_joint: child laser_link -> laser_frame
- joint left_caster_wheel_joint: origin xyz=-0.32 0.27 -0.062 rpy=1.5707963267948966 0 0 -> xyz=-0.32 0.27 -0.046999999999999986 rpy=1.5707963267948966 0 0
- joint left_wheel_joint: origin xyz=0.248 0.29 0 rpy=-1.5707963267948966 0 0 -> xyz=0.263 0.29 0 rpy=-1.5707963267948966 0 0
- joint right_caster_wheel_joint: origin xyz=-0.32 -0.27 -0.062 rpy=1.5707963267948966 0 0 -> xyz=-0.32 -0.27 -0.046999999999999986 rpy=1.5707963267948966 0 0
- joint right_wheel_joint: origin xyz=0.248 -0.29 0 rpy=1.5707963267948966 0 0 -> xyz=0.263 -0.29 0 rpy=1.5707963267948966 0 0
