Commit message: Update robot_core.xacro
Added imu_link to URDF

File: description/robot_core.xacro (robot description, xacro)
@@ -71,4 +71,23 @@
         <material>Gazebo/Orange</material>
     </gazebo>
+    <!-- *********************** IMU SETUP *********************************  -->
+    <!-- Each sensor must be attached to a link.                              -->
+    <link name="imu_link">
+        <visual>
+        <geometry>
+            <box size="0.1 0.1 0.1"/>
+        </geometry>
+        </visual>
+        <collision>
+        <geometry>
+            <box size="0.1 0.1 0.1"/>
+        </geometry>
+        </collision>
+    </link>
+    <joint name="imu_joint" type="fixed">
+        <parent link="chassis"/>
+        <child link="imu_link"/>
+        <origin xyz="0 0 0.01"/>
+    </joint>
     <!-- LEFT WHEEL LINK -->
     <joint name="left_wheel_joint" type="continuous">

Commit message: Wheels rotating from Joystick!

File: description/robot_core.xacro (robot description, xacro)
@@ -14,5 +14,5 @@
     <xacro:property name="wheel_offset_z" value="0.01"/>
     <xacro:property name="caster_wheel_radius" value="0.12"/>
-    <xacro:property name="caster_wheel_thickness" value="0.08"/>
+    <xacro:property name="caster_wheel_thickness" value="0.05"/>
     <xacro:property name="caster_wheel_mass" value="0.3"/>
     <xacro:property name="caster_wheel_offset_x" value="${-chassis_length/2 + caster_wheel_radius + 0.01}"/>

Commit message: Fixed collisions and wheel friction

File: description/robot_core.xacro (robot description, xacro)
@@ -62,5 +62,5 @@
         </visual>
         <collision>
-            <origin xyz="${chassis_length/2} 0 ${chassis_height/2}"/>
+            <origin xyz="0 0 ${chassis_height/2}" rpy="0 0 0"/>
             <geometry>
                 <box size="${chassis_length} ${chassis_width} ${chassis_height}"/>
@@ -68,5 +68,5 @@
         </collision>
         <xacro:inertial_box mass="0.5" x="${chassis_length}" y="${chassis_width}" z="${chassis_height}">
-            <origin xyz="${chassis_length/2} 0 ${chassis_height/2}" rpy="0 0 0"/>
+            <origin xyz="0 0 ${chassis_height/2}" rpy="0 0 0"/>
         </xacro:inertial_box>
     </link>
@@ -125,6 +125,22 @@
         <collision>
             <geometry>
-                <sphere radius="${wheel_radius}"/>
-            </geometry>
+                <cylinder radius="${wheel_radius}" length="${wheel_thickness}"/>
+            </geometry>
+            <max_contacts>1</max_contacts>
+            <surface>
+                <friction>
+                    <ode>
+                    <mu>0.4</mu>
+                    <mu2>0.6</mu2>
+                    </ode>
+                </friction>
+                <bounce/>
+                <contact>
+                    <ode>
+                    <min_depth>0.005</min_depth>
+                    <kp>1e8</kp>
+                    </ode>
+                </contact>
+            </surface>
         </collision>
         <xacro:inertial_cylinder mass="${wheel_mass}" length="${wheel_thickness}" radius="${wheel_radius}">
@@ -166,6 +182,22 @@
         <collision>
             <geometry>
-                <sphere radius="${wheel_radius}"/>
-            </geometry>
+                <cylinder radius="${wheel_radius}" length="${wheel_thickness}"/>
+            </geometry>
+            <max_contacts>1</max_contacts>
+            <surface>
+                <friction>
+                    <ode>
+                    <mu>0.4</mu>
+                    <mu2>0.6</mu2>
+                    </ode>
+                </friction>
+                <bounce/>
+                <contact>
+                    <ode>
+                    <min_depth>0.005</min_depth>
+                    <kp>1e8</kp>
+                    </ode>
+                </contact>
+            </surface>
         </collision>
         <xacro:inertial_cylinder mass="${wheel_mass}" length="${wheel_thickness}" radius="${wheel_radius}">
@@ -195,6 +227,16 @@
         <collision>
             <geometry>
-                <sphere radius="${caster_wheel_radius}"/>
-            </geometry>
+                <cylinder radius="${caster_wheel_radius}" length="${caster_wheel_thickness}"/>
+            </geometry>
+            <surface>
+                <friction>
+                    <ode>
+                    <mu>0</mu>
+                    <mu2>0</mu2>
+                    <slip1>1.0</slip1>
+                    <slip2>1.0</slip2>
+                    </ode>
+                </friction>
+            </surface>
         </collision>
         <xacro:inertial_sphere mass="${caster_wheel_mass}" radius="${caster_wheel_radius}">
@@ -223,6 +265,16 @@
         <collision>
             <geometry>
-                <sphere radius="${caster_wheel_radius}"/>
-            </geometry>
+                <cylinder radius="${caster_wheel_radius}" length="${caster_wheel_thickness}"/>
+            </geometry>
+            <surface>
+                <friction>
+                    <ode>
+                    <mu>0</mu>
+                    <mu2>0</mu2>
+                    <slip1>1.0</slip1>
+                    <slip2>1.0</slip2>
+                    </ode>
+                </friction>
+            </surface>
         </collision>
         <xacro:inertial_sphere mass="${caster_wheel_mass}" radius="${caster_wheel_radius}">
@@ -230,11 +282,3 @@
         </xacro:inertial_sphere>
     </link>
-    <!-- gazebo reference="right_caster_wheel">
-        <material>
-            <ambient>1.0 0.2 0.2 1</ambient>
-            <diffuse>1.0 0.1 0.1 1</diffuse>
-        </material>
-        <mu1 value="0.001"/>
-        <mu2 value="0.001"/>
-    </gazebo -->
 </robot>

Commit message: better footprint and initial pose defined

File: description/robot_core.xacro (robot description, xacro)
@@ -19,31 +19,30 @@
     <xacro:property name="caster_wheel_offset_y" value="0.270"/>
     <xacro:property name="caster_wheel_offset_z" value="${wheel_offset_z - wheel_radius + caster_wheel_radius}"/>
+    <!-- ********************** ROBOT BASE *********************************  -->
+    <link name="base_link">
+        <visual name="baselink_visual">
+            <origin xyz="0 0 0"/>
+            <geometry>
+                <sphere radius="0.03"/>
+            </geometry>
+            <material name="red"/>
+        </visual>
+    </link>
     <!-- ****************** ROBOT BASE FOOTPRINT ***************************  -->
     <!-- Define the center of the main robot chassis projected on the ground -->
-    <!-- link name="base_footprint"/ -->
     <link name="base_footprint">
         <visual name="footprint_visual">
             <origin xyz="0 0 0.01"/>
             <geometry>
-                <box size="${chassis_length} ${chassis_width} 0.02"/>
+                <box size="${chassis_length} ${wheel_offset_y * 2 + wheel_thickness} 0.02"/>
             </geometry>
             <material name="shadow_grey"/>
         </visual>
      </link>
-    <!-- ********************** ROBOT BASE *********************************  -->
-    <link name="base_link">
-        <visual name="footprint_visual">
-            <origin xyz="0 0 0"/>
-            <geometry>
-                <sphere radius="0.03"/>
-            </geometry>
-            <material name="red"/>
-        </visual>
-    </link>
     <!-- The base footprint of the robot is located underneath the chassis -->
     <joint name="base_joint" type="fixed">
-        <parent link="base_footprint"/>
-        <child link="base_link" />
-        <origin xyz="0 0 ${wheel_radius}" rpy="0 0 0"/>
+        <parent link="base_link"/>
+        <child link="base_footprint" />
+        <origin xyz="-${wheel_offset_x} 0 -${wheel_radius}" rpy="0 0 0"/>
     </joint>
     <!-- ********************** ROBOT BODY *********************************  -->

Commit message: Correct  enable_odom_tf: false and model wheels diameter

File: description/robot_core.xacro (robot description, xacro)
@@ -7,5 +7,5 @@
     <xacro:property name="chassis_height" value="0.50"/>
     <xacro:property name="chassis_mass" value="30.0"/>
-    <xacro:property name="wheel_radius" value="0.177"/>
+    <xacro:property name="wheel_radius" value="0.192"/>
     <xacro:property name="wheel_thickness" value="0.09"/>
     <xacro:property name="wheel_mass" value="1.0"/>

Commit message: Added Gazebo magnetometer sensor, as IMU doesn't deliver orientation

File: description/robot_core.xacro (robot description, xacro)
@@ -206,4 +206,47 @@
         </sensor>
     </gazebo>
+    <link name="magnetometer_link">
+        <visual>
+            <geometry>
+                <box size="0.1 0.1 0.1"/>
+            </geometry>
+            <material name="sensor_blue"/>
+        </visual>
+    </link>
+    <joint name="magnetometer_joint" type="fixed">
+        <parent link="chassis_link"/>
+        <child link="magnetometer_link"/>
+        <!-- we place Magnetometer next to IMU between the wheels -->
+        <origin xyz="${wheel_offset_x} 0 0.03" rpy="0 0 0"/>
+    </joint>
+    <gazebo reference="magnetometer_link">
+        <sensor name="magnetometer" type="magnetometer">
+          <always_on>1</always_on>
+          <update_rate>100</update_rate>
+          <visualize>true</visualize>
+          <topic>magnetometer</topic>
+          <enable_metrics>true</enable_metrics>
+          <magnetometer>
+            <x>
+              <noise type="gaussian">
+                <mean>0.0</mean>
+                <stddev>0.1</stddev>
+              </noise>
+            </x>
+            <y>
+              <noise type="gaussian">
+                <mean>0.0</mean>
+                <stddev>0.1</stddev>
+              </noise>
+            </y>
+            <z>
+              <noise type="gaussian">
+                <mean>0.0</mean>
+                <stddev>0.1</stddev>
+              </noise>
+            </z>
+          </magnetometer>
+        </sensor>
+    </gazebo>
     <!-- LEFT WHEEL LINK -->
     <joint name="left_wheel_joint" type="continuous">

Commit message: Update robot_core.xacro
corrected size of the base_link red sphere visual

File: description/robot_core.xacro (robot description, xacro)
@@ -24,5 +24,5 @@
             <origin xyz="0 0 0"/>
             <geometry>
-                <sphere radius="0.03"/>
+                <sphere radius="0.04"/>
             </geometry>
             <material name="red"/>

Commit message: Update robot_core.xacro
Proper handling of casters rotation in real Dragger and in SIM

File: description/robot_core.xacro (robot description, xacro)
@@ -19,4 +19,11 @@
     <xacro:property name="caster_wheel_offset_y" value="0.270"/>
     <xacro:property name="caster_wheel_offset_z" value="${wheel_offset_z - wheel_radius + caster_wheel_radius}"/>
+    <!-- we need the following because (unlike sim) real Dragger doesn't have a controller reporting caster's position -->
+    <xacro:if value="$(arg sim_mode)">
+        <xacro:property name="caster_joint_type" value="continuous"/>
+    </xacro:if>
+    <xacro:unless value="$(arg sim_mode)">
+        <xacro:property name="caster_joint_type" value="fixed"/>
+    </xacro:unless>
     <!-- ********************** ROBOT BASE *********************************  -->
     <link name="base_link">
@@ -368,5 +375,5 @@
     </link>
     <!-- CASTER WHEELS LINKS -->
-    <joint name="left_caster_wheel_joint" type="continuous">
+    <joint name="left_caster_wheel_joint" type="${caster_joint_type}">
         <parent link="chassis_link"/>
         <child link="left_caster_wheel"/>
@@ -406,5 +413,5 @@
         </xacro:inertial_cylinder>
     </link>
-    <joint name="right_caster_wheel_joint" type="continuous">
+    <joint name="right_caster_wheel_joint" type="${caster_joint_type}">
         <parent link="chassis_link"/>
         <child link="right_caster_wheel"/>

Commit message: Introduced wheel mesh for better looks

File: description/robot_core.xacro (robot description, xacro)
@@ -284,7 +284,21 @@
     </joint>
     <link name="left_wheel">
-        <visual name="left_wheel_visual">
-            <geometry>
-                <cylinder radius="${wheel_radius}" length="${wheel_thickness}"/>
+        <visual name="left_wheel_tire_gz_visual">
+            <origin xyz="0 0 0" rpy="${pi/2} 0 0" />
+            <geometry>
+                <mesh filename="model://meshes/wheel_link.STL" scale="${wheel_radius*12.7} ${wheel_thickness*10.2} ${wheel_radius*12.7}"/>
+            </geometry>
+            <material name="port_red"/>
+        </visual>
+        <visual name="left_wheel_tire_rviz_visual">
+            <origin xyz="0 0 0" rpy="${pi/2} 0 0" />
+            <geometry>
+                <mesh filename="package://articubot_one/description/meshes/wheel_link.STL" scale="${wheel_radius*12.7} ${wheel_thickness*10.2} ${wheel_radius*12.7}"/>
+            </geometry>
+            <material name="port_red"/>
+        </visual>
+        <visual name="left_wheel_solid_visual">
+            <geometry>
+                <cylinder radius="${wheel_radius}" length="${wheel_thickness/10.0}"/>
             </geometry>
             <material name="port_red"/>
@@ -341,7 +355,21 @@
     </joint>
     <link name="right_wheel">
-        <visual name="right_wheel_visual">
-            <geometry>
-                <cylinder radius="${wheel_radius}" length="${wheel_thickness}"/>
+        <visual name="right_wheel_tire_gz_visual">
+            <origin xyz="0 0 0" rpy="${pi/2} 0 0" />
+            <geometry>
+                <mesh filename="model://meshes/wheel_link.STL" scale="${wheel_radius*12.7} ${wheel_thickness*10.2} ${wheel_radius*12.7}"/>
+            </geometry>
+            <material name="starboard_green"/>
+        </visual>
+        <visual name="right_wheel_tire_rviz_visual">
+            <origin xyz="0 0 0" rpy="${pi/2} 0 0" />
+            <geometry>
+                <mesh filename="package://articubot_one/description/meshes/wheel_link.STL" scale="${wheel_radius*12.7} ${wheel_thickness*10.2} ${wheel_radius*12.7}"/>
+            </geometry>
+            <material name="starboard_green"/>
+        </visual>
+        <visual name="right_wheel_solid_visual">
+            <geometry>
+                <cylinder radius="${wheel_radius}" length="${wheel_thickness/10.0}"/>
             </geometry>
             <material name="starboard_green"/>

Commit message: Update robot_core.xacro
Proper orientation of the off-road tire on the right side

File: description/robot_core.xacro (robot description, xacro)
@@ -356,5 +356,5 @@
     <link name="right_wheel">
         <visual name="right_wheel_tire_gz_visual">
-            <origin xyz="0 0 0" rpy="${pi/2} 0 0" />
+            <origin xyz="0 0 0" rpy="${-pi/2} 0 0" />
             <geometry>
                 <mesh filename="model://meshes/wheel_link.STL" scale="${wheel_radius*12.7} ${wheel_thickness*10.2} ${wheel_radius*12.7}"/>
@@ -363,5 +363,5 @@
         </visual>
         <visual name="right_wheel_tire_rviz_visual">
-            <origin xyz="0 0 0" rpy="${pi/2} 0 0" />
+            <origin xyz="0 0 0" rpy="${-pi/2} 0 0" />
             <geometry>
                 <mesh filename="package://articubot_one/description/meshes/wheel_link.STL" scale="${wheel_radius*12.7} ${wheel_thickness*10.2} ${wheel_radius*12.7}"/>
