Commit message: Cartographer works, plucky/pluckysense launch files added

File: description/camera.xacro (robot description, xacro)
@@ -2,5 +2,5 @@
 <robot xmlns:xacro="http://www.ros.org/wiki/xacro" >
     <joint name="camera_joint" type="fixed">
-        <parent link="chassis"/>
+        <parent link="chassis_link"/>
         <child link="camera_link"/>
         <origin xyz="0.276 0 0.181" rpy="0 0.18 0"/>

File: description/depth_camera.xacro (robot description, xacro)
@@ -2,5 +2,5 @@
 <robot xmlns:xacro="http://www.ros.org/wiki/xacro" >
     <joint name="camera_joint" type="fixed">
-        <parent link="chassis"/>
+        <parent link="chassis_link"/>
         <child link="camera_link"/>
         <origin xyz="0.305 0 0.08" rpy="0 0 0"/>

File: description/face.xacro (robot description, xacro)
@@ -2,5 +2,5 @@
 <robot xmlns:xacro="http://www.ros.org/wiki/xacro" >
     <joint name="face_joint" type="fixed">
-        <parent link="chassis"/>
+        <parent link="chassis_link"/>
         <child link="face_link"/>
         <origin xyz="${chassis_length} 0 ${chassis_height/2}" rpy="0 0 0"/>

File: description/lidar.xacro (robot description, xacro)
@@ -2,5 +2,5 @@
 <robot xmlns:xacro="http://www.ros.org/wiki/xacro" >
     <joint name="laser_joint" type="fixed">
-        <parent link="chassis"/>
+        <parent link="base_link"/>
         <child link="laser_frame"/>
         <origin xyz="0.122 0 0.212" rpy="0 0 3.1459"/>

File: description/robot_core.xacro (robot description, xacro)
@@ -47,8 +47,8 @@
     <joint name="chassis_joint" type="fixed">
         <parent link="base_link"/>
-        <child link="chassis"/>
+        <child link="chassis_link"/>
         <origin xyz="${-wheel_offset_x} 0 ${-wheel_offset_z}"/>
     </joint>
-    <link name="chassis">
+    <link name="chassis_link">
         <visual>
             <origin xyz="${chassis_length/2} 0 ${chassis_height/2}"/>
@@ -68,5 +68,5 @@
         </xacro:inertial_box>
     </link>
-    <gazebo reference="chassis">
+    <gazebo reference="chassis_link">
         <material>Gazebo/Orange</material>
     </gazebo>
@@ -86,5 +86,5 @@
     </link>
     <joint name="imu_joint" type="fixed">
-        <parent link="chassis"/>
+        <parent link="base_link"/>
         <child link="imu_link"/>
         <origin xyz="0 0 0.01"/>
@@ -144,5 +144,5 @@
     <!-- CASTER WHEEL LINK -->
     <joint name="caster_wheel_joint" type="fixed">
-        <parent link="chassis"/>
+        <parent link="chassis_link"/>
         <child link="caster_wheel"/>
         <origin xyz="${caster_wheel_offset_x} 0 ${caster_wheel_offset_z}"/>

Commit message: Sim seems to work with all xacro files
Dragger model shows up. TODO: drive it with teleop

File: description/camera.xacro (robot description, xacro)
@@ -1,8 +1,10 @@
 <?xml version="1.0"?>
 <robot xmlns:xacro="http://www.ros.org/wiki/xacro" >
+    <xacro:property name="camera_offset_x" value="0.2"/>
+    <xacro:property name="camera_offset_z" value="0.55"/>
     <joint name="camera_joint" type="fixed">
-        <parent link="chassis_link"/>
+        <parent link="base_link"/>
         <child link="camera_link"/>
-        <origin xyz="0.276 0 0.181" rpy="0 0.18 0"/>
+        <origin xyz="${camera_offset_x} 0 ${camera_offset_z}" rpy="0 0.18 0"/>
     </joint>
     <link name="camera_link">
@@ -11,5 +13,4 @@
                 <box size="0.010 0.03 0.03"/>
             </geometry>
-            <material name="black"/>
         </visual>
         <visual>
@@ -18,5 +19,4 @@
                 <cylinder radius="0.002" length="0.1"/>
             </geometry>
-            <material name="black"/>
         </visual>
     </link>
@@ -27,6 +27,8 @@
     </joint>
     <link name="camera_link_optical"></link>
+    <gazebo reference="laser_frame">
+        <material>Gazebo/Grey</material>
+    </gazebo>
     <gazebo reference="camera_link">
-        <material>Gazebo/Black</material>
         <sensor name="camera" type="camera">
             <pose> 0 0 0 0 0 0 </pose>

File: description/gps.xacro (robot description, xacro)
@@ -1,22 +1,22 @@
 <?xml version="1.0"?>
 <robot xmlns:xacro="http://www.ros.org/wiki/xacro" >
+    <xacro:property name="gps_offset_x" value="-0.1"/>
+    <xacro:property name="gps_offset_z" value="0.65"/>
     <joint name="gps_joint" type="fixed">
         <parent link="base_link"/>
         <child link="gps_link"/>
-        <origin xyz="0.122 0 0.212" rpy="0 0 3.1459"/>
+        <origin xyz="${gps_offset_x} 0 ${gps_offset_z}" rpy="0 0 3.1459"/>
     </joint>
     <link name="gps_link">
         <visual>
             <geometry>
-                <cylinder radius="0.05" length="0.04"/>
+                <cylinder radius="0.05" length="0.02"/>
             </geometry>
-            <material name="black"/>
         </visual>
         <visual>
-            <origin xyz="0 0 -0.05"/>
+            <origin xyz="0 0 -0.1"/>
             <geometry>
-                <cylinder radius="0.01" length="0.1"/>
+                <cylinder radius="0.01" length="0.2"/>
             </geometry>
-            <material name="black"/>
         </visual>
         <collision>
@@ -25,11 +25,10 @@
             </geometry>
         </collision>
-        <xacro:inertial_cylinder mass="0.1" length="0.04" radius="0.05">
-            <origin xyz="0 0 0" rpy="0 0 0"/>
-        </xacro:inertial_cylinder>
     </link>
+    <gazebo reference="gps_link">
+        <material>Gazebo/Yellow</material>
+    </gazebo>
 	<!-- See https://medium.com/@bytesrobotics/a-review-of-the-ros2-urdf-gazebo-sensor-91e947c633d7 -->
 	<gazebo reference="gps_link">
-		<material>Gazebo/Grey</material>
 		<sensor name="gps_sensor" type="gps">
 			<always_on>true</always_on>

File: description/lidar.xacro (robot description, xacro)
@@ -1,15 +1,16 @@
 <?xml version="1.0"?>
 <robot xmlns:xacro="http://www.ros.org/wiki/xacro" >
+    <xacro:property name="laser_offset_x" value="-0.01"/>
+    <xacro:property name="laser_offset_z" value="0.57"/>
     <joint name="laser_joint" type="fixed">
         <parent link="base_link"/>
-        <child link="laser_frame"/>
-        <origin xyz="0.122 0 0.212" rpy="0 0 3.1459"/>
+        <child link="laser_link"/>
+        <origin xyz="${laser_offset_x} 0 ${laser_offset_z}" rpy="0 0 3.1459"/>
     </joint>
-    <link name="laser_frame">
+    <link name="laser_link">
         <visual>
             <geometry>
                 <cylinder radius="0.05" length="0.04"/>
             </geometry>
-            <material name="black"/>
         </visual>
         <visual>
@@ -18,5 +19,4 @@
                 <cylinder radius="0.01" length="0.1"/>
             </geometry>
-            <material name="black"/>
         </visual>
         <collision>
@@ -29,6 +29,9 @@
         </xacro:inertial_cylinder>
     </link>
-    <gazebo reference="laser_frame">
-        <material>Gazebo/Black</material>
+    <gazebo reference="laser_link">
+        <!-- Indigo Turquoise - see gazebo.material in gz-sim GitHub -->
+        <material>Gazebo/Indigo</material>
+    </gazebo>
+    <gazebo reference="laser_link">
         <sensor name="laser" type="ray">
             <pose> 0 0 0 0 0 0 </pose>
@@ -53,5 +56,5 @@
                 </ros>
                 <output_type>sensor_msgs/LaserScan</output_type>
-                <frame_name>laser_frame</frame_name>
+                <frame_name>laser_link</frame_name>
             </plugin>
         </sensor>

File: description/robot.urdf.xacro (robot description, xacro)
@@ -14,4 +14,4 @@
     <!-- <xacro:include filename="depth_camera.xacro" /> -->
     <xacro:include filename="gps.xacro" />
-    <xacro:include filename="face.xacro" />
+    <!-- xacro:include filename="face.xacro" / -->
 </robot>

File: description/robot_core.xacro (robot description, xacro)
@@ -4,16 +4,18 @@
 	<!-- Values corrected for Dragger robot -->
     <xacro:property name="chassis_length" value="0.90"/>
-    <xacro:property name="chassis_width" value="0.70"/>
-    <xacro:property name="chassis_height" value="0.75"/>
+    <xacro:property name="chassis_width" value="0.40"/>
+    <xacro:property name="chassis_height" value="0.50"/>
     <xacro:property name="chassis_mass" value="30.0"/>
     <xacro:property name="wheel_radius" value="0.192"/>
     <xacro:property name="wheel_thickness" value="0.09"/>
     <xacro:property name="wheel_mass" value="1.0"/>
-    <xacro:property name="wheel_offset_x" value="0.10"/>
+    <xacro:property name="wheel_offset_x" value="0.70"/>
     <xacro:property name="wheel_offset_y" value="0.290"/>
     <xacro:property name="wheel_offset_z" value="0.01"/>
     <xacro:property name="caster_wheel_radius" value="0.12"/>
+    <xacro:property name="caster_wheel_thickness" value="0.08"/>
     <xacro:property name="caster_wheel_mass" value="0.3"/>
-    <xacro:property name="caster_wheel_offset_x" value="0.48"/>
+    <xacro:property name="caster_wheel_offset_x" value="0.10"/>
+    <xacro:property name="caster_wheel_offset_y" value="0.280"/>
     <xacro:property name="caster_wheel_offset_z" value="${wheel_offset_z - wheel_radius + caster_wheel_radius}"/>
     <material name="white">
@@ -53,7 +55,14 @@
     <link name="chassis_link">
         <visual>
-            <origin xyz="${chassis_length/2} 0 ${chassis_height/2}"/>
-            <geometry>
-                <box size="${chassis_length} ${chassis_width} ${chassis_height}"/>
+            <origin xyz="${chassis_length/2} 0 ${chassis_height/4}"/>
+            <geometry>
+                <box size="${chassis_length} ${chassis_width} ${chassis_height/2}"/>
+            </geometry>
+            <material name="orange"/>
+        </visual>
+        <visual>
+            <origin xyz="${chassis_length*3/4} 0 ${chassis_height*3/4}"/>
+            <geometry>
+                <box size="${chassis_length/2} ${chassis_width} ${chassis_height/2}"/>
             </geometry>
             <material name="orange"/>
@@ -103,5 +112,4 @@
                 <cylinder radius="${wheel_radius}" length="${wheel_thickness}"/>
             </geometry>
-            <material name="blue"/>
         </visual>
         <collision>
@@ -115,5 +123,5 @@
     </link>
     <gazebo reference="left_wheel">
-        <material>Gazebo/Blue</material>
+        <material>Gazebo/Red</material>
     </gazebo>
     <!-- RIGHT WHEEL LINK -->
@@ -129,5 +137,4 @@
                 <cylinder radius="${wheel_radius}" length="${wheel_thickness}"/>
             </geometry>
-            <material name="blue"/>
         </visual>
         <collision>
@@ -141,23 +148,23 @@
     </link>
     <gazebo reference="right_wheel">
-        <material>Gazebo/Blue</material>
-    </gazebo>
-    <!-- CASTER WHEEL LINK -->
-    <joint name="caster_wheel_joint" type="fixed">
+        <material>Gazebo/Green</material>
+    </gazebo>
+    <!-- CASTER WHEELS LINKS -->
+    <joint name="left_caster_wheel_joint" type="fixed">
         <parent link="chassis_link"/>
-        <child link="caster_wheel"/>
-        <origin xyz="${caster_wheel_offset_x} 0 ${caster_wheel_offset_z}"/>
-    </joint>
-    <link name="caster_wheel">
-        <visual>
+        <child link="left_caster_wheel"/>
+        <origin xyz="${caster_wheel_offset_x} ${caster_wheel_offset_y} ${caster_wheel_offset_z}" rpy="${pi/2} 0 0" />
+        <axis xyz="0 0 1"/>
+    </joint>
+    <link name="left_caster_wheel">
+        <visual>
+            <geometry>
+               <cylinder radius="${caster_wheel_radius}" length="${caster_wheel_thickness}"/>
+            </geometry>
+        </visual>
+        <collision>
             <geometry>
                 <sphere radius="${caster_wheel_radius}"/>
             </geometry>
-            <material name="white"/>
-        </visual>
-        <collision>
-            <geometry>
-                <sphere radius="${caster_wheel_radius}"/>
-            </geometry>
         </collision>
         <xacro:inertial_sphere mass="${caster_wheel_mass}" radius="${caster_wheel_radius}">
@@ -165,8 +172,34 @@
         </xacro:inertial_sphere>
     </link>
-    <gazebo reference="caster_wheel">
-        <material>Gazebo/White</material>
+    <gazebo reference="left_caster_wheel">
+        <material>Gazebo/Red</material>
         <mu1 value="0.001"/>
         <mu2 value="0.001"/>
     </gazebo>
+    <joint name="right_caster_wheel_joint" type="fixed">
+        <parent link="chassis_link"/>
+        <child link="right_caster_wheel"/>
+        <origin xyz="${caster_wheel_offset_x} ${-caster_wheel_offset_y} ${caster_wheel_offset_z}" rpy="${pi/2} 0 0" />
+        <axis xyz="0 0 -1"/>
+    </joint>
+    <link name="right_caster_wheel">
+        <visual>
+            <geometry>
+               <cylinder radius="${caster_wheel_radius}" length="${caster_wheel_thickness}"/>
+            </geometry>
+        </visual>
+        <collision>
+            <geometry>
+                <sphere radius="${caster_wheel_radius}"/>
+            </geometry>
+        </collision>
+        <xacro:inertial_sphere mass="${caster_wheel_mass}" radius="${caster_wheel_radius}">
+            <origin xyz="0 0 0" rpy="0 0 0"/>
+        </xacro:inertial_sphere>
+    </link>
+    <gazebo reference="right_caster_wheel">
+        <material>Gazebo/Green</material>
+        <mu1 value="0.001"/>
+        <mu2 value="0.001"/>
+    </gazebo>
 </robot>
