Commit message: WIP - colors, wheel markers, plugins
commented out some launch nodes for now

File: description/camera.xacro (robot description, xacro)
@@ -13,4 +13,5 @@
                 <box size="0.010 0.03 0.03"/>
             </geometry>
+            <material name="sensor_blue"/>
         </visual>
         <visual>
@@ -19,4 +20,5 @@
                 <cylinder radius="0.002" length="0.1"/>
             </geometry>
+            <material name="sensor_blue"/>
         </visual>
     </link>
@@ -26,8 +28,23 @@
         <origin xyz="0 0 0" rpy="${-pi/2} 0 ${-pi/2}"/>
     </joint>
-    <link name="camera_link_optical"></link>
-    <gazebo reference="laser_frame">
-        <material>Gazebo/Grey</material>
-    </gazebo>
+    <link name="camera_link_optical">
+        <!-- sensor name="camera" type="camera">
+            <camera>
+                <horizontal_fov>1.047</horizontal_fov>
+                <image>
+                    <width>320</width>
+                    <height>240</height>
+                </image>
+                <clip>
+                    <near>0.1</near>
+                    <far>100</far>
+                </clip>
+            </camera>
+            <always_on>1</always_on>
+            <update_rate>30</update_rate>
+            <visualize>true</visualize>
+            <topic>camera</topic>
+        </sensor -->
+    </link>
     <gazebo reference="camera_link">
         <sensor name="camera" type="camera">

File: description/gps.xacro (robot description, xacro)
@@ -13,4 +13,5 @@
                 <cylinder radius="0.05" length="0.02"/>
             </geometry>
+            <material name="sensor_yellow"/>
         </visual>
         <visual>
@@ -19,4 +20,5 @@
                 <cylinder radius="0.01" length="0.2"/>
             </geometry>
+            <material name="sensor_yellow"/>
         </visual>
         <collision>
@@ -26,7 +28,4 @@
         </collision>
     </link>
-    <gazebo reference="gps_link">
-        <material>Gazebo/Yellow</material>
-    </gazebo>
 	<!-- See https://medium.com/@bytesrobotics/a-review-of-the-ros2-urdf-gazebo-sensor-91e947c633d7 -->
 	<gazebo reference="gps_link">

File: description/lidar.xacro (robot description, xacro)
@@ -13,4 +13,5 @@
                 <cylinder radius="0.05" length="0.04"/>
             </geometry>
+            <material name="sensor_blue"/>
         </visual>
         <visual>
@@ -19,4 +20,5 @@
                 <cylinder radius="0.01" length="0.1"/>
             </geometry>
+            <material name="sensor_blue"/>
         </visual>
         <collision>
@@ -29,8 +31,4 @@
         </xacro:inertial_cylinder>
     </link>
-    <gazebo reference="laser_link">
-        <!-- Indigo Turquoise - see gazebo.material in gz-sim GitHub -->
-        <material>Gazebo/Indigo</material>
-    </gazebo>
     <gazebo reference="laser_link">
         <sensor name="laser" type="ray">

File: description/robot.urdf.xacro (robot description, xacro)
@@ -1,4 +1,58 @@
 <?xml version="1.0"?>
 <robot xmlns:xacro="http://www.ros.org/wiki/xacro"  name="robot">
+    <!-- Gazebo Fortress (ROS Humble): -->
+    <plugin name="ignition::gazebo::systems::Physics" filename="libignition-gazebo-physics-system"/>
+    <plugin name="ignition::gazebo::systems::UserCommands" filename="libignition-gazebo-user-commands-system"/>
+    <plugin name="ignition::gazebo::systems::SceneBroadcaster" filename="libignition-gazebo-scene-broadcaster-system"/>
+    <plugin name="ignition::gazebo::systems::Contact" filename="libignition-gazebo-contact-system"/>
+    <plugin name="ignition::gazebo::systems::Imu" filename="libignition-gazebo-imu-system"/>
+    <plugin name="ignition::gazebo::systems::AirPressure" filename="libignition-gazebo-air-pressure-system"/>
+    <plugin name="ignition::gazebo::systems::ApplyLinkWrench" filename="libignition-gazebo-apply-link-wrench-system"/>
+    <plugin name="ignition::gazebo::systems::NavSat" filename="libignition-gazebo-navsat-system"/>
+    <plugin name="ignition::gazebo::systems::Sensors" filename="libignition-gazebo-sensors-system">
+      <render_engine>ogre2</render_engine>
+    </plugin>
+    <!-- Gazebo Garden (PX4): -->
+    <!-- plugin name="gz::sim::systems::Physics" filename="gz-sim-physics-system"/>
+    <plugin name="gz::sim::systems::UserCommands" filename="gz-sim-user-commands-system"/>
+    <plugin name="gz::sim::systems::SceneBroadcaster" filename="gz-sim-scene-broadcaster-system"/>
+    <plugin name="gz::sim::systems::Contact" filename="gz-sim-contact-system"/>
+    <plugin name="gz::sim::systems::Imu" filename="gz-sim-imu-system"/>
+    <plugin name="gz::sim::systems::AirPressure" filename="gz-sim-air-pressure-system"/>
+    <plugin name="gz::sim::systems::ApplyLinkWrench" filename="gz-sim-apply-link-wrench-system"/>
+    <plugin name="gz::sim::systems::NavSat" filename="gz-sim-navsat-system"/>
+    <plugin name="gz::sim::systems::Sensors" filename="gz-sim-sensors-system">
+      <render_engine>ogre2</render_engine>
+    </plugin -->
+    <!-- plugin filename="ignition-gazebo-sensors-system" name="gz::sim::systems::Sensors" -->
+    <!-- plugin filename="libignition-gazebo-sensors-system.so" name="ignition::gazebo::systems::Sensors">
+       <render_engine>ogre</render_engine>
+    </plugin -->
+    <material name="white">
+        <color rgba="1 1 1 1" />
+    </material>
+    <material name="black">
+        <color rgba="0 0 0 1"/>
+    </material>
+    <material name="blue">
+        <color rgba="0 0 1 1"/>
+    </material>
+    <material name="sensor_blue">
+        <color rgba="0.2 0.2 1 1"/>
+    </material>
+    <material name="sensor_yellow">
+        <color rgba="0.8 0.8 0.2 1"/>
+    </material>
+    <material name="body_color">
+        <color rgba="1 0.3 0.1 1"/>
+    </material>
+    <material name="port_red">
+        <color rgba="1 0.2 0.2 1"/>
+        <!-- ambient>1.0 0.2 0.2 1</ambient>
+        <diffuse>1.0 0.1 0.1 1</diffuse -->
+    </material>
+    <material name="starboard_green">
+        <color rgba="0.2 1 0.2 1"/>
+    </material>
     <xacro:arg name="use_ros2_control" default="true"/>
     <xacro:arg name="sim_mode" default="false"/>

File: description/robot_core.xacro (robot description, xacro)
@@ -19,19 +19,4 @@
     <xacro:property name="caster_wheel_offset_y" value="0.280"/>
     <xacro:property name="caster_wheel_offset_z" value="${wheel_offset_z - wheel_radius + caster_wheel_radius}"/>
-    <material name="white">
-        <color rgba="1 1 1 1" />
-    </material>
-    <material name="orange">
-        <color rgba="1 0.3 0.1 1"/>
-    </material>
-    <material name="blue">
-        <color rgba="0.2 0.2 1 1"/>
-    </material>
-    <material name="black">
-        <color rgba="0 0 0 1"/>
-    </material>
-    <material name="red">
-        <color rgba="1 0 0 1"/>
-    </material>
     <!-- ****************** ROBOT BASE FOOTPRINT ***************************  -->
     <!-- Define the center of the main robot chassis projected on the ground -->
@@ -54,17 +39,17 @@
     </joint>
     <link name="chassis_link">
-        <visual>
+        <visual name="chassis_visual">
             <origin xyz="${chassis_length/2} 0 ${chassis_height/4}"/>
             <geometry>
                 <box size="${chassis_length} ${chassis_width} ${chassis_height/2}"/>
             </geometry>
-            <material name="orange"/>
-        </visual>
-        <visual>
+            <material name="body_color"/>
+        </visual>
+        <visual name="chassis_top_visual">
             <origin xyz="${chassis_length*3/4} 0 ${chassis_height*3/4}"/>
             <geometry>
-                <box size="${chassis_length/2} ${chassis_width} ${chassis_height/2}"/>
-            </geometry>
-            <material name="orange"/>
+                <box size="${chassis_length*0.45} ${chassis_width*0.95} ${chassis_height/2}"/>
+            </geometry>
+            <material name="body_color"/>
         </visual>
         <collision>
@@ -78,7 +63,4 @@
         </xacro:inertial_box>
     </link>
-    <gazebo reference="chassis_link">
-        <material>Gazebo/Orange</material>
-    </gazebo>
     <!-- *********************** IMU SETUP *********************************  -->
     <!-- Each sensor must be attached to a link.                              -->
@@ -108,9 +90,28 @@
     </joint>
     <link name="left_wheel">
-        <visual>
+        <visual name="left_wheel_visual">
             <geometry>
                 <cylinder radius="${wheel_radius}" length="${wheel_thickness}"/>
             </geometry>
-        </visual>
+            <material name="port_red"/>
+        </visual>
+        <visual name="left_wheel_marker_visual">
+            <geometry>
+                <box size="${wheel_radius*0.5} ${wheel_radius*0.5} ${wheel_thickness*1.1}"/>
+            </geometry>
+            <material name="blue"/>
+        </visual>
+        <!-- visual name="left_wheel_marker_visual">
+            <pose>0.17 0 0 0 0 0</pose>
+            <geometry>
+                <box size=".10 .01 .21"/>
+            </geometry>
+            <material>
+                <ambient>1.0 0.2 0.2 1</ambient>
+                <diffuse>1.0 0.1 0.1 1</diffuse>
+                <specular>0 0 0 0</specular>
+                <emissive>0 0 0 1</emissive>
+            </material>
+        </visual -->
         <collision>
             <geometry>
@@ -122,7 +123,4 @@
         </xacro:inertial_cylinder>
     </link>
-    <gazebo reference="left_wheel">
-        <material>Gazebo/Red</material>
-    </gazebo>
     <!-- RIGHT WHEEL LINK -->
     <joint name="right_wheel_joint" type="continuous">
@@ -137,4 +135,11 @@
                 <cylinder radius="${wheel_radius}" length="${wheel_thickness}"/>
             </geometry>
+            <material name="starboard_green"/>
+        </visual>
+        <visual name="right_wheel_marker_visual">
+            <geometry>
+                <box size="${wheel_radius*0.5} ${wheel_radius*0.5} ${wheel_thickness*1.1}"/>
+            </geometry>
+            <material name="blue"/>
         </visual>
         <collision>
@@ -147,9 +152,6 @@
         </xacro:inertial_cylinder>
     </link>
-    <gazebo reference="right_wheel">
-        <material>Gazebo/Green</material>
-    </gazebo>
     <!-- CASTER WHEELS LINKS -->
-    <joint name="left_caster_wheel_joint" type="fixed">
+    <joint name="left_caster_wheel_joint" type="continuous">
         <parent link="chassis_link"/>
         <child link="left_caster_wheel"/>
@@ -162,4 +164,11 @@
                <cylinder radius="${caster_wheel_radius}" length="${caster_wheel_thickness}"/>
             </geometry>
+            <material name="port_red"/>
+        </visual>
+        <visual name="left_caster_marker_visual">
+            <geometry>
+                <box size="${caster_wheel_radius*0.5} ${caster_wheel_radius*0.5} ${caster_wheel_thickness*1.1}"/>
+            </geometry>
+            <material name="blue"/>
         </visual>
         <collision>
@@ -172,10 +181,5 @@
         </xacro:inertial_sphere>
     </link>
-    <gazebo reference="left_caster_wheel">
-        <material>Gazebo/Red</material>
-        <mu1 value="0.001"/>
-        <mu2 value="0.001"/>
-    </gazebo>
-    <joint name="right_caster_wheel_joint" type="fixed">
+    <joint name="right_caster_wheel_joint" type="continuous">
         <parent link="chassis_link"/>
         <child link="right_caster_wheel"/>
@@ -188,4 +192,11 @@
                <cylinder radius="${caster_wheel_radius}" length="${caster_wheel_thickness}"/>
             </geometry>
+            <material name="starboard_green"/>
+        </visual>
+        <visual name="left_caster_marker_visual">
+            <geometry>
+                <box size="${caster_wheel_radius*0.5} ${caster_wheel_radius*0.5} ${caster_wheel_thickness*1.1}"/>
+            </geometry>
+            <material name="blue"/>
         </visual>
         <collision>
@@ -198,8 +209,23 @@
         </xacro:inertial_sphere>
     </link>
-    <gazebo reference="right_caster_wheel">
+    <!-- gazebo reference="right_caster_wheel">
         <material>Gazebo/Green</material>
         <mu1 value="0.001"/>
         <mu2 value="0.001"/>
     </gazebo>
+    <gazebo reference="left_caster_wheel">
+        <material>Gazebo/Red</material>
+        <material>
+            <ambient>1.0 0.2 0.2 1</ambient>
+            <diffuse>1.0 0.1 0.1 1</diffuse>
+        </material>
+        <mu1 value="0.001"/>
+        <mu2 value="0.001"/>
+    </gazebo>
+    <gazebo reference="left_wheel">
+        <material>Gazebo/Red</material>
+    </gazebo>
+    <gazebo reference="right_wheel">
+        <material>Gazebo/Green</material>
+    </gazebo -->
 </robot>

File: description/ros2_control.xacro (robot description, xacro)
@@ -48,5 +48,5 @@
         <plugin filename="libign_ros2_control-system.so" name="ign_ros2_control::IgnitionROS2ControlPlugin">
         <!-- plugin filename="gz_ros2_control-system" name="gz_ros2_control::GazeboSimROS2ControlPlugin" -->
-            <!-- the following are just default parameters anyway. Skip them unless you want to reaasign them:
+            <!-- the following are just default parameters anyway. Skip them unless you want to reassign them:
             <robot_param>robot_description</robot_param>
             <robot_param_node>robot_state_publisher</robot_param_node> -->

Commit message: Better URDF - eliminated chassis joint

File: description/camera.xacro (robot description, xacro)
@@ -1,5 +1,5 @@
 <?xml version="1.0"?>
 <robot xmlns:xacro="http://www.ros.org/wiki/xacro" >
-    <xacro:property name="camera_offset_x" value="0.2"/>
+    <xacro:property name="camera_offset_x" value="${chassis_length/2 - 0.04}"/>
     <xacro:property name="camera_offset_z" value="0.55"/>
     <joint name="camera_joint" type="fixed">

File: description/gps.xacro (robot description, xacro)
@@ -1,5 +1,5 @@
 <?xml version="1.0"?>
 <robot xmlns:xacro="http://www.ros.org/wiki/xacro" >
-    <xacro:property name="gps_offset_x" value="-0.1"/>
+    <xacro:property name="gps_offset_x" value="0.05"/>
     <xacro:property name="gps_offset_z" value="0.65"/>
     <joint name="gps_joint" type="fixed">

File: description/lidar.xacro (robot description, xacro)
@@ -1,5 +1,5 @@
 <?xml version="1.0"?>
 <robot xmlns:xacro="http://www.ros.org/wiki/xacro" >
-    <xacro:property name="laser_offset_x" value="-0.01"/>
+    <xacro:property name="laser_offset_x" value="${chassis_length/4 + 0.05}"/>
     <xacro:property name="laser_offset_z" value="0.57"/>
     <joint name="laser_joint" type="fixed">
@@ -18,5 +18,5 @@
             <origin xyz="0 0 -0.05"/>
             <geometry>
-                <cylinder radius="0.01" length="0.1"/>
+                <cylinder radius="0.03" length="0.1"/>
             </geometry>
             <material name="sensor_blue"/>

File: description/robot.urdf.xacro (robot description, xacro)
@@ -7,4 +7,7 @@
     <material name="black">
         <color rgba="0 0 0 1"/>
+    </material>
+    <material name="shadow_grey">
+        <color rgba="0.3 0.3 0.3 0.5"/>
     </material>
     <material name="blue">

File: description/robot_core.xacro (robot description, xacro)
@@ -10,5 +10,5 @@
     <xacro:property name="wheel_thickness" value="0.09"/>
     <xacro:property name="wheel_mass" value="1.0"/>
-    <xacro:property name="wheel_offset_x" value="0.70"/>
+    <xacro:property name="wheel_offset_x" value="${chassis_length/2 - wheel_radius - 0.01}"/>
     <xacro:property name="wheel_offset_y" value="0.290"/>
     <xacro:property name="wheel_offset_z" value="0.01"/>
@@ -16,14 +16,19 @@
     <xacro:property name="caster_wheel_thickness" value="0.08"/>
     <xacro:property name="caster_wheel_mass" value="0.3"/>
-    <xacro:property name="caster_wheel_offset_x" value="0.10"/>
+    <xacro:property name="caster_wheel_offset_x" value="${-chassis_length/2 + caster_wheel_radius + 0.01}"/>
     <xacro:property name="caster_wheel_offset_y" value="0.280"/>
     <xacro:property name="caster_wheel_offset_z" value="${wheel_offset_z - wheel_radius + caster_wheel_radius}"/>
     <!-- ****************** ROBOT BASE FOOTPRINT ***************************  -->
     <!-- Define the center of the main robot chassis projected on the ground -->
+    <!-- link name="base_footprint"/ -->
     <link name="base_footprint">
-    </link>
-    <!-- ********************** ROBOT BASE *********************************  -->
-    <link name="base_link">
-    </link>
+        <visual name="footprint_visual">
+            <origin xyz="0 0 0.01"/>
+            <geometry>
+                <box size="${chassis_length} ${chassis_width} 0.02"/>
+            </geometry>
+            <material name="shadow_grey"/>
+        </visual>
+     </link>
     <!-- The base footprint of the robot is located underneath the chassis -->
     <joint name="base_joint" type="fixed">
@@ -32,13 +37,16 @@
         <origin xyz="0 0 ${wheel_radius}" rpy="0 0 0"/>
     </joint>
+    <!-- ********************** ROBOT BASE *********************************  -->
+    <!-- link name="base_link"/ -->
     <!-- CHASSIS LINK -->
-    <joint name="chassis_joint" type="fixed">
+    <!-- joint name="chassis_joint" type="fixed">
         <parent link="base_link"/>
         <child link="chassis_link"/>
         <origin xyz="${-wheel_offset_x} 0 ${-wheel_offset_z}"/>
-    </joint>
-    <link name="chassis_link">
+    </joint -->
+    <link name="base_link">
         <visual name="chassis_visual">
-            <origin xyz="${chassis_length/2} 0 ${chassis_height/4}"/>
+            <!-- origin xyz="${chassis_length/2} 0 ${chassis_height/4}"/ -->
+            <origin xyz="0 0 ${chassis_height/4}"/>
             <geometry>
                 <box size="${chassis_length} ${chassis_width} ${chassis_height/2}"/>
@@ -47,5 +55,5 @@
         </visual>
         <visual name="chassis_top_visual">
-            <origin xyz="${chassis_length*3/4} 0 ${chassis_height*3/4}"/>
+            <origin xyz="${chassis_length*1/4} 0 ${chassis_height*3/4}"/>
             <geometry>
                 <box size="${chassis_length*0.45} ${chassis_width*0.95} ${chassis_height/2}"/>
@@ -70,4 +78,5 @@
             <box size="0.1 0.1 0.1"/>
         </geometry>
+        <material name="sensor_blue"/>
         </visual>
         <collision>
@@ -80,5 +89,5 @@
         <parent link="base_link"/>
         <child link="imu_link"/>
-        <origin xyz="0 0 0.01"/>
+        <origin xyz="0 0 0.04"/>
     </joint>
     <!-- LEFT WHEEL LINK -->
@@ -86,6 +95,11 @@
         <parent link="base_link"/>
         <child link="left_wheel"/>
-        <origin xyz="0 ${wheel_offset_y} 0" rpy="-${pi/2} 0 0" />
-        <axis xyz="0 0 1"/>
+        <origin xyz="${wheel_offset_x} ${wheel_offset_y} 0" rpy="-${pi/2} 0 0" />
+        <axis xyz="0 0 1">
+          <limit>
+            <lower>-1.79769e+308</lower>
+            <upper>1.79769e+308</upper>
+          </limit>
+        </axis>
     </joint>
     <link name="left_wheel">
@@ -122,6 +136,11 @@
         <parent link="base_link"/>
         <child link="right_wheel"/>
-        <origin xyz="0 ${-wheel_offset_y} 0" rpy="${pi/2} 0 0" />
-        <axis xyz="0 0 -1"/>
+        <origin xyz="${wheel_offset_x} ${-wheel_offset_y} 0" rpy="${pi/2} 0 0" />
+        <axis xyz="0 0 -1">
+          <limit>
+            <lower>-1.79769e+308</lower>
+            <upper>1.79769e+308</upper>
+          </limit>
+        </axis>
     </joint>
     <link name="right_wheel">
@@ -156,5 +175,5 @@
     <!-- CASTER WHEELS LINKS -->
     <joint name="left_caster_wheel_joint" type="continuous">
-        <parent link="chassis_link"/>
+        <parent link="base_link"/>
         <child link="left_caster_wheel"/>
         <origin xyz="${caster_wheel_offset_x} ${caster_wheel_offset_y} ${caster_wheel_offset_z}" rpy="${pi/2} 0 0" />
@@ -184,5 +203,5 @@
     </link>
     <joint name="right_caster_wheel_joint" type="continuous">
-        <parent link="chassis_link"/>
+        <parent link="base_link"/>
         <child link="right_caster_wheel"/>
         <origin xyz="${caster_wheel_offset_x} ${-caster_wheel_offset_y} ${caster_wheel_offset_z}" rpy="${pi/2} 0 0" />
