Commit message: Sensors work, except IMU bridge. GPS needs work

File: description/camera.xacro (robot description, xacro)
@@ -26,46 +26,57 @@
         <parent link="camera_link"/>
         <child link="camera_link_optical"/>
-        <origin xyz="0 0 0" rpy="${-pi/2} 0 ${-pi/2}"/>
+        <origin xyz="0 0 0" rpy="0 0 0"/>
     </joint>
     <link name="camera_link_optical">
-        <sensor name="camera" type="camera">
-            <camera>
-                <horizontal_fov>1.047</horizontal_fov>
-                <image>
-                    <width>320</width>
-                    <height>240</height>
-                </image>
-                <clip>
-                    <near>0.1</near>
-                    <far>100</far>
-                </clip>
-            </camera>
-            <always_on>1</always_on>
-            <update_rate>30</update_rate>
-            <visualize>true</visualize>
-            <topic>camera</topic>
+    </link>
+	<gazebo reference="camera_link_optical">
+        <sensor name='camera' type='camera'>
+          <pose>0 0 0 0 0 0</pose>
+		  <always_on>true</always_on>
+          <topic>camera</topic>
+          <update_rate>30</update_rate>
+          <enable_metrics>false</enable_metrics>
+          <camera name='__default__'>
+            <pose>0 0 0 0 0 0</pose>
+            <horizontal_fov>1.0469999999999999</horizontal_fov>
+            <image>
+              <width>320</width>
+              <height>240</height>
+              <format>RGB_INT8</format>
+              <anti_aliasing>4</anti_aliasing>
+            </image>
+            <camera_info_topic>__default__</camera_info_topic>
+            <trigger_topic></trigger_topic>
+            <triggered>false</triggered>
+            <clip>
+              <near>0.10000000000000001</near>
+              <far>100</far>
+            </clip>
+            <save enabled='false'>
+              <path>__default__</path>
+            </save>
+            <visibility_mask>4294967295</visibility_mask>
+            <noise>
+              <type>none</type>
+              <mean>0</mean>
+              <stddev>0</stddev>
+            </noise>
+            <distortion>
+              <k1>0</k1>
+              <k2>0</k2>
+              <k3>0</k3>
+              <p1>0</p1>
+              <p2>0</p2>
+              <center>0.5 0.5</center>
+            </distortion>
+            <lens>
+              <type>stereographic</type>
+              <scale_to_hfov>true</scale_to_hfov>
+              <cutoff_angle>1.5707963267948966</cutoff_angle>
+              <env_texture_size>256</env_texture_size>
+            </lens>
+            <optical_frame_id></optical_frame_id>
+          </camera>
         </sensor>
-    </link>
-    <!-- gazebo reference="camera_link">
-        <sensor name="camera" type="camera">
-            <pose> 0 0 0 0 0 0 </pose>
-            <visualize>true</visualize>
-            <update_rate>10</update_rate>
-            <camera>
-                <horizontal_fov>1.089</horizontal_fov>
-                <image>
-                    <format>R8G8B8</format>
-                    <width>640</width>
-                    <height>480</height>
-                </image>
-                <clip>
-                    <near>0.05</near>
-                    <far>8.0</far>
-                </clip>
-            </camera>
-            <plugin name="camera_controller" filename="libgazebo_ros_camera.so">
-                <frame_name>camera_link_optical</frame_name>
-            </plugin>
-        </sensor>
-    </gazebo -->
+    </gazebo>
 </robot>

File: description/gps.xacro (robot description, xacro)
@@ -32,14 +32,8 @@
 		<sensor name="gps_sensor" type="gps">
 			<always_on>true</always_on>
+            <topic>navsat</topic>
 			<pose> 0 0 0 0 0 0 </pose>
 			<visualize>false</visualize>
 			<update_rate>5</update_rate>
-			<!-- plugin name="gps_controller" filename="libgazebo_ros_gps_sensor.so">
-				<ros>
-					< !- - <namespace>/br</namespace> - - >
-					<remapping>gps_controller/out:=gps</remapping>
-				</ros>
-				<frame_name>gps_link</frame_name>
-			</plugin -->
 		</sensor>
 	</gazebo>

File: description/lidar.xacro (robot description, xacro)
@@ -32,28 +32,37 @@
     </link>
     <gazebo reference="laser_link">
-        <sensor name="laser" type="ray">
-            <pose> 0 0 0 0 0 0 </pose>
-            <visualize>false</visualize>
-            <update_rate>10</update_rate>
-            <ray>
-                <scan>
-                    <horizontal>
-                        <samples>360</samples>
-                        <min_angle>-3.14</min_angle>
-                        <max_angle>3.14</max_angle>
-                    </horizontal>
-                </scan>
-                <range>
-                    <min>0.3</min>
-                    <max>12</max>
-                </range>
-            </ray>
-            <!-- plugin name="laser_controller" filename="libgazebo_ros_ray_sensor.so">
-                <ros>
-                    <argument>~/out:=scan</argument>
-                </ros>
-                <output_type>sensor_msgs/LaserScan</output_type>
-                <frame_name>laser_link</frame_name>
-            </plugin -->
+        <sensor name='front_laser' type='gpu_lidar'>
+          <pose>0 0 0 0 0 0</pose>
+          <always_on>1</always_on>
+          <update_rate>10</update_rate>
+          <topic>scan</topic>
+          <!-- frame_id>laser_frame</frame_id -->
+          <ray>
+            <scan>
+              <horizontal>
+                <samples>360</samples>
+                <resolution>1</resolution>
+                <min_angle>-3.1459</min_angle>
+                <max_angle>3.1459</max_angle>
+              </horizontal>
+              <vertical>
+                <samples>1</samples>
+                <resolution>1</resolution>
+                <min_angle>0.0</min_angle>
+                <max_angle>0.0</max_angle>
+              </vertical>
+            </scan>
+            <range>
+              <min>0.3</min>
+              <max>12.0</max>
+              <resolution>0.01</resolution>
+            </range>
+            <noise>
+              <type>gaussian</type>
+              <mean>0</mean>
+              <stddev>0.01</stddev>
+            </noise>
+          </ray>
+          <visualize>true</visualize>
         </sensor>
     </gazebo>

File: description/robot_core.xacro (robot description, xacro)
@@ -75,13 +75,13 @@
     <link name="imu_link">
         <visual>
-        <geometry>
-            <box size="0.1 0.1 0.1"/>
-        </geometry>
-        <material name="sensor_blue"/>
-        </visual>
-        <collision>
-        <geometry>
-            <box size="0.1 0.1 0.1"/>
-        </geometry>
+            <geometry>
+                <box size="0.1 0.1 0.1"/>
+            </geometry>
+            <material name="sensor_blue"/>
+        </visual>
+        <collision>
+            <geometry>
+                <box size="0.1 0.1 0.1"/>
+            </geometry>
         </collision>
     </link>
@@ -91,4 +91,84 @@
         <origin xyz="0 0 0.04"/>
     </joint>
+    <gazebo reference="imu_link">
+        <sensor name="imu_sensor" type="imu">
+        <always_on>1</always_on>
+        <topic>imu</topic>
+        <update_rate>250</update_rate>
+            <imu>
+                <enable_orientation>0</enable_orientation>
+                <angular_velocity>
+                    <x>
+                        <noise type="gaussian">
+                            <mean>0</mean>
+                            <stddev>0.009</stddev>
+                            <bias_mean>0.00075</bias_mean>
+                            <bias_stddev>0.005</bias_stddev>
+                            <dynamic_bias_stddev>0.00002</dynamic_bias_stddev>
+                            <dynamic_bias_correlation_time>400.0</dynamic_bias_correlation_time>
+                            <precision>0.00025</precision>
+                        </noise>
+                    </x>
+                    <y>
+                        <noise type="gaussian">
+                            <mean>0</mean>
+                            <stddev>0.009</stddev>
+                            <bias_mean>0.00075</bias_mean>
+                            <bias_stddev>0.005</bias_stddev>
+                            <dynamic_bias_stddev>0.00002</dynamic_bias_stddev>
+                            <dynamic_bias_correlation_time>400.0</dynamic_bias_correlation_time>
+                            <precision>0.00025</precision>
+                        </noise>
+                    </y>
+                    <z>
+                        <noise type="gaussian">
+                            <mean>0</mean>
+                            <stddev>0.009</stddev>
+                            <bias_mean>0.00075</bias_mean>
+                            <bias_stddev>0.005</bias_stddev>
+                            <dynamic_bias_stddev>0.00002</dynamic_bias_stddev>
+                            <dynamic_bias_correlation_time>400.0</dynamic_bias_correlation_time>
+                            <precision>0.00025</precision>
+                        </noise>
+                    </z>
+                </angular_velocity>
+                <linear_acceleration>
+                    <x>
+                        <noise type="gaussian">
+                            <mean>0</mean>
+                            <stddev>0.021</stddev>
+                            <bias_mean>0.05</bias_mean>
+                            <bias_stddev>0.0075</bias_stddev>
+                            <dynamic_bias_stddev>0.000375</dynamic_bias_stddev>
+                            <dynamic_bias_correlation_time>175.0</dynamic_bias_correlation_time>
+                            <precision>0.005</precision>
+                        </noise>
+                    </x>
+                    <y>
+                        <noise type="gaussian">
+                            <mean>0</mean>
+                            <stddev>0.021</stddev>
+                            <bias_mean>0.05</bias_mean>
+                            <bias_stddev>0.0075</bias_stddev>
+                            <dynamic_bias_stddev>0.000375</dynamic_bias_stddev>
+                            <dynamic_bias_correlation_time>175.0</dynamic_bias_correlation_time>
+                            <precision>0.005</precision>
+                        </noise>
+                    </y>
+                    <z>
+                        <noise type="gaussian">
+                            <mean>0</mean>
+                            <stddev>0.021</stddev>
+                            <bias_mean>0.05</bias_mean>
+                            <bias_stddev>0.0075</bias_stddev>
+                            <dynamic_bias_stddev>0.000375</dynamic_bias_stddev>
+                            <dynamic_bias_correlation_time>175.0</dynamic_bias_correlation_time>
+                            <precision>0.005</precision>
+                        </noise>
+                    </z>
+                </linear_acceleration>
+            </imu>
+        </sensor>
+    </gazebo>
     <!-- LEFT WHEEL LINK -->
     <joint name="left_wheel_joint" type="continuous">

Commit message: IMU sensor and bridge work in Gazebo

File: description/camera.xacro (robot description, xacro)
@@ -30,6 +30,7 @@
     <link name="camera_link_optical">
     </link>
+    <!-- gz model -m dragger -s rgb_camera -->
 	<gazebo reference="camera_link_optical">
-        <sensor name='camera' type='camera'>
+        <sensor name='rgb_camera' type='camera'>
           <pose>0 0 0 0 0 0</pose>
 		  <always_on>true</always_on>

File: description/depth_camera.xacro (robot description, xacro)
@@ -1,10 +1,10 @@
 <?xml version="1.0"?>
 <robot xmlns:xacro="http://www.ros.org/wiki/xacro" >
-    <joint name="camera_joint" type="fixed">
-        <parent link="chassis_link"/>
-        <child link="camera_link"/>
+    <joint name="depth_camera_joint" type="fixed">
+        <parent link="base_link"/>
+        <child link="depth_camera_link"/>
         <origin xyz="0.305 0 0.08" rpy="0 0 0"/>
     </joint>
-    <link name="camera_link">
+    <link name="depth_camera_link">
         <visual>
             <geometry>
@@ -14,13 +14,16 @@
         </visual>
     </link>
-    <joint name="camera_optical_joint" type="fixed">
-        <parent link="camera_link"/>
-        <child link="camera_link_optical"/>
+    <joint name="depth_camera_optical_joint" type="fixed">
+        <parent link="depth_camera_link"/>
+        <child link="depth_camera_link_optical"/>
         <origin xyz="0 0 0" rpy="${-pi/2} 0 ${-pi/2}"/>
     </joint>
-    <link name="camera_link_optical"></link>
-    <gazebo reference="camera_link">
+    <link name="depth_camera_link_optical">
+    </link>
+    <!-- gz model -m dragger -s depth_camera -->
+    <gazebo reference="depth_camera_link">
+        <!-- TODO: port to GZ Harmonic, add to gz_ros_brigde.yaml -->
         <material>Gazebo/Red</material>
-        <sensor name="camera" type="depth">
+        <sensor name="depth_camera" type="depth">
             <pose> 0 0 0 0 0 0 </pose>
             <visualize>true</visualize>

File: description/face.xacro (robot description, xacro)
@@ -2,5 +2,5 @@
 <robot xmlns:xacro="http://www.ros.org/wiki/xacro" >
     <joint name="face_joint" type="fixed">
-        <parent link="chassis_link"/>
+        <parent link="base_link"/>
         <child link="face_link"/>
         <origin xyz="${chassis_length} 0 ${chassis_height/2}" rpy="0 0 0"/>
@@ -29,6 +29,3 @@
         </visual>
     </link>
-    <gazebo reference="face_link">
-        <material>Gazebo/Black</material>
-    </gazebo>
 </robot>

File: description/gps.xacro (robot description, xacro)
@@ -29,4 +29,5 @@
     </link>
 	<!-- See https://medium.com/@bytesrobotics/a-review-of-the-ros2-urdf-gazebo-sensor-91e947c633d7 -->
+    <!-- gz model -m dragger -s gps_sensor -->
 	<gazebo reference="gps_link">
 		<sensor name="gps_sensor" type="gps">

File: description/lidar.xacro (robot description, xacro)
@@ -31,4 +31,5 @@
         </xacro:inertial_cylinder>
     </link>
+    <!-- gz model -m dragger -s front_laser -->
     <gazebo reference="laser_link">
         <sensor name='front_laser' type='gpu_lidar'>

File: description/robot_core.xacro (robot description, xacro)
@@ -91,4 +91,5 @@
         <origin xyz="0 0 0.04"/>
     </joint>
+    <!-- gz model -m dragger -s imu_sensor -->
     <gazebo reference="imu_link">
         <sensor name="imu_sensor" type="imu">

Commit message: Back to chassis_link, axles on chassis visual, namespace for nodes

File: description/camera.xacro (robot description, xacro)
@@ -4,5 +4,5 @@
     <xacro:property name="camera_offset_z" value="0.55"/>
     <joint name="camera_joint" type="fixed">
-        <parent link="base_link"/>
+        <parent link="chassis_link"/>
         <child link="camera_link"/>
         <origin xyz="${camera_offset_x} 0 ${camera_offset_z}" rpy="0 0.18 0"/>
@@ -77,5 +77,5 @@
               <env_texture_size>256</env_texture_size>
             </lens>
-            <optical_frame_id></optical_frame_id>
+            <optical_frame_id>camera_frame</optical_frame_id>
           </camera>
         </sensor>

File: description/depth_camera.xacro (robot description, xacro)
@@ -2,5 +2,5 @@
 <robot xmlns:xacro="http://www.ros.org/wiki/xacro" >
     <joint name="depth_camera_joint" type="fixed">
-        <parent link="base_link"/>
+        <parent link="chassis_link"/>
         <child link="depth_camera_link"/>
         <origin xyz="0.305 0 0.08" rpy="0 0 0"/>

File: description/face.xacro (robot description, xacro)
@@ -2,5 +2,5 @@
 <robot xmlns:xacro="http://www.ros.org/wiki/xacro" >
     <joint name="face_joint" type="fixed">
-        <parent link="base_link"/>
+        <parent link="chassis_link"/>
         <child link="face_link"/>
         <origin xyz="${chassis_length} 0 ${chassis_height/2}" rpy="0 0 0"/>

File: description/gps.xacro (robot description, xacro)
@@ -4,5 +4,5 @@
     <xacro:property name="gps_offset_z" value="0.65"/>
     <joint name="gps_joint" type="fixed">
-        <parent link="base_link"/>
+        <parent link="chassis_link"/>
         <child link="gps_link"/>
         <origin xyz="${gps_offset_x} 0 ${gps_offset_z}" rpy="0 0 3.1459"/>

File: description/lidar.xacro (robot description, xacro)
@@ -4,5 +4,5 @@
     <xacro:property name="laser_offset_z" value="0.57"/>
     <joint name="laser_joint" type="fixed">
-        <parent link="base_link"/>
+        <parent link="chassis_link"/>
         <child link="laser_link"/>
         <origin xyz="${laser_offset_x} 0 ${laser_offset_z}" rpy="0 0 3.1459"/>

File: description/robot.urdf.xacro (robot description, xacro)
@@ -10,4 +10,10 @@
     <material name="shadow_grey">
         <color rgba="0.3 0.3 0.3 0.5"/>
+    </material>
+    <material name="red">
+        <color rgba="1 0 0 1"/>
+    </material>
+    <material name="green">
+        <color rgba="0 1 0 1"/>
     </material>
     <material name="blue">

File: description/robot_core.xacro (robot description, xacro)
@@ -17,5 +17,5 @@
     <xacro:property name="caster_wheel_mass" value="0.3"/>
     <xacro:property name="caster_wheel_offset_x" value="${-chassis_length/2 + caster_wheel_radius + 0.01}"/>
-    <xacro:property name="caster_wheel_offset_y" value="0.280"/>
+    <xacro:property name="caster_wheel_offset_y" value="0.270"/>
     <xacro:property name="caster_wheel_offset_z" value="${wheel_offset_z - wheel_radius + caster_wheel_radius}"/>
     <!-- ****************** ROBOT BASE FOOTPRINT ***************************  -->
@@ -31,4 +31,14 @@
         </visual>
      </link>
+    <!-- ********************** ROBOT BASE *********************************  -->
+    <link name="base_link">
+        <visual name="footprint_visual">
+            <origin xyz="0 0 0"/>
+            <geometry>
+                <sphere radius="0.03"/>
+            </geometry>
+            <material name="red"/>
+        </visual>
+    </link>
     <!-- The base footprint of the robot is located underneath the chassis -->
     <joint name="base_joint" type="fixed">
@@ -37,13 +47,12 @@
         <origin xyz="0 0 ${wheel_radius}" rpy="0 0 0"/>
     </joint>
-    <!-- ********************** ROBOT BASE *********************************  -->
-    <!-- link name="base_link"/ -->
-    <!-- CHASSIS LINK -->
-    <!-- joint name="chassis_joint" type="fixed">
+    <!-- ********************** ROBOT BODY *********************************  -->
+    <joint name="chassis_joint" type="fixed">
         <parent link="base_link"/>
         <child link="chassis_link"/>
         <origin xyz="${-wheel_offset_x} 0 ${-wheel_offset_z}"/>
-    </joint -->
-    <link name="base_link">
+    </joint>
+    <!-- CHASSIS LINK -->
+    <link name="chassis_link">
         <visual name="chassis_visual">
             <!-- origin xyz="${chassis_length/2} 0 ${chassis_height/4}"/ -->
@@ -58,4 +67,32 @@
             <geometry>
                 <box size="${chassis_length*0.45} ${chassis_width*0.95} ${chassis_height/2}"/>
+            </geometry>
+            <material name="body_color"/>
+        </visual>
+        <visual name="chassis_front_axle_left">
+            <origin xyz="${wheel_offset_x} ${chassis_width*0.5} 0" rpy="-${pi/2} 0 0"/>
+            <geometry>
+                <cylinder radius="${0.06}" length="${chassis_width*0.5}"/>
+            </geometry>
+            <material name="body_color"/>
+        </visual>
+        <visual name="chassis_front_axle_right">
+            <origin xyz="${wheel_offset_x} ${-chassis_width*0.5} 0" rpy="${pi/2} 0 0"/>
+            <geometry>
+                <cylinder radius="${0.06}" length="${chassis_width*0.5}"/>
+            </geometry>
+            <material name="body_color"/>
+        </visual>
+        <visual name="chassis_caster_joint_left">
+            <origin xyz="${caster_wheel_offset_x} ${chassis_width*0.52} ${caster_wheel_offset_z}" rpy="0 0 0"/>
+            <geometry>
+                <sphere radius="${caster_wheel_offset_z*1.1}"/>
+            </geometry>
+            <material name="body_color"/>
+        </visual>
+        <visual name="chassis_caster_joint_right">
+            <origin xyz="${caster_wheel_offset_x} ${-chassis_width*0.51} ${caster_wheel_offset_z}" rpy="0 0 0"/>
+            <geometry>
+                <sphere radius="${caster_wheel_offset_z*1.1}"/>
             </geometry>
             <material name="body_color"/>
@@ -80,14 +117,10 @@
             <material name="sensor_blue"/>
         </visual>
-        <collision>
-            <geometry>
-                <box size="0.1 0.1 0.1"/>
-            </geometry>
-        </collision>
     </link>
     <joint name="imu_joint" type="fixed">
-        <parent link="base_link"/>
+        <parent link="chassis_link"/>
         <child link="imu_link"/>
-        <origin xyz="0 0 0.04"/>
+        <!-- we place IMU between the wheels -->
+        <origin xyz="${wheel_offset_x} 0 0.04" rpy="0 0 0"/>
     </joint>
     <!-- gz model -m dragger -s imu_sensor -->
@@ -174,5 +207,5 @@
     <!-- LEFT WHEEL LINK -->
     <joint name="left_wheel_joint" type="continuous">
-        <parent link="base_link"/>
+        <parent link="chassis_link"/>
         <child link="left_wheel"/>
         <origin xyz="${wheel_offset_x} ${wheel_offset_y} 0" rpy="-${pi/2} 0 0" />
@@ -231,5 +264,5 @@
     <!-- RIGHT WHEEL LINK -->
     <joint name="right_wheel_joint" type="continuous">
-        <parent link="base_link"/>
+        <parent link="chassis_link"/>
         <child link="right_wheel"/>
         <origin xyz="${wheel_offset_x} ${-wheel_offset_y} 0" rpy="${pi/2} 0 0" />
@@ -288,5 +321,5 @@
     <!-- CASTER WHEELS LINKS -->
     <joint name="left_caster_wheel_joint" type="continuous">
-        <parent link="base_link"/>
+        <parent link="chassis_link"/>
         <child link="left_caster_wheel"/>
         <origin xyz="${caster_wheel_offset_x} ${caster_wheel_offset_y} ${caster_wheel_offset_z}" rpy="${pi/2} 0 0" />
@@ -321,10 +354,10 @@
             </surface>
         </collision>
-        <xacro:inertial_sphere mass="${caster_wheel_mass}" radius="${caster_wheel_radius}">
+        <xacro:inertial_cylinder mass="${caster_wheel_mass}" length="${caster_wheel_thickness}" radius="${caster_wheel_radius}">
             <origin xyz="0 0 0" rpy="0 0 0"/>
-        </xacro:inertial_sphere>
+        </xacro:inertial_cylinder>
     </link>
     <joint name="right_caster_wheel_joint" type="continuous">
-        <parent link="base_link"/>
+        <parent link="chassis_link"/>
         <child link="right_caster_wheel"/>
         <origin xyz="${caster_wheel_offset_x} ${-caster_wheel_offset_y} ${caster_wheel_offset_z}" rpy="${pi/2} 0 0" />
@@ -359,7 +392,7 @@
             </surface>
         </collision>
-        <xacro:inertial_sphere mass="${caster_wheel_mass}" radius="${caster_wheel_radius}">
+        <xacro:inertial_cylinder mass="${caster_wheel_mass}" length="${caster_wheel_thickness}" radius="${caster_wheel_radius}">
             <origin xyz="0 0 0" rpy="0 0 0"/>
-        </xacro:inertial_sphere>
+        </xacro:inertial_cylinder>
     </link>
 </robot>
