Commit message: Adjusted code for "frame_id" coming from sensors

File: description/camera.xacro (robot description, xacro)
@@ -34,6 +34,8 @@
         <sensor name='rgb_camera' type='camera'>
           <pose>0 0 0 0 0 0</pose>
-		  <always_on>true</always_on>
+		      <always_on>true</always_on>
           <topic>camera</topic>
+          <!-- future Gazebo versions might require "<frame_id>" here. Must reference an actual link in .xacro -->
+          <!-- see <optical_frame_id> below     <gz_frame_id>camera_link_optical</gz_frame_id> -->
           <update_rate>30</update_rate>
           <enable_metrics>false</enable_metrics>
@@ -77,5 +79,5 @@
               <env_texture_size>256</env_texture_size>
             </lens>
-            <optical_frame_id>camera_frame</optical_frame_id>
+            <optical_frame_id>camera_link_optical</optical_frame_id>
           </camera>
         </sensor>

File: description/depth_camera.xacro (robot description, xacro)
@@ -29,4 +29,6 @@
             <visualize>true</visualize>
             <update_rate>10</update_rate>
+            <!-- future Gazebo versions might require "<frame_id>" here. Must reference an actual link in .xacro -->
+            <gz_frame_id>depth_camera_link</gz_frame_id>
             <camera>
                 <horizontal_fov>1.089</horizontal_fov>

File: description/gps.xacro (robot description, xacro)
@@ -34,4 +34,6 @@
 			<always_on>true</always_on>
             <topic>navsat</topic>
+            <!-- future Gazebo versions might require "<frame_id>" here. Must reference an actual link in .xacro -->
+            <gz_frame_id>gps_link</gz_frame_id>
 			<pose> 0 0 0 0 0 0 </pose>
 			<visualize>false</visualize>

File: description/lidar.xacro (robot description, xacro)
@@ -34,10 +34,12 @@
     <!-- gz model -m dragger -s front_laser -->
     <gazebo reference="laser_frame">
-        <sensor name='front_laser' type='gpu_lidar'>
+        <!-- name must be "laser_frame", specifically for lasers. Must reference an actual link in .xacro -->
+        <sensor name='laser_frame' type='gpu_lidar'>
           <pose>0 0 0 0 0 0</pose>
           <always_on>1</always_on>
           <update_rate>10</update_rate>
           <topic>scan</topic>
-          <!-- frame_id>laser_frame</frame_id -->
+          <!-- future Gazebo versions might require "<frame_id>" here. Must reference an actual link in .xacro -->
+          <gz_frame_id>laser_frame</gz_frame_id>
           <ray>
             <scan>

File: description/robot_core.xacro (robot description, xacro)
@@ -7,5 +7,5 @@
     <xacro:property name="chassis_height" value="0.50"/>
     <xacro:property name="chassis_mass" value="30.0"/>
-    <xacro:property name="wheel_radius" value="0.192"/>
+    <xacro:property name="wheel_radius" value="0.177"/>
     <xacro:property name="wheel_thickness" value="0.09"/>
     <xacro:property name="wheel_mass" value="1.0"/>
@@ -126,7 +126,9 @@
     <!-- gz model -m dragger -s imu_sensor -->
     <gazebo reference="imu_link">
-        <sensor name="imu_sensor" type="imu">
+        <sensor name="imu_link" type="imu">
         <always_on>1</always_on>
         <topic>imu</topic>
+        <!-- future Gazebo versions might require "<frame_id>" here. Must reference an actual link in .xacro -->
+        <gz_frame_id>imu_link</gz_frame_id>
         <update_rate>250</update_rate>
             <imu>

Commit message: Adding "gz" prefix to Gazebo topics, playing with depth camera

File: description/camera.xacro (robot description, xacro)
@@ -31,16 +31,17 @@
     </link>
     <!-- gz model -m dragger -s rgb_camera -->
-	<gazebo reference="camera_link_optical">
+	  <gazebo reference="camera_link_optical">
         <sensor name='rgb_camera' type='camera'>
           <pose>0 0 0 0 0 0</pose>
 		      <always_on>true</always_on>
-          <topic>camera</topic>
+          <topic>gz_camera</topic>
           <!-- future Gazebo versions might require "<frame_id>" here. Must reference an actual link in .xacro -->
           <!-- see <optical_frame_id> below     <gz_frame_id>camera_link_optical</gz_frame_id> -->
-          <update_rate>30</update_rate>
+          <update_rate>10</update_rate>
+          <visualize>true</visualize>
           <enable_metrics>false</enable_metrics>
           <camera name='__default__'>
             <pose>0 0 0 0 0 0</pose>
-            <horizontal_fov>1.0469999999999999</horizontal_fov>
+            <horizontal_fov>1.047</horizontal_fov>
             <image>
               <width>320</width>
@@ -49,5 +50,5 @@
               <anti_aliasing>4</anti_aliasing>
             </image>
-            <camera_info_topic>__default__</camera_info_topic>
+            <camera_info_topic>gz_camera_info</camera_info_topic>
             <trigger_topic></trigger_topic>
             <triggered>false</triggered>
@@ -76,5 +77,5 @@
               <type>stereographic</type>
               <scale_to_hfov>true</scale_to_hfov>
-              <cutoff_angle>1.5707963267948966</cutoff_angle>
+              <cutoff_angle>${pi/2}</cutoff_angle>
               <env_texture_size>256</env_texture_size>
             </lens>

File: description/depth_camera.xacro (robot description, xacro)
@@ -1,8 +1,10 @@
 <?xml version="1.0"?>
 <robot xmlns:xacro="http://www.ros.org/wiki/xacro" >
+    <xacro:property name="depth_camera_offset_x" value="${chassis_length/2 - 0.04}"/>
+    <xacro:property name="depth_camera_offset_z" value="0.55"/>
     <joint name="depth_camera_joint" type="fixed">
         <parent link="chassis_link"/>
         <child link="depth_camera_link"/>
-        <origin xyz="0.305 0 0.08" rpy="0 0 0"/>
+        <origin xyz="${depth_camera_offset_x} 0 ${depth_camera_offset_z}" rpy="0 0.18 0"/>
     </joint>
     <link name="depth_camera_link">
@@ -11,5 +13,12 @@
                 <box size="0.010 0.03 0.03"/>
             </geometry>
-            <material name="red"/>
+            <material name="sensor_blue"/>
+        </visual>
+        <visual>
+            <origin xyz="0 0 -0.05"/>
+            <geometry>
+                <cylinder radius="0.002" length="0.1"/>
+            </geometry>
+            <material name="sensor_blue"/>
         </visual>
     </link>
@@ -17,24 +26,27 @@
         <parent link="depth_camera_link"/>
         <child link="depth_camera_link_optical"/>
-        <origin xyz="0 0 0" rpy="${-pi/2} 0 ${-pi/2}"/>
+        <origin xyz="0 0 0" rpy="0 0 0"/>
     </joint>
     <link name="depth_camera_link_optical">
     </link>
     <!-- gz model -m dragger -s depth_camera -->
-    <gazebo reference="depth_camera_link">
-        <!-- TODO: port to GZ Harmonic, add to gz_ros_brigde.yaml -->
-        <material>Gazebo/Red</material>
+    <gazebo reference="depth_camera_link_optical">
         <sensor name="depth_camera" type="depth">
             <pose> 0 0 0 0 0 0 </pose>
+		    <always_on>true</always_on>
+            <topic>gz_depth_camera</topic>
+            <update_rate>10</update_rate>
             <visualize>true</visualize>
-            <update_rate>10</update_rate>
             <!-- future Gazebo versions might require "<frame_id>" here. Must reference an actual link in .xacro -->
-            <gz_frame_id>depth_camera_link</gz_frame_id>
+            <gz_frame_id>depth_camera_link_optical</gz_frame_id>
+            <frame_id>depth_camera_link_optical</frame_id>
             <camera>
-                <horizontal_fov>1.089</horizontal_fov>
+                <horizontal_fov>1.047</horizontal_fov>
+                <!-- camera_info_topic>gz_depth_camera_info</camera_info_topic -->
                 <image>
+                    <width>320</width>
+                    <height>240</height>
+                    <!--format>RGB_INT8</format -->
                     <format>B8G8R8</format>
-                    <width>640</width>
-                    <height>480</height>
                 </image>
                 <clip>
@@ -43,9 +55,4 @@
                 </clip>
             </camera>
-            <plugin name="camera_controller" filename="libgazebo_ros_camera.so">
-                <frame_name>camera_link_optical</frame_name>
-                <min_depth>0.1</min_depth>
-                <max_depth>100.0</max_depth>
-            </plugin>
         </sensor>
     </gazebo>

File: description/gps.xacro (robot description, xacro)
@@ -36,5 +36,5 @@
 			<always_on>true</always_on>
             <!-- topic defined in .../config/gz_ros_bridge.yaml -->
-            <topic>navsat</topic>
+            <topic>gz_navsat/fix</topic>
             <!-- future Gazebo versions might require "<frame_id>" here. Must reference an actual link in .xacro -->
             <gz_frame_id>gps_link</gz_frame_id>

File: description/imu.xacro (robot description, xacro)
@@ -23,5 +23,5 @@
         <sensor name="imu_link" type="imu">
         <always_on>1</always_on>
-        <topic>imu</topic>
+        <topic>gz_imu/data</topic>
         <!-- future Gazebo versions might require "<frame_id>" here. Must reference an actual link in .xacro -->
         <gz_frame_id>imu_link</gz_frame_id>

File: description/lidar.xacro (robot description, xacro)
@@ -41,5 +41,5 @@
           <always_on>1</always_on>
           <update_rate>10</update_rate>
-          <topic>scan</topic>
+          <topic>gz_scan</topic>
           <!-- future Gazebo versions might require "<frame_id>" here. Must reference an actual link in .xacro -->
           <gz_frame_id>laser_frame</gz_frame_id>

File: description/magnetometer.xacro (robot description, xacro)
@@ -24,5 +24,5 @@
           <update_rate>100</update_rate>
           <visualize>true</visualize>
-          <topic>magnetometer</topic>
+          <topic>gz_magnetometer/data</topic>
           <!-- future Gazebo versions might require "<frame_id>" here. Must reference an actual link in .xacro -->
           <gz_frame_id>magnetometer_link</gz_frame_id>

File: description/robot.urdf.xacro (robot description, xacro)
@@ -44,7 +44,7 @@
     <xacro:include filename="magnetometer.xacro" />
     <xacro:include filename="lidar.xacro" />
+    <xacro:include filename="gps.xacro" />
     <xacro:include filename="camera.xacro" />
-    <!-- <xacro:include filename="depth_camera.xacro" /> -->
-    <xacro:include filename="gps.xacro" />
+    <xacro:include filename="depth_camera.xacro" />
     <!-- xacro:include filename="face.xacro" / -->
     <xacro:include filename="ros2_control.xacro" />

Commit message: WIP: plucky and sensors *.xacro files

File: description/camera.xacro (robot description, xacro)
@@ -1,6 +1,4 @@
 <?xml version="1.0"?>
 <robot xmlns:xacro="http://www.ros.org/wiki/xacro" >
-    <xacro:property name="camera_offset_x" value="${chassis_length/2 - 0.04}"/>
-    <xacro:property name="camera_offset_z" value="0.55"/>
     <joint name="camera_joint" type="fixed">
         <parent link="chassis_link"/>

File: description/gps.xacro (robot description, xacro)
@@ -1,10 +1,8 @@
 <?xml version="1.0"?>
 <robot xmlns:xacro="http://www.ros.org/wiki/xacro" >
-    <xacro:property name="gps_offset_x" value="0.05"/>
-    <xacro:property name="gps_offset_z" value="0.65"/>
     <joint name="gps_joint" type="fixed">
         <parent link="chassis_link"/>
         <child link="gps_link"/>
-        <origin xyz="${gps_offset_x} 0 ${gps_offset_z}" rpy="0 0 0"/>
+        <origin xyz="${gps_offset_x} ${gps_offset_y} ${gps_offset_z}" rpy="0 0 0"/>
     </joint>
     <link name="gps_link">

File: description/imu.xacro (robot description, xacro)
@@ -1,6 +1,4 @@
 <?xml version="1.0"?>
 <robot xmlns:xacro="http://www.ros.org/wiki/xacro" >
-    <xacro:property name="imu_offset_x" value="${wheel_offset_x}"/>
-    <xacro:property name="imu_offset_z" value="0.04"/>
     <!-- *********************** IMU SETUP *********************************  -->
     <!-- Each sensor must be attached to a link.                              -->

File: description/lidar.xacro (robot description, xacro)
@@ -1,6 +1,4 @@
 <?xml version="1.0"?>
 <robot xmlns:xacro="http://www.ros.org/wiki/xacro" >
-    <xacro:property name="laser_offset_x" value="${chassis_length/4 + 0.05}"/>
-    <xacro:property name="laser_offset_z" value="0.57"/>
     <!-- ********************* LIDAR SETUP *********************************  -->
     <!-- Each sensor must be attached to a link.                              -->

File: robots/dragger/description/robot.urdf.xacro (robot description, xacro)
@@ -10,8 +10,17 @@
     <xacro:include filename="../../../description/common_properties.xacro" />
     <xacro:include filename="robot_core.xacro" />
+    <xacro:property name="imu_offset_x" value="${wheel_offset_x}"/>
+    <xacro:property name="imu_offset_z" value="0.04"/>
     <xacro:include filename="../../../description/imu.xacro" />
     <xacro:include filename="../../../description/magnetometer.xacro" />
+    <xacro:property name="laser_offset_x" value="${chassis_length/4 + 0.05}"/>
+    <xacro:property name="laser_offset_z" value="0.57"/>
     <xacro:include filename="../../../description/lidar.xacro" />
+    <xacro:property name="gps_offset_x" value="0.05"/>
+    <xacro:property name="gps_offset_y" value="0.0"/>
+    <xacro:property name="gps_offset_z" value="0.65"/>
     <xacro:include filename="../../../description/gps.xacro" />
+    <xacro:property name="camera_offset_x" value="${chassis_length/2 - 0.04}"/>
+    <xacro:property name="camera_offset_z" value="0.55"/>
     <xacro:include filename="../../../description/camera.xacro" />
     <!-- xacro:include filename="../../../description/depth_camera.xacro" / -->

File: robots/plucky/description/robot.urdf.xacro (robot description, xacro)
@@ -10,8 +10,17 @@
     <xacro:include filename="../../../description/common_properties.xacro" />
     <xacro:include filename="robot_core.xacro" />
+    <xacro:property name="imu_offset_x" value="${wheel_offset_x}"/>
+    <xacro:property name="imu_offset_z" value="0.01"/>
     <xacro:include filename="../../../description/imu.xacro" />
     <xacro:include filename="../../../description/magnetometer.xacro" />
+    <xacro:property name="laser_offset_x" value="${wheel_offset_x}"/>
+    <xacro:property name="laser_offset_z" value="0.50"/>
     <xacro:include filename="../../../description/lidar.xacro" />
+    <xacro:property name="gps_offset_x" value="${wheel_offset_x}"/>
+    <xacro:property name="gps_offset_y" value="-0.16"/>
+    <xacro:property name="gps_offset_z" value="0.45"/>
     <xacro:include filename="../../../description/gps.xacro" />
+    <xacro:property name="camera_offset_x" value="${wheel_offset_x + 0.05}"/>
+    <xacro:property name="camera_offset_z" value="0.45"/>
     <xacro:include filename="../../../description/camera.xacro" />
     <!-- xacro:include filename="../../../description/depth_camera.xacro" / -->

File: robots/plucky/description/robot_core.xacro (robot description, xacro)
@@ -3,19 +3,20 @@
     <xacro:include filename="../../../description/inertial_macros.xacro"/>
 	<!-- Values corrected for Plucky robot -->
-    <xacro:property name="chassis_length" value="0.90"/>
-    <xacro:property name="chassis_width" value="0.40"/>
-    <xacro:property name="chassis_height" value="0.50"/>
-    <xacro:property name="chassis_mass" value="30.0"/>
+    <xacro:property name="chassis_length" value="0.48"/>
+    <xacro:property name="chassis_width" value="0.42"/>
+    <xacro:property name="chassis_height" value="0.45"/>
+    <xacro:property name="chassis_mass" value="10.0"/>
+    <xacro:property name="chassis_top_length" value="0.095"/>
     <xacro:property name="wheel_radius" value="0.192"/>
-    <xacro:property name="wheel_thickness" value="0.09"/>
+    <xacro:property name="wheel_thickness" value="0.045"/>
     <xacro:property name="wheel_mass" value="1.0"/>
     <xacro:property name="wheel_offset_x" value="${chassis_length/2 - wheel_radius - 0.01}"/>
-    <xacro:property name="wheel_offset_y" value="0.290"/>
+    <xacro:property name="wheel_offset_y" value="0.300"/>
     <xacro:property name="wheel_offset_z" value="0.01"/>
-    <xacro:property name="caster_wheel_radius" value="0.12"/>
-    <xacro:property name="caster_wheel_thickness" value="0.05"/>
+    <xacro:property name="caster_wheel_radius" value="0.05"/>
+    <xacro:property name="caster_wheel_thickness" value="0.02"/>
     <xacro:property name="caster_wheel_mass" value="0.3"/>
-    <xacro:property name="caster_wheel_offset_x" value="${-chassis_length/2 + caster_wheel_radius + 0.01}"/>
-    <xacro:property name="caster_wheel_offset_y" value="0.270"/>
+    <xacro:property name="caster_wheel_offset_x" value="${-chassis_length/2 - 0.08}"/>
+    <xacro:property name="caster_wheel_offset_y" value="0.175"/>
     <xacro:property name="caster_wheel_offset_z" value="${wheel_offset_z - wheel_radius + caster_wheel_radius}"/>
     <!-- we need the following because (unlike sim) real Dragger doesn't have a controller reporting caster's position -->
@@ -82,7 +83,7 @@
         </visual>
         <visual name="chassis_top_visual">
-            <origin xyz="${chassis_length*1/4} 0 ${chassis_height*3/4}"/>
-            <geometry>
-                <box size="${chassis_length*0.45} ${chassis_width*0.95} ${chassis_height/2}"/>
+            <origin xyz="${wheel_offset_x} 0 ${chassis_height*3/4}"/>
+            <geometry>
+                <box size="${chassis_top_length} ${chassis_width} ${chassis_height/2}"/>
             </geometry>
             <material name="body_color"/>
@@ -103,14 +104,14 @@
         </visual>
         <visual name="chassis_caster_joint_left">
-            <origin xyz="${caster_wheel_offset_x} ${chassis_width*0.52} ${caster_wheel_offset_z}" rpy="0 0 0"/>
-            <geometry>
-                <sphere radius="${caster_wheel_offset_z*1.1}"/>
+            <origin xyz="${caster_wheel_offset_x} ${caster_wheel_offset_y*0.9} ${caster_wheel_offset_z}" rpy="0 0 0"/>
+            <geometry>
+                <sphere radius="0.02"/>
             </geometry>
             <material name="body_color"/>
         </visual>
         <visual name="chassis_caster_joint_right">
-            <origin xyz="${caster_wheel_offset_x} ${-chassis_width*0.51} ${caster_wheel_offset_z}" rpy="0 0 0"/>
-            <geometry>
-                <sphere radius="${caster_wheel_offset_z*1.1}"/>
+            <origin xyz="${caster_wheel_offset_x} ${-caster_wheel_offset_y*0.9} ${caster_wheel_offset_z}" rpy="0 0 0"/>
+            <geometry>
+                <sphere radius="0.02"/>
             </geometry>
             <material name="body_color"/>
@@ -161,5 +162,5 @@
         <visual name="left_wheel_axis_visual">
             <geometry>
-                <cylinder radius="${wheel_radius*0.1}" length="${wheel_thickness*1.1}"/>
+                <cylinder radius="${wheel_radius*0.05}" length="${wheel_thickness*1.1}"/>
             </geometry>
             <material name="blue"/>
@@ -232,5 +233,5 @@
         <visual name="right_wheel_axis_visual">
             <geometry>
-                <cylinder radius="${wheel_radius*0.1}" length="${wheel_thickness*1.1}"/>
+                <cylinder radius="${wheel_radius*0.05}" length="${wheel_thickness*1.1}"/>
             </geometry>
             <material name="blue"/>

File: robots/sim/description/robot.urdf.xacro (robot description, xacro)
@@ -10,8 +10,17 @@
     <xacro:include filename="../../../description/common_properties.xacro" />
     <xacro:include filename="robot_core.xacro" />
+    <xacro:property name="imu_offset_x" value="${wheel_offset_x}"/>
+    <xacro:property name="imu_offset_z" value="0.04"/>
     <xacro:include filename="../../../description/imu.xacro" />
     <xacro:include filename="../../../description/magnetometer.xacro" />
+    <xacro:property name="laser_offset_x" value="${chassis_length/4 + 0.05}"/>
+    <xacro:property name="laser_offset_z" value="0.57"/>
     <xacro:include filename="../../../description/lidar.xacro" />
+    <xacro:property name="gps_offset_x" value="0.05"/>
+    <xacro:property name="gps_offset_y" value="0.0"/>
+    <xacro:property name="gps_offset_z" value="0.65"/>
     <xacro:include filename="../../../description/gps.xacro" />
+    <xacro:property name="camera_offset_x" value="${chassis_length/2 - 0.04}"/>
+    <xacro:property name="camera_offset_z" value="0.55"/>
     <xacro:include filename="../../../description/camera.xacro" />
     <!-- xacro:include filename="../../../description/depth_camera.xacro" / -->

File: robots/turtle/description/robot.urdf.xacro (robot description, xacro)
@@ -14,7 +14,5 @@
     <xacro:include filename="../../../description/common_properties.xacro" />
     <xacro:include filename="create_1.urdf.xacro" />
-    <!-- xacro:include filename="../../../description/imu.xacro" />
-    <xacro:include filename="../../../description/magnetometer.xacro" />
-    <xacro:include filename="../../../description/turtle_sensors.xacro" / -->
+    <!-- <xacro:include filename="../../../description/turtle_sensors.xacro" / -->
     <xacro:include filename="ros2_control.xacro" />
 </robot>
