Commit message: WIP: four sim sonars/lasers in place

File: description/sonars.xacro (robot description, xacro)
@@ -81,8 +81,49 @@
         </visual>
     </link>
+    <!-- gz model -m dragger -s sonar_F_R_frame -->
+    <gazebo reference="sonar_F_R_frame">
+        <!-- name must be "sonar_F_R_frame", specifically for sonars. Must reference an actual link in .xacro -->
+        <sensor name='sonar_F_R_frame' type='gpu_lidar'>
+          <pose>0 0 0 0 0 0</pose>
+          <always_on>1</always_on>
+          <!-- 6 Hz for LD14 - see "frequency" in dual_ekf_navsat_parameters.yaml -->
+          <update_rate>6</update_rate>
+          <topic>gz_sonar_F_R</topic>
+          <!-- future Gazebo versions might require "<frame_id>" here. Must reference an actual link in .xacro -->
+          <gz_frame_id>sonar_F_R_frame</gz_frame_id>
+          <frame_id>sonar_F_R_frame</frame_id>
+          <ray>
+            <scan>
+              <horizontal>
+                <samples>10</samples>
+                <resolution>1</resolution>
+                <min_angle>-${pi/40}</min_angle>
+                <max_angle>${pi/40}</max_angle>
+              </horizontal>
+              <vertical>
+                <samples>1</samples>
+                <resolution>1</resolution>
+                <min_angle>0.0</min_angle>
+                <max_angle>0.0</max_angle>
+              </vertical>
+            </scan>
+            <range>
+              <min>0.3</min>
+              <max>3.0</max>
+              <resolution>0.01</resolution>
+            </range>
+            <noise>
+              <type>gaussian</type>
+              <mean>0</mean>
+              <stddev>0.01</stddev>
+            </noise>
+          </ray>
+          <visualize>true</visualize>
+        </sensor>
+    </gazebo>
     <joint name="sonar_B_L_joint" type="fixed">
         <parent link="chassis_link"/>
         <child link="sonar_B_L_frame"/>
-        <origin xyz="${-sonars_offset_x} ${sonars_offset_y} ${sonars_offset_z}" rpy="0 0 0"/>
+        <origin xyz="${-sonars_offset_x} ${sonars_offset_y} ${sonars_offset_z}" rpy="0 0 ${pi}"/>
     </joint>
     <!-- the name "sonar_B_L_frame" should correspond to /scan topic header->frame_id as defined in *.launch.py -->
@@ -96,8 +137,49 @@
         </visual>
     </link>
+    <!-- gz model -m dragger -s sonar_B_R_frame -->
+    <gazebo reference="sonar_B_L_frame">
+        <!-- name must be "sonar_B_L_frame", specifically for sonars. Must reference an actual link in .xacro -->
+        <sensor name='sonar_B_L_frame' type='gpu_lidar'>
+          <pose>0 0 0 0 0 0</pose>
+          <always_on>1</always_on>
+          <!-- 6 Hz for LD14 - see "frequency" in dual_ekf_navsat_parameters.yaml -->
+          <update_rate>6</update_rate>
+          <topic>gz_sonar_B_L</topic>
+          <!-- future Gazebo versions might require "<frame_id>" here. Must reference an actual link in .xacro -->
+          <gz_frame_id>sonar_B_L_frame</gz_frame_id>
+          <frame_id>sonar_B_L_frame</frame_id>
+          <ray>
+            <scan>
+              <horizontal>
+                <samples>10</samples>
+                <resolution>1</resolution>
+                <min_angle>-${pi/40}</min_angle>
+                <max_angle>${pi/40}</max_angle>
+              </horizontal>
+              <vertical>
+                <samples>1</samples>
+                <resolution>1</resolution>
+                <min_angle>0.0</min_angle>
+                <max_angle>0.0</max_angle>
+              </vertical>
+            </scan>
+            <range>
+              <min>0.3</min>
+              <max>3.0</max>
+              <resolution>0.01</resolution>
+            </range>
+            <noise>
+              <type>gaussian</type>
+              <mean>0</mean>
+              <stddev>0.01</stddev>
+            </noise>
+          </ray>
+          <visualize>true</visualize>
+        </sensor>
+    </gazebo>
     <joint name="sonar_B_R_joint" type="fixed">
         <parent link="chassis_link"/>
         <child link="sonar_B_R_frame"/>
-        <origin xyz="${-sonars_offset_x} ${-sonars_offset_y} ${sonars_offset_z}" rpy="0 0 0"/>
+        <origin xyz="${-sonars_offset_x} ${-sonars_offset_y} ${sonars_offset_z}" rpy="0 0 ${pi}"/>
     </joint>
     <!-- the name "sonar_B_R_frame" should correspond to /scan topic header->frame_id as defined in *.launch.py -->
@@ -111,3 +193,44 @@
         </visual>
     </link>
+    <!-- gz model -m dragger -s sonar_B_R_frame -->
+    <gazebo reference="sonar_B_R_frame">
+        <!-- name must be "sonar_B_R_frame", specifically for sonars. Must reference an actual link in .xacro -->
+        <sensor name='sonar_B_R_frame' type='gpu_lidar'>
+          <pose>0 0 0 0 0 0</pose>
+          <always_on>1</always_on>
+          <!-- 6 Hz for LD14 - see "frequency" in dual_ekf_navsat_parameters.yaml -->
+          <update_rate>6</update_rate>
+          <topic>gz_sonar_B_R</topic>
+          <!-- future Gazebo versions might require "<frame_id>" here. Must reference an actual link in .xacro -->
+          <gz_frame_id>sonar_B_R_frame</gz_frame_id>
+          <frame_id>sonar_B_R_frame</frame_id>
+          <ray>
+            <scan>
+              <horizontal>
+                <samples>10</samples>
+                <resolution>1</resolution>
+                <min_angle>-${pi/40}</min_angle>
+                <max_angle>${pi/40}</max_angle>
+              </horizontal>
+              <vertical>
+                <samples>1</samples>
+                <resolution>1</resolution>
+                <min_angle>0.0</min_angle>
+                <max_angle>0.0</max_angle>
+              </vertical>
+            </scan>
+            <range>
+              <min>0.3</min>
+              <max>3.0</max>
+              <resolution>0.01</resolution>
+            </range>
+            <noise>
+              <type>gaussian</type>
+              <mean>0</mean>
+              <stddev>0.01</stddev>
+            </noise>
+          </ray>
+          <visualize>true</visualize>
+        </sensor>
+    </gazebo>
 </robot>

Commit message: WIP: angle offset for sonars

File: description/sonars.xacro (robot description, xacro)
@@ -10,8 +10,9 @@
              https://medium.com/@bytesrobotics/a-review-of-the-ros2-urdf-gazebo-sensor-91e947c633d7
      -->
+    <xacro:property name="sonars_angle_offset" value="${pi/20}"/>
     <joint name="sonar_F_L_joint" type="fixed">
         <parent link="chassis_link"/>
         <child link="sonar_F_L_frame"/>
-        <origin xyz="${sonars_offset_x} ${sonars_offset_y} ${sonars_offset_z}" rpy="0 0 0"/>
+        <origin xyz="${sonars_offset_x} ${sonars_offset_y} ${sonars_offset_z}" rpy="0 0 ${sonars_angle_offset}"/>
     </joint>
     <!-- the name "sonar_F_L_frame" should correspond to /scan topic header->frame_id as defined in *.launch.py -->
@@ -69,5 +70,5 @@
         <parent link="chassis_link"/>
         <child link="sonar_F_R_frame"/>
-        <origin xyz="${sonars_offset_x} ${-sonars_offset_y} ${sonars_offset_z}" rpy="0 0 0"/>
+        <origin xyz="${sonars_offset_x} ${-sonars_offset_y} ${sonars_offset_z}" rpy="0 0 ${-sonars_angle_offset}"/>
     </joint>
     <!-- the name "sonar_F_R_frame" should correspond to /scan topic header->frame_id as defined in *.launch.py -->
@@ -125,5 +126,5 @@
         <parent link="chassis_link"/>
         <child link="sonar_B_L_frame"/>
-        <origin xyz="${-sonars_offset_x} ${sonars_offset_y} ${sonars_offset_z}" rpy="0 0 ${pi}"/>
+        <origin xyz="${-sonars_offset_x} ${sonars_offset_y} ${sonars_offset_z}" rpy="0 0 ${pi-sonars_angle_offset}"/>
     </joint>
     <!-- the name "sonar_B_L_frame" should correspond to /scan topic header->frame_id as defined in *.launch.py -->
@@ -181,5 +182,5 @@
         <parent link="chassis_link"/>
         <child link="sonar_B_R_frame"/>
-        <origin xyz="${-sonars_offset_x} ${-sonars_offset_y} ${sonars_offset_z}" rpy="0 0 ${pi}"/>
+        <origin xyz="${-sonars_offset_x} ${-sonars_offset_y} ${sonars_offset_z}" rpy="0 0 ${pi+sonars_angle_offset}"/>
     </joint>
     <!-- the name "sonar_B_R_frame" should correspond to /scan topic header->frame_id as defined in *.launch.py -->
