Commit message: base footprint circle > rectangle

File: description/magnetometer.xacro (robot description, xacro)
@@ -1,6 +1,6 @@
 <?xml version="1.0"?>
 <robot xmlns:xacro="http://www.ros.org/wiki/xacro" >
-    <xacro:property name="magnetometer_offset_x" value="${wheel_offset_x}"/>
-    <xacro:property name="magnetometer_offset_z" value="0.03"/>
+    <xacro:property name="magnetometer_offset_x" value="0.0"/>
+    <xacro:property name="magnetometer_offset_z" value="0.01"/>
     <!-- ******************* MAGNETOMETER SETUP ****************************  -->
     <!-- Each sensor must be attached to a link.                              -->
@@ -9,5 +9,5 @@
         <child link="magnetometer_link"/>
         <!-- we place Magnetometer next to IMU between the wheels -->
-        <origin xyz="${wheel_offset_x} 0 ${magnetometer_offset_z}" rpy="0 0 0"/>
+        <origin xyz="0.0 0.0 0.01" rpy="0 0 0"/>
     </joint>
     <link name="magnetometer_link">

File: robots/stingray/description/robot_core.xacro (robot description, xacro)
@@ -12,4 +12,6 @@
     <xacro:property name="wheel_mass" value="0.058"/>
     <xacro:property name="wheel_offset" value="0.13"/>
+    <xacro:property name="wheel_separation" value="0.26"/>
+    <xacro:property name="caster_radius" value="0.028"/>
     <xacro:property name="wheel_offset_x" value="0.13"/>
     <xacro:property name="wheel_offset_y" value="0.0"/>
@@ -39,5 +41,5 @@
             <origin xyz="0 0 0"/>
             <geometry>
-                <sphere radius="0.005"/>
+                <box size="0.01 0.01 0.01"/>
             </geometry>
             <material name="red"/>
@@ -53,10 +55,9 @@
     <link name="base_footprint">
         <visual name="footprint_visual">
-            <origin xyz="0 0 0.0001"/>
-            <geometry>
-                <!-- box size="${wheel_offset_y * 2 + wheel_thickness} ${wheel_offset_y * 2 + wheel_thickness} 0.02"/ -->
-                <cylinder radius="${wheel_offset_y + wheel_thickness + 0.03}" length="0.01"/>
-            </geometry>
-            <material name="shadow_grey"/>
+            <origin xyz="-${chassis_offset + caster_radius} 0.0 0.0"/>
+            <geometry>
+                <box size="${chassis_length + (caster_radius * 2)} ${wheel_separation + wheel_thickness} 0.001"/>
+            </geometry>
+            <material name="gray"/>
         </visual>
      </link>
@@ -105,5 +106,5 @@
         <parent link="base_link"/>
         <child link="left_wheel_link"/>
-        <origin xyz="0.0 ${wheel_offset} 0.0" rpy="-${pi/2} 0.0 0.0"/>
+        <origin xyz="0.0 ${wheel_offset} 0.0" rpy="${pi/2} 0.0 0.0"/>
         <axis xyz="0 0 1"/>
     </joint>
