Commit message: GPS SG>JP, LIDAR color, Mag color

File: description/JP_lidar.xacro (robot description, xacro)
@@ -16,5 +16,5 @@
                 <cylinder radius="${lidar_radius}" length="${lidar_height}"/>
             </geometry>
-            <material name="red"/>
+            <material name="blue"/>
         </visual>
         <collision>
@@ -28,6 +28,6 @@
     </link>
     <gazebo reference="laser_frame">
-        <material>Gazebo/Red</material>
-	    <sensor name="laser_frame" type="gpu_lidar">
+        <material>Gazebo/Blue</material>
+    	    <sensor name="laser_frame" type="gpu_lidar">
             <pose> 0.0 0.0 0.0 0.0 0.0 0.0 </pose>
             <visualize>true</visualize>

File: description/common_properties.xacro (robot description, xacro)
@@ -29,4 +29,7 @@
         <color rgba="0.8 0.8 0.2 1"/>
     </material>
+    <material name="sensor_green">
+        <color rgba="0.0 0.8 0.0 1"/>
+    </material>
     <material name="body_color">
         <color rgba="0.6 0.5 0.2 0.85"/>

File: description/magnetometer.xacro (robot description, xacro)
@@ -16,5 +16,5 @@
                 <box size="0.01 0.01 0.01"/>
             </geometry>
-            <material name="sensor_yellow"/>
+            <material name="sensor_green"/>
         </visual>
     </link>

File: robots/stingray/description/robot.urdf.xacro (robot description, xacro)
@@ -17,8 +17,8 @@
     <xacro:property name="laser_offset_z" value="0.50"/>
     <xacro:include filename="../../../description/JP_lidar.xacro" />
-    <xacro:property name="gps_offset_x" value="${wheel_offset_x}"/>
-    <xacro:property name="gps_offset_y" value="-0.16"/>
-    <xacro:property name="gps_offset_z" value="0.45"/>
-    <xacro:include filename="../../../description/gps.xacro" />
+    <xacro:property name="gps_offset_x" value="0.0"/>
+    <xacro:property name="gps_offset_y" value="0.0"/>
+    <xacro:property name="gps_offset_z" value="0.02"/>
+    <xacro:include filename="../../../description/JP_gps.xacro" />
     <xacro:property name="camera_offset_x" value="${front_panel_offset}"/>
     <xacro:property name="camera_offset_z" value="0.01525"/>
