Commit message: camera mass inertial, chassis mass

File: description/JP_camera.xacro (robot description, xacro)
@@ -4,4 +4,5 @@
     <xacro:property name="camera_width" value="0.040"/>
     <xacro:property name="camera_depth" value="0.0016"/>
+    <xacro:property name="camera_mass" value="0.012"/>
     <xacro:property name="camera_lens_radius" value="0.009"/>
     <xacro:property name="camera_lens_length" value="0.0256"/>
@@ -25,4 +26,7 @@
             </geometry>
         </collision>
+        <xacro:inertial_box mass="${camera_mass}" x="${camera_depth}" y="${camera_width}" z="${camera_height}">
+            <origin xyz="0 0 0" rpy="0 0 0"/>
+        </xacro:inertial_box>
     </link>
     <joint name="camera_lens_joint" type="fixed">

File: description/JP_lidar.xacro (robot description, xacro)
@@ -1,5 +1,5 @@
 <?xml version="1.0"?>
 <robot xmlns:xacro="http://www.ros.org/wiki/xacro" >
-    <xacro:property name="lidar_mass" value="0.207"/>
+    <xacro:property name="lidar_mass" value="0.164"/>
     <xacro:property name="lidar_radius" value="0.03025"/>
     <xacro:property name="lidar_height" value="0.016"/>

File: robots/stingray/description/robot_core.xacro (robot description, xacro)
@@ -6,10 +6,16 @@
     <xacro:property name="chassis_width" value="0.228"/>
     <xacro:property name="chassis_height" value="0.081"/>
-    <xacro:property name="chassis_mass" value="0.98"/>
+    <xacro:property name="chassis_mass" value="2.466"/>
     <xacro:property name="chassis_offset" value="0.0455"/>
     <xacro:property name="front_panel_offset" value="0.090"/>
+    <!-- <xacro:property name="chassis_mass" value="${stingray_total_mass}-2*${wheel_mass}-${caster_mass}-${lidar_mass}"
+    - ${OTHER_COMPONENTS_TO_BE_DETERMINED}/> -->
+    <!-- <xacro:property name="stingray_total_mass" value="2.915"/> -->
+    <!-- <xacro:property name="wheel_motor_assembly" value="0.375"/> -->
+    <!-- <xacro:property name="battery_mass" value="0.765"/> -->
+    <!-- <xacro:property name="wheel_motor_assembly" value="0.375"/> -->
     <xacro:property name="wheel_radius" value="0.0615"/>
     <xacro:property name="wheel_thickness" value="0.02"/>
-    <xacro:property name="wheel_mass" value="0.058"/>
+    <xacro:property name="wheel_mass" value="2.63"/>
     <xacro:property name="wheel_offset_x" value="0.13"/>
     <xacro:property name="wheel_separation" value="0.26"/>

Commit message: camera collision, chassis inertial, grey>gray

File: description/JP_camera.xacro (robot description, xacro)
@@ -22,4 +22,5 @@
         </visual>
         <collision>
+            <origin xyz="0 0 0" rpy="0 ${-pi/2} 0"/>
             <geometry>
                 <box size="${camera_height} ${camera_width} ${camera_depth}"/>
@@ -43,4 +44,5 @@
         </visual>
         <collision>
+            <origin xyz="${camera_lens_length/2} 0.0 0.0" rpy="0.0 ${pi/2} 0.0"/>
             <geometry>
                 <cylinder radius="${camera_lens_radius}" length="${camera_lens_length}"/>

File: description/common_properties.xacro (robot description, xacro)
@@ -17,8 +17,10 @@
         <color rgba="0 0 1 1"/>
     </material>
-    <material name="grey">
+    <!-- <material name="grey"> -->
+    <material name="gray">
         <color rgba="0.5 0.5 0.5 1"/>
     </material>
-    <material name="shadow_grey">
+    <!-- <material name="shadow_grey"> -->
+    <material name="shadow_gray">
         <color rgba="0.3 0.3 0.3 0.5"/>
     </material>

File: robots/stingray/description/robot_core.xacro (robot description, xacro)
@@ -80,5 +80,6 @@
             <origin xyz="0.0 0.0 0.0" rpy="0.0 0.0 0.0"/>
             <geometry>
-                <mesh filename="model://meshes/Stingray.stl" scale="0.001 0.001 0.001"/>
+                <!-- <mesh filename="model://meshes/Stingray.stl" scale="0.001 0.001 0.001"/> -->
+                <mesh filename="package://articubot_one/assets/meshes/Stingray.stl" scale="0.001 0.001 0.001"/>
             </geometry>
             <material name="acrylic"/>
@@ -87,5 +88,4 @@
              <origin xyz="0.0 0.0 0.0" rpy="0.0 0.0 0.0"/>
             <geometry>
-                <!-- box size="${chassis_length} ${chassis_width} ${chassis_height}"/ -->
                 <mesh filename="package://articubot_one/assets/meshes/Stingray.stl" scale="0.001 0.001 0.001"/>
             </geometry>
@@ -101,5 +101,5 @@
         </collision>
         <xacro:inertial_box mass="${chassis_mass}" x="${chassis_length}" y="${chassis_width}" z="${chassis_height}">
-            <origin xyz="0.0 0.0 0.0" rpy="0.0 0.0 0.0"/>
+            <origin xyz="${-chassis_offset} 0.0 0.0" rpy="0.0 0.0 0.0"/>
         </xacro:inertial_box>
     </link>
