Commit message: lidar support rotated

File: description/lidar_support.xacro (robot description, xacro)
@@ -10,5 +10,5 @@
     <link name="lidar_support_link">
         <visual name="lidar_support__gz_visual">
-            <origin xyz="${lidar_support_offset_x} ${lidar_support_offset_y} ${lidar_support_offset_z}" rpy="0.0 0.0 0.0"/>
+            <origin xyz="${lidar_support_offset_x} ${lidar_support_offset_y} ${lidar_support_offset_z}" rpy="0.0 0.0 ${pi/2}"/>
             <geometry>
                 <mesh filename="model://meshes/LIDAR_support.stl" scale="0.001 0.001 0.001"/>
@@ -16,6 +16,6 @@
             <material name="black"/>
         </visual>
-        <visual name="chassis_rviz_visual">
-            <origin xyz="0.0 0.0 0.0" rpy="0.0 0.0 0.0"/>
+        <visual name="lidar_support_rviz_visual">
+            <origin xyz="0.0 0.0 0.0" rpy="0.0 0.0 ${pi/2}"/>
             <geometry>
                 <mesh filename="package://articubot_one/assets/meshes/LIDAR_support.stl" scale="0.001 0.001 0.001"/>

File: robots/stingray/description/robot_core.xacro (robot description, xacro)
@@ -60,5 +60,5 @@
                 <box size="${chassis_length + (caster_radius * 2)} ${wheel_separation + wheel_thickness} 0.001"/>
             </geometry>
-            <material name="gray"/>
+            <material name="shadow_gray"/>
         </visual>
      </link>

Commit message: lidar support Rviz origin

File: description/lidar_support.xacro (robot description, xacro)
@@ -17,5 +17,6 @@
         </visual>
         <visual name="lidar_support_rviz_visual">
-            <origin xyz="0.0 0.0 0.0" rpy="0.0 0.0 ${pi/2}"/>
+            <!-- <origin xyz="0.0 0.0 0.0" rpy="0.0 0.0 ${pi/2}"/> -->
+            <origin xyz="${lidar_support_offset_x} ${lidar_support_offset_y} ${lidar_support_offset_z}" rpy="0.0 0.0 ${pi/2}"/>
             <geometry>
                 <mesh filename="package://articubot_one/assets/meshes/LIDAR_support.stl" scale="0.001 0.001 0.001"/>

File: robots/stingray/description/robot.urdf.xacro (robot description, xacro)
@@ -19,5 +19,4 @@
     <xacro:property name="lidar_support_offset_x" value="0.0"/>
     <xacro:property name="lidar_support_offset_y" value="0.0"/>
-    <!-- <xacro:property name="lidar_support_offset_z" value="0.0"/> -->
     <xacro:property name="lidar_support_offset_z" value="${chassis_height/2 + 0.00375}"/>
     <xacro:include filename="../../../description/lidar_support.xacro" />
