Commit message: Battery voltage and capacity in SIM is configurable now

File: description/battery.xacro (robot description, xacro)
@@ -19,5 +19,8 @@
         <state_interface name="capacity"/>
         <state_interface name="percentage"/>
-    </sensor>
+        <state_interface name="power_supply_status"/>
+        <state_interface name="power_supply_health"/>
+        <state_interface name="present"/>
+   </sensor>
   </ros2_control>
   <gazebo>
@@ -25,13 +28,17 @@
       <!--Li-ion battery spec from LIR18650 datasheet-->
       <battery_name>lithium_battery</battery_name>
-      <voltage>12.592</voltage>
-      <open_circuit_voltage_constant_coef>12.592</open_circuit_voltage_constant_coef>
+      <voltage>${open_circuit_voltage}</voltage>
+      <open_circuit_voltage_constant_coef>${open_circuit_voltage}</open_circuit_voltage_constant_coef>
       <open_circuit_voltage_linear_coef>-2.0</open_circuit_voltage_linear_coef>
-      <initial_charge>2.4</initial_charge>
-      <capacity>2.5 </capacity>
+      <initial_charge>${battery_capacity * 0.9}</initial_charge>
+      <capacity>${battery_capacity}</capacity>
       <resistance>0.07</resistance>
       <power_load>6.6</power_load>
       <smooth_current_tau>2.0</smooth_current_tau>
-      <fix_issue_225>true</fix_issue_225>
+      <!-- if "fix_issue_225" is true, percentage is reported in 1..100 range which is wrong.
+               see https://github.com/gazebosim/gz-sim/issues/225 -->
+      <fix_issue_225>false</fix_issue_225>
+      <!-- https://github.com/gazebosim/gz-sim/pull/2696 -->
+      <invert_current_sign>true</invert_current_sign>
       <enable_recharge>true</enable_recharge>
       <!-- charging I = c / t, discharging I = P / V,

File: robots/dragger/description/robot.urdf.xacro (robot description, xacro)
@@ -28,4 +28,6 @@
     <xacro:property name="camera_offset_z" value="0.55"/>
     <xacro:include filename="../../../description/camera.xacro" />
+    <xacro:property name="open_circuit_voltage" value="12.592"/>
+    <xacro:property name="battery_capacity" value="50.0"/>
     <xacro:include filename="../../../description/battery.xacro" />
     <!-- xacro:include filename="../../../description/depth_camera.xacro" / -->

File: robots/plucky/description/robot.urdf.xacro (robot description, xacro)
@@ -28,4 +28,6 @@
     <xacro:property name="camera_offset_z" value="0.45"/>
     <xacro:include filename="../../../description/camera.xacro" />
+    <xacro:property name="open_circuit_voltage" value="12.592"/>
+    <xacro:property name="battery_capacity" value="20.0"/>
     <xacro:include filename="../../../description/battery.xacro" />
     <!-- xacro:include filename="../../../description/depth_camera.xacro" / -->

File: robots/turtle/description/robot.urdf.xacro (robot description, xacro)
@@ -15,4 +15,6 @@
     <xacro:include filename="create_1.urdf.xacro" />
     <xacro:include filename="ros2_control.xacro" />
+    <xacro:property name="open_circuit_voltage" value="14.0"/>
+    <xacro:property name="battery_capacity" value="2.5"/>
     <xacro:include filename="../../../description/battery.xacro" />
 </robot>

Commit message: WIP: Seggy URDF - sensors

File: description/battery.xacro (robot description, xacro)
@@ -9,4 +9,6 @@
       Note: This is generic SIM battery. Copy to robots/<robot_model>/description/. and customize.
             Modify robot.urdf.xacro to include the customized version.
+      parameters: open_circuit_voltage
+                  battery_capacity
   -->
   <ros2_control name="BatteryState" type="diffdrive_arduino/DiffDriveArduino">

File: description/camera.xacro (robot description, xacro)
@@ -1,4 +1,6 @@
 <?xml version="1.0"?>
 <robot xmlns:xacro="http://www.ros.org/wiki/xacro" >
+    <!-- parameters: camera_offset_x
+                     camera_offset_z -->
     <joint name="camera_joint" type="fixed">
         <parent link="chassis_link"/>

File: description/depth_camera.xacro (robot description, xacro)
@@ -1,6 +1,6 @@
 <?xml version="1.0"?>
 <robot xmlns:xacro="http://www.ros.org/wiki/xacro" >
-    <xacro:property name="depth_camera_offset_x" value="${chassis_length/2 - 0.06}"/>
-    <xacro:property name="depth_camera_offset_z" value="0.58"/>
+    <!-- parameters: depth_camera_offset_x
+                     depth_camera_offset_z -->
     <joint name="depth_camera_joint" type="fixed">
         <parent link="chassis_link"/>
@@ -9,16 +9,37 @@
     </joint>
     <link name="depth_camera_link">
-        <visual>
+        <visual name ="depth_camera_visual_body">
             <geometry>
-                <box size="0.010 0.03 0.03"/>
+                <box size="0.020 0.095 0.030"/>
             </geometry>
             <material name="sensor_blue"/>
         </visual>
-        <visual>
+        <visual name="depth_camera_visual_lens_1">
+            <origin xyz="0.010 0 0.006" rpy="0 ${pi/2} 0"/>
+            <geometry>
+                <cylinder radius="0.005" length="0.002"/>
+            </geometry>
+            <material name="body_color"/>
+        </visual>
+        <visual name="depth_camera_visual_lens_2">
+            <origin xyz="0.010 0.040 0.006" rpy="0 ${pi/2} 0"/>
+            <geometry>
+                <cylinder radius="0.005" length="0.002"/>
+            </geometry>
+            <material name="body_color"/>
+        </visual>
+        <visual name="depth_camera_visual_lens_3">
+            <origin xyz="0.010 -0.040 0.006" rpy="0 ${pi/2} 0"/>
+            <geometry>
+                <cylinder radius="0.005" length="0.002"/>
+            </geometry>
+            <material name="body_color"/>
+        </visual>
+        <visual name="depth_camera_mounting_arm">
             <origin xyz="0 0 -0.05"/>
             <geometry>
-                <cylinder radius="0.002" length="0.1"/>
+                <cylinder radius="0.005" length="0.1"/>
             </geometry>
-            <material name="sensor_blue"/>
+            <material name="body_color"/>
         </visual>
     </link>

File: description/imu.xacro (robot description, xacro)
@@ -3,4 +3,7 @@
     <!-- *********************** IMU SETUP *********************************  -->
     <!-- Each sensor must be attached to a link.                              -->
+    <!-- parameters: imu_offset_x
+                     imu_offset_z
+                     imu_visual_size -->
     <joint name="imu_joint" type="fixed">
         <parent link="chassis_link"/>

File: description/lidar.xacro (robot description, xacro)
@@ -3,23 +3,36 @@
     <!-- ********************* LIDAR SETUP *********************************  -->
     <!-- Each sensor must be attached to a link.                              -->
+    <xacro:arg name="lidar_offset_x" default="0"/>
+    <xacro:arg name="lidar_offset_z" default="0"/>
+    <xacro:arg name="lidar_min_angle" default="-3.14159"/>
+    <xacro:arg name="lidar_max_angle" default="3.14159"/>
+    <xacro:arg name="lidar_base_length" default="0.003"/>
+    <xacro:property name="_lidar_base_length" value="$(arg lidar_base_length)"/>
     <joint name="laser_joint" type="fixed">
         <parent link="chassis_link"/>
         <child link="laser_frame"/>
-        <origin xyz="${laser_offset_x} 0 ${laser_offset_z}" rpy="0 0 0"/>
+        <origin xyz="$(arg lidar_offset_x) 0 $(arg lidar_offset_z)" rpy="0 0 0"/>
     </joint>
     <!-- the name "laser_frame" should correspond to /scan topic header->frame_id as defined in *.launch.py -->
     <link name="laser_frame">
-        <visual>
+        <visual name="lidar_visual_scanner">
             <geometry>
-                <cylinder radius="0.05" length="0.04"/>
+                <cylinder radius="0.03" length="0.02"/>
             </geometry>
             <material name="sensor_blue"/>
         </visual>
-        <visual>
-            <origin xyz="0 0 -0.05"/>
+        <visual name="lidar_visual_motor">
+            <origin xyz="0.03 0 -0.01"/>
             <geometry>
-                <cylinder radius="0.03" length="0.1"/>
+                <cylinder radius="0.012" length="0.01"/>
             </geometry>
             <material name="sensor_blue"/>
+        </visual>
+        <visual name="lidar_visual_base">
+            <origin xyz="0 0 -${_lidar_base_length/2+0.01}"/>
+            <geometry>
+                <cylinder radius="0.02" length="${_lidar_base_length}"/>
+            </geometry>
+            <material name="body_color"/>
         </visual>
         <collision>
@@ -49,12 +62,12 @@
                 <samples>360</samples>
                 <resolution>1</resolution>
-                <min_angle>-${pi}</min_angle>
-                <max_angle>${pi}</max_angle>
+                <min_angle>$(arg lidar_min_angle)</min_angle>
+                <max_angle>$(arg lidar_max_angle)</max_angle>
               </horizontal>
               <vertical>
                 <samples>1</samples>
                 <resolution>1</resolution>
-                <min_angle>0.0</min_angle>
-                <max_angle>0.0</max_angle>
+                <min_angle>0</min_angle>
+                <max_angle>0</max_angle>
               </vertical>
             </scan>

File: description/magnetometer.xacro (robot description, xacro)
@@ -1,9 +1,10 @@
 <?xml version="1.0"?>
 <robot xmlns:xacro="http://www.ros.org/wiki/xacro" >
-    <xacro:property name="magnetometer_offset_x" value="${wheel_offset_x}"/>
-    <xacro:property name="magnetometer_offset_z" value="0.03"/>
     <!-- ******************* MAGNETOMETER SETUP ********************************  -->
-    <!-- we are using IMU parameters here, as magnetometer is usually part of IMU -->
     <!-- Each sensor must be attached to a link.                                  -->
+    <!-- we are using IMU parameters here, as magnetometer is usually part of IMU:
+        parameters: imu_offset_x
+                     imu_offset_z
+                     imu_visual_size -->
     <joint name="magnetometer_joint" type="fixed">
         <parent link="chassis_link"/>

File: robots/seggy/description/robot.urdf.xacro (robot description, xacro)
@@ -10,17 +10,20 @@
     <xacro:include filename="../../../description/common_properties.xacro" />
     <xacro:include filename="robot_core.xacro" />
-    <xacro:property name="imu_offset_x" value="${wheel_offset_x + 0.09}"/>
-    <xacro:property name="imu_offset_z" value="0.1"/>
+    <xacro:property name="imu_offset_x" value="${wheel_offset_x - 0.0}"/>
+    <xacro:property name="imu_offset_z" value="${chassis_top_offset + 0.01}"/>
     <xacro:property name="imu_visual_size" value="0.01"/>
     <xacro:include filename="../../../description/imu.xacro" />
-    <xacro:include filename="../../../description/magnetometer.xacro" />
-    <xacro:property name="laser_offset_x" value="${wheel_offset_x + 0.05}"/>
-    <xacro:property name="laser_offset_z" value="0.27"/>
+    <!-- using arguments here, as that allows overriding default values -->
+    <xacro:arg name="lidar_offset_x" default="${wheel_offset_x + 0.05}"/>
+    <xacro:arg name="lidar_offset_z" default="0.27"/>
+    <xacro:arg name="lidar_min_angle" default="-${pi * 0.95}"/>
+    <xacro:arg name="lidar_max_angle" default="${pi * 0.95}"/>
+    <!-- xacro:arg name="lidar_base_length" default="0.04"/ -->
     <xacro:include filename="../../../description/lidar.xacro" />
     <xacro:property name="open_circuit_voltage" value="12.592"/>
     <xacro:property name="battery_capacity" value="20.0"/>
     <xacro:include filename="../../../description/battery.xacro" />
-    <xacro:property name="depth_camera_offset_x" value="${wheel_offset_x}"/>
-    <xacro:property name="depth_camera_offset_z" value="${chassis_top_offset + 0.12}"/>
+    <xacro:property name="depth_camera_offset_x" value="${wheel_offset_x + 0.03}"/>
+    <xacro:property name="depth_camera_offset_z" value="${chassis_top_offset + 0.11}"/>
     <xacro:include filename="../../../description/depth_camera.xacro"/>
     <xacro:unless value="$(arg sim_mode)">
