Commit message: Using new Lyrical BatteryState broadcaster and interfaces

File: description/battery.xacro (robot description, xacro)
@@ -12,18 +12,19 @@
                   battery_capacity
   -->
-  <ros2_control name="BatteryState" type="diffdrive_arduino/DiffDriveArduino">
-    <sensor name="main_battery">
-        <!-- See diffdrive_arduino/src/diffdrive_arduino.cpp export_state_interfaces()-->
-        <state_interface name="voltage"/>
-        <state_interface name="temperature"/>
-        <state_interface name="current"/>
-        <state_interface name="charge"/>
-        <state_interface name="capacity"/>
-        <state_interface name="percentage"/>
-        <state_interface name="power_supply_status"/>
-        <state_interface name="power_supply_health"/>
-        <state_interface name="present"/>
-   </sensor>
-  </ros2_control>
+  <!-- Included inside the real drive system's ros2_control element. Gazebo
+       publishes BatteryState through ros_gz_bridge instead of this broadcaster. -->
+  <xacro:macro name="battery_state_interfaces" params="battery_name:=main_battery">
+    <sensor name="${battery_name}">
+      <state_interface name="battery_voltage"/>
+      <state_interface name="battery_temperature"/>
+      <state_interface name="battery_current"/>
+      <state_interface name="battery_charge"/>
+      <state_interface name="battery_percentage"/>
+      <state_interface name="battery_power_supply_status"/>
+      <state_interface name="battery_power_supply_health"/>
+      <state_interface name="battery_present" data_type="bool"/>
+    </sensor>
+  </xacro:macro>
+  <xacro:if value="$(arg sim_mode)">
   <gazebo>
     <plugin name="gz::sim::systems::LinearBatteryPlugin" filename="gz-sim-linearbatteryplugin-system">
@@ -54,3 +55,4 @@
     </plugin>
   </gazebo>
+  </xacro:if>
 </robot>

File: robots/dragger/description/ros2_control.xacro (robot description, xacro)
@@ -74,4 +74,7 @@
             </joint>
         </xacro:if>
+        <xacro:unless value="$(arg sim_mode)">
+            <xacro:battery_state_interfaces battery_name="main_battery"/>
+        </xacro:unless>
     </ros2_control>
     <gazebo>

File: robots/fido/description/ros2_control.xacro (robot description, xacro)
@@ -49,4 +49,7 @@
             </joint>
         </xacro:if>
+        <xacro:unless value="$(arg sim_mode)">
+            <xacro:battery_state_interfaces battery_name="main_battery"/>
+        </xacro:unless>
     </ros2_control>
     <gazebo>

File: robots/plucky/description/ros2_control.xacro (robot description, xacro)
@@ -46,4 +46,7 @@
             </joint>
         </xacro:if>
+        <xacro:unless value="$(arg sim_mode)">
+            <xacro:battery_state_interfaces battery_name="main_battery"/>
+        </xacro:unless>
     </ros2_control>
     <gazebo>

File: robots/seggy/description/ros2_control.xacro (robot description, xacro)
@@ -49,4 +49,7 @@
             </joint>
         </xacro:if>
+        <xacro:unless value="$(arg sim_mode)">
+            <xacro:battery_state_interfaces battery_name="main_battery"/>
+        </xacro:unless>
     </ros2_control>
     <gazebo>
