Commit message: Trying Depth Camera SIM
strange orientation, cannot be fixed by tweaking rpy

File: description/depth_camera.xacro (robot description, xacro)
@@ -1,10 +1,10 @@
 <?xml version="1.0"?>
 <robot xmlns:xacro="http://www.ros.org/wiki/xacro" >
-    <xacro:property name="depth_camera_offset_x" value="${chassis_length/2 - 0.04}"/>
-    <xacro:property name="depth_camera_offset_z" value="0.55"/>
+    <xacro:property name="depth_camera_offset_x" value="${chassis_length/2 - 0.06}"/>
+    <xacro:property name="depth_camera_offset_z" value="0.58"/>
     <joint name="depth_camera_joint" type="fixed">
         <parent link="chassis_link"/>
         <child link="depth_camera_link"/>
-        <origin xyz="${depth_camera_offset_x} 0 ${depth_camera_offset_z}" rpy="0 0.18 0"/>
+        <origin xyz="${depth_camera_offset_x} 0 ${depth_camera_offset_z}" rpy="0 0 0"/>
     </joint>
     <link name="depth_camera_link">
@@ -24,35 +24,65 @@
     </link>
     <joint name="depth_camera_optical_joint" type="fixed">
-        <parent link="depth_camera_link"/>
+        <!-- parent link="depth_camera_link"/ -->
+        <parent link="chassis_link"/>
         <child link="depth_camera_link_optical"/>
-        <origin xyz="0 0 0" rpy="0 0 0"/>
+        <!-- origin xyz="0 0 0" rpy="0 0 0"/ -->
+        <origin xyz="${depth_camera_offset_x} 0 ${depth_camera_offset_z}" rpy="0 0 0"/>
     </joint>
     <link name="depth_camera_link_optical">
     </link>
     <!-- gz model -m dragger -s depth_camera -->
-    <gazebo reference="depth_camera_link_optical">
-        <sensor name="depth_camera" type="depth">
-            <pose> 0 0 0 0 0 0 </pose>
-		    <always_on>true</always_on>
-            <topic>gz_depth_camera</topic>
-            <update_rate>10</update_rate>
-            <visualize>true</visualize>
-            <!-- future Gazebo versions might require "<frame_id>" here. Must reference an actual link in .xacro -->
-            <gz_frame_id>depth_camera_link_optical</gz_frame_id>
-            <frame_id>depth_camera_link_optical</frame_id>
-            <camera>
-                <horizontal_fov>1.047</horizontal_fov>
-                <!-- camera_info_topic>gz_depth_camera_info</camera_info_topic -->
-                <image>
-                    <width>320</width>
-                    <height>240</height>
-                    <!--format>RGB_INT8</format -->
-                    <format>B8G8R8</format>
-                </image>
-                <clip>
-                    <near>0.05</near>
-                    <far>8.0</far>
-                </clip>
-            </camera>
+	  <gazebo reference="depth_camera_link">
+        <sensor name='depth_camera' type='depth'>
+          <pose>0 0 0 0 0 0</pose>
+		      <always_on>true</always_on>
+          <topic>gz_depth_camera</topic>
+          <!-- future Gazebo versions might require "<frame_id>" here. Must reference an actual link in .xacro -->
+          <!-- see <optical_frame_id> below     <gz_frame_id>depth_camera_link_optical</gz_frame_id> -->
+          <update_rate>10</update_rate>
+          <visualize>true</visualize>
+          <enable_metrics>false</enable_metrics>
+          <camera name='__default__'>
+            <pose>0 0 0 0 0 0</pose>
+            <horizontal_fov>1.047</horizontal_fov>
+            <image>
+              <width>320</width>
+              <height>240</height>
+              <!--format>RGB_INT8</format -->
+              <format>B8G8R8</format>
+              <anti_aliasing>4</anti_aliasing>
+            </image>
+            <camera_info_topic>gz_depth_camera_info</camera_info_topic>
+            <trigger_topic></trigger_topic>
+            <triggered>false</triggered>
+            <clip>
+              <near>0.1</near>
+              <far>8</far>
+            </clip>
+            <save enabled='false'>
+              <path>__default__</path>
+            </save>
+            <visibility_mask>4294967295</visibility_mask>
+            <noise>
+              <type>none</type>
+              <mean>0</mean>
+              <stddev>0</stddev>
+            </noise>
+            <distortion>
+              <k1>0</k1>
+              <k2>0</k2>
+              <k3>0</k3>
+              <p1>0</p1>
+              <p2>0</p2>
+              <center>0.5 0.5</center>
+            </distortion>
+            <lens>
+              <type>stereographic</type>
+              <scale_to_hfov>true</scale_to_hfov>
+              <cutoff_angle>${pi/2}</cutoff_angle>
+              <env_texture_size>256</env_texture_size>
+            </lens>
+            <optical_frame_id>depth_camera_link_optical</optical_frame_id>
+          </camera>
         </sensor>
     </gazebo>

File: description/robot.urdf.xacro (robot description, xacro)
@@ -46,5 +46,5 @@
     <xacro:include filename="gps.xacro" />
     <xacro:include filename="camera.xacro" />
-    <xacro:include filename="depth_camera.xacro" />
+    <!-- xacro:include filename="depth_camera.xacro" / -->
     <!-- xacro:include filename="face.xacro" / -->
     <xacro:include filename="ros2_control.xacro" />

Commit message: OAK-D for Plucky

File: description/depth_camera.xacro (robot description, xacro)
@@ -30,6 +30,9 @@
         <origin xyz="${depth_camera_offset_x} 0 ${depth_camera_offset_z}" rpy="0 0 0"/>
     </joint>
-    <link name="depth_camera_link_optical">
-    </link>
+    <xacro:if value="$(arg sim_mode)">
+      <!-- OAK-D depthai_descr.urdf.xacro generates its own "parent_frame", in our case we want it to be "depth_camera_link_optical" -->
+      <link name="depth_camera_link_optical">
+      </link>
+    </xacro:if>
     <!-- gz model -m dragger -s depth_camera -->
 	  <gazebo reference="depth_camera_link">

File: robots/plucky/description/robot.urdf.xacro (robot description, xacro)
@@ -32,6 +32,11 @@
     <xacro:property name="battery_capacity" value="20.0"/>
     <xacro:include filename="../../../description/battery.xacro" />
-    <!-- xacro:include filename="../../../description/depth_camera.xacro" / -->
-    <!-- xacro:include filename="../../../description/face.xacro" / -->
+    <xacro:property name="depth_camera_offset_x" value="${wheel_offset_x}"/>
+    <xacro:property name="depth_camera_offset_z" value="0.45"/>
+    <xacro:include filename="../../../description/depth_camera.xacro"/>
+    <xacro:unless value="$(arg sim_mode)">
+        <xacro:arg name="parent_frame" default="depth_camera_link_optical" />
+        <xacro:include filename="$(find depthai_descriptions)/urdf/depthai_descr.urdf.xacro"/>
+    </xacro:unless>
     <xacro:include filename="ros2_control.xacro" />
 </robot>

Commit message: Dev to Main merge - new Seggy robot, many small adjustments, all sims work (#5) - squashed merge
* Dragger's nav2_params.yaml updated from Plucky's

* Let action_server_result_timeout be default

* Update nav2_params.yaml

Turtle params

* Update dragger.launch.py

LD-19P has 230400 baud rate and "LDLiDAR_LD14P" setting works for LD-19P LIDAR

* Dragger LIDAR: added min_intensity; Nav2: removed range_sensor_layer from global costmap

* Added 'do_filtering' and "do_triplets to dragger.launch.py

* Update dual_ekf_navsat_params.yaml

Added headers to covariances for better understanding of their meaning

* Update dual_ekf_navsat_params.yaml

Using https://github.com/cra-ros-pkg/robot_localization/blob/ros2/params/dual_ekf_navsat_example.yaml

* Update dragger.launch.py

For now, NearFilter doesn't work for LD-19 LIDAR

* OAK-D for Plucky

* Update dual_ekf_navsat_params.yaml

GPS localization works in sim very well

* Update dual_ekf_navsat_params.yaml

* Dragger parameters adjusted

* Adjusted Nav2 parameters for Dragger

* Create oakd.launch.py

* Created robots/seggy folder, cloned from Plucky, did all renaming

* Seggy: removed navsat/GPS, sonars

* Actual values for Seggy - wheels, tics/rev, acceleration limits

* Update controllers.yaml

* Update ros2_control.xacro

* Adjusted rates and frequencies for Nav2, ekf2 and controllers. Ignore compass in IMU

* Update seggy.launch.py

* WIP: Seggy URDF

* WIP: Seggy URDF

* WIP: Seggy URDF - sensors

* Plucky and Dragger URDFs adjusted to latest parameters changes

* Using namespace='' everywhere

* Update nav2_params.yaml

* Update seggy_sim.launch.py

* Using /odometry/local instead of /diff_cont/odom in Nav2

* Update nav2_params.yaml

Adjusted footprint

* Adjusted robot_radius, removed footprint. WIP: remapping for controller components

* WIP: trying proper remappings in controller_manager

* Update seggy.launch.py

* Final working version of remappings in controller_manager components

* Update seggy_sim.launch.py

* Parameter replaced: diff_cont/odom -> odometry/local in launch files

* consider_footprint - setting to false, used to work with "true" before Oct 2025

* Update seggy_sim_nav.launch.py

'odom_topic': 'odometry/local', using composition

* Update controllers.yaml

velocity_limits adjusted for Seggy robot

* Update main.rviz

* Update seggy_sim.launch.py

* Merged recent Seggy changes into Plucky and Dragger launch files

* Merged latest Seggy nav2 parameters into Plucky and Dragger's

* Merged recent changes from Seggy to Turtle launch files

* Update turtle_nav.launch.py

* Update nav2_params.yaml

* Update turtle_nav.launch.py

File: description/depth_camera.xacro (robot description, xacro)
@@ -1,6 +1,6 @@
 <?xml version="1.0"?>
 <robot xmlns:xacro="http://www.ros.org/wiki/xacro" >
-    <xacro:property name="depth_camera_offset_x" value="${chassis_length/2 - 0.06}"/>
-    <xacro:property name="depth_camera_offset_z" value="0.58"/>
+    <!-- parameters: depth_camera_offset_x
+                     depth_camera_offset_z -->
     <joint name="depth_camera_joint" type="fixed">
         <parent link="chassis_link"/>
@@ -9,16 +9,37 @@
     </joint>
     <link name="depth_camera_link">
-        <visual>
+        <visual name ="depth_camera_visual_body">
             <geometry>
-                <box size="0.010 0.03 0.03"/>
+                <box size="0.020 0.095 0.030"/>
             </geometry>
             <material name="sensor_blue"/>
         </visual>
-        <visual>
+        <visual name="depth_camera_visual_lens_1">
+            <origin xyz="0.010 0 0.006" rpy="0 ${pi/2} 0"/>
+            <geometry>
+                <cylinder radius="0.005" length="0.002"/>
+            </geometry>
+            <material name="body_color"/>
+        </visual>
+        <visual name="depth_camera_visual_lens_2">
+            <origin xyz="0.010 0.040 0.006" rpy="0 ${pi/2} 0"/>
+            <geometry>
+                <cylinder radius="0.005" length="0.002"/>
+            </geometry>
+            <material name="body_color"/>
+        </visual>
+        <visual name="depth_camera_visual_lens_3">
+            <origin xyz="0.010 -0.040 0.006" rpy="0 ${pi/2} 0"/>
+            <geometry>
+                <cylinder radius="0.005" length="0.002"/>
+            </geometry>
+            <material name="body_color"/>
+        </visual>
+        <visual name="depth_camera_mounting_arm">
             <origin xyz="0 0 -0.05"/>
             <geometry>
-                <cylinder radius="0.002" length="0.1"/>
+                <cylinder radius="0.005" length="0.1"/>
             </geometry>
-            <material name="sensor_blue"/>
+            <material name="body_color"/>
         </visual>
     </link>
@@ -30,6 +51,9 @@
         <origin xyz="${depth_camera_offset_x} 0 ${depth_camera_offset_z}" rpy="0 0 0"/>
     </joint>
-    <link name="depth_camera_link_optical">
-    </link>
+    <xacro:if value="$(arg sim_mode)">
+      <!-- OAK-D depthai_descr.urdf.xacro generates its own "parent_frame", in our case we want it to be "depth_camera_link_optical" -->
+      <link name="depth_camera_link_optical">
+      </link>
+    </xacro:if>
     <!-- gz model -m dragger -s depth_camera -->
 	  <gazebo reference="depth_camera_link">

File: robots/plucky/description/robot.urdf.xacro (robot description, xacro)
@@ -15,6 +15,8 @@
     <xacro:include filename="../../../description/imu.xacro" />
     <xacro:include filename="../../../description/magnetometer.xacro" />
-    <xacro:property name="laser_offset_x" value="${wheel_offset_x}"/>
-    <xacro:property name="laser_offset_z" value="0.50"/>
+    <!-- using arguments here, as that allows overriding default values -->
+    <xacro:arg name="lidar_offset_x" default="${wheel_offset_x}"/>
+    <xacro:arg name="lidar_offset_z" default="0.47"/>
+    <xacro:arg name="lidar_base_length" default="0.01"/>
     <xacro:include filename="../../../description/lidar.xacro" />
     <xacro:property name="sonars_offset_x" value="${chassis_length/2 + 0.005}"/>
@@ -26,12 +28,17 @@
     <xacro:property name="gps_offset_z" value="0.45"/>
     <xacro:include filename="../../../description/gps.xacro" />
-    <xacro:property name="camera_offset_x" value="${wheel_offset_x + 0.05}"/>
-    <xacro:property name="camera_offset_z" value="0.45"/>
+    <xacro:property name="camera_offset_x" value="${wheel_offset_x + 0.1}"/>
+    <xacro:property name="camera_offset_z" value="0.25"/>
     <xacro:include filename="../../../description/camera.xacro" />
     <xacro:property name="open_circuit_voltage" value="12.592"/>
     <xacro:property name="battery_capacity" value="20.0"/>
     <xacro:include filename="../../../description/battery.xacro" />
-    <!-- xacro:include filename="../../../description/depth_camera.xacro" / -->
-    <!-- xacro:include filename="../../../description/face.xacro" / -->
+    <xacro:property name="depth_camera_offset_x" value="${wheel_offset_x + 0.045}"/>
+    <xacro:property name="depth_camera_offset_z" value="0.4"/>
+    <xacro:include filename="../../../description/depth_camera.xacro"/>
+    <xacro:unless value="$(arg sim_mode)">
+        <xacro:arg name="parent_frame" default="depth_camera_link_optical" />
+        <xacro:include filename="$(find depthai_descriptions)/urdf/depthai_descr.urdf.xacro"/>
+    </xacro:unless>
     <xacro:include filename="ros2_control.xacro" />
 </robot>
