Commit message: Adjusted Create_1 URDF model

File: description/common_properties.xacro (robot description, xacro)
@@ -16,4 +16,7 @@
     <material name="blue">
         <color rgba="0 0 1 1"/>
+    </material>
+    <material name="grey">
+        <color rgba="0.5 0.5 0.5 1"/>
     </material>
     <material name="shadow_grey">

File: robots/turtle/description/create_base.urdf.xacro (robot description, xacro)
@@ -14,4 +14,5 @@
           <cylinder radius="${wheel_radius}" length="${wheel_width}"/>
         </geometry>
+        <material name="grey"/>
       </visual>
       <collision>
@@ -24,6 +25,6 @@
     <!-- joint name="${prefix}_wheel_joint" type="fixed" -->
     <joint name="${prefix}_wheel_joint" type="continuous">
-      <origin xyz="0 ${y_offset} 0.015" rpy="0 0 0"/>
-      <parent link="base_link"/>
+      <origin xyz="0 ${y_offset} ${-wheel_radius}" rpy="0 0 0"/>
+      <parent link="chassis_link"/>
       <child link="${prefix}_wheel_link"/>
       <axis xyz="0 1 0"/>
@@ -38,5 +39,5 @@
           <origin xyz="0 0 0"/>
           <geometry>
-              <sphere radius="0.04"/>
+              <sphere radius="0.01"/>
           </geometry>
           <material name="red"/>
@@ -46,5 +47,5 @@
     <link name="base_footprint">
       <visual name="footprint_visual">
-          <origin xyz="0 0 0.001"/>
+          <origin xyz="0 0 0"/>
           <geometry>
               <cylinder radius="${base_diameter/2 + 0.01}" length="0.003"/>
@@ -62,5 +63,5 @@
       <parent link="base_link"/>
       <child link="chassis_link"/>
-      <origin xyz="0 0 0"/>
+      <origin xyz="0 0 ${wheel_radius}"/>
     </joint>
     <!-- CHASSIS LINK -->
@@ -72,5 +73,5 @@
       </inertial>
       <visual>
-        <origin xyz=" 0 0 0.0308" rpy="0 0 0"/>
+        <origin xyz=" 0 0 -0.015" rpy="0 0 0"/>
         <geometry>
           <xacro:insert_block name="mesh"/>
@@ -78,7 +79,7 @@
       </visual>
       <collision>
-        <origin xyz="0.0 0.0 0.0308" rpy="0 0 0"/>
-        <geometry>
-          <cylinder length="0.0611632" radius="0.16495"/>
+        <origin xyz="0.0 0.0 0" rpy="0 0 0"/>
+        <geometry>
+          <cylinder length="0.0611632" radius="${base_diameter/2}"/>
         </geometry>
       </collision>
@@ -121,30 +122,30 @@
     <joint name="base_wall_sensor_joint" type="fixed">
       <origin xyz="0.09 -0.120 0.042" rpy="0 0 -1.0"/>
-      <parent link="base_link"/>
+      <parent link="chassis_link"/>
       <child link="wall_sensor_link"/>
     </joint>
     <joint name="base_left_cliff_sensor_joint" type="fixed">
       <origin xyz="0.07 0.14 0.01" rpy="0 ${PI/2} 0"/>
-      <parent link="base_link"/>
+      <parent link="chassis_link"/>
       <child link="left_cliff_sensor_link"/>
     </joint>
     <joint name="base_right_cliff_sensor_joint" type="fixed">
       <origin xyz="0.07 -0.14 0.01" rpy="0 ${PI/2} 0"/>
-      <parent link="base_link"/>
+      <parent link="chassis_link"/>
       <child link="right_cliff_sensor_link"/>
     </joint>
     <joint name="base_leftfront_cliff_sensor_joint" type="fixed">
       <origin xyz="0.15 0.04 0.01" rpy="0 ${PI/2} 0"/>
-      <parent link="base_link"/>
+      <parent link="chassis_link"/>
       <child link="leftfront_cliff_sensor_link"/>
     </joint>
     <joint name="base_rightfront_cliff_sensor_joint" type="fixed">
       <origin xyz="0.15 -0.04 0.01" rpy="0 ${PI/2} 0"/>
-      <parent link="base_link"/>
+      <parent link="chassis_link"/>
       <child link="rightfront_cliff_sensor_link"/>
     </joint>
     <xacro:create_wheel prefix="left" y_offset="${wheel_separation / 2}" wheel_radius="${wheel_radius}" wheel_width="${wheel_width}"/>
     <xacro:create_wheel prefix="right" y_offset="${wheel_separation / -2}" wheel_radius="${wheel_radius}" wheel_width="${wheel_width}"/>
-    <link name="front_wheel_link">
+    <link name="front_castor_link">
       <inertial>
         <origin xyz="0 0 0"/>
@@ -157,4 +158,5 @@
           <sphere radius="0.018"/>
         </geometry>
+        <material name="grey"/>
       </visual>
       <collision>
@@ -167,11 +169,11 @@
     <!-- fixed because there's no transmission -->
     <joint name="front_castor_joint" type="fixed">
-      <origin xyz="0.13 0 0.0" rpy="0 0 0"/>
-      <parent link="base_link"/>
-      <child link="front_wheel_link"/>
+      <origin xyz="0.13 0 -0.048" rpy="0 0 0"/>
+      <parent link="chassis_link"/>
+      <child link="front_castor_link"/>
       <axis xyz="0 1 0"/>
     </joint>
     <joint name="imu_joint" type="fixed">
-      <parent link="base_link"/>
+      <parent link="chassis_link"/>
       <child link="imu_link"/>
       <origin xyz="0.0 0 0.068" rpy="0 0 0"/>
@@ -179,7 +181,7 @@
     <link name="imu_link"/>
     <joint name="scan_joint" type="fixed">
-      <parent link="base_link"/>
+      <parent link="chassis_link"/>
       <child link="laser_frame"/>
-      <origin xyz="0.085 0 0.08" rpy="0 0 0"/>
+      <origin xyz="0.085 0 0.033" rpy="0 0 0"/>
     </joint>
     <link name="laser_frame">

Commit message: add chassis collision, inertia, change properties

File: description/common_properties.xacro (robot description, xacro)
@@ -38,4 +38,7 @@
         <color rgba="0.2 1 0.2 1"/>
     </material>
+    <material name="acrylic">
+        <color rgba="1.0 1.0 1.0 0.3"/>
+    </material>
     <xacro:arg name="sim_mode" default="false"/>
 </robot>

File: robots/stingray/description/robot_core.xacro (robot description, xacro)
@@ -3,8 +3,12 @@
     <xacro:include filename="../../../description/inertial_macros.xacro"/>
 	<!-- Values corrected for stingray robot -->
-    <xacro:property name="chassis_length" value="0.48"/>
-    <xacro:property name="chassis_width" value="0.42"/>
-    <xacro:property name="chassis_height" value="0.45"/>
-    <xacro:property name="chassis_mass" value="10.0"/>
+    <!-- <xacro:property name="chassis_length" value="0.48"/> -->
+    <!-- <xacro:property name="chassis_width" value="0.42"/> -->
+    <!-- <xacro:property name="chassis_height" value="0.45"/> -->
+    <!-- <xacro:property name="chassis_mass" value="10.0"/> -->
+    <xacro:property name="chassis_length" value="0.266"/>
+    <xacro:property name="chassis_width" value="0.228"/>
+    <xacro:property name="chassis_height" value="0.081"/>
+    <xacro:property name="chassis_mass" value="0.98"/>
     <xacro:property name="chassis_top_length" value="0.095"/>
     <xacro:property name="wheel_radius" value="0.192"/>
@@ -52,5 +56,5 @@
     <link name="base_footprint">
         <visual name="footprint_visual">
-            <origin xyz="0 0 0.01"/>
+            <origin xyz="0 0 0.001"/>
             <geometry>
                 <!-- box size="${wheel_offset_y * 2 + wheel_thickness} ${wheel_offset_y * 2 + wheel_thickness} 0.02"/ -->
@@ -80,5 +84,5 @@
                 <mesh filename="model://meshes/Stingray.stl" scale="0.001 0.001 0.001"/>
             </geometry>
-            <material name="grey"/>
+            <material name="acrylic"/>
         </visual>
         <visual name="chassis_rviz_visual">
@@ -89,6 +93,16 @@
                 <mesh filename="package://articubot_one/assets/meshes/Stingray.stl" scale="0.001 0.001 0.001"/>
             </geometry>
-            <material name="grey"/>
-        </visual>
+            <material name="acrylic"/>
+        </visual>
+        <collision>
+            <origin xyz="0.0 0.0 0.0" rpy="0.0 0.0 0.0"/>
+            <geometry>
+		        <!-- collision doesn't need to be a mesh, a box is sufficient -->
+                <box size="${chassis_length} ${chassis_width} ${chassis_height}"/>
+            </geometry>
+        </collision>
+        <xacro:inertial_box mass="${chassis_mass}" x="${chassis_length}" y="${chassis_width}" z="${chassis_height}">
+            <origin xyz="0.0 0.0 0.0" rpy="0.0 0.0 0.0"/>
+        </xacro:inertial_box>
         <visual name="chassis_front_axle_left">
             <origin xyz="${wheel_offset_x} ${chassis_width*0.5} 0" rpy="-${pi/2} 0 0"/>

Commit message: right caster removed, acrylic redefined

File: description/common_properties.xacro (robot description, xacro)
@@ -39,5 +39,5 @@
     </material>
     <material name="acrylic">
-        <color rgba="1.0 1.0 1.0 0.3"/>
+        <color rgba="1.0 1.0 1.0 0.5"/>
     </material>
     <xacro:arg name="sim_mode" default="false"/>

File: robots/stingray/description/robot_core.xacro (robot description, xacro)
@@ -109,5 +109,5 @@
         <parent link="base_link"/>
         <child link="left_wheel_link"/>
-        <origin xyz="0.0 ${wheel_offset} 0.0" rpy="${pi/2} 0.0 0.0"/>
+        <origin xyz="0.0 ${wheel_offset} 0.0" rpy="-${pi/2} 0.0 0.0"/>
         <axis xyz="0 0 1"/>
     </joint>
@@ -189,38 +189,4 @@
             <geometry>
                 <sphere radius="${caster_radius}"/>
-            </geometry>
-        </collision>
-        <xacro:inertial_sphere mass="${caster_mass}" radius="${caster_radius}">
-            <origin xyz="0.0 0.0 0.0" rpy="0.0 0.0 0.0"/>
-        </xacro:inertial_sphere>
-    </link>
-    <!-- CASTER WHEELS LINKS -->
-<!--
-    <joint name="left_caster_wheel_joint" type="${caster_joint_type}">
-        <parent link="chassis_link"/>
-        <child link="left_caster_wheel"/>
-        <origin xyz="${caster_wheel_offset_x} ${caster_wheel_offset_y} ${caster_wheel_offset_z}" rpy="${pi/2} 0 0" />
-        <axis xyz="0 0 1"/>
-    </joint>
- -->
-    <!-- <link name="left_caster_wheel"> -->
-<!--
-        <visual name="left_caster_visual">
-            <geometry>
-               <cylinder radius="${caster_wheel_radius}" length="${caster_wheel_thickness}"/>
-            </geometry>
-            <material name="port_red"/>
-        </visual>
-        <visual name="left_caster_marker_visual">
-            <geometry>
-                <box size="${caster_wheel_radius*0.5} ${caster_wheel_radius*0.5} ${caster_wheel_thickness*1.1}"/>
-            </geometry>
-            <material name="blue"/>
-        </visual>
- -->
-        <!--
-        <collision>
-            <geometry>
-                <cylinder radius="${caster_wheel_radius}" length="${caster_wheel_thickness}"/>
             </geometry>
             <surface>
@@ -235,25 +201,27 @@
             </surface>
         </collision>
-        -->
-<!--
-        <xacro:inertial_cylinder mass="${caster_wheel_mass}" length="${caster_wheel_thickness}" radius="${caster_wheel_radius}">
-            <origin xyz="0 0 0" rpy="0 0 0"/>
-        </xacro:inertial_cylinder>
--->
-    <!-- </link> -->
-    <joint name="right_caster_wheel_joint" type="${caster_joint_type}">
+        <xacro:inertial_sphere mass="${caster_mass}" radius="${caster_radius}">
+            <origin xyz="0.0 0.0 0.0" rpy="0.0 0.0 0.0"/>
+        </xacro:inertial_sphere>
+    </link>
+    <!-- CASTER WHEELS LINKS -->
+    <!-- LEFT CASTER WHEEL -->
+<!--
+    <joint name="left_caster_wheel_joint" type="${caster_joint_type}">
         <parent link="chassis_link"/>
-        <child link="right_caster_wheel"/>
-        <origin xyz="${caster_wheel_offset_x} ${-caster_wheel_offset_y} ${caster_wheel_offset_z}" rpy="${pi/2} 0 0" />
-        <axis xyz="0 0 -1"/>
-    </joint>
-    <link name="right_caster_wheel">
-        <visual name="right_caster_visual">
+        <child link="left_caster_wheel"/>
+        <origin xyz="${caster_wheel_offset_x} ${caster_wheel_offset_y} ${caster_wheel_offset_z}" rpy="${pi/2} 0 0" />
+        <axis xyz="0 0 1"/>
+    </joint>
+ -->
+    <!-- <link name="left_caster_wheel"> -->
+<!--
+        <visual name="left_caster_visual">
             <geometry>
                <cylinder radius="${caster_wheel_radius}" length="${caster_wheel_thickness}"/>
             </geometry>
-            <material name="starboard_green"/>
-        </visual>
-        <visual name="right_caster_marker_visual">
+            <material name="port_red"/>
+        </visual>
+        <visual name="left_caster_marker_visual">
             <geometry>
                 <box size="${caster_wheel_radius*0.5} ${caster_wheel_radius*0.5} ${caster_wheel_thickness*1.1}"/>
@@ -261,4 +229,6 @@
             <material name="blue"/>
         </visual>
+ -->
+        <!--
         <collision>
             <geometry>
@@ -276,7 +246,57 @@
             </surface>
         </collision>
+        -->
+<!--
         <xacro:inertial_cylinder mass="${caster_wheel_mass}" length="${caster_wheel_thickness}" radius="${caster_wheel_radius}">
             <origin xyz="0 0 0" rpy="0 0 0"/>
         </xacro:inertial_cylinder>
-    </link>
+-->
+    <!-- </link> -->
+    <!-- RIGHT CASTER WHEEL -->
+<!--
+    <joint name="right_caster_wheel_joint" type="${caster_joint_type}">
+        <parent link="chassis_link"/>
+        <child link="right_caster_wheel"/>
+        <origin xyz="${caster_wheel_offset_x} ${-caster_wheel_offset_y} ${caster_wheel_offset_z}" rpy="${pi/2} 0 0" />
+        <axis xyz="0 0 -1"/>
+    </joint>
+ -->
+    <!-- <link name="right_caster_wheel"> -->
+<!--
+        <visual name="right_caster_visual">
+            <geometry>
+               <cylinder radius="${caster_wheel_radius}" length="${caster_wheel_thickness}"/>
+            </geometry>
+            <material name="starboard_green"/>
+        </visual>
+        <visual name="right_caster_marker_visual">
+            <geometry>
+                <box size="${caster_wheel_radius*0.5} ${caster_wheel_radius*0.5} ${caster_wheel_thickness*1.1}"/>
+            </geometry>
+            <material name="blue"/>
+        </visual>
+ -->
+<!--
+        <collision>
+            <geometry>
+                <cylinder radius="${caster_wheel_radius}" length="${caster_wheel_thickness}"/>
+            </geometry>
+            <surface>
+                <friction>
+                    <ode>
+                    <mu>0</mu>
+                    <mu2>0</mu2>
+                    <slip1>1.0</slip1>
+                    <slip2>1.0</slip2>
+                    </ode>
+                </friction>
+            </surface>
+        </collision>
+ -->
+<!--
+        <xacro:inertial_cylinder mass="${caster_wheel_mass}" length="${caster_wheel_thickness}" radius="${caster_wheel_radius}">
+            <origin xyz="0 0 0" rpy="0 0 0"/>
+        </xacro:inertial_cylinder>
+ -->
+    <!-- </link> -->
 </robot>
