Commit message: Added camera_stereo for RPi5 dual camera depth+inference on Dragger

File: description/common_properties.xacro (robot description, xacro)
@@ -26,4 +26,7 @@
         <color rgba="0.2 0.2 1 1"/>
     </material>
+    <material name="sensor_lens_blue">
+        <color rgba="0.26 0.34 0.55 1"/>
+    </material>
     <material name="sensor_yellow">
         <color rgba="0.8 0.8 0.2 1"/>

File: robots/dragger/description/robot.urdf.xacro (robot description, xacro)
@@ -30,4 +30,7 @@
     <xacro:property name="camera_offset_z" value="0.55"/>
     <xacro:include filename="../../../description/camera.xacro" />
+    <xacro:property name="camera_stereo_offset_x" value="${wheel_offset_x + 0.19}"/>
+    <xacro:property name="camera_stereo_offset_z" value="0.2"/>
+    <xacro:include filename="../../../description/camera_stereo.xacro" />
     <xacro:property name="open_circuit_voltage" value="12.592"/>
     <xacro:property name="battery_capacity" value="50.0"/>
