Commit message: WIP: turtle sim drives and shows scan and imu topics

File: description/imu.xacro (robot description, xacro)
@@ -19,5 +19,5 @@
         </visual>
     </link>
-    <!-- gz model -m dragger -s imu_sensor -->
+    <!-- gz model -m dragger -s imu_link -->
     <gazebo reference="imu_link">
         <sensor name="imu_link" type="imu">

File: description/lidar.xacro (robot description, xacro)
@@ -34,5 +34,5 @@
         </xacro:inertial_cylinder>
     </link>
-    <!-- gz model -m dragger -s front_laser -->
+    <!-- gz model -m dragger -s laser_frame -->
     <gazebo reference="laser_frame">
         <!-- name must be "laser_frame", specifically for lasers. Must reference an actual link in .xacro -->

File: robots/turtle/description/create_base.urdf.xacro (robot description, xacro)
@@ -18,5 +18,5 @@
       </collision>
       <xacro:inertial_cylinder mass="0.01" length="${wheel_width}" radius="${wheel_radius}">
-          <origin xyz="0 0 0" rpy="0 0 0"/>
+        <origin xyz="0 0 0" rpy="0 0 0"/>
       </xacro:inertial_cylinder>
     </link>
@@ -66,5 +66,11 @@
     <!-- CHASSIS LINK -->
     <link name="chassis_link">
-      <visual>
+      <visual name="chassis_gz_visual">
+        <origin xyz=" 0 0 -0.015" rpy="0 0 0"/>
+        <geometry>
+            <mesh filename="model://meshes/create_1.dae"/>
+        </geometry>
+      </visual>
+      <visual name="chassis_rviz_visual">
         <origin xyz=" 0 0 -0.015" rpy="0 0 0"/>
         <geometry>
@@ -79,5 +85,6 @@
       </collision>
       <xacro:inertial_cylinder mass="${mass_kg}" length="0.0611632" radius="${base_diameter/2}">
-          <origin xyz="0 0 -0.015" rpy="0 0 0"/>
+        <!-- cheat: origin moved forward a bit, so that center mass is forward of the wheels axis -->
+        <origin xyz="0.03 0 0" rpy="0 0 0"/>
       </xacro:inertial_cylinder>
     </link>
@@ -134,5 +141,5 @@
       </collision>
       <xacro:inertial_sphere mass="0.01" radius="0.018">
-          <origin xyz="0 0 0" rpy="0 0 0"/>
+        <origin xyz="0 0 0" rpy="0 0 0"/>
       </xacro:inertial_sphere>
     </link>
@@ -150,4 +157,92 @@
     </joint>
     <link name="imu_link"/>
+    <!-- gz model -m turtle -s imu_link -->
+    <gazebo reference="imu_link">
+        <sensor name="imu_link" type="imu">
+        <always_on>1</always_on>
+        <topic>gz_imu/data</topic>
+        <!-- future Gazebo versions might require "<frame_id>" here. Must reference an actual link in .xacro -->
+        <gz_frame_id>imu_link</gz_frame_id>
+        <frame_id>imu_link</frame_id>
+        <update_rate>250</update_rate>
+            <imu>
+                <orientation_reference_frame>
+                  <localization>ENU</localization>
+                  <!-- custom_rpy parent_frame='world'>1.570795 0 0</custom_rpy -->
+                </orientation_reference_frame>
+                <enable_orientation>1</enable_orientation>
+                <angular_velocity>
+                    <x>
+                        <noise type="gaussian">
+                            <mean>0</mean>
+                            <stddev>0.009</stddev>
+                            <bias_mean>0.00075</bias_mean>
+                            <bias_stddev>0.005</bias_stddev>
+                            <dynamic_bias_stddev>0.00002</dynamic_bias_stddev>
+                            <dynamic_bias_correlation_time>400.0</dynamic_bias_correlation_time>
+                            <precision>0.00025</precision>
+                        </noise>
+                    </x>
+                    <y>
+                        <noise type="gaussian">
+                            <mean>0</mean>
+                            <stddev>0.009</stddev>
+                            <bias_mean>0.00075</bias_mean>
+                            <bias_stddev>0.005</bias_stddev>
+                            <dynamic_bias_stddev>0.00002</dynamic_bias_stddev>
+                            <dynamic_bias_correlation_time>400.0</dynamic_bias_correlation_time>
+                            <precision>0.00025</precision>
+                        </noise>
+                    </y>
+                    <z>
+                        <noise type="gaussian">
+                            <mean>0</mean>
+                            <stddev>0.009</stddev>
+                            <bias_mean>0.00075</bias_mean>
+                            <bias_stddev>0.005</bias_stddev>
+                            <dynamic_bias_stddev>0.00002</dynamic_bias_stddev>
+                            <dynamic_bias_correlation_time>400.0</dynamic_bias_correlation_time>
+                            <precision>0.00025</precision>
+                        </noise>
+                    </z>
+                </angular_velocity>
+                <linear_acceleration>
+                    <x>
+                        <noise type="gaussian">
+                            <mean>0</mean>
+                            <stddev>0.021</stddev>
+                            <bias_mean>0.05</bias_mean>
+                            <bias_stddev>0.0075</bias_stddev>
+                            <dynamic_bias_stddev>0.000375</dynamic_bias_stddev>
+                            <dynamic_bias_correlation_time>175.0</dynamic_bias_correlation_time>
+                            <precision>0.005</precision>
+                        </noise>
+                    </x>
+                    <y>
+                        <noise type="gaussian">
+                            <mean>0</mean>
+                            <stddev>0.021</stddev>
+                            <bias_mean>0.05</bias_mean>
+                            <bias_stddev>0.0075</bias_stddev>
+                            <dynamic_bias_stddev>0.000375</dynamic_bias_stddev>
+                            <dynamic_bias_correlation_time>175.0</dynamic_bias_correlation_time>
+                            <precision>0.005</precision>
+                        </noise>
+                    </y>
+                    <z>
+                        <noise type="gaussian">
+                            <mean>0</mean>
+                            <stddev>0.021</stddev>
+                            <bias_mean>0.05</bias_mean>
+                            <bias_stddev>0.0075</bias_stddev>
+                            <dynamic_bias_stddev>0.000375</dynamic_bias_stddev>
+                            <dynamic_bias_correlation_time>175.0</dynamic_bias_correlation_time>
+                            <precision>0.005</precision>
+                        </noise>
+                    </z>
+                </linear_acceleration>
+            </imu>
+        </sensor>
+    </gazebo>
     <joint name="scan_joint" type="fixed">
       <parent link="chassis_link"/>
@@ -170,4 +265,45 @@
       </visual>
     </link>
+    <!-- gz model -m turtle -s laser_frame -->
+    <gazebo reference="laser_frame">
+        <!-- name must be "laser_frame", specifically for lasers. Must reference an actual link in .xacro -->
+        <sensor name='laser_frame' type='gpu_lidar'>
+          <pose>0 0 0 0 0 0</pose>
+          <always_on>1</always_on>
+          <!-- 6 Hz for LD14 - see "frequency" in dual_ekf_navsat_parameters.yaml -->
+          <update_rate>6</update_rate>
+          <topic>gz_scan</topic>
+          <!-- future Gazebo versions might require "<frame_id>" here. Must reference an actual link in .xacro -->
+          <gz_frame_id>laser_frame</gz_frame_id>
+          <frame_id>laser_frame</frame_id>
+          <ray>
+            <scan>
+              <horizontal>
+                <samples>360</samples>
+                <resolution>1</resolution>
+                <min_angle>-${pi}</min_angle>
+                <max_angle>${pi}</max_angle>
+              </horizontal>
+              <vertical>
+                <samples>1</samples>
+                <resolution>1</resolution>
+                <min_angle>0.0</min_angle>
+                <max_angle>0.0</max_angle>
+              </vertical>
+            </scan>
+            <range>
+              <min>0.3</min>
+              <max>12.0</max>
+              <resolution>0.01</resolution>
+            </range>
+            <noise>
+              <type>gaussian</type>
+              <mean>0</mean>
+              <stddev>0.01</stddev>
+            </noise>
+          </ray>
+          <visualize>true</visualize>
+        </sensor>
+    </gazebo>
   </xacro:macro>
 </robot>

Commit message: resize & move IMU Mag

File: description/imu.xacro (robot description, xacro)
@@ -12,5 +12,6 @@
         <visual>
             <geometry>
-                <box size="0.1 0.1 0.1"/>
+                <!-- <box size="0.1 0.1 0.1"/> -->
+                <box size="0.016 0.020 0.004"/>
             </geometry>
             <material name="sensor_blue"/>

File: description/magnetometer.xacro (robot description, xacro)
@@ -14,7 +14,7 @@
         <visual>
             <geometry>
-                <box size="0.1 0.1 0.1"/>
+                <box size="0.01 0.01 0.01"/>
             </geometry>
-            <material name="sensor_blue"/>
+            <material name="sensor_yellow"/>
         </visual>
     </link>

File: robots/stingray/description/robot.urdf.xacro (robot description, xacro)
@@ -10,6 +10,6 @@
     <xacro:include filename="../../../description/common_properties.xacro" />
     <xacro:include filename="robot_core.xacro" />
-    <xacro:property name="imu_offset_x" value="${wheel_offset_x}"/>
-    <xacro:property name="imu_offset_z" value="0.01"/>
+    <xacro:property name="imu_offset_x" value="0.0"/>
+    <xacro:property name="imu_offset_z" value="0.0"/>
     <xacro:include filename="../../../description/imu.xacro" />
     <xacro:include filename="../../../description/magnetometer.xacro" />

File: robots/stingray/description/robot_core.xacro (robot description, xacro)
@@ -3,8 +3,4 @@
     <xacro:include filename="../../../description/inertial_macros.xacro"/>
 	<!-- Values corrected for stingray robot -->
-    <!-- <xacro:property name="chassis_length" value="0.48"/> -->
-    <!-- <xacro:property name="chassis_width" value="0.42"/> -->
-    <!-- <xacro:property name="chassis_height" value="0.45"/> -->
-    <!-- <xacro:property name="chassis_mass" value="10.0"/> -->
     <xacro:property name="chassis_length" value="0.266"/>
     <xacro:property name="chassis_width" value="0.228"/>
@@ -12,8 +8,4 @@
     <xacro:property name="chassis_mass" value="0.98"/>
     <xacro:property name="chassis_offset" value="0.0455"/>
-    <!-- <xacro:property name="chassis_top_length" value="0.095"/> -->
-    <!-- <xacro:property name="wheel_radius" value="0.192"/> -->
-    <!-- <xacro:property name="wheel_thickness" value="0.045"/> -->
-    <!-- <xacro:property name="wheel_mass" value="1.0"/> -->
     <xacro:property name="wheel_radius" value="0.0615"/>
     <xacro:property name="wheel_thickness" value="0.02"/>
@@ -47,5 +39,5 @@
             <origin xyz="0 0 0"/>
             <geometry>
-                <sphere radius="0.04"/>
+                <sphere radius="0.005"/>
             </geometry>
             <material name="red"/>
@@ -86,5 +78,4 @@
             <origin xyz="0.0 0.0 0.0" rpy="0.0 0.0 0.0"/>
             <geometry>
-                <!-- <mesh filename="file://$(find stingray)/description/Stingray.stl" scale="0.001 0.001 0.001"/> -->
                 <mesh filename="model://meshes/Stingray.stl" scale="0.001 0.001 0.001"/>
             </geometry>
@@ -95,5 +86,4 @@
             <geometry>
                 <!-- box size="${chassis_length} ${chassis_width} ${chassis_height}"/ -->
-                <!-- <mesh filename="file://$(find stingray)/description/meshes/Stingray.stl" scale="0.001 0.001 0.001"/> -->
                 <mesh filename="package://articubot_one/assets/meshes/Stingray.stl" scale="0.001 0.001 0.001"/>
             </geometry>
@@ -112,15 +102,4 @@
     </link>
     <!-- LEFT WHEEL JOINT -->
-    <!-- <joint name="left_wheel_joint" type="continuous">
-        <parent link="chassis_link"/>
-        <child link="left_wheel"/>
-        <origin xyz="${wheel_offset_x} ${wheel_offset_y} 0" rpy="-${pi/2 - 0.15} 0 0" />
-        <axis xyz="0 0 1">
-          <limit>
-            <lower>-1.79769e+308</lower>
-            <upper>1.79769e+308</upper>
-          </limit>
-        </axis>
-    </joint> -->
     <joint name="left_wheel_joint" type="continuous">
         <parent link="base_link"/>
@@ -131,61 +110,4 @@
     <!-- LEFT WHEEL LINK -->
     <link name="left_wheel_link">
-        <!-- <visual name="left_wheel_tire_gz_visual">
-            <origin xyz="0 0 0" rpy="${pi/2} 0 0" />
-            <geometry>
-                <mesh filename="model://meshes/wheel_link.STL" scale="${wheel_radius*12.7} ${wheel_thickness*10.2} ${wheel_radius*12.7}"/>
-            </geometry>
-            <material name="port_red"/>
-        </visual> -->
-        <!-- <visual name="left_wheel_tire_rviz_visual">
-            <origin xyz="0 0 0" rpy="${pi/2} 0 0" />
-            <geometry>
-                <mesh filename="package://articubot_one/assets/meshes/wheel_link.STL" scale="${wheel_radius*12.7} ${wheel_thickness*10.2} ${wheel_radius*12.7}"/>
-            </geometry>
-            <material name="port_red"/>
-        </visual> -->
-        <!-- <visual name="left_wheel_solid_visual">
-            <geometry>
-                <cylinder radius="${wheel_radius}" length="${wheel_thickness/10.0}"/>
-            </geometry>
-            <material name="port_red"/>
-        </visual> -->
-        <!-- <visual name="left_wheel_axis_visual">
-            <geometry>
-                <cylinder radius="${wheel_radius*0.05}" length="${wheel_thickness*1.1}"/>
-            </geometry>
-            <material name="blue"/>
-        </visual> -->
-        <!-- <visual name="left_wheel_marker_visual">
-            <origin xyz="0 ${wheel_radius*0.7} 0" rpy="0 0 0" />
-            <geometry>
-                <box size="${wheel_radius*0.2} ${wheel_radius*0.3} ${wheel_thickness*1.1}"/>
-            </geometry>
-            <material name="blue"/>
-        </visual> -->
-        <!-- <collision>
-            <geometry>
-                <cylinder radius="${wheel_radius}" length="${wheel_thickness}"/>
-            </geometry>
-            <max_contacts>1</max_contacts>
-            <surface>
-                <friction>
-                    <ode>
-                    <mu>0.4</mu>
-                    <mu2>0.6</mu2>
-                    </ode>
-                </friction>
-                <bounce/>
-                <contact>
-                    <ode>
-                    <min_depth>0.005</min_depth>
-                    <kp>1e8</kp>
-                    </ode>
-                </contact>
-            </surface>
-        </collision> -->
-        <!-- <xacro:inertial_cylinder mass="${wheel_mass}" length="${wheel_thickness}" radius="${wheel_radius}">
-            <origin xyz="0 0 0" rpy="0 0 0"/>
-        </xacro:inertial_cylinder> -->
         <visual name="left_wheel_visual">
             <geometry>
@@ -219,61 +141,4 @@
     <!-- RIGHT WHEEL LINK -->
     <link name="right_wheel_link">
-        <!-- <visual name="right_wheel_tire_gz_visual">
-            <origin xyz="0 0 0" rpy="${-pi/2} 0 0" />
-            <geometry>
-                <mesh filename="model://meshes/wheel_link.STL" scale="${wheel_radius*12.7} ${wheel_thickness*10.2} ${wheel_radius*12.7}"/>
-            </geometry>
-            <material name="starboard_green"/>
-        </visual> -->
-        <!-- <visual name="right_wheel_tire_rviz_visual">
-            <origin xyz="0 0 0" rpy="${-pi/2} 0 0" />
-            <geometry>
-                <mesh filename="package://articubot_one/assets/meshes/wheel_link.STL" scale="${wheel_radius*12.7} ${wheel_thickness*10.2} ${wheel_radius*12.7}"/>
-            </geometry>
-            <material name="starboard_green"/>
-        </visual> -->
-        <!-- <visual name="right_wheel_solid_visual">
-            <geometry>
-                <cylinder radius="${wheel_radius}" length="${wheel_thickness/10.0}"/>
-            </geometry>
-            <material name="starboard_green"/>
-        </visual> -->
-        <!-- <visual name="right_wheel_axis_visual">
-            <geometry>
-                <cylinder radius="${wheel_radius*0.05}" length="${wheel_thickness*1.1}"/>
-            </geometry>
-            <material name="blue"/>
-        </visual> -->
-        <!-- <visual name="right_wheel_marker_visual">
-            <origin xyz="0 ${-wheel_radius*0.7} 0" rpy="0 0 0" />
-            <geometry>
-                <box size="${wheel_radius*0.2} ${wheel_radius*0.3} ${wheel_thickness*1.1}"/>
-            </geometry>
-            <material name="blue"/>
-        </visual> -->
-        <!-- <collision>
-            <geometry>
-                <cylinder radius="${wheel_radius}" length="${wheel_thickness}"/>
-            </geometry>
-            <max_contacts>1</max_contacts>
-            <surface>
-                <friction>
-                    <ode>
-                    <mu>0.4</mu>
-                    <mu2>0.6</mu2>
-                    </ode>
-                </friction>
-                <bounce/>
-                <contact>
-                    <ode>
-                    <min_depth>0.005</min_depth>
-                    <kp>1e8</kp>
-                    </ode>
-                </contact>
-            </surface>
-        </collision> -->
-        <!-- <xacro:inertial_cylinder mass="${wheel_mass}" length="${wheel_thickness}" radius="${wheel_radius}">
-            <origin xyz="0 0 0" rpy="0 0 0"/>
-        </xacro:inertial_cylinder> -->
         <visual name="right_wheel_visual">
             <geometry>
