Commit message: Better placement of IMU and other sensors in .xacro files

File: description/imu.xacro (robot description, xacro)
@@ -6,5 +6,5 @@
         <parent link="chassis_link"/>
         <child link="imu_link"/>
-        <!-- we place IMU between the wheels -->
+        <!-- we want to place IMU closely between the wheels, at center mass -->
         <origin xyz="${imu_offset_x} 0 ${imu_offset_z}" rpy="0 0 0"/>
     </joint>
@@ -12,5 +12,5 @@
         <visual>
             <geometry>
-                <box size="0.1 0.1 0.1"/>
+                <box size="${imu_visual_size} ${imu_visual_size} ${imu_visual_size}"/>
             </geometry>
             <material name="sensor_blue"/>

File: description/magnetometer.xacro (robot description, xacro)
@@ -3,16 +3,17 @@
     <xacro:property name="magnetometer_offset_x" value="${wheel_offset_x}"/>
     <xacro:property name="magnetometer_offset_z" value="0.03"/>
-    <!-- ******************* MAGNETOMETER SETUP ****************************  -->
-    <!-- Each sensor must be attached to a link.                              -->
+    <!-- ******************* MAGNETOMETER SETUP ********************************  -->
+    <!-- we are using IMU parameters here, as magnetometer is usually part of IMU -->
+    <!-- Each sensor must be attached to a link.                                  -->
     <joint name="magnetometer_joint" type="fixed">
         <parent link="chassis_link"/>
         <child link="magnetometer_link"/>
-        <!-- we place Magnetometer next to IMU between the wheels -->
-        <origin xyz="${wheel_offset_x} 0 ${magnetometer_offset_z}" rpy="0 0 0"/>
+        <!-- we want to place Magnetometer next to IMU between the wheels, at center mass -->
+        <origin xyz="${imu_offset_x} 0 ${imu_offset_z}" rpy="0 0 0"/>
     </joint>
     <link name="magnetometer_link">
         <visual>
             <geometry>
-                <box size="0.1 0.1 0.1"/>
+              <cylinder radius="${imu_visual_size * 0.85}" length="${imu_visual_size / 4}"/>
             </geometry>
             <material name="sensor_blue"/>

File: robots/dragger/description/robot.urdf.xacro (robot description, xacro)
@@ -10,9 +10,10 @@
     <xacro:include filename="../../../description/common_properties.xacro" />
     <xacro:include filename="robot_core.xacro" />
-    <xacro:property name="imu_offset_x" value="${wheel_offset_x}"/>
-    <xacro:property name="imu_offset_z" value="0.04"/>
+    <xacro:property name="imu_offset_x" value="${wheel_offset_x + 0.04}"/>
+    <xacro:property name="imu_offset_z" value="0.52"/>
+    <xacro:property name="imu_visual_size" value="0.01"/>
     <xacro:include filename="../../../description/imu.xacro" />
     <xacro:include filename="../../../description/magnetometer.xacro" />
-    <xacro:property name="laser_offset_x" value="${chassis_length/4 + 0.05}"/>
+    <xacro:property name="laser_offset_x" value="${wheel_offset_x - 0.14}"/>
     <xacro:property name="laser_offset_z" value="0.57"/>
     <xacro:include filename="../../../description/lidar.xacro" />
@@ -21,9 +22,9 @@
     <xacro:property name="sonars_offset_z" value="0.05"/>
     <xacro:include filename="../../../description/sonars.xacro" />
-    <xacro:property name="gps_offset_x" value="0.05"/>
+    <xacro:property name="gps_offset_x" value="${wheel_offset_x}"/>
     <xacro:property name="gps_offset_y" value="0.0"/>
     <xacro:property name="gps_offset_z" value="0.65"/>
     <xacro:include filename="../../../description/gps.xacro" />
-    <xacro:property name="camera_offset_x" value="${chassis_length/2 - 0.04}"/>
+    <xacro:property name="camera_offset_x" value="${wheel_offset_x + 0.14}"/>
     <xacro:property name="camera_offset_z" value="0.55"/>
     <xacro:include filename="../../../description/camera.xacro" />

File: robots/plucky/description/robot.urdf.xacro (robot description, xacro)
@@ -10,6 +10,7 @@
     <xacro:include filename="../../../description/common_properties.xacro" />
     <xacro:include filename="robot_core.xacro" />
-    <xacro:property name="imu_offset_x" value="${wheel_offset_x}"/>
-    <xacro:property name="imu_offset_z" value="0.01"/>
+    <xacro:property name="imu_offset_x" value="${wheel_offset_x + 0.09}"/>
+    <xacro:property name="imu_offset_z" value="0.1"/>
+    <xacro:property name="imu_visual_size" value="0.01"/>
     <xacro:include filename="../../../description/imu.xacro" />
     <xacro:include filename="../../../description/magnetometer.xacro" />

File: robots/turtle/description/create_1.urdf.xacro (robot description, xacro)
@@ -2,10 +2,11 @@
 <robot name="create_1" xmlns:xacro="http://ros.org/wiki/xacro">
   <xacro:include filename="create_base.urdf.xacro" />
-  <xacro:property name="imu_offset_x" value="0"/>
+  <xacro:property name="imu_offset_x" value="-0.04"/>
   <xacro:property name="imu_offset_z" value="0"/>
+  <xacro:property name="imu_visual_size" value="0.01"/>
+  <xacro:include filename="../../../description/imu.xacro" />
   <xacro:property name="laser_offset_x" value="0.085"/>
   <xacro:property name="laser_offset_z" value="0.033"/>
   <xacro:include filename="create_sensors.urdf.xacro" />
-  <xacro:include filename="create_1_gazebo.urdf.xacro" />
   <!-- wheel_separation - distance between left and right wheels, defined in ~/create_robot_ws/src/libcreate/src/types.cpp -->
   <xacro:create_base wheel_separation="0.258" base_diameter="0.3302" wheel_radius="0.033" wheel_width="0.024" mass_kg="3.5">

File: robots/turtle/description/create_sensors.urdf.xacro (robot description, xacro)
@@ -1,18 +1,8 @@
 <?xml version="1.0" ?>
 <robot xmlns:xacro="http://ros.org/wiki/xacro">
-    <joint name="imu_joint" type="fixed">
-      <parent link="chassis_link"/>
-      <child link="imu_link"/>
-      <!-- we place IMU between the wheels -->
-      <origin xyz="${imu_offset_x} 0 ${imu_offset_z}" rpy="0 0 0"/>
-    </joint>
-    <link name="imu_link">
-      <visual>
-        <geometry>
-          <box size="0.01 0.01 0.01"/>
-        </geometry>
-        <material name="sensor_blue"/>
-      </visual>
-    </link>
+<!--
+We want Turtle's LIDAR (XV-11) to look a bit different, so we don't use common description.
+meld ~/robot_ws/src/articubot_one/robots/turtle/description/create_sensors.urdf.xacro ~/robot_ws/src/articubot_one/description/lidar.xacro
+-->
     <joint name="laser_joint" type="fixed">
       <parent link="chassis_link"/>
@@ -35,3 +25,44 @@
       </visual>
     </link>
+    <!-- gz model -m turtle -s laser_frame -->
+    <gazebo reference="laser_frame">
+        <!-- name must be "laser_frame", specifically for lasers. Must reference an actual link in .xacro -->
+        <sensor name='laser_frame' type='gpu_lidar'>
+          <pose>0 0 0 0 0 0</pose>
+          <always_on>1</always_on>
+          <!-- 6 Hz for LD14 - see "frequency" in dual_ekf_navsat_parameters.yaml -->
+          <update_rate>6</update_rate>
+          <topic>gz_scan</topic>
+          <!-- future Gazebo versions might require "<frame_id>" here. Must reference an actual link in .xacro -->
+          <gz_frame_id>laser_frame</gz_frame_id>
+          <frame_id>laser_frame</frame_id>
+          <ray>
+            <scan>
+              <horizontal>
+                <samples>360</samples>
+                <resolution>1</resolution>
+                <min_angle>-${pi}</min_angle>
+                <max_angle>${pi}</max_angle>
+              </horizontal>
+              <vertical>
+                <samples>1</samples>
+                <resolution>1</resolution>
+                <min_angle>0.0</min_angle>
+                <max_angle>0.0</max_angle>
+              </vertical>
+            </scan>
+            <range>
+              <min>0.3</min>
+              <max>12.0</max>
+              <resolution>0.01</resolution>
+            </range>
+            <noise>
+              <type>gaussian</type>
+              <mean>0</mean>
+              <stddev>0.01</stddev>
+            </noise>
+          </ray>
+          <visualize>true</visualize>
+        </sensor>
+    </gazebo>
 </robot>

Commit message: Dev to main merge (#3)
* bno055_driver_node for Plucky

* Added missing <pose>0 0 0 0 0 0</pose> to sensors definitions

* Update imu.xacro

* Better placement of IMU and other sensors in .xacro files

* Commenting on addresses for BNO055

* Update controllers.yaml

* wheels_pwm_factor adjusted for Plucky, battery parameters added for Dragger

* Update nav2_params.yaml

* Update plucky.launch.py

* Update package.xml

added some dependencies

* Adjusted cmd_vel_timeout: 0.2

File: description/imu.xacro (robot description, xacro)
@@ -6,5 +6,5 @@
         <parent link="chassis_link"/>
         <child link="imu_link"/>
-        <!-- we place IMU between the wheels -->
+        <!-- we want to place IMU closely between the wheels, at center mass -->
         <origin xyz="${imu_offset_x} 0 ${imu_offset_z}" rpy="0 0 0"/>
     </joint>
@@ -12,5 +12,5 @@
         <visual>
             <geometry>
-                <box size="0.1 0.1 0.1"/>
+                <box size="${imu_visual_size} ${imu_visual_size} ${imu_visual_size}"/>
             </geometry>
             <material name="sensor_blue"/>
@@ -20,4 +20,5 @@
     <gazebo reference="imu_link">
         <sensor name="imu_link" type="imu">
+        <pose>0 0 0 0 0 0</pose>
         <always_on>1</always_on>
         <topic>gz_imu/data</topic>

File: description/magnetometer.xacro (robot description, xacro)
@@ -3,16 +3,17 @@
     <xacro:property name="magnetometer_offset_x" value="${wheel_offset_x}"/>
     <xacro:property name="magnetometer_offset_z" value="0.03"/>
-    <!-- ******************* MAGNETOMETER SETUP ****************************  -->
-    <!-- Each sensor must be attached to a link.                              -->
+    <!-- ******************* MAGNETOMETER SETUP ********************************  -->
+    <!-- we are using IMU parameters here, as magnetometer is usually part of IMU -->
+    <!-- Each sensor must be attached to a link.                                  -->
     <joint name="magnetometer_joint" type="fixed">
         <parent link="chassis_link"/>
         <child link="magnetometer_link"/>
-        <!-- we place Magnetometer next to IMU between the wheels -->
-        <origin xyz="${wheel_offset_x} 0 ${magnetometer_offset_z}" rpy="0 0 0"/>
+        <!-- we want to place Magnetometer next to IMU between the wheels, at center mass -->
+        <origin xyz="${imu_offset_x} 0 ${imu_offset_z}" rpy="0 0 0"/>
     </joint>
     <link name="magnetometer_link">
         <visual>
             <geometry>
-                <box size="0.1 0.1 0.1"/>
+              <cylinder radius="${imu_visual_size * 0.85}" length="${imu_visual_size / 4}"/>
             </geometry>
             <material name="sensor_blue"/>
@@ -21,4 +22,5 @@
     <gazebo reference="magnetometer_link">
         <sensor name="magnetometer" type="magnetometer">
+          <pose>0 0 0 0 0 0</pose>
           <always_on>1</always_on>
           <update_rate>100</update_rate>

Commit message: Adjusted Magnetometer in Gazebo topic, sharing IMU link, merged two Turtle xacro files in one

File: description/imu.xacro (robot description, xacro)
@@ -22,4 +22,6 @@
     <!-- gz model -m dragger -s imu_link -->
     <gazebo reference="imu_link">
+        <!-- IMU sensor, with "enable_orientation" publishes /imu/data, without - /imu/data_raw
+             See https://github.com/CCNYRoboticsLab/imu_tools -->
         <sensor name="imu_link" type="imu">
         <pose>0 0 0 0 0 0</pose>
@@ -108,4 +110,36 @@
             </imu>
         </sensor>
+        <!-- Magnetometer sharing the IMU link, taking magnetic field from "gz::sim::systems::Magnetometer" Gazebo plugin -->
+        <sensor name="magnetometer" type="magnetometer">
+          <pose>0 0 0 0 0 0</pose>
+          <always_on>1</always_on>
+          <update_rate>100</update_rate>
+          <visualize>true</visualize>
+          <topic>gz_magnetometer/data</topic>
+          <!-- future Gazebo versions might require "<frame_id>" here. Must reference an actual link in .xacro -->
+          <gz_frame_id>imu_link</gz_frame_id>
+          <frame_id>imu_link</frame_id>
+          <enable_metrics>true</enable_metrics>
+          <magnetometer>
+            <x>
+              <noise type="gaussian">
+                <mean>0.0</mean>
+                <stddev>0.001</stddev>
+              </noise>
+            </x>
+            <y>
+              <noise type="gaussian">
+                <mean>0.0</mean>
+                <stddev>0.001</stddev>
+              </noise>
+            </y>
+            <z>
+              <noise type="gaussian">
+                <mean>0.0</mean>
+                <stddev>0.001</stddev>
+              </noise>
+            </z>
+          </magnetometer>
+        </sensor>
     </gazebo>
 </robot>

File: robots/dragger/description/robot.urdf.xacro (robot description, xacro)
@@ -14,5 +14,4 @@
     <xacro:property name="imu_visual_size" value="0.01"/>
     <xacro:include filename="../../../description/imu.xacro" />
-    <xacro:include filename="../../../description/magnetometer.xacro" />
     <!-- using arguments here, as that allows overriding default values -->
     <xacro:arg name="lidar_offset_x" default="${wheel_offset_x - 0.14}"/>

File: robots/plucky/description/robot.urdf.xacro (robot description, xacro)
@@ -14,5 +14,4 @@
     <xacro:property name="imu_visual_size" value="0.01"/>
     <xacro:include filename="../../../description/imu.xacro" />
-    <xacro:include filename="../../../description/magnetometer.xacro" />
     <!-- using arguments here, as that allows overriding default values -->
     <xacro:arg name="lidar_offset_x" default="${wheel_offset_x}"/>

File: robots/turtle/description/robot.urdf.xacro (robot description, xacro)
@@ -11,10 +11,23 @@
              The AutonomyLab *.xacro files are moved here because robot_description topic is published on the Desktop, not the robot RPi
     -->
+    <xacro:include filename="../../../description/common_properties.xacro" />
+    <!-- =========== an equivalent of "robot_core.xacro" here: ============== -->
     <xacro:include filename="../../../description/inertial_macros.xacro" />
-    <xacro:include filename="../../../description/common_properties.xacro" />
-    <xacro:include filename="create_1.urdf.xacro" />
+    <!-- wheel_separation - distance between left and right wheels, defined in ~/create_robot_ws/src/libcreate/src/types.cpp -->
+    <xacro:include filename="create_base.urdf.xacro" />
+    <xacro:create_base wheel_separation="0.258" base_diameter="0.3302" wheel_radius="0.033" wheel_width="0.024" mass_kg="3.5">
+        <mesh filename="package://articubot_one/assets/meshes/create_1.dae" />
+    </xacro:create_base>
+    <!-- ===================================================================== -->
+    <xacro:property name="imu_offset_x" value="-0.04"/>
+    <xacro:property name="imu_offset_z" value="0"/>
+    <xacro:property name="imu_visual_size" value="0.01"/>
+    <xacro:include filename="../../../description/imu.xacro" />
+    <xacro:property name="laser_offset_x" value="0.085"/>
+    <xacro:property name="laser_offset_z" value="0.033"/>
     <xacro:include filename="ros2_control.xacro" />
     <xacro:property name="open_circuit_voltage" value="14.0"/>
     <xacro:property name="battery_capacity" value="2.5"/>
     <xacro:include filename="../../../description/battery.xacro" />
+    <xacro:include filename="create_sensors.urdf.xacro" />
 </robot>
