Commit message: the name "laser_frame" should correspond to /scan topic header->frame_id

File: description/lidar.xacro (robot description, xacro)
@@ -5,8 +5,9 @@
     <joint name="laser_joint" type="fixed">
         <parent link="chassis_link"/>
-        <child link="laser_link"/>
+        <child link="laser_frame"/>
         <origin xyz="${laser_offset_x} 0 ${laser_offset_z}" rpy="0 0 3.1459"/>
     </joint>
-    <link name="laser_link">
+    <!-- the name "laser_frame" should correspond to /scan topic header->frame_id as defined in *.launch.py -->
+    <link name="laser_frame">
         <visual>
             <geometry>
@@ -32,5 +33,5 @@
     </link>
     <!-- gz model -m dragger -s front_laser -->
-    <gazebo reference="laser_link">
+    <gazebo reference="laser_frame">
         <sensor name='front_laser' type='gpu_lidar'>
           <pose>0 0 0 0 0 0</pose>

Commit message: Proper LIDAR orientation, separate xacro files for IMU and magnetometer

File: description/lidar.xacro (robot description, xacro)
@@ -3,8 +3,10 @@
     <xacro:property name="laser_offset_x" value="${chassis_length/4 + 0.05}"/>
     <xacro:property name="laser_offset_z" value="0.57"/>
+    <!-- ********************* LIDAR SETUP *********************************  -->
+    <!-- Each sensor must be attached to a link.                              -->
     <joint name="laser_joint" type="fixed">
         <parent link="chassis_link"/>
         <child link="laser_frame"/>
-        <origin xyz="${laser_offset_x} 0 ${laser_offset_z}" rpy="0 0 ${pi}"/>
+        <origin xyz="${laser_offset_x} 0 ${laser_offset_z}" rpy="0 0 0"/>
     </joint>
     <!-- the name "laser_frame" should correspond to /scan topic header->frame_id as defined in *.launch.py -->

File: description/robot.urdf.xacro (robot description, xacro)
@@ -38,4 +38,6 @@
     <xacro:include filename="robot_core.xacro" />
     <xacro:include filename="ros2_control.xacro" />
+    <xacro:include filename="imu.xacro" />
+    <xacro:include filename="magnetometer.xacro" />
     <xacro:include filename="lidar.xacro" />
     <xacro:include filename="camera.xacro" />

File: description/robot_core.xacro (robot description, xacro)
@@ -126,150 +126,4 @@
         </xacro:inertial_box>
     </link>
-    <!-- *********************** IMU SETUP *********************************  -->
-    <!-- Each sensor must be attached to a link.                              -->
-    <link name="imu_link">
-        <visual>
-            <geometry>
-                <box size="0.1 0.1 0.1"/>
-            </geometry>
-            <material name="sensor_blue"/>
-        </visual>
-    </link>
-    <joint name="imu_joint" type="fixed">
-        <parent link="chassis_link"/>
-        <child link="imu_link"/>
-        <!-- we place IMU between the wheels -->
-        <origin xyz="${wheel_offset_x} 0 0.04" rpy="0 0 0"/>
-    </joint>
-    <!-- gz model -m dragger -s imu_sensor -->
-    <gazebo reference="imu_link">
-        <sensor name="imu_link" type="imu">
-        <always_on>1</always_on>
-        <topic>imu/data</topic>
-        <!-- future Gazebo versions might require "<frame_id>" here. Must reference an actual link in .xacro -->
-        <gz_frame_id>imu_link</gz_frame_id>
-        <update_rate>250</update_rate>
-            <imu>
-                <orientation_reference_frame>
-                  <localization>ENU</localization>
-                  <!-- custom_rpy parent_frame='world'>1.570795 0 0</custom_rpy -->
-                </orientation_reference_frame>
-                <enable_orientation>1</enable_orientation>
-                <angular_velocity>
-                    <x>
-                        <noise type="gaussian">
-                            <mean>0</mean>
-                            <stddev>0.009</stddev>
-                            <bias_mean>0.00075</bias_mean>
-                            <bias_stddev>0.005</bias_stddev>
-                            <dynamic_bias_stddev>0.00002</dynamic_bias_stddev>
-                            <dynamic_bias_correlation_time>400.0</dynamic_bias_correlation_time>
-                            <precision>0.00025</precision>
-                        </noise>
-                    </x>
-                    <y>
-                        <noise type="gaussian">
-                            <mean>0</mean>
-                            <stddev>0.009</stddev>
-                            <bias_mean>0.00075</bias_mean>
-                            <bias_stddev>0.005</bias_stddev>
-                            <dynamic_bias_stddev>0.00002</dynamic_bias_stddev>
-                            <dynamic_bias_correlation_time>400.0</dynamic_bias_correlation_time>
-                            <precision>0.00025</precision>
-                        </noise>
-                    </y>
-                    <z>
-                        <noise type="gaussian">
-                            <mean>0</mean>
-                            <stddev>0.009</stddev>
-                            <bias_mean>0.00075</bias_mean>
-                            <bias_stddev>0.005</bias_stddev>
-                            <dynamic_bias_stddev>0.00002</dynamic_bias_stddev>
-                            <dynamic_bias_correlation_time>400.0</dynamic_bias_correlation_time>
-                            <precision>0.00025</precision>
-                        </noise>
-                    </z>
-                </angular_velocity>
-                <linear_acceleration>
-                    <x>
-                        <noise type="gaussian">
-                            <mean>0</mean>
-                            <stddev>0.021</stddev>
-                            <bias_mean>0.05</bias_mean>
-                            <bias_stddev>0.0075</bias_stddev>
-                            <dynamic_bias_stddev>0.000375</dynamic_bias_stddev>
-                            <dynamic_bias_correlation_time>175.0</dynamic_bias_correlation_time>
-                            <precision>0.005</precision>
-                        </noise>
-                    </x>
-                    <y>
-                        <noise type="gaussian">
-                            <mean>0</mean>
-                            <stddev>0.021</stddev>
-                            <bias_mean>0.05</bias_mean>
-                            <bias_stddev>0.0075</bias_stddev>
-                            <dynamic_bias_stddev>0.000375</dynamic_bias_stddev>
-                            <dynamic_bias_correlation_time>175.0</dynamic_bias_correlation_time>
-                            <precision>0.005</precision>
-                        </noise>
-                    </y>
-                    <z>
-                        <noise type="gaussian">
-                            <mean>0</mean>
-                            <stddev>0.021</stddev>
-                            <bias_mean>0.05</bias_mean>
-                            <bias_stddev>0.0075</bias_stddev>
-                            <dynamic_bias_stddev>0.000375</dynamic_bias_stddev>
-                            <dynamic_bias_correlation_time>175.0</dynamic_bias_correlation_time>
-                            <precision>0.005</precision>
-                        </noise>
-                    </z>
-                </linear_acceleration>
-            </imu>
-        </sensor>
-    </gazebo>
-    <link name="magnetometer_link">
-        <visual>
-            <geometry>
-                <box size="0.1 0.1 0.1"/>
-            </geometry>
-            <material name="sensor_blue"/>
-        </visual>
-    </link>
-    <joint name="magnetometer_joint" type="fixed">
-        <parent link="chassis_link"/>
-        <child link="magnetometer_link"/>
-        <!-- we place Magnetometer next to IMU between the wheels -->
-        <origin xyz="${wheel_offset_x} 0 0.03" rpy="0 0 0"/>
-    </joint>
-    <gazebo reference="magnetometer_link">
-        <sensor name="magnetometer" type="magnetometer">
-          <always_on>1</always_on>
-          <update_rate>100</update_rate>
-          <visualize>true</visualize>
-          <topic>magnetometer</topic>
-          <enable_metrics>true</enable_metrics>
-          <magnetometer>
-            <x>
-              <noise type="gaussian">
-                <mean>0.0</mean>
-                <stddev>0.001</stddev>
-              </noise>
-            </x>
-            <y>
-              <noise type="gaussian">
-                <mean>0.0</mean>
-                <stddev>0.001</stddev>
-              </noise>
-            </y>
-            <z>
-              <noise type="gaussian">
-                <mean>0.0</mean>
-                <stddev>0.001</stddev>
-              </noise>
-            </z>
-          </magnetometer>
-        </sensor>
-    </gazebo>
     <!-- LEFT WHEEL LINK -->
     <joint name="left_wheel_joint" type="continuous">

Commit message: WIP: trying to fix turtle slam_toolbox

File: description/lidar.xacro (robot description, xacro)
@@ -49,6 +49,6 @@
                 <samples>360</samples>
                 <resolution>1</resolution>
-                <min_angle>-${pi}</min_angle>
-                <max_angle>${pi}</max_angle>
+                <min_angle>-${PI}</min_angle>
+                <max_angle>${PI}</max_angle>
               </horizontal>
               <vertical>

File: robots/turtle/description/create_1.urdf.xacro (robot description, xacro)
@@ -2,4 +2,8 @@
 <robot name="create_1" xmlns:xacro="http://ros.org/wiki/xacro">
   <xacro:include filename="create_base.urdf.xacro" />
+  <xacro:property name="imu_offset_x" value="0"/>
+  <xacro:property name="imu_offset_z" value="0"/>
+  <xacro:property name="laser_offset_x" value="0.085"/>
+  <xacro:property name="laser_offset_z" value="0.033"/>
   <xacro:include filename="create_sensors.urdf.xacro" />
   <xacro:include filename="create_1_gazebo.urdf.xacro" />

File: robots/turtle/description/create_sensors.urdf.xacro (robot description, xacro)
@@ -4,11 +4,19 @@
       <parent link="chassis_link"/>
       <child link="imu_link"/>
-      <origin xyz="0.0 0 0.068" rpy="0 0 0"/>
+      <!-- we place IMU between the wheels -->
+      <origin xyz="${imu_offset_x} 0 ${imu_offset_z}" rpy="0 0 0"/>
     </joint>
-    <link name="imu_link"/>
-    <joint name="scan_joint" type="fixed">
+    <link name="imu_link">
+      <visual>
+        <geometry>
+          <box size="0.01 0.01 0.01"/>
+        </geometry>
+        <material name="sensor_blue"/>
+      </visual>
+    </link>
+    <joint name="laser_joint" type="fixed">
       <parent link="chassis_link"/>
       <child link="laser_frame"/>
-      <origin xyz="0.085 0 0.033" rpy="0 0 0"/>
+      <origin xyz="${laser_offset_x} 0 ${laser_offset_z}" rpy="0 0 0"/>
     </joint>
     <link name="laser_frame">

Commit message: Cartographer and slam_toolbox now work with ekf_odom filter

File: description/lidar.xacro (robot description, xacro)
@@ -49,6 +49,6 @@
                 <samples>360</samples>
                 <resolution>1</resolution>
-                <min_angle>-${PI}</min_angle>
-                <max_angle>${PI}</max_angle>
+                <min_angle>-${pi}</min_angle>
+                <max_angle>${pi}</max_angle>
               </horizontal>
               <vertical>

File: robots/turtle/description/create_1_gazebo.urdf.xacro (robot description, xacro)
@@ -106,6 +106,6 @@
                 <samples>360</samples>
                 <resolution>1</resolution>
-                <min_angle>-${PI}</min_angle>
-                <max_angle>${PI}</max_angle>
+                <min_angle>-${pi}</min_angle>
+                <max_angle>${pi}</max_angle>
               </horizontal>
               <vertical>

File: robots/turtle/description/create_base.urdf.xacro (robot description, xacro)
@@ -1,9 +1,8 @@
 ﻿<?xml version="1.0" encoding="UTF-8"?>
 <robot xmlns:xacro="http://ros.org/wiki/xacro">
-  <xacro:property name="PI" value="3.1415926535897931"/>
   <xacro:macro name="create_wheel" params="prefix y_offset wheel_radius wheel_width">
     <link name="${prefix}_wheel_link">
       <visual>
-        <origin xyz="0 0 0" rpy="0 ${PI/2} ${PI/2}"/>
+        <origin xyz="0 0 0" rpy="0 ${pi/2} ${pi/2}"/>
         <geometry>
           <cylinder radius="${wheel_radius}" length="${wheel_width}"/>
@@ -12,5 +11,5 @@
       </visual>
       <collision>
-        <origin xyz="0 0 0" rpy="0 ${PI/2} ${PI/2}"/>
+        <origin xyz="0 0 0" rpy="0 ${pi/2} ${pi/2}"/>
         <geometry>
           <cylinder radius="${wheel_radius}" length="${wheel_width}"/>
@@ -105,20 +104,20 @@
     </joint>
     <joint name="base_left_cliff_sensor_joint" type="fixed">
-      <origin xyz="0.07 0.14 0.01" rpy="0 ${PI/2} 0"/>
+      <origin xyz="0.07 0.14 0.01" rpy="0 ${pi/2} 0"/>
       <parent link="chassis_link"/>
       <child link="left_cliff_sensor_link"/>
     </joint>
     <joint name="base_right_cliff_sensor_joint" type="fixed">
-      <origin xyz="0.07 -0.14 0.01" rpy="0 ${PI/2} 0"/>
+      <origin xyz="0.07 -0.14 0.01" rpy="0 ${pi/2} 0"/>
       <parent link="chassis_link"/>
       <child link="right_cliff_sensor_link"/>
     </joint>
     <joint name="base_leftfront_cliff_sensor_joint" type="fixed">
-      <origin xyz="0.15 0.04 0.01" rpy="0 ${PI/2} 0"/>
+      <origin xyz="0.15 0.04 0.01" rpy="0 ${pi/2} 0"/>
       <parent link="chassis_link"/>
       <child link="leftfront_cliff_sensor_link"/>
     </joint>
     <joint name="base_rightfront_cliff_sensor_joint" type="fixed">
-      <origin xyz="0.15 -0.04 0.01" rpy="0 ${PI/2} 0"/>
+      <origin xyz="0.15 -0.04 0.01" rpy="0 ${pi/2} 0"/>
       <parent link="chassis_link"/>
       <child link="rightfront_cliff_sensor_link"/>
@@ -128,5 +127,5 @@
     <link name="front_castor_link">
       <visual>
-        <origin xyz="0 0 0" rpy="0 ${PI/2} ${PI/2}"/>
+        <origin xyz="0 0 0" rpy="0 ${pi/2} ${pi/2}"/>
         <geometry>
           <sphere radius="0.018"/>
@@ -135,5 +134,5 @@
       </visual>
       <collision>
-        <origin xyz="0 0 0" rpy="0 ${PI/2} ${PI/2}"/>
+        <origin xyz="0 0 0" rpy="0 ${pi/2} ${pi/2}"/>
         <geometry>
           <sphere radius="0.018"/>

Commit message: Manual copy/merge dev->main

File: description/lidar.xacro (robot description, xacro)
@@ -7,6 +7,6 @@
     <xacro:arg name="lidar_min_angle" default="-3.14159"/>
     <xacro:arg name="lidar_max_angle" default="3.14159"/>
-    <xacro:arg name="lidar_base_length" default="0.003"/>
-    <xacro:property name="_lidar_base_length" value="$(arg lidar_base_length)"/>
+    <xacro:arg name="lidar_pedestal_height" default="0.003"/>
+    <xacro:property name="_lidar_pedestal_height" value="$(arg lidar_pedestal_height)"/>
     <joint name="laser_joint" type="fixed">
         <parent link="chassis_link"/>
@@ -30,7 +30,7 @@
         </visual>
         <visual name="lidar_visual_base">
-            <origin xyz="0 0 -${_lidar_base_length/2+0.01}"/>
+            <origin xyz="0 0 -${_lidar_pedestal_height/2+0.01}"/>
             <geometry>
-                <cylinder radius="0.02" length="${_lidar_base_length}"/>
+                <cylinder radius="0.02" length="${_lidar_pedestal_height}"/>
             </geometry>
             <material name="body_color"/>

File: robots/dragger/description/robot.urdf.xacro (robot description, xacro)
@@ -18,5 +18,5 @@
     <xacro:arg name="lidar_offset_x" default="${wheel_offset_x - 0.14}"/>
     <xacro:arg name="lidar_offset_z" default="0.57"/>
-    <xacro:arg name="lidar_base_length" default="0.06"/>
+    <xacro:arg name="lidar_pedestal_height" default="0.06"/>
     <xacro:include filename="../../../description/lidar.xacro" />
     <xacro:property name="sonars_offset_x" value="${chassis_length/2 + 0.005}"/>

File: robots/plucky/description/robot.urdf.xacro (robot description, xacro)
@@ -18,5 +18,5 @@
     <xacro:arg name="lidar_offset_x" default="${wheel_offset_x}"/>
     <xacro:arg name="lidar_offset_z" default="0.47"/>
-    <xacro:arg name="lidar_base_length" default="0.01"/>
+    <xacro:arg name="lidar_pedestal_height" default="0.01"/>
     <xacro:include filename="../../../description/lidar.xacro" />
     <xacro:property name="sonars_offset_x" value="${chassis_length/2 + 0.005}"/>

File: robots/seggy/description/robot.urdf.xacro (robot description, xacro)
@@ -19,5 +19,5 @@
     <xacro:arg name="lidar_min_angle" default="-${pi * 0.95}"/>
     <xacro:arg name="lidar_max_angle" default="${pi * 0.95}"/>
-    <!-- xacro:arg name="lidar_base_length" default="0.04"/ -->
+    <!-- xacro:arg name="lidar_pedestal_height" default="0.04"/ -->
     <xacro:include filename="../../../description/lidar.xacro" />
     <xacro:property name="open_circuit_voltage" value="12.592"/>

Commit message: Dev -> JP magnetometer and IMU related changes

File: description/lidar.xacro (robot description, xacro)
@@ -74,5 +74,5 @@
             <range>
               <min>0.3</min>
-              <max>12.0</max>
+              <max>24.0</max>
               <resolution>0.01</resolution>
             </range>

File: robots/dragger/description/robot_core.xacro (robot description, xacro)
@@ -56,5 +56,5 @@
                 <cylinder radius="${wheel_offset_y + wheel_thickness / 2}" length="0.02"/>
             </geometry>
-            <material name="shadow_gray"/>
+            <material name="shadow_grey"/>
         </visual>
      </link>

File: robots/plucky/description/robot_core.xacro (robot description, xacro)
@@ -57,5 +57,5 @@
                 <cylinder radius="${wheel_offset_y + wheel_thickness + 0.03}" length="0.01"/>
             </geometry>
-            <material name="shadow_gray"/>
+            <material name="shadow_grey"/>
         </visual>
      </link>

File: robots/seggy/description/robot_core.xacro (robot description, xacro)
@@ -59,5 +59,5 @@
                 <cylinder radius="${wheel_offset_y + wheel_thickness + 0.03}" length="0.01"/>
             </geometry>
-            <material name="shadow_gray"/>
+            <material name="shadow_grey"/>
         </visual>
      </link>

File: robots/turtle/description/create_base.urdf.xacro (robot description, xacro)
@@ -8,5 +8,5 @@
           <cylinder radius="${wheel_radius}" length="${wheel_width}"/>
         </geometry>
-        <material name="gray"/>
+        <material name="grey"/>
       </visual>
       <collision>
@@ -47,5 +47,5 @@
               <cylinder radius="${base_diameter/2 + 0.01}" length="0.003"/>
           </geometry>
-          <material name="shadow_gray"/>
+          <material name="shadow_grey"/>
       </visual>
     </link>
@@ -129,5 +129,5 @@
           <sphere radius="0.018"/>
         </geometry>
-        <material name="gray"/>
+        <material name="grey"/>
       </visual>
       <collision>
