Commit message: WIP: simulated stereo_camera for RTAB-Map

File: description/camera_stereo.xacro (robot description, xacro)
@@ -37,63 +37,38 @@
         <parent link="camera_stereo_link"/>
         <child link="camera_stereo_link_optical"/>
-        <origin xyz="0 0 0" rpy="0 0 0"/>
+        <origin xyz="0 0 0" rpy="${-pi/2} 0 ${-pi/2}"/>
     </joint>
     <link name="camera_stereo_link_optical">
     </link>
     <!-- gz model -m dragger -s depth_camera -->
-	  <gazebo reference="camera_stereo_link_optical">
-        <sensor name='depth_camera' type='depth'>
-          <pose>0 0 0 0 0 0</pose>
-		      <always_on>true</always_on>
-          <topic>gz_depth_camera</topic>
-          <!-- future Gazebo versions might require "<frame_id>" here. Must reference an actual link in .xacro -->
-          <!-- see <optical_frame_id> below     <gz_frame_id>depth_camera_link_optical</gz_frame_id> -->
-          <update_rate>10</update_rate>
-          <visualize>true</visualize>
-          <enable_metrics>false</enable_metrics>
-          <camera name='__default__'>
-            <pose>0 0 0 0 0 0</pose>
-            <horizontal_fov>1.047</horizontal_fov>
-            <image>
-              <width>320</width>
-              <height>240</height>
-              <!--format>RGB_INT8</format -->
-              <!--format>B8G8R8</format -->
-              <format>L_INT16</format>
-              <anti_aliasing>4</anti_aliasing>
-            </image>
-            <camera_info_topic>gz_depth_camera_info</camera_info_topic>
-            <trigger_topic></trigger_topic>
-            <triggered>false</triggered>
-            <clip>
-              <near>0.1</near>
-              <far>8</far>
-            </clip>
-            <save enabled='false'>
-              <path>__default__</path>
-            </save>
-            <visibility_mask>4294967295</visibility_mask>
-            <noise>
-              <type>none</type>
-              <mean>0</mean>
-              <stddev>0</stddev>
-            </noise>
-            <distortion>
-              <k1>0</k1>
-              <k2>0</k2>
-              <k3>0</k3>
-              <p1>0</p1>
-              <p2>0</p2>
-              <center>0.5 0.5</center>
-            </distortion>
-            <lens>
-              <type>stereographic</type>
-              <scale_to_hfov>true</scale_to_hfov>
-              <cutoff_angle>${pi/2}</cutoff_angle>
-              <env_texture_size>256</env_texture_size>
-            </lens>
-            <optical_frame_id>camera_stereo_link_optical</optical_frame_id>
-          </camera>
-        </sensor>
+    <gazebo reference="camera_stereo_link_optical">
+      <!-- This sensor type is optimized for use with RTAB-Map on Dragger and Seggy ronots
+           See https://github.com/slgrobotics/articubot_one/wiki/Visual-SLAM-with-RTAB%E2%80%90Map -->
+      <sensor name="rgbd_camera" type="rgbd">
+        <always_on>true</always_on>
+        <update_rate>10</update_rate>
+        <visualize>true</visualize>
+        <topic>/camera_stereo</topic>
+        <camera_info_topic>/camera_stereo/camera_info</camera_info_topic>
+        <camera>
+          <horizontal_fov>1.047</horizontal_fov>
+          <image>
+            <!-- Use full size 820x616 or a 0.5 scale 408x308 -->
+            <width>820</width>
+            <height>616</height>
+            <format>R8G8B8</format>
+          </image>
+          <clip>
+            <near>0.1</near>
+            <far>8.0</far>
+          </clip>
+          <optical_frame_id>camera_stereo_link_optical</optical_frame_id>
+          <noise>
+            <type>gaussian</type>
+            <mean>0</mean>
+            <stddev>0.005</stddev>
+          </noise>
+        </camera>
+      </sensor>
     </gazebo>
 </robot>

File: description/depth_camera.xacro (robot description, xacro)
@@ -77,5 +77,5 @@
               <anti_aliasing>4</anti_aliasing>
             </image>
-            <camera_info_topic>gz_depth_camera_info</camera_info_topic>
+            <camera_info_topic>/gz_depth_camera_info</camera_info_topic>
             <trigger_topic></trigger_topic>
             <triggered>false</triggered>

Commit message: Update camera_stereo.xacro

File: description/camera_stereo.xacro (robot description, xacro)
@@ -37,5 +37,5 @@
         <parent link="camera_stereo_link"/>
         <child link="camera_stereo_link_optical"/>
-        <origin xyz="0 0 0" rpy="${-pi/2} 0 ${-pi/2}"/>
+        <origin xyz="0 0 0" rpy="0 0 0"/>
     </joint>
     <link name="camera_stereo_link_optical">

Commit message: Update camera_stereo.xacro

File: description/camera_stereo.xacro (robot description, xacro)
@@ -34,4 +34,10 @@
         </visual>
     </link>
+    <!-- REP-103 defines a Right-Handed, Z-Up coordinate system.
+        - X-Axis (Red in RViz):   Points Forward (the direction the robot drives)
+        - Y-Axis (Green in RViz): Points Left
+        - Z-Axis (Blue in RViz):  Points Up (against gravity)
+      The Gazebo camera is operating in that frame, with no rotation needed
+    -->
     <joint name="camera_stereo_optical_joint" type="fixed">
         <parent link="camera_stereo_link"/>
@@ -40,4 +46,20 @@
     </joint>
     <link name="camera_stereo_link_optical">
+    </link>
+    <!--  The Optical Coordinate System (For Cameras and Sensors)
+      Cameras view the world from a pixel grid perspective rather than a driving perspective.
+      Because of this, REP-103 defines a completely different axis standard for optical frames:
+      When looking out through the camera lens:
+        - Z-Axis: Points Forward (into the scene, acting as the Depth axis)
+        - X-Axis: Points Right   (horizontal pixel axis)
+        - Y-Axis: Points Down    (vertical pixel axis)
+      RTAB-Map relies on this standard to calculate visual odometry and project depth pixels into a 3D world
+    -->
+    <joint name="camera_stereo_optical2_joint" type="fixed">
+        <parent link="camera_stereo_link"/>
+        <child link="camera_stereo_link_optical2"/>
+        <origin xyz="0 0 0" rpy="${-pi/2} 0 ${-pi/2}"/>
+    </joint>
+    <link name="camera_stereo_link_optical2">
     </link>
     <!-- gz model -m dragger -s depth_camera -->
@@ -69,5 +91,5 @@
             <far>5.0</far>
           </clip>
-          <optical_frame_id>camera_stereo_link_optical</optical_frame_id>
+          <optical_frame_id>camera_stereo_link_optical2</optical_frame_id>
           <noise>
             <type>gaussian</type>

Commit message: Update camera_stereo.xacro

File: description/camera_stereo.xacro (robot description, xacro)
@@ -40,10 +40,10 @@
       The Gazebo camera is operating in that frame, with no rotation needed
     -->
-    <joint name="camera_stereo_optical_joint" type="fixed">
+    <joint name="camera_stereo_head_joint" type="fixed">
         <parent link="camera_stereo_link"/>
-        <child link="camera_stereo_link_optical"/>
+        <child link="camera_stereo_link_head"/>
         <origin xyz="0 0 0" rpy="0 0 0"/>
     </joint>
-    <link name="camera_stereo_link_optical">
+    <link name="camera_stereo_link_head">
     </link>
     <!--  The Optical Coordinate System (For Cameras and Sensors)
@@ -56,13 +56,13 @@
       RTAB-Map relies on this standard to calculate visual odometry and project depth pixels into a 3D world
     -->
-    <joint name="camera_stereo_optical2_joint" type="fixed">
+    <joint name="camera_stereo_optical_joint" type="fixed">
         <parent link="camera_stereo_link"/>
-        <child link="camera_stereo_link_optical2"/>
+        <child link="camera_stereo_link_optical"/>
         <origin xyz="0 0 0" rpy="${-pi/2} 0 ${-pi/2}"/>
     </joint>
-    <link name="camera_stereo_link_optical2">
+    <link name="camera_stereo_link_optical">
     </link>
     <!-- gz model -m dragger -s depth_camera -->
-    <gazebo reference="camera_stereo_link_optical">
+    <gazebo reference="camera_stereo_link_head">
       <!-- This sensor type is optimized for use with RTAB-Map on Dragger and Seggy robots
            See https://github.com/slgrobotics/articubot_one/wiki/Visual-SLAM-with-RTAB%E2%80%90Map
@@ -91,5 +91,5 @@
             <far>5.0</far>
           </clip>
-          <optical_frame_id>camera_stereo_link_optical2</optical_frame_id>
+          <optical_frame_id>camera_stereo_link_optical</optical_frame_id>
           <noise>
             <type>gaussian</type>

Commit message: Update camera_stereo.xacro

File: description/camera_stereo.xacro (robot description, xacro)
@@ -34,17 +34,4 @@
         </visual>
     </link>
-    <!-- REP-103 defines a Right-Handed, Z-Up coordinate system.
-        - X-Axis (Red in RViz):   Points Forward (the direction the robot drives)
-        - Y-Axis (Green in RViz): Points Left
-        - Z-Axis (Blue in RViz):  Points Up (against gravity)
-      The Gazebo camera is operating in that frame, with no rotation needed
-    -->
-    <joint name="camera_stereo_head_joint" type="fixed">
-        <parent link="camera_stereo_link"/>
-        <child link="camera_stereo_link_head"/>
-        <origin xyz="0 0 0" rpy="0 0 0"/>
-    </joint>
-    <link name="camera_stereo_link_head">
-    </link>
     <!--  The Optical Coordinate System (For Cameras and Sensors)
       Cameras view the world from a pixel grid perspective rather than a driving perspective.
@@ -55,4 +42,5 @@
         - Y-Axis: Points Down    (vertical pixel axis)
       RTAB-Map relies on this standard to calculate visual odometry and project depth pixels into a 3D world
+      So, we use <optical_frame_id>camera_stereo_link_optical</optical_frame_id> to force frame_id in message headers.
     -->
     <joint name="camera_stereo_optical_joint" type="fixed">
@@ -63,6 +51,12 @@
     <link name="camera_stereo_link_optical">
     </link>
-    <!-- gz model -m dragger -s depth_camera -->
-    <gazebo reference="camera_stereo_link_head">
+    <!-- REP-103 defines a Right-Handed, Z-Up coordinate system.
+        - X-Axis (Red in RViz):   Points Forward (the direction the robot drives)
+        - Y-Axis (Green in RViz): Points Left
+        - Z-Axis (Blue in RViz):  Points Up (against gravity)
+      The Gazebo camera is operating in that frame, with no rotation needed (uses camera_stereo_link)
+    -->
+    <!-- gz model -m dragger -s rgbd_camera -->
+    <gazebo reference="camera_stereo_link">
       <!-- This sensor type is optimized for use with RTAB-Map on Dragger and Seggy robots
            See https://github.com/slgrobotics/articubot_one/wiki/Visual-SLAM-with-RTAB%E2%80%90Map
