Commit message: Update camera_oakd.xacro

File: description/camera_oakd.xacro (robot description, xacro)
@@ -56,6 +56,9 @@
         <origin xyz="0 0 0" rpy="${-pi/2} 0 ${-pi/2}"/>
     </joint>
-    <link name="camera_oakd_link_optical">
-    </link>
+    <xacro:if value="$(arg sim_mode)">
+      <!-- OAK-D depthai_descr.urdf.xacro generates its own "parent_frame", in our case we want it to be "depth_camera_link_optical" -->
+      <link name="camera_oakd_link_optical">
+      </link>
+    </xacro:if>
     <!-- REP-103 defines a Right-Handed, Z-Up coordinate system.
         - X-Axis (Red in RViz):   Points Forward (the direction the robot drives)

Commit message: Rendering OAK-D Lite camera using DepthAI package STLs

File: description/camera_oakd.xacro (robot description, xacro)
@@ -13,4 +13,19 @@
     </joint>
     <link name="camera_oakd_link">
+        <visual name="oak-d_visual">
+            <origin xyz="0.007 0 0.005" rpy="${pi/2} 0 ${pi/2}" />
+            <geometry>
+                <mesh filename="model:/opt/ros/jazzy/share/depthai_descriptions/urdf/models/OAK-D-LITE.stl" scale="1.0 1.0 1.0"/>
+            </geometry>
+            <material name="dark_grey"/>
+        </visual>
+        <visual name="oak-d_visual_rviz">
+            <origin xyz="0.007 0 0.005" rpy="${pi/2} 0 ${pi/2}" />
+            <geometry>
+                <mesh filename="package://depthai_descriptions/urdf/models/OAK-D-LITE.stl" scale="1.0 1.0 1.0"/>
+            </geometry>
+            <material name="dark_grey"/>
+        </visual>
+        <!-- Use this when STL doesn't work:
         <visual>
             <geometry>
@@ -19,4 +34,5 @@
             <material name="sensor_blue"/>
         </visual>
+        -->
         <visual name="stereo_camera_visual_lens_center">
             <origin xyz="0.010 0 0.005" rpy="0 ${pi/2} 0"/>

File: description/common_properties.xacro (robot description, xacro)
@@ -19,4 +19,7 @@
     <material name="grey">
         <color rgba="0.5 0.5 0.5 1"/>
+    </material>
+    <material name="dark_grey">
+        <color rgba="0.15 0.15 0.15 0.9"/>
     </material>
     <material name="shadow_grey">

File: robots/seggy/description/robot.urdf.xacro (robot description, xacro)
@@ -37,5 +37,5 @@
             <visual>
             <geometry>
-                <box size="0.002 0.07 0.115"/>
+                <box size="0.005 0.07 0.115"/>
             </geometry>
             <material name="body_color"/>

Commit message: Update camera_oakd.xacro

File: description/camera_oakd.xacro (robot description, xacro)
@@ -70,5 +70,12 @@
         <parent link="camera_oakd_link"/>
         <child link="camera_oakd_link_optical"/>
-        <origin xyz="0 0 0" rpy="${-pi/2} 0 ${-pi/2}"/>
+        <xacro:if value="$(arg sim_mode)">
+          <!-- for Gazebo we need to rotate 'camera_oakd_link_optical' -->
+          <origin xyz="0 0 0" rpy="${-pi/2} 0 ${-pi/2}"/>
+        </xacro:if>
+        <xacro:unless value="$(arg sim_mode)">
+          <!-- real OAK-D camera creates 'camera_oakd_link_optical' already rotated -->
+          <origin xyz="0 0 0" rpy="0 0 0"/>
+        </xacro:unless>
     </joint>
     <xacro:if value="$(arg sim_mode)">

Commit message: Solving duplicate URDF mesh definitions

File: description/camera_oakd.xacro (robot description, xacro)
@@ -14,11 +14,4 @@
     <link name="camera_oakd_link">
         <visual name="oak-d_visual">
-            <origin xyz="0.007 0 0.005" rpy="${pi/2} 0 ${pi/2}" />
-            <geometry>
-                <mesh filename="model:/opt/ros/jazzy/share/depthai_descriptions/urdf/models/OAK-D-LITE.stl" scale="1.0 1.0 1.0"/>
-            </geometry>
-            <material name="dark_grey"/>
-        </visual>
-        <visual name="oak-d_visual_rviz">
             <origin xyz="0.007 0 0.005" rpy="${pi/2} 0 ${pi/2}" />
             <geometry>
