Commit message: Moved around files to "robots" directory to support multiple robot models

File: robots/sim/description/robot.urdf.xacro (robot description, xacro)
@@ -41,11 +41,11 @@
     <xacro:arg name="sim_mode" default="false"/>
     <xacro:include filename="robot_core.xacro" />
-    <xacro:include filename="imu.xacro" />
-    <xacro:include filename="magnetometer.xacro" />
-    <xacro:include filename="lidar.xacro" />
-    <xacro:include filename="gps.xacro" />
-    <xacro:include filename="camera.xacro" />
-    <!-- xacro:include filename="depth_camera.xacro" / -->
-    <!-- xacro:include filename="face.xacro" / -->
+    <xacro:include filename="../../../description/imu.xacro" />
+    <xacro:include filename="../../../description/magnetometer.xacro" />
+    <xacro:include filename="../../../description/lidar.xacro" />
+    <xacro:include filename="../../../description/gps.xacro" />
+    <xacro:include filename="../../../description/camera.xacro" />
+    <!-- xacro:include filename="../../../description/depth_camera.xacro" / -->
+    <!-- xacro:include filename="../../../description/face.xacro" / -->
     <xacro:include filename="ros2_control.xacro" />
 </robot>

File: robots/sim/description/robot_core.xacro (robot description, xacro)
@@ -1,5 +1,5 @@
 <?xml version="1.0"?>
 <robot xmlns:xacro="http://www.ros.org/wiki/xacro" >
-    <xacro:include filename="inertial_macros.xacro"/>
+    <xacro:include filename="../../../description/inertial_macros.xacro"/>
 	<!-- Values corrected for Dragger robot -->
     <xacro:property name="chassis_length" value="0.90"/>
@@ -149,5 +149,5 @@
             <origin xyz="0 0 0" rpy="${pi/2} 0 0" />
             <geometry>
-                <mesh filename="package://articubot_one/description/meshes/wheel_link.STL" scale="${wheel_radius*12.7} ${wheel_thickness*10.2} ${wheel_radius*12.7}"/>
+                <mesh filename="package://articubot_one/assets/meshes/wheel_link.STL" scale="${wheel_radius*12.7} ${wheel_thickness*10.2} ${wheel_radius*12.7}"/>
             </geometry>
             <material name="port_red"/>
@@ -220,5 +220,5 @@
             <origin xyz="0 0 0" rpy="${-pi/2} 0 0" />
             <geometry>
-                <mesh filename="package://articubot_one/description/meshes/wheel_link.STL" scale="${wheel_radius*12.7} ${wheel_thickness*10.2} ${wheel_radius*12.7}"/>
+                <mesh filename="package://articubot_one/assets/meshes/wheel_link.STL" scale="${wheel_radius*12.7} ${wheel_thickness*10.2} ${wheel_radius*12.7}"/>
             </geometry>
             <material name="starboard_green"/>

File: robots/sim/description/ros2_control.xacro (robot description, xacro)
@@ -75,6 +75,5 @@
             <robot_param>robot_description</robot_param>
             <robot_param_node>robot_state_publisher</robot_param_node> -->
-            <parameters>$(find articubot_one)/config/gaz_ros2_ctl_use_sim.yaml</parameters>
-            <parameters>$(find articubot_one)/config/controllers_sim.yaml</parameters>
+            <parameters>$(find articubot_one)/robots/sim/config/controllers.yaml</parameters>
         </plugin>
     </gazebo>
