Commit message: WIP: Create_1 shows up in RViz with Cartographer, wheels need work

File: robots/turtle/description/create_base.urdf.xacro (robot description, xacro)
@@ -29,5 +29,5 @@
     </joint>
   </xacro:macro>
-  <xacro:macro name="create_base" params="diffdrive_update_rate:=40 wheel_separation wheel_radius:=0.036 wheel_width:=0.024 wheel_torque:=1.0 wheel_accel:=1.8 mass_kg:=3.5 base_diameter *mesh">
+  <xacro:macro name="create_base" params="diffdrive_update_rate:=40 wheel_separation:=0.262 wheel_radius:=0.033 wheel_width:=0.024 wheel_torque:=1.0 wheel_accel:=1.8 mass_kg:=3.5 base_diameter *mesh">
     <xacro:include filename="$(find articubot_one)/robots/turtle/description/create_base_gazebo.urdf.xacro" />
     <link name="base_footprint">
@@ -35,7 +35,7 @@
       <origin xyz="0 0 0" rpy="0 0 0" />
       <geometry>
-        <box size="0.001 0.001 0.001" />
-      </geometry>
-      <material name="Green" />
+        <box size="0.005 0.005 0.005" />
+      </geometry>
+      <material name="green" />
     </visual>
     <collision>
@@ -184,16 +184,29 @@
       <axis xyz="0 1 0" />
     </joint>
-    <joint name="gyro_joint" type="fixed">
-      <axis xyz="0 1 0" />
-      <origin xyz="0 0 0.04" rpy="0 0 0" />
-      <parent link="base_link" />
-      <child link="gyro_link" />
-    </joint>
-    <link name="gyro_link">
-    <inertial>
-      <mass value="0.001" />
-      <origin xyz="0 0 0" rpy="0 0 0" />
-      <inertia ixx="0.0001" ixy="0" ixz="0" iyy="0.000001" iyz="0" izz="0.0001" />
-    </inertial>
+    <joint name="imu_joint" type="fixed">
+      <parent link="base_link"/>
+      <child link="imu_link"/>
+      <origin xyz="0.0 0 0.068" rpy="0 0 0"/>
+    </joint>
+    <link name="imu_link"/>
+    <joint name="scan_joint" type="fixed">
+      <parent link="base_link"/>
+      <child link="base_scan"/>
+      <origin xyz="-0.064 0 0.09" rpy="0 0 0"/>
+    </joint>
+    <link name="base_scan">
+      <visual>
+          <geometry>
+              <cylinder radius="0.0375" length="0.03"/>
+          </geometry>
+          <material name="sensor_blue"/>
+      </visual>
+      <visual>
+          <origin xyz="0 0 -0.01"/>
+          <geometry>
+              <cylinder radius="0.01" length="0.02"/>
+          </geometry>
+          <material name="sensor_blue"/>
+      </visual>
     </link>
     <!-- Simulation sensors -->

File: robots/turtle/description/robot.urdf.xacro (robot description, xacro)
@@ -14,7 +14,5 @@
     <xacro:arg name="sim_mode" default="false"/>
     <!-- xacro:include filename="common_properties.urdf" / -->
-    <material name="Green">
-        <color rgba="0.0 0.8 0.0 1.0"/>
-    </material>
+    <xacro:include filename="../../../description/common_properties.xacro" />
     <xacro:include filename="create_1.urdf.xacro" />
     <!-- xacro:include filename="../../../description/imu.xacro" />

Commit message: WIP: Create_1 turtle in the works

File: robots/turtle/description/create_base.urdf.xacro (robot description, xacro)
@@ -22,4 +22,5 @@
     </collision>
     </link>
+   <!-- joint name="${prefix}_wheel_joint" type="fixed" -->
    <joint name="${prefix}_wheel_joint" type="continuous">
       <origin xyz="0 ${y_offset} 0.015" rpy="0 0 0" />
@@ -193,10 +194,10 @@
       <parent link="base_link"/>
       <child link="base_scan"/>
-      <origin xyz="-0.064 0 0.09" rpy="0 0 0"/>
+      <origin xyz="0.085 0 0.08" rpy="0 0 0"/>
     </joint>
     <link name="base_scan">
       <visual>
           <geometry>
-              <cylinder radius="0.0375" length="0.03"/>
+              <cylinder radius="0.0375" length="0.025"/>
           </geometry>
           <material name="sensor_blue"/>

File: robots/turtle/description/robot.urdf.xacro (robot description, xacro)
@@ -8,7 +8,7 @@
           xacro install/articubot_one/share/articubot_one/robots/turtle/description/robot.urdf.xacro sim_mode:=false > src/articubot_one/robots/turtle/description/robot.urdf.generated.xml
     -->
-    <!-- See https://github.com/ROBOTIS-GIT/turtlebot3/tree/main/turtlebot3_description/urdf
-             https://github.com/slgrobotics/turtlebot3/commit/3df7ba0ea8944014ee9d2f29a438f830e2a0a031#diff-0de49a4761b9e2ca43e7f6e85e6f022224b347a9d374b30d4bf45ef4cc2fcf8b
-             ~/turtlebot3_ws/src/turtlebot3/turtlebot3/turtlebot3_description/urdf  -->
+    <!-- See https://github.com/slgrobotics/create_robot/tree/jazzy/create_description/urdf
+             The AutonomyLab *.xacro files are moved here because robot_description topic is published on the Desktop, not the robot RPi
+    -->
     <!-- xacro:include filename="../../../description/inertial_macros.xacro"/ -->
     <xacro:arg name="sim_mode" default="false"/>

Commit message: WIP: trying to use slam_toolbox on turtle

File: robots/turtle/description/create_base.urdf.xacro (robot description, xacro)
@@ -32,19 +32,4 @@
   <xacro:macro name="create_base" params="diffdrive_update_rate:=40 wheel_separation:=0.262 wheel_radius:=0.033 wheel_width:=0.024 wheel_torque:=1.0 wheel_accel:=1.8 mass_kg:=3.5 base_diameter *mesh">
     <xacro:include filename="$(find articubot_one)/robots/turtle/description/create_base_gazebo.urdf.xacro" />
-    <link name="base_footprint">
-    <visual>
-      <origin xyz="0 0 0" rpy="0 0 0" />
-      <geometry>
-        <box size="0.005 0.005 0.005" />
-      </geometry>
-      <material name="green" />
-    </visual>
-    <collision>
-      <origin xyz="0 0 0.017" rpy="0 0 0" />
-      <geometry>
-        <box size="0.001 0.001 0.001" />
-      </geometry>
-    </collision>
-    </link>
     <link name="base_link">
     <inertial>
@@ -53,57 +38,72 @@
       <inertia ixx="0.01" ixy="0.0" ixz="0.0" iyy="0.01" iyz="0.0" izz="0.5" />
     </inertial>
-    <visual>
-      <origin xyz=" 0 0 0.0308" rpy="0 0 0" />
-      <geometry>
-        <xacro:insert_block name="mesh" />
-      </geometry>
-    </visual>
-    <collision>
-      <origin xyz="0.0 0.0 0.0308" rpy="0 0 0" />
-      <geometry>
-        <cylinder length="0.0611632" radius="0.16495" />
-      </geometry>
-    </collision>
-    </link>
-    <link name="wall_sensor_link">
-    <inertial>
-      <mass value="0.01" />
-      <origin xyz="0 0 0" />
-      <inertia ixx="0.001" ixy="0.0" ixz="0.0" iyy="0.001" iyz="0.0" izz="0.001" />
-    </inertial>
-    </link>
-    <link name="left_cliff_sensor_link">
-    <inertial>
-      <mass value="0.01" />
-      <origin xyz="0 0 0" />
-      <inertia ixx="0.001" ixy="0.0" ixz="0.0" iyy="0.001" iyz="0.0" izz="0.001" />
-    </inertial>
-    </link>
-    <link name="right_cliff_sensor_link">
-    <inertial>
-      <mass value="0.01" />
-      <origin xyz="0 0 0" />
-      <inertia ixx="0.001" ixy="0.0" ixz="0.0" iyy="0.001" iyz="0.0" izz="0.001" />
-    </inertial>
-    </link>
-    <link name="leftfront_cliff_sensor_link">
-    <inertial>
-      <mass value="0.01" />
-      <origin xyz="0 0 0" />
-      <inertia ixx="1.0" ixy="0.0" ixz="0.0" iyy="0.01" iyz="0.0" izz="0.01" />
-    </inertial>
-    </link>
-    <link name="rightfront_cliff_sensor_link">
-    <inertial>
-      <mass value="0.01" />
-      <origin xyz="0 0 0" />
-      <inertia ixx="0.001" ixy="0.0" ixz="0.0" iyy="0.001" iyz="0.0" izz="0.001" />
-    </inertial>
-    </link>
+    <link name="base_footprint">
+    <visual>
+      <origin xyz="0 0 0" rpy="0 0 0" />
+      <geometry>
+        <box size="0.005 0.005 0.005" />
+      </geometry>
+      <material name="green" />
+    </visual>
     <joint name="base_footprint_joint" type="fixed">
       <origin xyz="0 0 0.017" rpy="0 0 0" />
-      <parent link="base_footprint" />
-      <child link="base_link" />
-    </joint>
+      <parent link="base_link" />
+      <child link="base_footprint" />
+    </joint>
+    <collision>
+      <origin xyz="0 0 0.017" rpy="0 0 0" />
+      <geometry>
+        <box size="0.001 0.001 0.001" />
+      </geometry>
+    </collision>
+    </link>
+    <visual>
+      <origin xyz=" 0 0 0.0308" rpy="0 0 0" />
+      <geometry>
+        <xacro:insert_block name="mesh" />
+      </geometry>
+    </visual>
+    <collision>
+      <origin xyz="0.0 0.0 0.0308" rpy="0 0 0" />
+      <geometry>
+        <cylinder length="0.0611632" radius="0.16495" />
+      </geometry>
+    </collision>
+    </link>
+    <link name="wall_sensor_link">
+    <inertial>
+      <mass value="0.01" />
+      <origin xyz="0 0 0" />
+      <inertia ixx="0.001" ixy="0.0" ixz="0.0" iyy="0.001" iyz="0.0" izz="0.001" />
+    </inertial>
+    </link>
+    <link name="left_cliff_sensor_link">
+    <inertial>
+      <mass value="0.01" />
+      <origin xyz="0 0 0" />
+      <inertia ixx="0.001" ixy="0.0" ixz="0.0" iyy="0.001" iyz="0.0" izz="0.001" />
+    </inertial>
+    </link>
+    <link name="right_cliff_sensor_link">
+    <inertial>
+      <mass value="0.01" />
+      <origin xyz="0 0 0" />
+      <inertia ixx="0.001" ixy="0.0" ixz="0.0" iyy="0.001" iyz="0.0" izz="0.001" />
+    </inertial>
+    </link>
+    <link name="leftfront_cliff_sensor_link">
+    <inertial>
+      <mass value="0.01" />
+      <origin xyz="0 0 0" />
+      <inertia ixx="1.0" ixy="0.0" ixz="0.0" iyy="0.01" iyz="0.0" izz="0.01" />
+    </inertial>
+    </link>
+    <link name="rightfront_cliff_sensor_link">
+    <inertial>
+      <mass value="0.01" />
+      <origin xyz="0 0 0" />
+      <inertia ixx="0.001" ixy="0.0" ixz="0.0" iyy="0.001" iyz="0.0" izz="0.001" />
+    </inertial>
+    </link>
     <joint name="base_wall_sensor_joint" type="fixed">
       <origin xyz="0.09 -0.120 0.042" rpy="0 0 -1.0" />

Commit message: Pretty-printed and improved create_base.urdf.xacro

File: robots/turtle/description/create_base.urdf.xacro (robot description, xacro)
@@ -1,133 +1,142 @@
-<?xml version="1.0" ?>
+﻿<?xml version="1.0" encoding="UTF-8"?>
 <robot xmlns:xacro="http://ros.org/wiki/xacro">
-  <xacro:property name="PI" value="3.1415926535897931" />
+  <xacro:property name="PI" value="3.1415926535897931"/>
   <xacro:macro name="create_wheel" params="prefix y_offset wheel_radius wheel_width">
     <link name="${prefix}_wheel_link">
-    <inertial>
-      <origin xyz="0 0 0" />
-      <mass value="0.01" />
-      <inertia ixx="0.001" ixy="0.0" ixz="0.0" iyy="0.001" iyz="0.0" izz="0.001" />
-    </inertial>
-    <visual>
-      <origin xyz="0 0 0" rpy="0 ${PI/2} ${PI/2}" />
-      <geometry>
-        <cylinder radius="${wheel_radius}" length="${wheel_width}" />
-      </geometry>
-    </visual>
-    <collision>
-      <origin xyz="0 0 0" rpy="0 ${PI/2} ${PI/2}" />
-      <geometry>
-        <cylinder radius="${wheel_radius}" length="${wheel_width}" />
-      </geometry>
-    </collision>
-    </link>
-   <!-- joint name="${prefix}_wheel_joint" type="fixed" -->
-   <joint name="${prefix}_wheel_joint" type="continuous">
-      <origin xyz="0 ${y_offset} 0.015" rpy="0 0 0" />
-      <parent link="base_link" />
-      <child link="${prefix}_wheel_link" />
-      <axis xyz="0 1 0" />
+      <inertial>
+        <origin xyz="0 0 0"/>
+        <mass value="0.01"/>
+        <inertia ixx="0.001" ixy="0.0" ixz="0.0" iyy="0.001" iyz="0.0" izz="0.001"/>
+      </inertial>
+      <visual>
+        <origin xyz="0 0 0" rpy="0 ${PI/2} ${PI/2}"/>
+        <geometry>
+          <cylinder radius="${wheel_radius}" length="${wheel_width}"/>
+        </geometry>
+      </visual>
+      <collision>
+        <origin xyz="0 0 0" rpy="0 ${PI/2} ${PI/2}"/>
+        <geometry>
+          <cylinder radius="${wheel_radius}" length="${wheel_width}"/>
+        </geometry>
+      </collision>
+    </link>
+    <!-- joint name="${prefix}_wheel_joint" type="fixed" -->
+    <joint name="${prefix}_wheel_joint" type="continuous">
+      <origin xyz="0 ${y_offset} 0.015" rpy="0 0 0"/>
+      <parent link="base_link"/>
+      <child link="${prefix}_wheel_link"/>
+      <axis xyz="0 1 0"/>
     </joint>
   </xacro:macro>
   <xacro:macro name="create_base" params="diffdrive_update_rate:=40 wheel_separation:=0.262 wheel_radius:=0.033 wheel_width:=0.024 wheel_torque:=1.0 wheel_accel:=1.8 mass_kg:=3.5 base_diameter *mesh">
-    <xacro:include filename="$(find articubot_one)/robots/turtle/description/create_base_gazebo.urdf.xacro" />
+    <xacro:include filename="$(find articubot_one)/robots/turtle/description/create_base_gazebo.urdf.xacro"/>
     <link name="base_link">
-    <inertial>
-      <mass value="2" />
-      <origin xyz="0 0 0.0" />
-      <inertia ixx="0.01" ixy="0.0" ixz="0.0" iyy="0.01" iyz="0.0" izz="0.5" />
-    </inertial>
+      <visual name="baselink_visual">
+          <origin xyz="0 0 0"/>
+          <geometry>
+              <sphere radius="0.04"/>
+          </geometry>
+          <material name="red"/>
+      </visual>
+    </link>
     <link name="base_footprint">
-    <visual>
-      <origin xyz="0 0 0" rpy="0 0 0" />
-      <geometry>
-        <box size="0.005 0.005 0.005" />
-      </geometry>
-      <material name="green" />
-    </visual>
+      <visual name="footprint_visual">
+          <origin xyz="0 0 0.001"/>
+          <geometry>
+              <cylinder radius="0.16495" length="0.002"/>
+          </geometry>
+          <material name="shadow_grey"/>
+      </visual>
+    </link>
     <joint name="base_footprint_joint" type="fixed">
-      <origin xyz="0 0 0.017" rpy="0 0 0" />
-      <parent link="base_link" />
-      <child link="base_footprint" />
-    </joint>
-    <collision>
-      <origin xyz="0 0 0.017" rpy="0 0 0" />
-      <geometry>
-        <box size="0.001 0.001 0.001" />
-      </geometry>
-    </collision>
-    </link>
-    <visual>
-      <origin xyz=" 0 0 0.0308" rpy="0 0 0" />
-      <geometry>
-        <xacro:insert_block name="mesh" />
-      </geometry>
-    </visual>
-    <collision>
-      <origin xyz="0.0 0.0 0.0308" rpy="0 0 0" />
-      <geometry>
-        <cylinder length="0.0611632" radius="0.16495" />
-      </geometry>
-    </collision>
+      <origin xyz="0 0 0.017" rpy="0 0 0"/>
+      <parent link="base_link"/>
+      <child link="base_footprint"/>
+    </joint>
+    <joint name="chassis_joint" type="fixed">
+      <parent link="base_link"/>
+      <child link="chassis_link"/>
+      <origin xyz="0 0 0"/>
+    </joint>
+    <!-- CHASSIS LINK -->
+    <link name="chassis_link">
+      <inertial>
+        <mass value="${mass_kg}"/>
+        <origin xyz="0 0 0.0"/>
+        <inertia ixx="0.01" ixy="0.0" ixz="0.0" iyy="0.01" iyz="0.0" izz="0.5"/>
+      </inertial>
+      <visual>
+        <origin xyz=" 0 0 0.0308" rpy="0 0 0"/>
+        <geometry>
+          <xacro:insert_block name="mesh"/>
+        </geometry>
+      </visual>
+      <collision>
+        <origin xyz="0.0 0.0 0.0308" rpy="0 0 0"/>
+        <geometry>
+          <cylinder length="0.0611632" radius="0.16495"/>
+        </geometry>
+      </collision>
     </link>
     <link name="wall_sensor_link">
-    <inertial>
-      <mass value="0.01" />
-      <origin xyz="0 0 0" />
-      <inertia ixx="0.001" ixy="0.0" ixz="0.0" iyy="0.001" iyz="0.0" izz="0.001" />
-    </inertial>
+      <inertial>
+        <mass value="0.01"/>
+        <origin xyz="0 0 0"/>
+        <inertia ixx="0.001" ixy="0.0" ixz="0.0" iyy="0.001" iyz="0.0" izz="0.001"/>
+      </inertial>
     </link>
     <link name="left_cliff_sensor_link">
-    <inertial>
-      <mass value="0.01" />
-      <origin xyz="0 0 0" />
-      <inertia ixx="0.001" ixy="0.0" ixz="0.0" iyy="0.001" iyz="0.0" izz="0.001" />
-    </inertial>
+      <inertial>
+        <mass value="0.01"/>
+        <origin xyz="0 0 0"/>
+        <inertia ixx="0.001" ixy="0.0" ixz="0.0" iyy="0.001" iyz="0.0" izz="0.001"/>
+      </inertial>
     </link>
     <link name="right_cliff_sensor_link">
-    <inertial>
-      <mass value="0.01" />
-      <origin xyz="0 0 0" />
-      <inertia ixx="0.001" ixy="0.0" ixz="0.0" iyy="0.001" iyz="0.0" izz="0.001" />
-    </inertial>
+      <inertial>
+        <mass value="0.01"/>
+        <origin xyz="0 0 0"/>
+        <inertia ixx="0.001" ixy="0.0" ixz="0.0" iyy="0.001" iyz="0.0" izz="0.001"/>
+      </inertial>
     </link>
     <link name="leftfront_cliff_sensor_link">
-    <inertial>
-      <mass value="0.01" />
-      <origin xyz="0 0 0" />
-      <inertia ixx="1.0" ixy="0.0" ixz="0.0" iyy="0.01" iyz="0.0" izz="0.01" />
-    </inertial>
+      <inertial>
+        <mass value="0.01"/>
+        <origin xyz="0 0 0"/>
+        <inertia ixx="1.0" ixy="0.0" ixz="0.0" iyy="0.01" iyz="0.0" izz="0.01"/>
+      </inertial>
     </link>
     <link name="rightfront_cliff_sensor_link">
-    <inertial>
-      <mass value="0.01" />
-      <origin xyz="0 0 0" />
-      <inertia ixx="0.001" ixy="0.0" ixz="0.0" iyy="0.001" iyz="0.0" izz="0.001" />
-    </inertial>
+      <inertial>
+        <mass value="0.01"/>
+        <origin xyz="0 0 0"/>
+        <inertia ixx="0.001" ixy="0.0" ixz="0.0" iyy="0.001" iyz="0.0" izz="0.001"/>
+      </inertial>
     </link>
     <joint name="base_wall_sensor_joint" type="fixed">
-      <origin xyz="0.09 -0.120 0.042" rpy="0 0 -1.0" />
-      <parent link="base_link" />
-      <child link="wall_sensor_link" />
+      <origin xyz="0.09 -0.120 0.042" rpy="0 0 -1.0"/>
+      <parent link="base_link"/>
+      <child link="wall_sensor_link"/>
     </joint>
     <joint name="base_left_cliff_sensor_joint" type="fixed">
-      <origin xyz="0.07 0.14 0.01" rpy="0 ${PI/2} 0" />
-      <parent link="base_link" />
-      <child link="left_cliff_sensor_link" />
+      <origin xyz="0.07 0.14 0.01" rpy="0 ${PI/2} 0"/>
+      <parent link="base_link"/>
+      <child link="left_cliff_sensor_link"/>
     </joint>
     <joint name="base_right_cliff_sensor_joint" type="fixed">
-      <origin xyz="0.07 -0.14 0.01" rpy="0 ${PI/2} 0" />
-      <parent link="base_link" />
-      <child link="right_cliff_sensor_link" />
+      <origin xyz="0.07 -0.14 0.01" rpy="0 ${PI/2} 0"/>
+      <parent link="base_link"/>
+      <child link="right_cliff_sensor_link"/>
     </joint>
     <joint name="base_leftfront_cliff_sensor_joint" type="fixed">
-      <origin xyz="0.15 0.04 0.01" rpy="0 ${PI/2} 0" />
-      <parent link="base_link" />
-      <child link="leftfront_cliff_sensor_link" />
+      <origin xyz="0.15 0.04 0.01" rpy="0 ${PI/2} 0"/>
+      <parent link="base_link"/>
+      <child link="leftfront_cliff_sensor_link"/>
     </joint>
     <joint name="base_rightfront_cliff_sensor_joint" type="fixed">
-      <origin xyz="0.15 -0.04 0.01" rpy="0 ${PI/2} 0" />
-      <parent link="base_link" />
-      <child link="rightfront_cliff_sensor_link" />
+      <origin xyz="0.15 -0.04 0.01" rpy="0 ${PI/2} 0"/>
+      <parent link="base_link"/>
+      <child link="rightfront_cliff_sensor_link"/>
     </joint>
     <xacro:create_wheel prefix="left" y_offset="${wheel_separation / 2}" wheel_radius="${wheel_radius}" wheel_width="${wheel_width}"/>
@@ -160,28 +169,28 @@
     </joint>-->
     <link name="front_wheel_link">
-    <inertial>
-      <origin xyz="0 0 0" />
-      <mass value="0.01" />
-      <inertia ixx="0.001" ixy="0.0" ixz="0.0" iyy="0.001" iyz="0.0" izz="0.001" />
-    </inertial>
-    <visual>
-      <origin xyz="0 0 0" rpy="0 ${PI/2} ${PI/2}" />
-      <geometry>
-        <sphere radius="0.018" />
-      </geometry>
-    </visual>
-    <collision>
-      <origin xyz="0 0 0" rpy="0 ${PI/2} ${PI/2}" />
-      <geometry>
-        <sphere radius="0.018" />
-      </geometry>
-    </collision>
+      <inertial>
+        <origin xyz="0 0 0"/>
+        <mass value="0.01"/>
+        <inertia ixx="0.001" ixy="0.0" ixz="0.0" iyy="0.001" iyz="0.0" izz="0.001"/>
+      </inertial>
+      <visual>
+        <origin xyz="0 0 0" rpy="0 ${PI/2} ${PI/2}"/>
+        <geometry>
+          <sphere radius="0.018"/>
+        </geometry>
+      </visual>
+      <collision>
+        <origin xyz="0 0 0" rpy="0 ${PI/2} ${PI/2}"/>
+        <geometry>
+          <sphere radius="0.018"/>
+        </geometry>
+      </collision>
     </link>
     <!-- fixed because there's no transmission -->
     <joint name="front_castor_joint" type="fixed">
-      <origin xyz="0.13 0 0.0" rpy="0 0 0" />
-      <parent link="base_link" />
-      <child link="front_wheel_link" />
-      <axis xyz="0 1 0" />
+      <origin xyz="0.13 0 0.0" rpy="0 0 0"/>
+      <parent link="base_link"/>
+      <child link="front_wheel_link"/>
+      <axis xyz="0 1 0"/>
     </joint>
     <joint name="imu_joint" type="fixed">
@@ -198,15 +207,15 @@
     <link name="base_scan">
       <visual>
-          <geometry>
-              <cylinder radius="0.0375" length="0.025"/>
-          </geometry>
-          <material name="sensor_blue"/>
-      </visual>
-      <visual>
-          <origin xyz="0 0 -0.01"/>
-          <geometry>
-              <cylinder radius="0.01" length="0.02"/>
-          </geometry>
-          <material name="sensor_blue"/>
+        <geometry>
+          <cylinder radius="0.0375" length="0.025"/>
+        </geometry>
+        <material name="sensor_blue"/>
+      </visual>
+      <visual>
+        <origin xyz="0 0 -0.01"/>
+        <geometry>
+          <cylinder radius="0.01" length="0.02"/>
+        </geometry>
+        <material name="sensor_blue"/>
       </visual>
     </link>
