Commit message: Updated create_1 xacro file

File: robots/turtle/description/create_base.urdf.xacro (robot description, xacro)
@@ -30,6 +30,8 @@
     </joint>
   </xacro:macro>
-  <xacro:macro name="create_base" params="diffdrive_update_rate:=40 wheel_separation:=0.262 wheel_radius:=0.033 wheel_width:=0.024 wheel_torque:=1.0 wheel_accel:=1.8 mass_kg:=3.5 base_diameter *mesh">
+  <xacro:macro name="create_base"
+               params="diffdrive_update_rate:=40 wheel_separation wheel_radius:=0.033 wheel_width:=0.024 wheel_torque:=1.0 wheel_accel:=1.8 mass_kg:=3.5 base_diameter *mesh">
     <xacro:include filename="$(find articubot_one)/robots/turtle/description/create_base_gazebo.urdf.xacro"/>
+    <!-- The coordinate frame called base_link is rigidly attached to the robot root body. -->
     <link name="base_link">
       <visual name="baselink_visual">
@@ -41,17 +43,19 @@
       </visual>
     </link>
+    <!-- Define the center of the main robot chassis projected on the ground -->
     <link name="base_footprint">
       <visual name="footprint_visual">
           <origin xyz="0 0 0.001"/>
           <geometry>
-              <cylinder radius="0.16495" length="0.002"/>
+              <cylinder radius="${base_diameter/2 + 0.01}" length="0.003"/>
           </geometry>
           <material name="shadow_grey"/>
       </visual>
     </link>
+    <!-- The base footprint of the robot is located underneath the chassis -->
     <joint name="base_footprint_joint" type="fixed">
-      <origin xyz="0 0 0.017" rpy="0 0 0"/>
-      <parent link="base_link"/>
-      <child link="base_footprint"/>
+      <parent link="base_link"/>
+      <child link="base_footprint" />
+      <origin xyz="0 0 -${wheel_radius}" rpy="0 0 0"/>
     </joint>
     <joint name="chassis_joint" type="fixed">
@@ -142,30 +146,4 @@
     <xacro:create_wheel prefix="left" y_offset="${wheel_separation / 2}" wheel_radius="${wheel_radius}" wheel_width="${wheel_width}"/>
     <xacro:create_wheel prefix="right" y_offset="${wheel_separation / -2}" wheel_radius="${wheel_radius}" wheel_width="${wheel_width}"/>
-    <!--<link name="rear_wheel_link">
-    <inertial>
-      <origin xyz="0 0 0"/>
-      <mass value="0.001" />
-      <inertia ixx="0.0001" ixy="0.0" ixz="0.0"
-        iyy="0.0001" iyz="0.0" izz="0.0001" />
-    </inertial>
-    <visual>
-      <origin xyz="0 0 0" rpy="0 ${PI/2} ${PI/2}"/>
-      <geometry>
-        <sphere radius="0.015" />
-      </geometry>
-    </visual>
-    <collision>
-      <origin xyz="0 0 0" rpy="0 ${PI/2} ${PI/2}" />
-      <geometry>
-        <sphere radius="0.015" />
-      </geometry>
-    </collision>
-    </link>
-    <joint name="rear_castor_joint" type="fixed">
-      <origin xyz="-0.13 0 0.0" rpy="0 0 0"/>
-      <parent link="base_link"/>
-      <child link="rear_wheel_link"/>
-      <axis xyz="0 1 0"/>
-    </joint>-->
     <link name="front_wheel_link">
       <inertial>

Commit message: Launch files cleanup; Turtle shows all right in RViz

File: robots/turtle/description/create_base.urdf.xacro (robot description, xacro)
@@ -180,8 +180,8 @@
     <joint name="scan_joint" type="fixed">
       <parent link="base_link"/>
-      <child link="base_scan"/>
+      <child link="laser_frame"/>
       <origin xyz="0.085 0 0.08" rpy="0 0 0"/>
     </joint>
-    <link name="base_scan">
+    <link name="laser_frame">
       <visual>
         <geometry>

Commit message: WIP: turtle inertias replaced with macros

File: robots/turtle/description/create_base.urdf.xacro (robot description, xacro)
@@ -4,9 +4,4 @@
   <xacro:macro name="create_wheel" params="prefix y_offset wheel_radius wheel_width">
     <link name="${prefix}_wheel_link">
-      <inertial>
-        <origin xyz="0 0 0"/>
-        <mass value="0.01"/>
-        <inertia ixx="0.001" ixy="0.0" ixz="0.0" iyy="0.001" iyz="0.0" izz="0.001"/>
-      </inertial>
       <visual>
         <origin xyz="0 0 0" rpy="0 ${PI/2} ${PI/2}"/>
@@ -22,4 +17,7 @@
         </geometry>
       </collision>
+      <xacro:inertial_cylinder mass="0.01" length="${wheel_width}" radius="${wheel_radius}">
+          <origin xyz="0 0 0" rpy="0 0 0"/>
+      </xacro:inertial_cylinder>
     </link>
     <!-- joint name="${prefix}_wheel_joint" type="fixed" -->
@@ -68,9 +66,4 @@
     <!-- CHASSIS LINK -->
     <link name="chassis_link">
-      <inertial>
-        <mass value="${mass_kg}"/>
-        <origin xyz="0 0 0.0"/>
-        <inertia ixx="0.01" ixy="0.0" ixz="0.0" iyy="0.01" iyz="0.0" izz="0.5"/>
-      </inertial>
       <visual>
         <origin xyz=" 0 0 -0.015" rpy="0 0 0"/>
@@ -85,39 +78,17 @@
         </geometry>
       </collision>
+      <xacro:inertial_cylinder mass="${mass_kg}" length="0.0611632" radius="${base_diameter/2}">
+          <origin xyz="0 0 -0.015" rpy="0 0 0"/>
+      </xacro:inertial_cylinder>
     </link>
     <link name="wall_sensor_link">
-      <inertial>
-        <mass value="0.01"/>
-        <origin xyz="0 0 0"/>
-        <inertia ixx="0.001" ixy="0.0" ixz="0.0" iyy="0.001" iyz="0.0" izz="0.001"/>
-      </inertial>
     </link>
     <link name="left_cliff_sensor_link">
-      <inertial>
-        <mass value="0.01"/>
-        <origin xyz="0 0 0"/>
-        <inertia ixx="0.001" ixy="0.0" ixz="0.0" iyy="0.001" iyz="0.0" izz="0.001"/>
-      </inertial>
     </link>
     <link name="right_cliff_sensor_link">
-      <inertial>
-        <mass value="0.01"/>
-        <origin xyz="0 0 0"/>
-        <inertia ixx="0.001" ixy="0.0" ixz="0.0" iyy="0.001" iyz="0.0" izz="0.001"/>
-      </inertial>
     </link>
     <link name="leftfront_cliff_sensor_link">
-      <inertial>
-        <mass value="0.01"/>
-        <origin xyz="0 0 0"/>
-        <inertia ixx="1.0" ixy="0.0" ixz="0.0" iyy="0.01" iyz="0.0" izz="0.01"/>
-      </inertial>
     </link>
     <link name="rightfront_cliff_sensor_link">
-      <inertial>
-        <mass value="0.01"/>
-        <origin xyz="0 0 0"/>
-        <inertia ixx="0.001" ixy="0.0" ixz="0.0" iyy="0.001" iyz="0.0" izz="0.001"/>
-      </inertial>
     </link>
     <joint name="base_wall_sensor_joint" type="fixed">
@@ -149,9 +120,4 @@
     <xacro:create_wheel prefix="right" y_offset="${wheel_separation / -2}" wheel_radius="${wheel_radius}" wheel_width="${wheel_width}"/>
     <link name="front_castor_link">
-      <inertial>
-        <origin xyz="0 0 0"/>
-        <mass value="0.01"/>
-        <inertia ixx="0.001" ixy="0.0" ixz="0.0" iyy="0.001" iyz="0.0" izz="0.001"/>
-      </inertial>
       <visual>
         <origin xyz="0 0 0" rpy="0 ${PI/2} ${PI/2}"/>
@@ -167,4 +133,7 @@
         </geometry>
       </collision>
+      <xacro:inertial_sphere mass="0.01" radius="0.018">
+          <origin xyz="0 0 0" rpy="0 0 0"/>
+      </xacro:inertial_sphere>
     </link>
     <!-- fixed because there's no transmission -->

File: robots/turtle/description/create_base_gazebo.urdf.xacro (robot description, xacro)
@@ -1,4 +1,4 @@
 <?xml version="1.0" ?>
-<!-- replaced with ros2_control.xacro -->
+<!-- not used - replaced with ros2_control.xacro -->
 <robot xmlns:xacro="http://ros.org/wiki/xacro">
   <xacro:macro name="sim_create_base">

File: robots/turtle/description/robot.urdf.xacro (robot description, xacro)
@@ -11,5 +11,5 @@
              The AutonomyLab *.xacro files are moved here because robot_description topic is published on the Desktop, not the robot RPi
     -->
-    <!-- xacro:include filename="../../../description/inertial_macros.xacro"/ -->
+    <xacro:include filename="../../../description/inertial_macros.xacro" />
     <xacro:include filename="../../../description/common_properties.xacro" />
     <xacro:include filename="create_1.urdf.xacro" />
