Commit message: Rearranged turtle URDF files

File: robots/turtle/description/create_1.urdf.xacro (robot description, xacro)
@@ -1,6 +1,7 @@
 ﻿<?xml version="1.0" ?>
 <robot name="create_1" xmlns:xacro="http://ros.org/wiki/xacro">
-  <xacro:include filename="$(find articubot_one)/robots/turtle/description/create_base.urdf.xacro" />
-  <xacro:include filename="$(find articubot_one)/robots/turtle/description/create_1_gazebo.urdf.xacro" />
+  <xacro:include filename="create_base.urdf.xacro" />
+  <xacro:include filename="create_sensors.urdf.xacro" />
+  <xacro:include filename="create_1_gazebo.urdf.xacro" />
   <xacro:create_base wheel_separation="0.26" base_diameter="0.3302">
     <mesh filename="package://articubot_one/assets/meshes/create_1.dae" />

File: robots/turtle/description/create_1_gazebo.urdf.xacro (robot description, xacro)
@@ -1,3 +1,132 @@
 <?xml version="1.0" ?>
 <robot xmlns:xacro="http://ros.org/wiki/xacro">
+    <!-- gz model -m turtle -s imu_link -->
+    <gazebo reference="imu_link">
+        <sensor name="imu_link" type="imu">
+        <always_on>1</always_on>
+        <topic>gz_imu/data</topic>
+        <!-- future Gazebo versions might require "<frame_id>" here. Must reference an actual link in .xacro -->
+        <gz_frame_id>imu_link</gz_frame_id>
+        <frame_id>imu_link</frame_id>
+        <update_rate>250</update_rate>
+            <imu>
+                <orientation_reference_frame>
+                  <localization>ENU</localization>
+                  <!-- custom_rpy parent_frame='world'>1.570795 0 0</custom_rpy -->
+                </orientation_reference_frame>
+                <enable_orientation>1</enable_orientation>
+                <angular_velocity>
+                    <x>
+                        <noise type="gaussian">
+                            <mean>0</mean>
+                            <stddev>0.009</stddev>
+                            <bias_mean>0.00075</bias_mean>
+                            <bias_stddev>0.005</bias_stddev>
+                            <dynamic_bias_stddev>0.00002</dynamic_bias_stddev>
+                            <dynamic_bias_correlation_time>400.0</dynamic_bias_correlation_time>
+                            <precision>0.00025</precision>
+                        </noise>
+                    </x>
+                    <y>
+                        <noise type="gaussian">
+                            <mean>0</mean>
+                            <stddev>0.009</stddev>
+                            <bias_mean>0.00075</bias_mean>
+                            <bias_stddev>0.005</bias_stddev>
+                            <dynamic_bias_stddev>0.00002</dynamic_bias_stddev>
+                            <dynamic_bias_correlation_time>400.0</dynamic_bias_correlation_time>
+                            <precision>0.00025</precision>
+                        </noise>
+                    </y>
+                    <z>
+                        <noise type="gaussian">
+                            <mean>0</mean>
+                            <stddev>0.009</stddev>
+                            <bias_mean>0.00075</bias_mean>
+                            <bias_stddev>0.005</bias_stddev>
+                            <dynamic_bias_stddev>0.00002</dynamic_bias_stddev>
+                            <dynamic_bias_correlation_time>400.0</dynamic_bias_correlation_time>
+                            <precision>0.00025</precision>
+                        </noise>
+                    </z>
+                </angular_velocity>
+                <linear_acceleration>
+                    <x>
+                        <noise type="gaussian">
+                            <mean>0</mean>
+                            <stddev>0.021</stddev>
+                            <bias_mean>0.05</bias_mean>
+                            <bias_stddev>0.0075</bias_stddev>
+                            <dynamic_bias_stddev>0.000375</dynamic_bias_stddev>
+                            <dynamic_bias_correlation_time>175.0</dynamic_bias_correlation_time>
+                            <precision>0.005</precision>
+                        </noise>
+                    </x>
+                    <y>
+                        <noise type="gaussian">
+                            <mean>0</mean>
+                            <stddev>0.021</stddev>
+                            <bias_mean>0.05</bias_mean>
+                            <bias_stddev>0.0075</bias_stddev>
+                            <dynamic_bias_stddev>0.000375</dynamic_bias_stddev>
+                            <dynamic_bias_correlation_time>175.0</dynamic_bias_correlation_time>
+                            <precision>0.005</precision>
+                        </noise>
+                    </y>
+                    <z>
+                        <noise type="gaussian">
+                            <mean>0</mean>
+                            <stddev>0.021</stddev>
+                            <bias_mean>0.05</bias_mean>
+                            <bias_stddev>0.0075</bias_stddev>
+                            <dynamic_bias_stddev>0.000375</dynamic_bias_stddev>
+                            <dynamic_bias_correlation_time>175.0</dynamic_bias_correlation_time>
+                            <precision>0.005</precision>
+                        </noise>
+                    </z>
+                </linear_acceleration>
+            </imu>
+        </sensor>
+    </gazebo>
+    <!-- gz model -m turtle -s laser_frame -->
+    <gazebo reference="laser_frame">
+        <!-- name must be "laser_frame", specifically for lasers. Must reference an actual link in .xacro -->
+        <sensor name='laser_frame' type='gpu_lidar'>
+          <pose>0 0 0 0 0 0</pose>
+          <always_on>1</always_on>
+          <!-- 6 Hz for LD14 - see "frequency" in dual_ekf_navsat_parameters.yaml -->
+          <update_rate>6</update_rate>
+          <topic>gz_scan</topic>
+          <!-- future Gazebo versions might require "<frame_id>" here. Must reference an actual link in .xacro -->
+          <gz_frame_id>laser_frame</gz_frame_id>
+          <frame_id>laser_frame</frame_id>
+          <ray>
+            <scan>
+              <horizontal>
+                <samples>360</samples>
+                <resolution>1</resolution>
+                <min_angle>-${PI}</min_angle>
+                <max_angle>${PI}</max_angle>
+              </horizontal>
+              <vertical>
+                <samples>1</samples>
+                <resolution>1</resolution>
+                <min_angle>0.0</min_angle>
+                <max_angle>0.0</max_angle>
+              </vertical>
+            </scan>
+            <range>
+              <min>0.3</min>
+              <max>12.0</max>
+              <resolution>0.01</resolution>
+            </range>
+            <noise>
+              <type>gaussian</type>
+              <mean>0</mean>
+              <stddev>0.01</stddev>
+            </noise>
+          </ray>
+          <visualize>true</visualize>
+        </sensor>
+    </gazebo>
 </robot>

File: robots/turtle/description/create_base.urdf.xacro (robot description, xacro)
@@ -151,159 +151,4 @@
       <axis xyz="0 1 0"/>
     </joint>
-    <joint name="imu_joint" type="fixed">
-      <parent link="chassis_link"/>
-      <child link="imu_link"/>
-      <origin xyz="0.0 0 0.068" rpy="0 0 0"/>
-    </joint>
-    <link name="imu_link"/>
-    <!-- gz model -m turtle -s imu_link -->
-    <gazebo reference="imu_link">
-        <sensor name="imu_link" type="imu">
-        <always_on>1</always_on>
-        <topic>gz_imu/data</topic>
-        <!-- future Gazebo versions might require "<frame_id>" here. Must reference an actual link in .xacro -->
-        <gz_frame_id>imu_link</gz_frame_id>
-        <frame_id>imu_link</frame_id>
-        <update_rate>250</update_rate>
-            <imu>
-                <orientation_reference_frame>
-                  <localization>ENU</localization>
-                  <!-- custom_rpy parent_frame='world'>1.570795 0 0</custom_rpy -->
-                </orientation_reference_frame>
-                <enable_orientation>1</enable_orientation>
-                <angular_velocity>
-                    <x>
-                        <noise type="gaussian">
-                            <mean>0</mean>
-                            <stddev>0.009</stddev>
-                            <bias_mean>0.00075</bias_mean>
-                            <bias_stddev>0.005</bias_stddev>
-                            <dynamic_bias_stddev>0.00002</dynamic_bias_stddev>
-                            <dynamic_bias_correlation_time>400.0</dynamic_bias_correlation_time>
-                            <precision>0.00025</precision>
-                        </noise>
-                    </x>
-                    <y>
-                        <noise type="gaussian">
-                            <mean>0</mean>
-                            <stddev>0.009</stddev>
-                            <bias_mean>0.00075</bias_mean>
-                            <bias_stddev>0.005</bias_stddev>
-                            <dynamic_bias_stddev>0.00002</dynamic_bias_stddev>
-                            <dynamic_bias_correlation_time>400.0</dynamic_bias_correlation_time>
-                            <precision>0.00025</precision>
-                        </noise>
-                    </y>
-                    <z>
-                        <noise type="gaussian">
-                            <mean>0</mean>
-                            <stddev>0.009</stddev>
-                            <bias_mean>0.00075</bias_mean>
-                            <bias_stddev>0.005</bias_stddev>
-                            <dynamic_bias_stddev>0.00002</dynamic_bias_stddev>
-                            <dynamic_bias_correlation_time>400.0</dynamic_bias_correlation_time>
-                            <precision>0.00025</precision>
-                        </noise>
-                    </z>
-                </angular_velocity>
-                <linear_acceleration>
-                    <x>
-                        <noise type="gaussian">
-                            <mean>0</mean>
-                            <stddev>0.021</stddev>
-                            <bias_mean>0.05</bias_mean>
-                            <bias_stddev>0.0075</bias_stddev>
-                            <dynamic_bias_stddev>0.000375</dynamic_bias_stddev>
-                            <dynamic_bias_correlation_time>175.0</dynamic_bias_correlation_time>
-                            <precision>0.005</precision>
-                        </noise>
-                    </x>
-                    <y>
-                        <noise type="gaussian">
-                            <mean>0</mean>
-                            <stddev>0.021</stddev>
-                            <bias_mean>0.05</bias_mean>
-                            <bias_stddev>0.0075</bias_stddev>
-                            <dynamic_bias_stddev>0.000375</dynamic_bias_stddev>
-                            <dynamic_bias_correlation_time>175.0</dynamic_bias_correlation_time>
-                            <precision>0.005</precision>
-                        </noise>
-                    </y>
-                    <z>
-                        <noise type="gaussian">
-                            <mean>0</mean>
-                            <stddev>0.021</stddev>
-                            <bias_mean>0.05</bias_mean>
-                            <bias_stddev>0.0075</bias_stddev>
-                            <dynamic_bias_stddev>0.000375</dynamic_bias_stddev>
-                            <dynamic_bias_correlation_time>175.0</dynamic_bias_correlation_time>
-                            <precision>0.005</precision>
-                        </noise>
-                    </z>
-                </linear_acceleration>
-            </imu>
-        </sensor>
-    </gazebo>
-    <joint name="scan_joint" type="fixed">
-      <parent link="chassis_link"/>
-      <child link="laser_frame"/>
-      <origin xyz="0.085 0 0.033" rpy="0 0 0"/>
-    </joint>
-    <link name="laser_frame">
-      <visual>
-        <geometry>
-          <cylinder radius="0.0375" length="0.025"/>
-        </geometry>
-        <material name="sensor_blue"/>
-      </visual>
-      <visual>
-        <origin xyz="0 0 -0.01"/>
-        <geometry>
-          <cylinder radius="0.01" length="0.02"/>
-        </geometry>
-        <material name="sensor_blue"/>
-      </visual>
-    </link>
-    <!-- gz model -m turtle -s laser_frame -->
-    <gazebo reference="laser_frame">
-        <!-- name must be "laser_frame", specifically for lasers. Must reference an actual link in .xacro -->
-        <sensor name='laser_frame' type='gpu_lidar'>
-          <pose>0 0 0 0 0 0</pose>
-          <always_on>1</always_on>
-          <!-- 6 Hz for LD14 - see "frequency" in dual_ekf_navsat_parameters.yaml -->
-          <update_rate>6</update_rate>
-          <topic>gz_scan</topic>
-          <!-- future Gazebo versions might require "<frame_id>" here. Must reference an actual link in .xacro -->
-          <gz_frame_id>laser_frame</gz_frame_id>
-          <frame_id>laser_frame</frame_id>
-          <ray>
-            <scan>
-              <horizontal>
-                <samples>360</samples>
-                <resolution>1</resolution>
-                <min_angle>-${pi}</min_angle>
-                <max_angle>${pi}</max_angle>
-              </horizontal>
-              <vertical>
-                <samples>1</samples>
-                <resolution>1</resolution>
-                <min_angle>0.0</min_angle>
-                <max_angle>0.0</max_angle>
-              </vertical>
-            </scan>
-            <range>
-              <min>0.3</min>
-              <max>12.0</max>
-              <resolution>0.01</resolution>
-            </range>
-            <noise>
-              <type>gaussian</type>
-              <mean>0</mean>
-              <stddev>0.01</stddev>
-            </noise>
-          </ray>
-          <visualize>true</visualize>
-        </sensor>
-    </gazebo>
   </xacro:macro>
 </robot>

File: robots/turtle/description/robot.urdf.xacro (robot description, xacro)
@@ -14,5 +14,4 @@
     <xacro:include filename="../../../description/common_properties.xacro" />
     <xacro:include filename="create_1.urdf.xacro" />
-    <!-- <xacro:include filename="../../../description/turtle_sensors.xacro" / -->
     <xacro:include filename="ros2_control.xacro" />
 </robot>

Commit message: Squashed commit of the following:
commit acd97cc2fa5e48a904368bcf2d6176365d0ee769
Author: Sergei Grichine <msghub@hotmail.com>
Date:   Mon Jan 13 12:55:40 2025 -0600

    Create roomba.py

commit cee4fa63c3025132680a3fdc0b334ec82b7926bf
Author: Sergei Grichine <msghub@hotmail.com>
Date:   Sun Jan 12 12:47:05 2025 -0600

    Corrections after calibrating Turtle odometry

commit 8af54e0db978ef9e17ff873393f51a1849040a96
Author: Sergei Grichine <msghub@hotmail.com>
Date:   Sat Jan 11 10:22:38 2025 -0600

    Create 1 wheel_separation="0.258"

commit bbd023543a4e7ecd13fb67facaa005934dc7054d
Author: Sergei Grichine <msghub@hotmail.com>
Date:   Thu Jan 9 12:44:32 2025 -0600

    Update myturtle.py

commit b7aa92f43571797722c2c9c5cd5ead2c371d39c4
Author: Sergei Grichine <msghub@hotmail.com>
Date:   Wed Jan 8 21:48:11 2025 -0600

    Turtle files added

commit a7125edb6aeb7f900629f3f71924bc5d7020ec23
Merge: cd58e4d b20aaa5
Author: Sergei Grichine <msghub@hotmail.com>
Date:   Wed Jan 8 17:27:21 2025 -0600

    Merge branch 'dev' of https://github.com/slgrobotics/articubot_one into dev

commit cd58e4d6b71186f6b6032aa6b0a1d6adbe2e22ea
Author: Sergei Grichine <msghub@hotmail.com>
Date:   Wed Jan 8 17:27:06 2025 -0600

    Update turtle_sim.launch.py

commit c80ea3802ed111b7fe36ba916635e842e547e929
Author: Sergei Grichine <msghub@hotmail.com>
Date:   Wed Jan 8 11:21:08 2025 -0600

    Streamlined Create1 xacro files

commit b20aaa5a0669b48c27116ff1db8687d55ca870bd
Author: Sergei Grichine <msghub@hotmail.com>
Date:   Wed Jan 8 09:16:54 2025 -0600

    Update turtle.launch.py

commit 8cc1fc31cf4f426dc8a53a75823ce70bd4f10de9
Author: Sergei Grichine <msghub@hotmail.com>
Date:   Tue Jan 7 21:55:05 2025 -0600

    Create 1 driver uses "wheel_left_joint" and "wheel_right_joint" names

commit b584a5a47f7843c3f6acd38ca6ab9646644177bb
Author: Sergei Grichine <msghub@hotmail.com>
Date:   Tue Jan 7 18:52:24 2025 -0600

    WIP: turtle nav

File: robots/turtle/description/create_1.urdf.xacro (robot description, xacro)
@@ -8,5 +8,6 @@
   <xacro:include filename="create_sensors.urdf.xacro" />
   <xacro:include filename="create_1_gazebo.urdf.xacro" />
-  <xacro:create_base wheel_separation="0.26" base_diameter="0.3302">
+  <!-- wheel_separation - distance between left and right wheels, defined in ~/create_robot_ws/src/libcreate/src/types.cpp -->
+  <xacro:create_base wheel_separation="0.258" base_diameter="0.3302" wheel_radius="0.033" wheel_width="0.024" mass_kg="3.5">
     <mesh filename="package://articubot_one/assets/meshes/create_1.dae" />
   </xacro:create_base>

File: robots/turtle/description/create_base.urdf.xacro (robot description, xacro)
@@ -21,5 +21,5 @@
     </link>
     <!-- joint name="${prefix}_wheel_joint" type="fixed" -->
-    <joint name="${prefix}_wheel_joint" type="continuous">
+    <joint name="wheel_${prefix}_joint" type="continuous">
       <origin xyz="0 ${y_offset} ${-wheel_radius}" rpy="0 0 0"/>
       <parent link="chassis_link"/>
@@ -29,7 +29,5 @@
   </xacro:macro>
   <xacro:macro name="create_base"
-               params="diffdrive_update_rate:=40 wheel_separation wheel_radius:=0.033 wheel_width:=0.024 wheel_torque:=1.0 wheel_accel:=1.8 mass_kg:=3.5 base_diameter *mesh">
-    <!-- replaced with ros2_control.xacro -->
-    <!-- xacro:include filename="$(find articubot_one)/robots/turtle/description/create_base_gazebo.urdf.xacro"/ -->
+               params="wheel_separation base_diameter wheel_radius wheel_width mass_kg *mesh">
     <!-- The coordinate frame called base_link is rigidly attached to the robot root body. -->
     <link name="base_link">

File: robots/turtle/description/ros2_control.xacro (robot description, xacro)
@@ -4,9 +4,14 @@
         <!-- Wheel geometry information - see controllers.yaml -->
         <hardware>
+            <xacro:unless value="$(arg sim_mode)">
+                <!-- Actual Create 1 base hardware driver runs on the Turtlebot Raspberry Pi 3B
+                     It publishes /joint_states [wheel_left_joint, wheel_right_joint] <- ! note the names !
+                     see https://github.com/slgrobotics/robots_bringup/tree/main/Docs/Create1 -->
+            </xacro:unless>
             <xacro:if value="$(arg sim_mode)">
                 <plugin>gz_ros2_control/GazeboSimSystem</plugin>
             </xacro:if>
         </hardware>
-        <joint name="left_wheel_joint">
+        <joint name="wheel_left_joint">
             <command_interface name="velocity">
                 <param name="min">-10</param>
@@ -23,5 +28,5 @@
             </state_interface -->
         </joint>
-        <joint name="right_wheel_joint">
+        <joint name="wheel_right_joint">
             <command_interface name="velocity">
                 <param name="min">-10</param>
