Commit message: Update robot_core.xacro

File: robots/plucky/description/robot_core.xacro (robot description, xacro)
@@ -55,5 +55,5 @@
             <geometry>
                 <!-- box size="${wheel_offset_y * 2 + wheel_thickness} ${wheel_offset_y * 2 + wheel_thickness} 0.02"/ -->
-                <cylinder radius="${wheel_offset_y + wheel_thickness / 2}" length="0.02"/>
+                <cylinder radius="${wheel_offset_y + wheel_thickness + 0.03}" length="0.01"/>
             </geometry>
             <material name="shadow_grey"/>
@@ -92,5 +92,5 @@
             <origin xyz="${wheel_offset_x} ${chassis_width*0.5} 0" rpy="-${pi/2} 0 0"/>
             <geometry>
-                <cylinder radius="${0.06}" length="${chassis_width*0.5}"/>
+                <cylinder radius="0.03" length="${chassis_width*0.5}"/>
             </geometry>
             <material name="body_color"/>
@@ -99,5 +99,12 @@
             <origin xyz="${wheel_offset_x} ${-chassis_width*0.5} 0" rpy="${pi/2} 0 0"/>
             <geometry>
-                <cylinder radius="${0.06}" length="${chassis_width*0.5}"/>
+                <cylinder radius="0.03" length="${chassis_width*0.5}"/>
+            </geometry>
+            <material name="body_color"/>
+        </visual>
+        <visual name="chassis_caster_holder_left">
+            <origin xyz="${caster_wheel_offset_x+0.09} ${caster_wheel_offset_y*0.85} ${caster_wheel_offset_z*0.42}" rpy="0 ${pi/4} 0"/>
+            <geometry>
+                <cylinder radius="0.012" length="0.23"/>
             </geometry>
             <material name="body_color"/>
@@ -106,5 +113,12 @@
             <origin xyz="${caster_wheel_offset_x} ${caster_wheel_offset_y*0.9} ${caster_wheel_offset_z}" rpy="0 0 0"/>
             <geometry>
-                <sphere radius="0.02"/>
+                <sphere radius="0.03"/>
+            </geometry>
+            <material name="body_color"/>
+        </visual>
+        <visual name="chassis_caster_holder_right">
+            <origin xyz="${caster_wheel_offset_x+0.09} ${-caster_wheel_offset_y*0.85} ${caster_wheel_offset_z*0.42}" rpy="0 ${pi/4} 0"/>
+            <geometry>
+                <cylinder radius="0.012" length="0.23"/>
             </geometry>
             <material name="body_color"/>
@@ -113,5 +127,5 @@
             <origin xyz="${caster_wheel_offset_x} ${-caster_wheel_offset_y*0.9} ${caster_wheel_offset_z}" rpy="0 0 0"/>
             <geometry>
-                <sphere radius="0.02"/>
+                <sphere radius="0.03"/>
             </geometry>
             <material name="body_color"/>
@@ -131,5 +145,5 @@
         <parent link="chassis_link"/>
         <child link="left_wheel"/>
-        <origin xyz="${wheel_offset_x} ${wheel_offset_y} 0" rpy="-${pi/2} 0 0" />
+        <origin xyz="${wheel_offset_x} ${wheel_offset_y} 0" rpy="-${pi/2 - 0.15} 0 0" />
         <axis xyz="0 0 1">
           <limit>
@@ -202,5 +216,5 @@
         <parent link="chassis_link"/>
         <child link="right_wheel"/>
-        <origin xyz="${wheel_offset_x} ${-wheel_offset_y} 0" rpy="${pi/2} 0 0" />
+        <origin xyz="${wheel_offset_x} ${-wheel_offset_y} 0" rpy="${pi/2 - 0.15} 0 0" />
         <axis xyz="0 0 -1">
           <limit>

Commit message: Update robot_core.xacro

File: robots/plucky/description/robot_core.xacro (robot description, xacro)
@@ -74,9 +74,22 @@
     <!-- CHASSIS LINK -->
     <link name="chassis_link">
-        <visual name="chassis_visual">
-            <!-- origin xyz="${chassis_length/2} 0 ${chassis_height/4}"/ -->
-            <origin xyz="0 0 ${chassis_height/4}"/>
-            <geometry>
-                <box size="${chassis_length} ${chassis_width} ${chassis_height/2}"/>
+        <visual name="chassis_visual_bottom">
+            <origin xyz="0 0 ${chassis_height/8}"/>
+            <geometry>
+                <box size="${chassis_length} ${chassis_width} ${chassis_height/4}"/>
+            </geometry>
+            <material name="body_color"/>
+        </visual>
+        <visual name="chassis_visual_front">
+            <origin xyz="0.15 0 ${chassis_height/2-0.03}" rpy="0 ${pi/4} 0"/>
+            <geometry>
+                <box size="0.25 ${chassis_width} 0.01"/>
+            </geometry>
+            <material name="body_color"/>
+        </visual>
+        <visual name="chassis_visual_back">
+            <origin xyz="-0.07 0 ${chassis_height/2-0.03}" rpy="0 -${pi/4} 0"/>
+            <geometry>
+                <box size="0.25 ${chassis_width} 0.01"/>
             </geometry>
             <material name="body_color"/>

Commit message: Update robot_core.xacro
wheels Y offset 0.280 for Plucky

File: robots/plucky/description/robot_core.xacro (robot description, xacro)
@@ -12,5 +12,5 @@
     <xacro:property name="wheel_mass" value="1.0"/>
     <xacro:property name="wheel_offset_x" value="${chassis_length/2 - wheel_radius - 0.01}"/>
-    <xacro:property name="wheel_offset_y" value="0.300"/>
+    <xacro:property name="wheel_offset_y" value="0.280"/>
     <xacro:property name="wheel_offset_z" value="0.01"/>
     <xacro:property name="caster_wheel_radius" value="0.05"/>
