Commit message: WIP: turtle sim

File: robots/dragger/description/ros2_control.xacro (robot description, xacro)
@@ -2,5 +2,5 @@
 <robot xmlns:xacro="http://www.ros.org/wiki/xacro">
     <ros2_control name="DraggerRobot" type="system">
-        <!-- Wheel geometry information - see controllers_*.yaml -->
+        <!-- Wheel geometry information - see controllers.yaml -->
         <hardware>
             <xacro:unless value="$(arg sim_mode)">

File: robots/sim/description/ros2_control.xacro (robot description, xacro)
@@ -2,5 +2,5 @@
 <robot xmlns:xacro="http://www.ros.org/wiki/xacro">
     <ros2_control name="DraggerSimRobot" type="system">
-        <!-- Wheel geometry information - see controllers_*.yaml -->
+        <!-- Wheel geometry information - see controllers.yaml -->
         <hardware>
             <xacro:unless value="$(arg sim_mode)">

File: robots/turtle/description/create_base.urdf.xacro (robot description, xacro)
@@ -33,5 +33,6 @@
   <xacro:macro name="create_base"
                params="diffdrive_update_rate:=40 wheel_separation wheel_radius:=0.033 wheel_width:=0.024 wheel_torque:=1.0 wheel_accel:=1.8 mass_kg:=3.5 base_diameter *mesh">
-    <xacro:include filename="$(find articubot_one)/robots/turtle/description/create_base_gazebo.urdf.xacro"/>
+    <!-- replaced with ros2_control.xacro -->
+    <!-- xacro:include filename="$(find articubot_one)/robots/turtle/description/create_base_gazebo.urdf.xacro"/ -->
     <!-- The coordinate frame called base_link is rigidly attached to the robot root body. -->
     <link name="base_link">
@@ -200,9 +201,4 @@
       </visual>
     </link>
-    <!-- Simulation sensors -->
-    <xacro:sim_create_base/>
-    <xacro:sim_create_wall_sensor/>
-    <xacro:sim_create_cliff_sensors/>
-    <xacro:sim_imu/>
   </xacro:macro>
 </robot>

File: robots/turtle/description/create_base_gazebo.urdf.xacro (robot description, xacro)
@@ -1,3 +1,4 @@
 <?xml version="1.0" ?>
+<!-- replaced with ros2_control.xacro -->
 <robot xmlns:xacro="http://ros.org/wiki/xacro">
   <xacro:macro name="sim_create_base">

File: robots/turtle/description/robot.urdf.xacro (robot description, xacro)
@@ -12,6 +12,4 @@
     -->
     <!-- xacro:include filename="../../../description/inertial_macros.xacro"/ -->
-    <xacro:arg name="sim_mode" default="false"/>
-    <!-- xacro:include filename="common_properties.urdf" / -->
     <xacro:include filename="../../../description/common_properties.xacro" />
     <xacro:include filename="create_1.urdf.xacro" />
@@ -19,3 +17,4 @@
     <xacro:include filename="../../../description/magnetometer.xacro" />
     <xacro:include filename="../../../description/turtle_sensors.xacro" / -->
+    <xacro:include filename="ros2_control.xacro" />
 </robot>

File: robots/turtle/description/ros2_control.xacro (robot description, xacro)
@@ -1,19 +1,7 @@
 <?xml version="1.0"?>
 <robot xmlns:xacro="http://www.ros.org/wiki/xacro">
-    <ros2_control name="PluckyRobot" type="system">
+    <ros2_control name="TurtleSimRobot" type="system">
         <!-- Wheel geometry information - see controllers.yaml -->
         <hardware>
-            <xacro:unless value="$(arg sim_mode)">
-                <!-- Values corrected for Dragger robot -->
-                <plugin>diffdrive_arduino/DiffDriveArduino</plugin>
-                <param name="left_wheel_name">left_wheel_joint</param>
-                <param name="right_wheel_name">right_wheel_joint</param>
-                <param name="loop_rate">30</param>
-                <param name="device">/dev/ttyACM0</param>
-                <param name="baud_rate">115200</param>
-                <param name="timeout">1000</param>
-                <param name="enc_counts_per_rev">13730</param>
-                <param name="wheels_pwm_factor">1.0</param>
-            </xacro:unless>
             <xacro:if value="$(arg sim_mode)">
                 <plugin>gz_ros2_control/GazeboSimSystem</plugin>
@@ -50,23 +38,4 @@
             </state_interface -->
         </joint>
-        <xacro:if value="$(arg sim_mode)">
-            <!-- we need this for Rviz to reflect rotations of joints published by broad_cont in Gazebo -->
-            <joint name="left_caster_wheel_joint">
-                <state_interface name="velocity">
-                    <param name="initial_value">0.0</param>
-                </state_interface>
-                <state_interface name="position">
-                    <param name="initial_value">0.0</param>
-                </state_interface>
-            </joint>
-            <joint name="right_caster_wheel_joint">
-                <state_interface name="velocity">
-                    <param name="initial_value">0.0</param>
-                </state_interface>
-                <state_interface name="position">
-                    <param name="initial_value">0.0</param>
-                </state_interface>
-            </joint>
-        </xacro:if>
     </ros2_control>
     <gazebo>
@@ -75,5 +44,5 @@
             <robot_param>robot_description</robot_param>
             <robot_param_node>robot_state_publisher</robot_param_node> -->
-            <parameters>$(find articubot_one)/robots/sim/config/controllers.yaml</parameters>
+            <parameters>$(find articubot_one)/robots/turtle/config/controllers.yaml</parameters>
         </plugin>
     </gazebo>

Commit message: new branch HBRC ROS meeting

File: robots/dragger/description/ros2_control.xacro (robot description, xacro)
@@ -75,5 +75,5 @@
             <robot_param>robot_description</robot_param>
             <robot_param_node>robot_state_publisher</robot_param_node> -->
-            <parameters>$(find articubot_one)/robots/dragger/config/controllers.yaml</parameters>
+            <parameters>/home/ubuntu/ros_ws/install/articubot_one/share/articubot_one/robots/dragger/config/controllers.yaml</parameters>
         </plugin>
     </gazebo>

File: robots/stingray/description/JP_camera.xacro (robot description, xacro)
@@ -79,5 +79,7 @@
             <camera name='__default__'>
                 <pose>0 0 0 0 0 0</pose>
-                <horizontal_fov>1.047</horizontal_fov>
+                <!-- <horizontal_fov>${pi/2}</horizontal_fov> -->
+                <horizontal_fov>1.40</horizontal_fov>
+                <!-- <vertical_fov>${pi}</horizontal_fov> -->
                 <image>
                     <width>640</width>

File: robots/stingray/description/JP_imu.xacro (robot description, xacro)
@@ -7,5 +7,5 @@
         <child link="imu_link"/>
         <!-- we place IMU between the wheels -->
-        <origin xyz="${imu_offset_x} 0 ${imu_offset_z}" rpy="0 0 0"/>
+        <origin xyz="${imu_offset_x} ${imu_offset_y} ${imu_offset_z}" rpy="${imu_rotation_x} ${imu_rotation_y} ${imu_rotation_z}"/>
     </joint>
     <link name="imu_link">

File: robots/stingray/description/JP_lidar.xacro (robot description, xacro)
@@ -4,10 +4,14 @@
     <xacro:property name="lidar_radius" value="0.03025"/>
     <xacro:property name="lidar_height" value="0.016"/>
-    <xacro:property name="lidar_stand_height" value="0.0424"/>
+    <xacro:property name="lidar_support_height" value="0.0424"/>
     <xacro:property name="lidar_offset_x" value="0.045"/>
+    <xacro:property name="lidar_offset_y" value="0.0"/>
+    <xacro:property name="lidar_rotation_x" value="${pi}"/>
+    <xacro:property name="lidar_rotation_y" value="0.0"/>
+    <xacro:property name="lidar_rotation_z" value="${pi/2}"/>
     <joint name="laser_joint" type="fixed">
-        <parent link="chassis_link"/>
+        <parent link="lidar_support_link"/>
         <child link="laser_frame"/>
-        <origin xyz="${lidar_offset_x} 0 ${(chassis_height/2) + (lidar_stand_height) + (lidar_height/2)}" rpy="0 0 0"/>
+        <origin xyz="${lidar_offset_x} ${lidar_offset_y} ${(chassis_height/2) + (lidar_support_height) + (lidar_height/2)}" rpy="${lidar_rotation_x} ${lidar_rotation_y} ${lidar_rotation_z}"/>
     </joint>
     <link name="laser_frame">

File: robots/stingray/description/lidar_support.xacro (robot description, xacro)
@@ -3,9 +3,13 @@
     <!-- LIDAR SUPPORT JOINT -->
     <joint name="lidar_support_joint" type="fixed">
-        <parent link="base_link"/>
+        <parent link="chassis_link"/>
         <child link="lidar_support_link"/>
         <origin xyz="0.0 0.0 0.0"/>
     </joint>
     <!-- LIDAR SUPPORT LINK -->
+    <!-- 'Front' of YDLidar is the drive motor end
+    which in this instance points to the left of the robot
+    thus the rotation of the support link by pi/2 radians
+    -->
     <link name="lidar_support_link">
         <visual name="lidar_support__gz_visual">
@@ -17,5 +21,4 @@
         </visual>
         <visual name="lidar_support_rviz_visual">
-            <!-- <origin xyz="0.0 0.0 0.0" rpy="0.0 0.0 ${pi/2}"/> -->
             <origin xyz="${lidar_support_offset_x} ${lidar_support_offset_y} ${lidar_support_offset_z}" rpy="0.0 0.0 ${pi/2}"/>
             <geometry>

File: robots/stingray/description/robot.urdf.xacro (robot description, xacro)
@@ -1,4 +1,16 @@
 <?xml version="1.0"?>
 <robot xmlns:xacro="http://www.ros.org/wiki/xacro"  name="robot">
+    <!-- robot.urdf.xacro
+    imports
+        robot_core.xacro
+        common_properties.xacro
+        individual sensors - each with their positions
+            JP_lidar.xacro
+            JP_imu.xacro
+            JP_camera.xacro
+        other components
+            battery.xacro
+            ros2_control.xacro
+    -->
     <!-- See common Gazebo pugins in the world file -->
     <!--
@@ -9,35 +21,32 @@
     -->
     <!-- COMMON -->
-    <xacro:include filename="../../../description/common_properties.xacro" />
+    <xacro:include filename="$(find articubot_one)/description/common_properties.xacro" />
     <!-- CORE -->
     <xacro:include filename="robot_core.xacro" />
-    <!-- CAMERA -->
+    <!-- USB FISHEYE CAMERA -->
     <xacro:property name="camera_offset_x" value="${front_panel_offset}"/>
     <xacro:property name="camera_offset_z" value="0.01525"/>
-    <xacro:include filename="../../../description/JP_camera.xacro" />
+    <xacro:include filename="$(find articubot_one)/robots/stingray/description/JP_camera.xacro" />
+    <xacro:property name="camera_rotation_y" value="-0.1571"/>    <!-- =9 degrees -->
     <!-- LIDAR -->
-    <xacro:property name="lidar_support_offset_x" value="0.0"/>
-    <xacro:property name="lidar_support_offset_y" value="0.0"/>
+    <xacro:property name="lidar_support_offset_x" value="0.042"/>
+    <xacro:property name="lidar_support_offset_y" value="-0.02"/>
     <xacro:property name="lidar_support_offset_z" value="${chassis_height/2 + 0.00375}"/>
-    <xacro:include filename="../../../description/lidar_support.xacro" />
-    <xacro:property name="laser_offset_x" value="${wheel_offset_x}"/>
-    <xacro:property name="laser_offset_z" value="0.50"/>
-    <xacro:include filename="../../../description/JP_lidar.xacro" />
-    <!-- GPS -->
-    <xacro:property name="gps_offset_x" value="0.0"/>
-    <xacro:property name="gps_offset_y" value="0.0"/>
-    <xacro:property name="gps_offset_z" value="0.02"/>
-    <xacro:include filename="../../../description/JP_gps.xacro" />
+    <xacro:include filename="$(find articubot_one)/robots/stingray/description/lidar_support.xacro"/>
+    <!-- <xacro:property name="laser_offset_x" value="${wheel_offset_x}"/> -->
+    <!-- <xacro:property name="laser_offset_z" value="0.50"/> -->
+    <xacro:include filename="$(find articubot_one)/robots/stingray/description/JP_lidar.xacro" />
     <!-- IMU -->
     <xacro:property name="imu_offset_x" value="0.0"/>
+    <xacro:property name="imu_offset_y" value="0.0"/>
     <xacro:property name="imu_offset_z" value="0.0"/>
-    <xacro:include filename="../../../description/imu.xacro" />
-    <!-- MAG -->
-    <xacro:include filename="../../../description/magnetometer.xacro" />
+    <xacro:property name="imu_rotation_x" value="0.0"/>
+    <xacro:property name="imu_rotation_y" value="0.0"/>
+    <xacro:property name="imu_rotation_z" value="0.0"/>
+    <xacro:include filename="$(find articubot_one)/robots/stingray/description/JP_imu.xacro"/>
     <!-- BATTERY -->
-    <xacro:include filename="../../../description/battery.xacro" />
+    <xacro:include filename="$(find articubot_one)/robots/stingray/description/Zeee_LiPo_battery.xacro" />
     <!-- OPTIONAL -->
     <!-- xacro:include filename="../../../description/depth_camera.xacro" / -->
-    <!-- xacro:include filename="../../../description/face.xacro" / -->
     <!-- ROS2 CONTROL -->
     <xacro:include filename="ros2_control.xacro" />

File: robots/stingray/description/robot_core.xacro (robot description, xacro)
@@ -1,7 +1,15 @@
 <?xml version="1.0"?>
 <robot xmlns:xacro="http://www.ros.org/wiki/xacro" >
-    <xacro:include filename="../../../description/inertial_macros.xacro"/>
+    <!-- robot_core.xacro -->
+    <!-- This file contains the core components of the
+    Stingray robot, including the chassis, wheels, and joints.
+    It is included in the main robot.urdf.xacro file
+    to modularize the robot description.
+    Additional components such as sensors and actuators
+    are in robot.urdf.xacro -->
     <!-- TEMPLATE -->
     <xacro:property name="TEMPLATE" value="0.0"/>
+    <!-- INERTIAL -->
+    <xacro:include filename="../../../description/inertial_macros.xacro"/>
     <!-- CHASSIS -->
     <xacro:property name="chassis_length" value="0.266"/>
@@ -11,6 +19,6 @@
     <xacro:property name="front_panel_offset" value="0.090"/>
     <xacro:property name="chassis_mass" value="2.466"/>
-    <!-- <xacro:property name="chassis_mass" value="${stingray_total_mass}-2*${wheel_mass}-${caster_mass}-${lidar_mass}"
-    - ${OTHER_COMPONENTS_TO_BE_DETERMINED}/> -->
+    <!-- <xacro:property name="chassis_mass" value="${stingray_total_mass}-2*${wheel_mass}-${caster_mass}-${lidar_mass}" -->
+    <!-- ${OTHER_COMPONENTS_TO_BE_DETERMINED}/> -->
     <!-- <xacro:property name="stingray_total_mass" value="2.915"/> -->
     <!-- <xacro:property name="wheel_motor_assembly" value="0.375"/> -->
@@ -28,13 +36,4 @@
     <xacro:property name="caster_z_offset" value="-0.035"/>
     <xacro:property name="caster_mass" value="0.022"/>
-    <!-- we need the following because (unlike sim) real Dragger doesn't have a controller reporting caster's position -->
-<!--
-    <xacro:if value="$(arg sim_mode)">
-        <xacro:property name="caster_joint_type" value="continuous"/>
-    </xacro:if>
-    <xacro:unless value="$(arg sim_mode)">
-        <xacro:property name="caster_joint_type" value="fixed"/>
-    </xacro:unless>
- -->
     <!-- ********************** ROBOT BASE *********************************  -->
     <!-- The coordinate frame called base_link is rigidly attached to the robot root body.
@@ -48,5 +47,5 @@
             <origin xyz="0 0 0"/>
             <geometry>
-                <box size="0.01 0.01 0.01"/>
+                <sphere radius="0.005"/>
             </geometry>
             <material name="red"/>
@@ -58,11 +57,15 @@
          The translation component of the frame should be the barycenter of the feet projections on the floor.
          With respect to the odom frame, the roll and pitch angles should be zero and the yaw angle should correspond to the base_link yaw angle.
-         Rationale: base_footprint provides a fairly stable 2D planar representation of the humanoid even while walking and swaying with the base_link. -->
+         Rationale: base_footprint provides a fairly stable 2D planar representation of the humanoid even while walking and swaying with the base_link.
+    -->
+    <!-- base_footprint radius = ~0.19 -->
     <!-- Define the center of the main robot chassis projected on the ground -->
     <link name="base_footprint">
         <visual name="footprint_visual">
-            <origin xyz="-${chassis_offset + caster_radius} 0.0 0.0"/>
-            <geometry>
-                <box size="${chassis_length + (caster_radius * 2)} ${wheel_separation + wheel_thickness} 0.001"/>
+            <!-- <origin xyz="-${chassis_offset + caster_radius} 0.0 0.0"/> -->
+            <origin xyz="-${chassis_offset} 0.0 0.0"/>
+            <geometry>
+                <!-- <box size="${chassis_length + (caster_radius * 2)} ${wheel_separation + wheel_thickness} 0.001"/> -->
+                <cylinder radius="0.19" length="0.001"/>
             </geometry>
             <material name="shadow_gray"/>
@@ -98,5 +101,4 @@
         </visual>
         <collision>
-            <!-- <origin xyz="0.0 0.0 0.0" rpy="0.0 0.0 0.0"/> -->
             <origin xyz="${-chassis_offset} 0.0 0.0" rpy="0.0 0.0 0.0"/>
             <geometry>
@@ -111,5 +113,5 @@
     <!-- LEFT WHEEL JOINT -->
     <joint name="left_wheel_joint" type="continuous">
-        <parent link="base_link"/>
+        <parent link="chassis_link"/>
         <child link="left_wheel_link"/>
         <origin xyz="0.0 ${wheel_offset_x} 0.0" rpy="-${pi/2} 0.0 0.0"/>
@@ -175,5 +177,5 @@
     <joint name="caster_wheel_joint" type="fixed">
         <origin xyz="${caster_x_offset} 0.0 ${caster_z_offset}" rpy="0.0 0.0 0.0"/>
-        <parent link="base_link"/>
+        <parent link="chassis_link"/>
         <child link="caster_wheel_link"/>
         <axis xyz="0.0 0.0 0.0"/>

File: robots/stingray/description/ros2_control.xacro (robot description, xacro)
@@ -4,16 +4,4 @@
         <!-- Wheel geometry information - see controllers.yaml -->
         <hardware>
-            <xacro:unless value="$(arg sim_mode)">
-                <!-- Values corrected for Dragger robot -->
-                <plugin>diffdrive_arduino/DiffDriveArduino</plugin>
-                <param name="left_wheel_name">left_wheel_joint</param>
-                <param name="right_wheel_name">right_wheel_joint</param>
-                <param name="loop_rate">30</param>
-                <param name="device">/dev/ttyACM0</param>
-                <param name="baud_rate">115200</param>
-                <param name="timeout">1000</param>
-                <param name="enc_counts_per_rev">2506</param>
-                <param name="wheels_pwm_factor">1.0</param>
-            </xacro:unless>
             <xacro:if value="$(arg sim_mode)">
                 <plugin>gz_ros2_control/GazeboSimSystem</plugin>
@@ -30,22 +18,8 @@
             <state_interface name="position" />
         </joint>
-        <!-- <xacro:if value="$(arg sim_mode)"> -->
-            <!-- we need this for Rviz to reflect rotations of joints published by broad_cont in Gazebo -->
-            <!-- <joint name="left_caster_wheel_joint">
-                <state_interface name="velocity" />
-                <state_interface name="position" />
-            </joint> -->
-            <!-- <joint name="right_caster_wheel_joint">
-                <state_interface name="velocity" />
-                <state_interface name="position" />
-            </joint> -->
-        <!-- </xacro:if> -->
     </ros2_control>
     <gazebo>
         <plugin filename="libgz_ros2_control-system.so" name="gz_ros2_control::GazeboSimROS2ControlPlugin">
-            <!-- the following are just default parameters anyway. Skip them unless you want to reassign them:
-            <robot_param>robot_description</robot_param>
-            <robot_param_node>robot_state_publisher</robot_param_node> -->
-            <parameters>$(find articubot_one)/robots/stingray/config/controllers.yaml</parameters>
+            <parameters>/home/ubuntu/ros_ws/install/articubot_one/share/articubot_one/robots/stingray/config/controllers.yaml</parameters>
         </plugin>
     </gazebo>

File: robots/turtle/description/ros2_control.xacro (robot description, xacro)
@@ -49,5 +49,5 @@
             <robot_param>robot_description</robot_param>
             <robot_param_node>robot_state_publisher</robot_param_node> -->
-            <parameters>$(find articubot_one)/robots/turtle/config/controllers.yaml</parameters>
+            <parameters>/home/ubuntu/ros_ws/install/articubot_one/share/articubot_one/robots/turtle/config/controllers.yaml</parameters>
         </plugin>
     </gazebo>
