Commit message: Moved cURDF colors to common_properties.xacro

File: robots/dragger/description/robot.urdf.xacro (robot description, xacro)
@@ -3,41 +3,10 @@
     <!-- See common Gazebo pugins in the world file -->
     <!--
-        To re-generate robot.urdf manually for troubleshooting:
-          xacro ~/robot_ws/install/articubot_one/share/articubot_one/description/robot.urdf.xacro sim_mode:=true > ~/robot_ws/src/articubot_one/description/robot.urdf
+        To re-generate robot.urdf.generated.xml manually for troubleshooting:
+          cd ~/robot_ws
+          colcon build
+          xacro install/articubot_one/share/articubot_one/robots/dragger/description/robot.urdf.xacro sim_mode:=false > src/articubot_one/robots/dragger/description/robot.urdf.generated.xml
     -->
-    <material name="white">
-        <color rgba="1 1 1 1" />
-    </material>
-    <material name="black">
-        <color rgba="0 0 0 1"/>
-    </material>
-    <material name="shadow_grey">
-        <color rgba="0.3 0.3 0.3 0.5"/>
-    </material>
-    <material name="red">
-        <color rgba="1 0 0 1"/>
-    </material>
-    <material name="green">
-        <color rgba="0 1 0 1"/>
-    </material>
-    <material name="blue">
-        <color rgba="0 0 1 1"/>
-    </material>
-    <material name="sensor_blue">
-        <color rgba="0.2 0.2 1 1"/>
-    </material>
-    <material name="sensor_yellow">
-        <color rgba="0.8 0.8 0.2 1"/>
-    </material>
-    <material name="body_color">
-        <color rgba="1 0.3 0.1 1"/>
-    </material>
-    <material name="port_red">
-        <color rgba="1 0.2 0.2 1"/>
-    </material>
-    <material name="starboard_green">
-        <color rgba="0.2 1 0.2 1"/>
-    </material>
-    <xacro:arg name="sim_mode" default="false"/>
+    <xacro:include filename="../../../description/common_properties.xacro" />
     <xacro:include filename="robot_core.xacro" />
     <xacro:include filename="../../../description/imu.xacro" />

File: robots/plucky/description/robot.urdf.xacro (robot description, xacro)
@@ -3,41 +3,10 @@
     <!-- See common Gazebo pugins in the world file -->
     <!--
-        To re-generate robot.urdf manually for troubleshooting:
-          xacro ~/robot_ws/install/articubot_one/share/articubot_one/description/robot.urdf.xacro sim_mode:=true > ~/robot_ws/src/articubot_one/description/robot.urdf
+        To re-generate robot.urdf.generated.xml manually for troubleshooting:
+          cd ~/robot_ws
+          colcon build
+          xacro install/articubot_one/share/articubot_one/robots/plucky/description/robot.urdf.xacro sim_mode:=false > src/articubot_one/robots/plucky/description/robot.urdf.generated.xml
     -->
-    <material name="white">
-        <color rgba="1 1 1 1" />
-    </material>
-    <material name="black">
-        <color rgba="0 0 0 1"/>
-    </material>
-    <material name="shadow_grey">
-        <color rgba="0.3 0.3 0.3 0.5"/>
-    </material>
-    <material name="red">
-        <color rgba="1 0 0 1"/>
-    </material>
-    <material name="green">
-        <color rgba="0 1 0 1"/>
-    </material>
-    <material name="blue">
-        <color rgba="0 0 1 1"/>
-    </material>
-    <material name="sensor_blue">
-        <color rgba="0.2 0.2 1 1"/>
-    </material>
-    <material name="sensor_yellow">
-        <color rgba="0.8 0.8 0.2 1"/>
-    </material>
-    <material name="body_color">
-        <color rgba="1 0.3 0.1 1"/>
-    </material>
-    <material name="port_red">
-        <color rgba="1 0.2 0.2 1"/>
-    </material>
-    <material name="starboard_green">
-        <color rgba="0.2 1 0.2 1"/>
-    </material>
-    <xacro:arg name="sim_mode" default="false"/>
+    <xacro:include filename="../../../description/common_properties.xacro" />
     <xacro:include filename="robot_core.xacro" />
     <xacro:include filename="../../../description/imu.xacro" />

File: robots/sim/description/robot.urdf.xacro (robot description, xacro)
@@ -3,41 +3,10 @@
     <!-- See common Gazebo pugins in the world file -->
     <!--
-        To re-generate robot.urdf manually for troubleshooting:
-          xacro ~/robot_ws/install/articubot_one/share/articubot_one/description/robot.urdf.xacro sim_mode:=true > ~/robot_ws/src/articubot_one/description/robot.urdf
+        To re-generate robot.urdf.generated.xml manually for troubleshooting:
+          cd ~/robot_ws
+          colcon build
+          xacro install/articubot_one/share/articubot_one/robots/sim/description/robot.urdf.xacro sim_mode:=true > src/articubot_one/robots/sim/description/robot.urdf.generated.xml
     -->
-    <material name="white">
-        <color rgba="1 1 1 1" />
-    </material>
-    <material name="black">
-        <color rgba="0 0 0 1"/>
-    </material>
-    <material name="shadow_grey">
-        <color rgba="0.3 0.3 0.3 0.5"/>
-    </material>
-    <material name="red">
-        <color rgba="1 0 0 1"/>
-    </material>
-    <material name="green">
-        <color rgba="0 1 0 1"/>
-    </material>
-    <material name="blue">
-        <color rgba="0 0 1 1"/>
-    </material>
-    <material name="sensor_blue">
-        <color rgba="0.2 0.2 1 1"/>
-    </material>
-    <material name="sensor_yellow">
-        <color rgba="0.8 0.8 0.2 1"/>
-    </material>
-    <material name="body_color">
-        <color rgba="1 0.3 0.1 1"/>
-    </material>
-    <material name="port_red">
-        <color rgba="1 0.2 0.2 1"/>
-    </material>
-    <material name="starboard_green">
-        <color rgba="0.2 1 0.2 1"/>
-    </material>
-    <xacro:arg name="sim_mode" default="false"/>
+    <xacro:include filename="../../../description/common_properties.xacro" />
     <xacro:include filename="robot_core.xacro" />
     <xacro:include filename="../../../description/imu.xacro" />

File: robots/turtle/description/robot.urdf.xacro (robot description, xacro)
@@ -6,5 +6,5 @@
           cd ~/robot_ws
           colcon build
-          xacro install/articubot_one/share/articubot_one/robots/turtle/description/robot.urdf.xacro sim_mode:=true > src/articubot_one/robots/turtle/description/robot.urdf.generated.xml
+          xacro install/articubot_one/share/articubot_one/robots/turtle/description/robot.urdf.xacro sim_mode:=false > src/articubot_one/robots/turtle/description/robot.urdf.generated.xml
     -->
     <!-- See https://github.com/ROBOTIS-GIT/turtlebot3/tree/main/turtlebot3_description/urdf

Commit message: WIP: sonars initial check-in

File: robots/dragger/description/robot.urdf.xacro (robot description, xacro)
@@ -17,4 +17,8 @@
     <xacro:property name="laser_offset_z" value="0.57"/>
     <xacro:include filename="../../../description/lidar.xacro" />
+    <xacro:property name="sonars_offset_x" value="${chassis_length/2 + 0.005}"/>
+    <xacro:property name="sonars_offset_y" value="${chassis_width/2 - 0.02}"/>
+    <xacro:property name="sonars_offset_z" value="0.05"/>
+    <xacro:include filename="../../../description/sonars.xacro" />
     <xacro:property name="gps_offset_x" value="0.05"/>
     <xacro:property name="gps_offset_y" value="0.0"/>

File: robots/plucky/description/robot.urdf.xacro (robot description, xacro)
@@ -17,4 +17,8 @@
     <xacro:property name="laser_offset_z" value="0.50"/>
     <xacro:include filename="../../../description/lidar.xacro" />
+    <xacro:property name="sonars_offset_x" value="${chassis_length/2 + 0.005}"/>
+    <xacro:property name="sonars_offset_y" value="${chassis_width/2 - 0.02}"/>
+    <xacro:property name="sonars_offset_z" value="0.05"/>
+    <xacro:include filename="../../../description/sonars.xacro" />
     <xacro:property name="gps_offset_x" value="${wheel_offset_x}"/>
     <xacro:property name="gps_offset_y" value="-0.16"/>

Commit message: Plucky and Dragger URDFs adjusted to latest parameters changes

File: robots/dragger/description/robot.urdf.xacro (robot description, xacro)
@@ -15,6 +15,8 @@
     <xacro:include filename="../../../description/imu.xacro" />
     <xacro:include filename="../../../description/magnetometer.xacro" />
-    <xacro:property name="laser_offset_x" value="${wheel_offset_x - 0.14}"/>
-    <xacro:property name="laser_offset_z" value="0.57"/>
+    <!-- using arguments here, as that allows overriding default values -->
+    <xacro:arg name="lidar_offset_x" default="${wheel_offset_x - 0.14}"/>
+    <xacro:arg name="lidar_offset_z" default="0.57"/>
+    <xacro:arg name="lidar_base_length" default="0.06"/>
     <xacro:include filename="../../../description/lidar.xacro" />
     <xacro:property name="sonars_offset_x" value="${chassis_length/2 + 0.005}"/>

File: robots/plucky/description/robot.urdf.xacro (robot description, xacro)
@@ -15,6 +15,8 @@
     <xacro:include filename="../../../description/imu.xacro" />
     <xacro:include filename="../../../description/magnetometer.xacro" />
-    <xacro:property name="laser_offset_x" value="${wheel_offset_x}"/>
-    <xacro:property name="laser_offset_z" value="0.50"/>
+    <!-- using arguments here, as that allows overriding default values -->
+    <xacro:arg name="lidar_offset_x" default="${wheel_offset_x}"/>
+    <xacro:arg name="lidar_offset_z" default="0.47"/>
+    <xacro:arg name="lidar_base_length" default="0.01"/>
     <xacro:include filename="../../../description/lidar.xacro" />
     <xacro:property name="sonars_offset_x" value="${chassis_length/2 + 0.005}"/>
@@ -26,12 +28,12 @@
     <xacro:property name="gps_offset_z" value="0.45"/>
     <xacro:include filename="../../../description/gps.xacro" />
-    <xacro:property name="camera_offset_x" value="${wheel_offset_x + 0.05}"/>
-    <xacro:property name="camera_offset_z" value="0.45"/>
+    <xacro:property name="camera_offset_x" value="${wheel_offset_x + 0.1}"/>
+    <xacro:property name="camera_offset_z" value="0.25"/>
     <xacro:include filename="../../../description/camera.xacro" />
     <xacro:property name="open_circuit_voltage" value="12.592"/>
     <xacro:property name="battery_capacity" value="20.0"/>
     <xacro:include filename="../../../description/battery.xacro" />
-    <xacro:property name="depth_camera_offset_x" value="${wheel_offset_x}"/>
-    <xacro:property name="depth_camera_offset_z" value="0.45"/>
+    <xacro:property name="depth_camera_offset_x" value="${wheel_offset_x + 0.045}"/>
+    <xacro:property name="depth_camera_offset_z" value="0.4"/>
     <xacro:include filename="../../../description/depth_camera.xacro"/>
     <xacro:unless value="$(arg sim_mode)">
