Commit message: camera_oakd works in sim

File: robots/dragger/description/robot.urdf.xacro (robot description, xacro)
@@ -36,5 +36,4 @@
     <xacro:property name="battery_capacity" value="50.0"/>
     <xacro:include filename="../../../description/battery.xacro" />
-    <!-- xacro:include filename="../../../description/depth_camera.xacro" / -->
     <!-- xacro:include filename="../../../description/face.xacro" / -->
     <xacro:include filename="ros2_control.xacro" />

File: robots/seggy/description/robot.urdf.xacro (robot description, xacro)
@@ -24,9 +24,25 @@
     <xacro:property name="battery_capacity" value="20.0"/>
     <xacro:include filename="../../../description/battery.xacro" />
-    <xacro:property name="depth_camera_offset_x" value="${wheel_offset_x + 0.03}"/>
-    <xacro:property name="depth_camera_offset_z" value="${chassis_top_offset + 0.11}"/>
-    <xacro:include filename="../../../description/depth_camera.xacro"/>
+    <xacro:property name="camera_oakd_offset_x" value="${wheel_offset_x + 0.03}"/>
+    <xacro:property name="camera_oakd_offset_z" value="${chassis_top_offset + 0.115}"/>
+    <!-- URDF definitions for OAK-D Lite camera and Gazebo sim sensor -->
+    <xacro:include filename="../../../description/camera_oakd.xacro"/>
+    <!-- add a visual - mount for OAK-D Lite -->
+    <joint name="camera_oakd_mount_joint" type="fixed">
+        <parent link="chassis_link"/>
+        <child link="camera_oakd_mount_link"/>
+        <origin xyz="${camera_oakd_offset_x - 0.01} 0 ${camera_oakd_offset_z - 0.057}" rpy="0 0 0"/>
+    </joint>
+    <link name="camera_oakd_mount_link">
+            <visual>
+            <geometry>
+                <box size="0.002 0.07 0.115"/>
+            </geometry>
+            <material name="body_color"/>
+        </visual>
+    </link>
     <xacro:unless value="$(arg sim_mode)">
-        <xacro:arg name="parent_frame" default="depth_camera_link_optical" />
+        <!-- real OAK-D Lite camera -->
+        <xacro:arg name="parent_frame" default="camera_oakd_link_optical" />
         <xacro:include filename="$(find depthai_descriptions)/urdf/depthai_descr.urdf.xacro"/>
     </xacro:unless>

Commit message: Added OAK-D camera to Dragger

File: robots/dragger/description/robot.urdf.xacro (robot description, xacro)
@@ -30,10 +30,16 @@
     <xacro:property name="camera_offset_z" value="0.55"/>
     <xacro:include filename="../../../description/camera.xacro" />
+    <!--
     <xacro:property name="camera_stereo_offset_x" value="${wheel_offset_x + 0.19}"/>
     <xacro:property name="camera_stereo_offset_z" value="0.2"/>
     <xacro:include filename="../../../description/camera_stereo.xacro" />
+    -->
     <xacro:property name="open_circuit_voltage" value="12.592"/>
     <xacro:property name="battery_capacity" value="50.0"/>
     <xacro:include filename="../../../description/battery.xacro" />
+    <xacro:property name="camera_oakd_offset_x" value="${wheel_offset_x + 0.19}"/>
+    <xacro:property name="camera_oakd_offset_z" value="0.48"/>
+    <!-- URDF definitions for OAK-D Lite camera and Gazebo sim sensor -->
+    <xacro:include filename="../../../description/camera_oakd.xacro"/>
     <!-- xacro:include filename="../../../description/face.xacro" / -->
     <xacro:include filename="ros2_control.xacro" />

Commit message: Separated robot hardware parameters into a YAML file

File: robots/dragger/description/robot.urdf.xacro (robot description, xacro)
@@ -1,4 +1,7 @@
 <?xml version="1.0"?>
 <robot xmlns:xacro="http://www.ros.org/wiki/xacro"  name="robot">
+    <!-- Override this path for machine-specific real-hardware calibration. -->
+    <xacro:arg name="hardware_config"
+               default="$(find articubot_one)/robots/dragger/config/hardware.yaml"/>
     <!-- See common Gazebo pugins in the world file -->
     <!--

File: robots/dragger/description/ros2_control.xacro (robot description, xacro)
@@ -5,19 +5,20 @@
         <hardware>
             <xacro:unless value="$(arg sim_mode)">
-                <!-- Values corrected for Dragger robot -->
+                <!-- Load only for real hardware; simulation needs no hardware YAML. -->
+                <xacro:property name="hw" value="${xacro.load_yaml('$(arg hardware_config)')}"/>
                 <plugin>diffdrive_arduino/DiffDriveArduino</plugin>
                 <param name="left_wheel_name">left_wheel_joint</param>
                 <param name="right_wheel_name">right_wheel_joint</param>
                 <param name="loop_rate">30</param>
-                <param name="device">/dev/ttyACM0</param>
-                <param name="baud_rate">115200</param>
-                <param name="timeout">1000</param>
-                <param name="enc_counts_per_rev">13730</param>
-                <param name="wheels_pwm_factor">60.0</param>
+                <param name="device">${hw['device']}</param>
+                <param name="baud_rate">${hw['baud_rate']}</param>
+                <param name="timeout">${hw['timeout']}</param>
+                <param name="enc_counts_per_rev">${hw['enc_counts_per_rev']}</param>
+                <param name="wheels_pwm_factor">${hw['wheels_pwm_factor']}</param>
                 <!-- See https://docs.ros.org/en/jazzy/p/sensor_msgs/interfaces/msg/BatteryState.html -->
                 <param name="battery_name">main_battery</param>
-                <param name="battery_num_cells">4</param>
-                <param name="battery_technology">4</param>
-                <param name="battery_design_capacity">50</param>
+                <param name="battery_num_cells">${hw['battery_num_cells']}</param>
+                <param name="battery_technology">${hw['battery_technology']}</param>
+                <param name="battery_design_capacity">${hw['battery_design_capacity']}</param>
                 <!-- A workaround for sonar no-return ".inf" values
                  Set sonar_broadcaster's max_range: 5.1 in robots/dragger/config/controllers.yaml

File: robots/fido/description/robot.urdf.xacro (robot description, xacro)
@@ -1,4 +1,7 @@
 <?xml version="1.0"?>
 <robot xmlns:xacro="http://www.ros.org/wiki/xacro"  name="robot">
+    <!-- Override this path for machine-specific real-hardware calibration. -->
+    <xacro:arg name="hardware_config"
+               default="$(find articubot_one)/robots/fido/config/hardware.yaml"/>
     <!-- See common Gazebo pugins in the world file -->
     <!--

File: robots/fido/description/ros2_control.xacro (robot description, xacro)
@@ -6,21 +6,22 @@
             <!-- See https://github.com/slgrobotics/diffdrive_arduino-->
             <xacro:unless value="$(arg sim_mode)">
-                <!-- Values corrected for Fido robot -->
+                <!-- Load only for real hardware; simulation needs no hardware YAML. -->
+                <xacro:property name="hw" value="${xacro.load_yaml('$(arg hardware_config)')}"/>
                 <plugin>diffdrive_arduino/DiffDriveArduino</plugin>
                 <param name="left_wheel_name">left_wheel_joint</param>
                 <param name="right_wheel_name">right_wheel_joint</param>
                 <param name="loop_rate">30</param>
-                <param name="device">/dev/ttyACM0</param>
-                <param name="baud_rate">115200</param>
-                <param name="timeout">1000</param>
-                <param name="enc_counts_per_rev">60</param>
+                <param name="device">${hw['device']}</param>
+                <param name="baud_rate">${hw['baud_rate']}</param>
+                <param name="timeout">${hw['timeout']}</param>
+                <param name="enc_counts_per_rev">${hw['enc_counts_per_rev']}</param>
                 <!-- Arduino expects wheel speed setpoints in the range -100..100 (percent of max speed)
                      Use wheels_pwm_factor parameter (multiplier) to bring interface speed input into this range -->
-                <param name="wheels_pwm_factor">60.0</param>
+                <param name="wheels_pwm_factor">${hw['wheels_pwm_factor']}</param>
                 <!-- See https://docs.ros.org/en/jazzy/p/sensor_msgs/interfaces/msg/BatteryState.html -->
                 <param name="battery_name">main_battery</param>
-                <param name="battery_num_cells">4</param>
-                <param name="battery_technology">4</param>
-                <param name="battery_design_capacity">20</param>
+                <param name="battery_num_cells">${hw['battery_num_cells']}</param>
+                <param name="battery_technology">${hw['battery_technology']}</param>
+                <param name="battery_design_capacity">${hw['battery_design_capacity']}</param>
             </xacro:unless>
             <xacro:if value="$(arg sim_mode)">

File: robots/seggy/description/robot.urdf.xacro (robot description, xacro)
@@ -1,4 +1,7 @@
 <?xml version="1.0"?>
 <robot xmlns:xacro="http://www.ros.org/wiki/xacro"  name="robot">
+    <!-- Override this path for machine-specific real-hardware calibration. -->
+    <xacro:arg name="hardware_config"
+               default="$(find articubot_one)/robots/seggy/config/hardware.yaml"/>
     <!-- See common Gazebo pugins in the world file -->
     <!--

File: robots/seggy/description/ros2_control.xacro (robot description, xacro)
@@ -6,21 +6,22 @@
             <!-- See https://github.com/slgrobotics/diffdrive_arduino-->
             <xacro:unless value="$(arg sim_mode)">
-                <!-- Values corrected for Seggy robot -->
+                <!-- Load only for real hardware; simulation needs no hardware YAML. -->
+                <xacro:property name="hw" value="${xacro.load_yaml('$(arg hardware_config)')}"/>
                 <plugin>diffdrive_arduino/DiffDriveArduino</plugin>
                 <param name="left_wheel_name">left_wheel_joint</param>
                 <param name="right_wheel_name">right_wheel_joint</param>
                 <param name="loop_rate">30</param>
-                <param name="device">/dev/ttyACM0</param>
-                <param name="baud_rate">115200</param>
-                <param name="timeout">1000</param>
-                <param name="enc_counts_per_rev">60</param>
+                <param name="device">${hw['device']}</param>
+                <param name="baud_rate">${hw['baud_rate']}</param>
+                <param name="timeout">${hw['timeout']}</param>
+                <param name="enc_counts_per_rev">${hw['enc_counts_per_rev']}</param>
                 <!-- Arduino expects wheel speed setpoints in the range -100..100 (percent of max speed)
                      Use wheels_pwm_factor parameter (multiplier) to bring interface speed input into this range -->
-                <param name="wheels_pwm_factor">60.0</param>
+                <param name="wheels_pwm_factor">${hw['wheels_pwm_factor']}</param>
                 <!-- See https://docs.ros.org/en/jazzy/p/sensor_msgs/interfaces/msg/BatteryState.html -->
                 <param name="battery_name">main_battery</param>
-                <param name="battery_num_cells">4</param>
-                <param name="battery_technology">4</param>
-                <param name="battery_design_capacity">20</param>
+                <param name="battery_num_cells">${hw['battery_num_cells']}</param>
+                <param name="battery_technology">${hw['battery_technology']}</param>
+                <param name="battery_design_capacity">${hw['battery_design_capacity']}</param>
             </xacro:unless>
             <xacro:if value="$(arg sim_mode)">
