Commit message: typo fixed

File: robots/dragger/description/robot_core.xacro (robot description, xacro)
@@ -110,5 +110,5 @@
         </visual>
         <visual name="chassis_caster_joint_right">
-            <origin xyz="${caster_wheel_offset_x} ${-chassis_width*0.51} ${caster_wheel_offset_z}" rpy="0 0 0"/>
+            <origin xyz="${caster_wheel_offset_x} ${-chassis_width*0.52} ${caster_wheel_offset_z}" rpy="0 0 0"/>
             <geometry>
                 <sphere radius="${caster_wheel_offset_z*1.1}"/>

Commit message: Update robot_core.xacro

File: robots/dragger/description/robot_core.xacro (robot description, xacro)
@@ -105,5 +105,5 @@
             <origin xyz="${caster_wheel_offset_x} ${chassis_width*0.52} ${caster_wheel_offset_z}" rpy="0 0 0"/>
             <geometry>
-                <sphere radius="${caster_wheel_offset_z*1.1}"/>
+                <sphere radius="${caster_wheel_radius*0.7}"/>
             </geometry>
             <material name="body_color"/>
@@ -112,5 +112,5 @@
             <origin xyz="${caster_wheel_offset_x} ${-chassis_width*0.52} ${caster_wheel_offset_z}" rpy="0 0 0"/>
             <geometry>
-                <sphere radius="${caster_wheel_offset_z*1.1}"/>
+                <sphere radius="${caster_wheel_radius*0.7}"/>
             </geometry>
             <material name="body_color"/>
