Commit message: URDF: resolve package://articubot_one/... resources in Gazebo as well as RViz

File: robots/dragger/description/robot_core.xacro (robot description, xacro)
@@ -139,12 +139,5 @@
     </joint>
     <link name="left_wheel">
-        <visual name="left_wheel_tire_gz_visual">
-            <origin xyz="0 0 0" rpy="${pi/2} 0 0" />
-            <geometry>
-                <mesh filename="model://meshes/wheel_link.STL" scale="${wheel_radius*12.7} ${wheel_thickness*10.2} ${wheel_radius*12.7}"/>
-            </geometry>
-            <material name="port_red"/>
-        </visual>
-        <visual name="left_wheel_tire_rviz_visual">
+        <visual name="left_wheel_tire_visual">
             <origin xyz="0 0 0" rpy="${pi/2} 0 0" />
             <geometry>
@@ -210,12 +203,5 @@
     </joint>
     <link name="right_wheel">
-        <visual name="right_wheel_tire_gz_visual">
-            <origin xyz="0 0 0" rpy="${-pi/2} 0 0" />
-            <geometry>
-                <mesh filename="model://meshes/wheel_link.STL" scale="${wheel_radius*12.7} ${wheel_thickness*10.2} ${wheel_radius*12.7}"/>
-            </geometry>
-            <material name="starboard_green"/>
-        </visual>
-        <visual name="right_wheel_tire_rviz_visual">
+        <visual name="right_wheel_tire_visual">
             <origin xyz="0 0 0" rpy="${-pi/2} 0 0" />
             <geometry>

File: robots/fido/description/robot_core.xacro (robot description, xacro)
@@ -162,12 +162,5 @@
     </joint>
     <link name="left_wheel">
-        <visual name="left_wheel_tire_gz_visual">
-            <origin xyz="0 0 0" rpy="${pi/2} 0 0" />
-            <geometry>
-                <mesh filename="model://meshes/wheel_link.STL" scale="${wheel_radius*12.7} ${wheel_thickness*10.2} ${wheel_radius*12.7}"/>
-            </geometry>
-            <material name="port_red"/>
-        </visual>
-        <visual name="left_wheel_tire_rviz_visual">
+        <visual name="left_wheel_tire_visual">
             <origin xyz="0 0 0" rpy="${pi/2} 0 0" />
             <geometry>
@@ -233,12 +226,5 @@
     </joint>
     <link name="right_wheel">
-        <visual name="right_wheel_tire_gz_visual">
-            <origin xyz="0 0 0" rpy="${-pi/2} 0 0" />
-            <geometry>
-                <mesh filename="model://meshes/wheel_link.STL" scale="${wheel_radius*12.7} ${wheel_thickness*10.2} ${wheel_radius*12.7}"/>
-            </geometry>
-            <material name="starboard_green"/>
-        </visual>
-        <visual name="right_wheel_tire_rviz_visual">
+        <visual name="right_wheel_tire_visual">
             <origin xyz="0 0 0" rpy="${-pi/2} 0 0" />
             <geometry>

File: robots/plucky/description/robot_core.xacro (robot description, xacro)
@@ -167,12 +167,5 @@
     </joint>
     <link name="left_wheel">
-        <visual name="left_wheel_tire_gz_visual">
-            <origin xyz="0 0 0" rpy="${pi/2} 0 0" />
-            <geometry>
-                <mesh filename="model://meshes/wheel_link.STL" scale="${wheel_radius*12.7} ${wheel_thickness*10.2} ${wheel_radius*12.7}"/>
-            </geometry>
-            <material name="port_red"/>
-        </visual>
-        <visual name="left_wheel_tire_rviz_visual">
+        <visual name="left_wheel_tire_visual">
             <origin xyz="0 0 0" rpy="${pi/2} 0 0" />
             <geometry>
@@ -238,12 +231,5 @@
     </joint>
     <link name="right_wheel">
-        <visual name="right_wheel_tire_gz_visual">
-            <origin xyz="0 0 0" rpy="${-pi/2} 0 0" />
-            <geometry>
-                <mesh filename="model://meshes/wheel_link.STL" scale="${wheel_radius*12.7} ${wheel_thickness*10.2} ${wheel_radius*12.7}"/>
-            </geometry>
-            <material name="starboard_green"/>
-        </visual>
-        <visual name="right_wheel_tire_rviz_visual">
+        <visual name="right_wheel_tire_visual">
             <origin xyz="0 0 0" rpy="${-pi/2} 0 0" />
             <geometry>

File: robots/seggy/description/robot_core.xacro (robot description, xacro)
@@ -162,12 +162,5 @@
     </joint>
     <link name="left_wheel">
-        <visual name="left_wheel_tire_gz_visual">
-            <origin xyz="0 0 0" rpy="${pi/2} 0 0" />
-            <geometry>
-                <mesh filename="model://meshes/wheel_link.STL" scale="${wheel_radius*12.7} ${wheel_thickness*10.2} ${wheel_radius*12.7}"/>
-            </geometry>
-            <material name="port_red"/>
-        </visual>
-        <visual name="left_wheel_tire_rviz_visual">
+        <visual name="left_wheel_tire_visual">
             <origin xyz="0 0 0" rpy="${pi/2} 0 0" />
             <geometry>
@@ -233,12 +226,5 @@
     </joint>
     <link name="right_wheel">
-        <visual name="right_wheel_tire_gz_visual">
-            <origin xyz="0 0 0" rpy="${-pi/2} 0 0" />
-            <geometry>
-                <mesh filename="model://meshes/wheel_link.STL" scale="${wheel_radius*12.7} ${wheel_thickness*10.2} ${wheel_radius*12.7}"/>
-            </geometry>
-            <material name="starboard_green"/>
-        </visual>
-        <visual name="right_wheel_tire_rviz_visual">
+        <visual name="right_wheel_tire_visual">
             <origin xyz="0 0 0" rpy="${-pi/2} 0 0" />
             <geometry>

File: robots/turtle/description/create_base.urdf.xacro (robot description, xacro)
@@ -63,11 +63,5 @@
     <!-- CHASSIS LINK -->
     <link name="chassis_link">
-      <visual name="chassis_gz_visual">
-        <origin xyz=" 0 0 -0.015" rpy="0 0 0"/>
-        <geometry>
-            <mesh filename="model://meshes/create_1.dae"/>
-        </geometry>
-      </visual>
-      <visual name="chassis_rviz_visual">
+      <visual name="chassis_visual">
         <origin xyz=" 0 0 -0.015" rpy="0 0 0"/>
         <geometry>
