Commit message: commented out Gazebo visuals

File: robots/stingray/description/lidar_support.xacro (robot description, xacro)
@@ -13,5 +13,5 @@
     -->
     <link name="lidar_support_link">
-        <visual name="lidar_support__gz_visual">
+        <!-- <visual name="lidar_support__gz_visual">
             <origin xyz="${lidar_support_offset_x} ${lidar_support_offset_y} ${lidar_support_offset_z}" rpy="0.0 0.0 ${pi/2}"/>
             <geometry>
@@ -19,5 +19,5 @@
             </geometry>
             <material name="black"/>
-        </visual>
+        </visual> -->
         <visual name="lidar_support_rviz_visual">
             <origin xyz="${lidar_support_offset_x} ${lidar_support_offset_y} ${lidar_support_offset_z}" rpy="0.0 0.0 ${pi/2}"/>

File: robots/stingray/description/robot_core.xacro (robot description, xacro)
@@ -86,5 +86,5 @@
     <!-- CHASSIS LINK -->
     <link name="chassis_link">
-        <visual name="chassis_gz_visual">
+        <!-- <visual name="chassis_gz_visual">
             <origin xyz="0.0 0.0 0.0" rpy="0.0 0.0 0.0"/>
             <geometry>
@@ -92,5 +92,5 @@
             </geometry>
             <material name="acrylic"/>
-        </visual>
+        </visual> -->
         <visual name="chassis_rviz_visual">
              <origin xyz="0.0 0.0 0.0" rpy="0.0 0.0 0.0"/>
