Commit message: delete Plucky body

File: robots/stingray/description/robot_core.xacro (robot description, xacro)
@@ -74,5 +74,5 @@
     <!-- CHASSIS LINK -->
     <link name="chassis_link">
-        <visual name="chassis_visual_bottom">
+        <!-- <visual name="chassis_visual_bottom">
             <origin xyz="0 0 ${chassis_height/8}"/>
             <geometry>
@@ -101,5 +101,5 @@
             </geometry>
             <material name="body_color"/>
-        </visual>
+        </visual> -->
         <visual name="chassis_front_axle_left">
             <origin xyz="${wheel_offset_x} ${chassis_width*0.5} 0" rpy="-${pi/2} 0 0"/>

Commit message: add Stingray .mesh body

File: robots/stingray/description/robot_core.xacro (robot description, xacro)
@@ -74,32 +74,21 @@
     <!-- CHASSIS LINK -->
     <link name="chassis_link">
-        <!-- <visual name="chassis_visual_bottom">
-            <origin xyz="0 0 ${chassis_height/8}"/>
-            <geometry>
-                <box size="${chassis_length} ${chassis_width} ${chassis_height/4}"/>
-            </geometry>
-            <material name="body_color"/>
-        </visual>
-        <visual name="chassis_visual_front">
-            <origin xyz="0.15 0 ${chassis_height/2-0.03}" rpy="0 ${pi/4} 0"/>
-            <geometry>
-                <box size="0.25 ${chassis_width} 0.01"/>
-            </geometry>
-            <material name="body_color"/>
-        </visual>
-        <visual name="chassis_visual_back">
-            <origin xyz="-0.07 0 ${chassis_height/2-0.03}" rpy="0 -${pi/4} 0"/>
-            <geometry>
-                <box size="0.25 ${chassis_width} 0.01"/>
-            </geometry>
-            <material name="body_color"/>
-        </visual>
-        <visual name="chassis_top_visual">
-            <origin xyz="${wheel_offset_x} 0 ${chassis_height*3/4}"/>
-            <geometry>
-                <box size="${chassis_top_length} ${chassis_width} ${chassis_height/2}"/>
-            </geometry>
-            <material name="body_color"/>
-        </visual> -->
+        <visual name="chassis_gz_visual">
+            <origin xyz="0.0 0.0 0.0" rpy="0.0 0.0 0.0"/>
+            <geometry>
+                <!-- <mesh filename="file://$(find stingray)/description/Stingray.stl" scale="0.001 0.001 0.001"/> -->
+                <mesh filename="model://meshes/Stingray.stl" scale="0.001 0.001 0.001"/>
+            </geometry>
+            <material name="grey"/>
+        </visual>
+        <visual name="chassis_rviz_visual">
+             <origin xyz="0.0 0.0 0.0" rpy="0.0 0.0 0.0"/>
+            <geometry>
+                <!-- box size="${chassis_length} ${chassis_width} ${chassis_height}"/ -->
+                <!-- <mesh filename="file://$(find stingray)/description/meshes/Stingray.stl" scale="0.001 0.001 0.001"/> -->
+                <mesh filename="package://articubot_one/assets/meshes/Stingray.stl" scale="0.001 0.001 0.001"/>
+            </geometry>
+            <material name="grey"/>
+        </visual>
         <visual name="chassis_front_axle_left">
             <origin xyz="${wheel_offset_x} ${chassis_width*0.5} 0" rpy="-${pi/2} 0 0"/>

Commit message: chassis & wheel properties

File: robots/stingray/description/robot_core.xacro (robot description, xacro)
@@ -12,7 +12,11 @@
     <xacro:property name="chassis_mass" value="0.98"/>
     <xacro:property name="chassis_top_length" value="0.095"/>
-    <xacro:property name="wheel_radius" value="0.192"/>
-    <xacro:property name="wheel_thickness" value="0.045"/>
-    <xacro:property name="wheel_mass" value="1.0"/>
+    <!-- <xacro:property name="wheel_radius" value="0.192"/> -->
+    <!-- <xacro:property name="wheel_thickness" value="0.045"/> -->
+    <!-- <xacro:property name="wheel_mass" value="1.0"/> -->
+    <xacro:property name="wheel_radius" value="0.0615"/>
+    <xacro:property name="wheel_thickness" value="0.02"/>
+    <xacro:property name="wheel_mass" value="0.058"/>
+    <xacro:property name="wheel_offset" value="0.13"/>
     <xacro:property name="wheel_offset_x" value="${chassis_length/2 - wheel_radius - 0.01}"/>
     <xacro:property name="wheel_offset_y" value="0.280"/>

Commit message: remove Left wheel except empty link

File: robots/stingray/description/robot_core.xacro (robot description, xacro)
@@ -11,5 +11,5 @@
     <xacro:property name="chassis_height" value="0.081"/>
     <xacro:property name="chassis_mass" value="0.98"/>
-    <xacro:property name="chassis_top_length" value="0.095"/>
+    <!-- <xacro:property name="chassis_top_length" value="0.095"/> -->
     <!-- <xacro:property name="wheel_radius" value="0.192"/> -->
     <!-- <xacro:property name="wheel_thickness" value="0.045"/> -->
@@ -60,5 +60,5 @@
     <link name="base_footprint">
         <visual name="footprint_visual">
-            <origin xyz="0 0 0.001"/>
+            <origin xyz="0 0 0.0001"/>
             <geometry>
                 <!-- box size="${wheel_offset_y * 2 + wheel_thickness} ${wheel_offset_y * 2 + wheel_thickness} 0.02"/ -->
@@ -108,55 +108,4 @@
         <xacro:inertial_box mass="${chassis_mass}" x="${chassis_length}" y="${chassis_width}" z="${chassis_height}">
             <origin xyz="0.0 0.0 0.0" rpy="0.0 0.0 0.0"/>
-        </xacro:inertial_box>
-        <visual name="chassis_front_axle_left">
-            <origin xyz="${wheel_offset_x} ${chassis_width*0.5} 0" rpy="-${pi/2} 0 0"/>
-            <geometry>
-                <cylinder radius="0.03" length="${chassis_width*0.5}"/>
-            </geometry>
-            <material name="body_color"/>
-        </visual>
-        <visual name="chassis_front_axle_right">
-            <origin xyz="${wheel_offset_x} ${-chassis_width*0.5} 0" rpy="${pi/2} 0 0"/>
-            <geometry>
-                <cylinder radius="0.03" length="${chassis_width*0.5}"/>
-            </geometry>
-            <material name="body_color"/>
-        </visual>
-        <visual name="chassis_caster_holder_left">
-            <origin xyz="${caster_wheel_offset_x+0.09} ${caster_wheel_offset_y*0.85} ${caster_wheel_offset_z*0.42}" rpy="0 ${pi/4} 0"/>
-            <geometry>
-                <cylinder radius="0.012" length="0.23"/>
-            </geometry>
-            <material name="body_color"/>
-        </visual>
-        <visual name="chassis_caster_joint_left">
-            <origin xyz="${caster_wheel_offset_x} ${caster_wheel_offset_y*0.9} ${caster_wheel_offset_z}" rpy="0 0 0"/>
-            <geometry>
-                <sphere radius="0.03"/>
-            </geometry>
-            <material name="body_color"/>
-        </visual>
-        <visual name="chassis_caster_holder_right">
-            <origin xyz="${caster_wheel_offset_x+0.09} ${-caster_wheel_offset_y*0.85} ${caster_wheel_offset_z*0.42}" rpy="0 ${pi/4} 0"/>
-            <geometry>
-                <cylinder radius="0.012" length="0.23"/>
-            </geometry>
-            <material name="body_color"/>
-        </visual>
-        <visual name="chassis_caster_joint_right">
-            <origin xyz="${caster_wheel_offset_x} ${-caster_wheel_offset_y*0.9} ${caster_wheel_offset_z}" rpy="0 0 0"/>
-            <geometry>
-                <sphere radius="0.03"/>
-            </geometry>
-            <material name="body_color"/>
-        </visual>
-        <collision>
-            <origin xyz="0 0 ${chassis_height/2}" rpy="0 0 0"/>
-            <geometry>
-                <box size="${chassis_length} ${chassis_width} ${chassis_height}"/>
-            </geometry>
-        </collision>
-        <xacro:inertial_box mass="0.5" x="${chassis_length}" y="${chassis_width}" z="${chassis_height}">
-            <origin xyz="0 0 ${chassis_height/2}" rpy="0 0 0"/>
         </xacro:inertial_box>
     </link>
@@ -174,5 +123,5 @@
     </joint>
     <link name="left_wheel">
-        <visual name="left_wheel_tire_gz_visual">
+        <!-- <visual name="left_wheel_tire_gz_visual">
             <origin xyz="0 0 0" rpy="${pi/2} 0 0" />
             <geometry>
@@ -180,6 +129,6 @@
             </geometry>
             <material name="port_red"/>
-        </visual>
-        <visual name="left_wheel_tire_rviz_visual">
+        </visual> -->
+        <!-- <visual name="left_wheel_tire_rviz_visual">
             <origin xyz="0 0 0" rpy="${pi/2} 0 0" />
             <geometry>
@@ -187,18 +136,18 @@
             </geometry>
             <material name="port_red"/>
-        </visual>
-        <visual name="left_wheel_solid_visual">
+        </visual> -->
+        <!-- <visual name="left_wheel_solid_visual">
             <geometry>
                 <cylinder radius="${wheel_radius}" length="${wheel_thickness/10.0}"/>
             </geometry>
             <material name="port_red"/>
-        </visual>
-        <visual name="left_wheel_axis_visual">
+        </visual> -->
+        <!-- <visual name="left_wheel_axis_visual">
             <geometry>
                 <cylinder radius="${wheel_radius*0.05}" length="${wheel_thickness*1.1}"/>
             </geometry>
             <material name="blue"/>
-        </visual>
-        <visual name="left_wheel_marker_visual">
+        </visual> -->
+        <!-- <visual name="left_wheel_marker_visual">
             <origin xyz="0 ${wheel_radius*0.7} 0" rpy="0 0 0" />
             <geometry>
@@ -206,6 +155,6 @@
             </geometry>
             <material name="blue"/>
-        </visual>
-        <collision>
+        </visual> -->
+        <!-- <collision>
             <geometry>
                 <cylinder radius="${wheel_radius}" length="${wheel_thickness}"/>
@@ -227,8 +176,8 @@
                 </contact>
             </surface>
-        </collision>
-        <xacro:inertial_cylinder mass="${wheel_mass}" length="${wheel_thickness}" radius="${wheel_radius}">
+        </collision> -->
+        <!-- <xacro:inertial_cylinder mass="${wheel_mass}" length="${wheel_thickness}" radius="${wheel_radius}">
             <origin xyz="0 0 0" rpy="0 0 0"/>
-        </xacro:inertial_cylinder>
+        </xacro:inertial_cylinder> -->
     </link>
     <!-- RIGHT WHEEL LINK -->

Commit message: delete right wheel collision

File: robots/stingray/description/robot_core.xacro (robot description, xacro)
@@ -227,5 +227,5 @@
             <material name="blue"/>
         </visual>
-        <collision>
+        <!-- <collision>
             <geometry>
                 <cylinder radius="${wheel_radius}" length="${wheel_thickness}"/>
@@ -247,5 +247,5 @@
                 </contact>
             </surface>
-        </collision>
+        </collision> -->
         <xacro:inertial_cylinder mass="${wheel_mass}" length="${wheel_thickness}" radius="${wheel_radius}">
             <origin xyz="0 0 0" rpy="0 0 0"/>

Commit message: delete right wheel marker

File: robots/stingray/description/robot_core.xacro (robot description, xacro)
@@ -220,5 +220,5 @@
             <material name="blue"/>
         </visual>
-        <visual name="right_wheel_marker_visual">
+        <!-- <visual name="right_wheel_marker_visual">
             <origin xyz="0 ${-wheel_radius*0.7} 0" rpy="0 0 0" />
             <geometry>
@@ -226,5 +226,5 @@
             </geometry>
             <material name="blue"/>
-        </visual>
+        </visual> -->
         <!-- <collision>
             <geometry>

Commit message: delete right wheel completely

File: robots/stingray/description/robot_core.xacro (robot description, xacro)
@@ -194,5 +194,5 @@
     </joint>
     <link name="right_wheel">
-        <visual name="right_wheel_tire_gz_visual">
+        <!-- <visual name="right_wheel_tire_gz_visual">
             <origin xyz="0 0 0" rpy="${-pi/2} 0 0" />
             <geometry>
@@ -200,6 +200,6 @@
             </geometry>
             <material name="starboard_green"/>
-        </visual>
-        <visual name="right_wheel_tire_rviz_visual">
+        </visual> -->
+        <!-- <visual name="right_wheel_tire_rviz_visual">
             <origin xyz="0 0 0" rpy="${-pi/2} 0 0" />
             <geometry>
@@ -207,17 +207,17 @@
             </geometry>
             <material name="starboard_green"/>
-        </visual>
-        <visual name="right_wheel_solid_visual">
+        </visual> -->
+        <!-- <visual name="right_wheel_solid_visual">
             <geometry>
                 <cylinder radius="${wheel_radius}" length="${wheel_thickness/10.0}"/>
             </geometry>
             <material name="starboard_green"/>
-        </visual>
-        <visual name="right_wheel_axis_visual">
+        </visual> -->
+        <!-- <visual name="right_wheel_axis_visual">
             <geometry>
                 <cylinder radius="${wheel_radius*0.05}" length="${wheel_thickness*1.1}"/>
             </geometry>
             <material name="blue"/>
-        </visual>
+        </visual> -->
         <!-- <visual name="right_wheel_marker_visual">
             <origin xyz="0 ${-wheel_radius*0.7} 0" rpy="0 0 0" />

Commit message: P>S L wheel joint, add _link to empty wheel def

File: robots/stingray/description/robot_core.xacro (robot description, xacro)
@@ -110,6 +110,6 @@
         </xacro:inertial_box>
     </link>
-    <!-- LEFT WHEEL LINK -->
-    <joint name="left_wheel_joint" type="continuous">
+    <!-- LEFT WHEEL JOINT -->
+    <!-- <joint name="left_wheel_joint" type="continuous">
         <parent link="chassis_link"/>
         <child link="left_wheel"/>
@@ -121,6 +121,13 @@
           </limit>
         </axis>
-    </joint>
-    <link name="left_wheel">
+    </joint> -->
+    <joint name="left_wheel_joint" type="continuous">
+        <parent link="base_link"/>
+        <child link="left_wheel_link"/>
+        <origin xyz="0.0 0.13 0.0" rpy="-${pi/2} 0.0 0.0"/>
+        <axis xyz="0 0 1"/>
+    </joint>
+    <!-- LEFT WHEEL LINK -->
+    <link name="left_wheel_link">
         <!-- <visual name="left_wheel_tire_gz_visual">
             <origin xyz="0 0 0" rpy="${pi/2} 0 0" />
@@ -248,7 +255,7 @@
             </surface>
         </collision> -->
-        <xacro:inertial_cylinder mass="${wheel_mass}" length="${wheel_thickness}" radius="${wheel_radius}">
+        <!-- <xacro:inertial_cylinder mass="${wheel_mass}" length="${wheel_thickness}" radius="${wheel_radius}">
             <origin xyz="0 0 0" rpy="0 0 0"/>
-        </xacro:inertial_cylinder>
+        </xacro:inertial_cylinder> -->
     </link>
     <!-- CASTER WHEELS LINKS -->

Commit message: add right wheel

File: robots/stingray/description/robot_core.xacro (robot description, xacro)
@@ -19,7 +19,7 @@
     <xacro:property name="wheel_mass" value="0.058"/>
     <xacro:property name="wheel_offset" value="0.13"/>
-    <xacro:property name="wheel_offset_x" value="${chassis_length/2 - wheel_radius - 0.01}"/>
-    <xacro:property name="wheel_offset_y" value="0.280"/>
-    <xacro:property name="wheel_offset_z" value="0.01"/>
+    <xacro:property name="wheel_offset_x" value="0.13"/>
+    <xacro:property name="wheel_offset_y" value="0.0"/>
+    <xacro:property name="wheel_offset_z" value="0.0"/>
     <xacro:property name="caster_wheel_radius" value="0.05"/>
     <xacro:property name="caster_wheel_thickness" value="0.02"/>
@@ -125,5 +125,5 @@
         <parent link="base_link"/>
         <child link="left_wheel_link"/>
-        <origin xyz="0.0 0.13 0.0" rpy="-${pi/2} 0.0 0.0"/>
+        <origin xyz="0.0 ${wheel_offset} 0.0" rpy="-${pi/2} 0.0 0.0"/>
         <axis xyz="0 0 1"/>
     </joint>
@@ -187,18 +187,40 @@
             <origin xyz="0 0 0" rpy="0 0 0"/>
         </xacro:inertial_cylinder> -->
-    </link>
-    <!-- RIGHT WHEEL LINK -->
+        <visual name="left_wheel_visual">
+            <geometry>
+                <cylinder radius="${wheel_radius}" length="${wheel_thickness}"/>
+            </geometry>
+            <material name="blue"/>
+        </visual>
+        <visual name="left_wheel_marker_visual">
+            <origin xyz="0 ${wheel_radius*0.7} 0" rpy="0 0 0" />
+            <geometry>
+                <box size="${wheel_radius*0.2} ${wheel_radius*0.3} ${wheel_thickness*1.1}"/>
+            </geometry>
+            <material name="white"/>
+        </visual>
+        <collision>
+            <geometry>
+                <cylinder radius="${wheel_radius}" length="${wheel_thickness}"/>
+            </geometry>
+        </collision>
+        <xacro:inertial_cylinder mass="0.141" length="${wheel_thickness}" radius="${wheel_radius}">
+            <origin xyz="0.0 0.0 0.0" rpy="0.0 0.0 0.0"/>
+        </xacro:inertial_cylinder>
+    </link>
+    <!-- RIGHT WHEEL JOINT -->
     <joint name="right_wheel_joint" type="continuous">
         <parent link="chassis_link"/>
-        <child link="right_wheel"/>
-        <origin xyz="${wheel_offset_x} ${-wheel_offset_y} 0" rpy="${pi/2 - 0.15} 0 0" />
+        <child link="right_wheel_link"/>
+        <origin xyz="0.0 ${-wheel_offset} 0.0" rpy="${pi/2} 0 0"/>
         <axis xyz="0 0 -1">
-          <limit>
+          <!-- <limit>
             <lower>-1.79769e+308</lower>
             <upper>1.79769e+308</upper>
-          </limit>
+          </limit> -->
         </axis>
     </joint>
-    <link name="right_wheel">
+    <!-- RIGHT WHEEL LINK -->
+    <link name="right_wheel_link">
         <!-- <visual name="right_wheel_tire_gz_visual">
             <origin xyz="0 0 0" rpy="${-pi/2} 0 0" />
@@ -258,4 +280,18 @@
             <origin xyz="0 0 0" rpy="0 0 0"/>
         </xacro:inertial_cylinder> -->
+        <visual name="right_wheel_visual">
+            <geometry>
+                <cylinder radius="${wheel_radius}" length="${wheel_thickness}"/>
+            </geometry>
+            <material name="blue"/>
+        </visual>
+        <collision>
+            <geometry>
+                <cylinder radius="${wheel_radius}" length="${wheel_thickness}"/>
+            </geometry>
+        </collision>
+        <xacro:inertial_cylinder mass="0.141" length="${wheel_thickness}" radius="${wheel_radius}">
+            <origin xyz="0.0 0.0 0.0" rpy="0.0 0.0 0.0"/>
+        </xacro:inertial_cylinder>
     </link>
     <!-- CASTER WHEELS LINKS -->

Commit message: fixed left wheel

File: robots/stingray/description/robot_core.xacro (robot description, xacro)
@@ -11,4 +11,5 @@
     <xacro:property name="chassis_height" value="0.081"/>
     <xacro:property name="chassis_mass" value="0.98"/>
+    <xacro:property name="chassis_offset" value="0.0455"/>
     <!-- <xacro:property name="chassis_top_length" value="0.095"/> -->
     <!-- <xacro:property name="wheel_radius" value="0.192"/> -->
@@ -78,5 +79,5 @@
         <parent link="base_link"/>
         <child link="chassis_link"/>
-        <origin xyz="${-wheel_offset_x} 0 ${-wheel_offset_z}"/>
+        <origin xyz="0.0 0.0 0.0"/>
     </joint>
     <!-- CHASSIS LINK -->
@@ -214,10 +215,5 @@
         <child link="right_wheel_link"/>
         <origin xyz="0.0 ${-wheel_offset} 0.0" rpy="${pi/2} 0 0"/>
-        <axis xyz="0 0 -1">
-          <!-- <limit>
-            <lower>-1.79769e+308</lower>
-            <upper>1.79769e+308</upper>
-          </limit> -->
-        </axis>
+        <axis xyz="0 0 -1"/>
     </joint>
     <!-- RIGHT WHEEL LINK -->
@@ -286,4 +282,11 @@
             <material name="blue"/>
         </visual>
+        <visual name="right_wheel_marker_visual">
+            <origin xyz="0 ${wheel_radius*0.7} 0" rpy="0 0 0" />
+            <geometry>
+                <box size="${wheel_radius*0.2} ${wheel_radius*0.3} ${wheel_thickness*1.1}"/>
+            </geometry>
+            <material name="white"/>
+        </visual>
         <collision>
             <geometry>

Commit message: add fixed center caster

File: robots/stingray/description/robot_core.xacro (robot description, xacro)
@@ -14,4 +14,7 @@
     <xacro:property name="wheel_separation" value="0.26"/>
     <xacro:property name="caster_radius" value="0.028"/>
+    <xacro:property name="caster_x_offset" value="-0.207"/>
+    <xacro:property name="caster_z_offset" value="-0.035"/>
+    <xacro:property name="caster_mass" value="0.022"/>
     <xacro:property name="wheel_offset_x" value="0.13"/>
     <xacro:property name="wheel_offset_y" value="0.0"/>
@@ -164,4 +167,36 @@
         </xacro:inertial_cylinder>
     </link>
+    <!-- CASTER WHEEL center JHP -->
+    <!-- CASTER WHEEL JOINT-->
+    <joint name="caster_wheel_joint" type="fixed">
+        <origin xyz="${caster_x_offset} 0.0 ${caster_z_offset}" rpy="0.0 0.0 0.0"/>
+        <parent link="base_link"/>
+        <child link="caster_wheel_link"/>
+        <axis xyz="0.0 0.0 0.0"/>
+        <limit lower="0.0" upper="0.0" effort="0.0" velocity="0.0"/>
+    </joint>
+    <!-- CASTER WHEEL LINK -->
+    <link name="caster_wheel_link">
+        <visual name="">
+            <origin xyz="0.0 0.0 0.0" rpy="0.0 0.0 0.0"/>
+            <geometry>
+                <sphere radius="${caster_radius}"/>
+            </geometry>
+            <material name="white"/>
+        </visual>
+<!--
+        <collision>
+            <origin xyz="0.0 0.0 0.0" rpy="0.0 0.0 0.0"/>
+            <geometry>
+                <sphere radius="${caster_radius}"/>
+            </geometry>
+        </collision>
+ -->
+<!--
+        <xacro:inertial_sphere mass="${caster_mass}" radius="${caster_radius}">
+            <origin xyz="0.0 0.0 0.0" rpy="0.0 0.0 0.0"/>
+        </xacro:inertial_sphere>
+ -->
+    </link>
     <!-- CASTER WHEELS LINKS -->
     <joint name="left_caster_wheel_joint" type="${caster_joint_type}">
