Commit message: left caster removed

File: robots/stingray/description/robot_core.xacro (robot description, xacro)
@@ -196,4 +196,5 @@
     </link>
     <!-- CASTER WHEELS LINKS -->
+<!--
     <joint name="left_caster_wheel_joint" type="${caster_joint_type}">
         <parent link="chassis_link"/>
@@ -202,5 +203,7 @@
         <axis xyz="0 0 1"/>
     </joint>
-    <link name="left_caster_wheel">
+ -->
+    <!-- <link name="left_caster_wheel"> -->
+<!--
         <visual name="left_caster_visual">
             <geometry>
@@ -215,4 +218,6 @@
             <material name="blue"/>
         </visual>
+ -->
+        <!--
         <collision>
             <geometry>
@@ -230,8 +235,11 @@
             </surface>
         </collision>
+        -->
+<!--
         <xacro:inertial_cylinder mass="${caster_wheel_mass}" length="${caster_wheel_thickness}" radius="${caster_wheel_radius}">
             <origin xyz="0 0 0" rpy="0 0 0"/>
         </xacro:inertial_cylinder>
-    </link>
+-->
+    <!-- </link> -->
     <joint name="right_caster_wheel_joint" type="${caster_joint_type}">
         <parent link="chassis_link"/>

File: robots/stingray/description/ros2_control.xacro (robot description, xacro)
@@ -30,15 +30,15 @@
             <state_interface name="position" />
         </joint>
-        <xacro:if value="$(arg sim_mode)">
+        <!-- <xacro:if value="$(arg sim_mode)"> -->
             <!-- we need this for Rviz to reflect rotations of joints published by broad_cont in Gazebo -->
-            <joint name="left_caster_wheel_joint">
+            <!-- <joint name="left_caster_wheel_joint">
                 <state_interface name="velocity" />
                 <state_interface name="position" />
-            </joint>
-            <joint name="right_caster_wheel_joint">
+            </joint> -->
+            <!-- <joint name="right_caster_wheel_joint">
                 <state_interface name="velocity" />
                 <state_interface name="position" />
-            </joint>
-        </xacro:if>
+            </joint> -->
+        <!-- </xacro:if> -->
     </ros2_control>
     <gazebo>

Commit message: deleted commented out code

File: robots/stingray/description/robot_core.xacro (robot description, xacro)
@@ -205,98 +205,3 @@
         </xacro:inertial_sphere>
     </link>
-    <!-- CASTER WHEELS LINKS -->
-    <!-- LEFT CASTER WHEEL -->
-<!--
-    <joint name="left_caster_wheel_joint" type="${caster_joint_type}">
-        <parent link="chassis_link"/>
-        <child link="left_caster_wheel"/>
-        <origin xyz="${caster_wheel_offset_x} ${caster_wheel_offset_y} ${caster_wheel_offset_z}" rpy="${pi/2} 0 0" />
-        <axis xyz="0 0 1"/>
-    </joint>
- -->
-    <!-- <link name="left_caster_wheel"> -->
-<!--
-        <visual name="left_caster_visual">
-            <geometry>
-               <cylinder radius="${caster_wheel_radius}" length="${caster_wheel_thickness}"/>
-            </geometry>
-            <material name="port_red"/>
-        </visual>
-        <visual name="left_caster_marker_visual">
-            <geometry>
-                <box size="${caster_wheel_radius*0.5} ${caster_wheel_radius*0.5} ${caster_wheel_thickness*1.1}"/>
-            </geometry>
-            <material name="blue"/>
-        </visual>
- -->
-        <!--
-        <collision>
-            <geometry>
-                <cylinder radius="${caster_wheel_radius}" length="${caster_wheel_thickness}"/>
-            </geometry>
-            <surface>
-                <friction>
-                    <ode>
-                    <mu>0</mu>
-                    <mu2>0</mu2>
-                    <slip1>1.0</slip1>
-                    <slip2>1.0</slip2>
-                    </ode>
-                </friction>
-            </surface>
-        </collision>
-        -->
-<!--
-        <xacro:inertial_cylinder mass="${caster_wheel_mass}" length="${caster_wheel_thickness}" radius="${caster_wheel_radius}">
-            <origin xyz="0 0 0" rpy="0 0 0"/>
-        </xacro:inertial_cylinder>
--->
-    <!-- </link> -->
-    <!-- RIGHT CASTER WHEEL -->
-<!--
-    <joint name="right_caster_wheel_joint" type="${caster_joint_type}">
-        <parent link="chassis_link"/>
-        <child link="right_caster_wheel"/>
-        <origin xyz="${caster_wheel_offset_x} ${-caster_wheel_offset_y} ${caster_wheel_offset_z}" rpy="${pi/2} 0 0" />
-        <axis xyz="0 0 -1"/>
-    </joint>
- -->
-    <!-- <link name="right_caster_wheel"> -->
-<!--
-        <visual name="right_caster_visual">
-            <geometry>
-               <cylinder radius="${caster_wheel_radius}" length="${caster_wheel_thickness}"/>
-            </geometry>
-            <material name="starboard_green"/>
-        </visual>
-        <visual name="right_caster_marker_visual">
-            <geometry>
-                <box size="${caster_wheel_radius*0.5} ${caster_wheel_radius*0.5} ${caster_wheel_thickness*1.1}"/>
-            </geometry>
-            <material name="blue"/>
-        </visual>
- -->
-<!--
-        <collision>
-            <geometry>
-                <cylinder radius="${caster_wheel_radius}" length="${caster_wheel_thickness}"/>
-            </geometry>
-            <surface>
-                <friction>
-                    <ode>
-                    <mu>0</mu>
-                    <mu2>0</mu2>
-                    <slip1>1.0</slip1>
-                    <slip2>1.0</slip2>
-                    </ode>
-                </friction>
-            </surface>
-        </collision>
- -->
-<!--
-        <xacro:inertial_cylinder mass="${caster_wheel_mass}" length="${caster_wheel_thickness}" radius="${caster_wheel_radius}">
-            <origin xyz="0 0 0" rpy="0 0 0"/>
-        </xacro:inertial_cylinder>
- -->
-    <!-- </link> -->
 </robot>

Commit message: chassis collision corrected

File: robots/stingray/description/robot_core.xacro (robot description, xacro)
@@ -93,5 +93,6 @@
         </visual>
         <collision>
-            <origin xyz="0.0 0.0 0.0" rpy="0.0 0.0 0.0"/>
+            <!-- <origin xyz="0.0 0.0 0.0" rpy="0.0 0.0 0.0"/> -->
+            <origin xyz="${-chassis_offset} 0.0 0.0" rpy="0.0 0.0 0.0"/>
             <geometry>
 		        <!-- collision doesn't need to be a mesh, a box is sufficient -->

Commit message: organized robot_core.xacro

File: robots/stingray/description/robot_core.xacro (robot description, xacro)
@@ -2,11 +2,11 @@
 <robot xmlns:xacro="http://www.ros.org/wiki/xacro" >
     <xacro:include filename="../../../description/inertial_macros.xacro"/>
-	<!-- Values corrected for stingray robot -->
+    <!-- CHASSIS -->
     <xacro:property name="chassis_length" value="0.266"/>
     <xacro:property name="chassis_width" value="0.228"/>
     <xacro:property name="chassis_height" value="0.081"/>
-    <xacro:property name="chassis_mass" value="2.466"/>
     <xacro:property name="chassis_offset" value="0.0455"/>
     <xacro:property name="front_panel_offset" value="0.090"/>
+    <xacro:property name="chassis_mass" value="2.466"/>
     <!-- <xacro:property name="chassis_mass" value="${stingray_total_mass}-2*${wheel_mass}-${caster_mass}-${lidar_mass}"
     - ${OTHER_COMPONENTS_TO_BE_DETERMINED}/> -->
@@ -15,4 +15,5 @@
     <!-- <xacro:property name="battery_mass" value="0.765"/> -->
     <!-- <xacro:property name="wheel_motor_assembly" value="0.375"/> -->
+    <!-- WHEELS -->
     <xacro:property name="wheel_radius" value="0.0615"/>
     <xacro:property name="wheel_thickness" value="0.02"/>
@@ -20,4 +21,5 @@
     <xacro:property name="wheel_offset_x" value="0.13"/>
     <xacro:property name="wheel_separation" value="0.26"/>
+    <!-- CASTER -->
     <xacro:property name="caster_radius" value="0.028"/>
     <xacro:property name="caster_x_offset" value="-0.207"/>
@@ -25,4 +27,5 @@
     <xacro:property name="caster_mass" value="0.022"/>
     <!-- we need the following because (unlike sim) real Dragger doesn't have a controller reporting caster's position -->
+<!--
     <xacro:if value="$(arg sim_mode)">
         <xacro:property name="caster_joint_type" value="continuous"/>
@@ -31,4 +34,5 @@
         <xacro:property name="caster_joint_type" value="fixed"/>
     </xacro:unless>
+ -->
     <!-- ********************** ROBOT BASE *********************************  -->
     <!-- The coordinate frame called base_link is rigidly attached to the robot root body.

Commit message: update odom params

File: robots/stingray/description/robot_core.xacro (robot description, xacro)
@@ -26,5 +26,5 @@
     <!-- <xacro:property name="wheel_motor_assembly" value="0.375"/> -->
     <!-- WHEELS -->
-    <xacro:property name="wheel_radius" value="0.0615"/>
+    <xacro:property name="wheel_radius" value="0.062"/>
     <xacro:property name="wheel_thickness" value="0.02"/>
     <xacro:property name="wheel_mass" value="2.63"/>
