Commit message: extensive Claude-Sonnet-4.5 dialog re navigation

File: robots/stingray/description/JP_lidar.xacro (robot description, xacro)
@@ -7,4 +7,5 @@
     <xacro:property name="lidar_offset_x" value="0.045"/>
     <xacro:property name="lidar_offset_y" value="0.0"/>
+    <xacro:property name="lidar_offset_z" value="${(chassis_height/2) + (lidar_support_height) + (lidar_height/2) + 0.015}"/>
     <xacro:property name="lidar_rotation_x" value="${pi}"/>
     <xacro:property name="lidar_rotation_y" value="0.0"/>
@@ -13,5 +14,5 @@
         <parent link="lidar_support_link"/>
         <child link="laser_frame"/>
-        <origin xyz="${lidar_offset_x} ${lidar_offset_y} ${(chassis_height/2) + (lidar_support_height) + (lidar_height/2)}" rpy="${lidar_rotation_x} ${lidar_rotation_y} ${lidar_rotation_z}"/>
+        <origin xyz="${lidar_offset_x} ${lidar_offset_y} ${lidar_offset_z}" rpy="${lidar_rotation_x} ${lidar_rotation_y} ${lidar_rotation_z}"/>
     </joint>
     <link name="laser_frame">

File: robots/stingray/description/Zeee_LiPo_battery.xacro (robot description, xacro)
@@ -7,5 +7,5 @@
     <xacro:property name="battery_offset_x" value="-0.05654"/>
     <xacro:property name="battery_offset_y" value="0.0"/>
-    <xacro:property name="battery_offset_z" value="${chassis_height/2 + battery_height/2}"/>
+    <xacro:property name="battery_offset_z" value="${chassis_height/2 + battery_height/2 + 0.005}"/>
     <joint name="battery_joint" type="fixed">
         <parent link="chassis_link"/>

File: robots/stingray/description/robot.urdf.xacro (robot description, xacro)
@@ -9,5 +9,5 @@
             JP_imu.xacro
             JP_camera.xacro
-        other components
+            OAK-D camera
             battery.xacro
             ros2_control.xacro
@@ -25,8 +25,10 @@
     <xacro:include filename="robot_core.xacro" />
     <!-- USB FISHEYE CAMERA -->
+    <!--
     <xacro:property name="camera_offset_x" value="${front_panel_offset}"/>
     <xacro:property name="camera_offset_z" value="0.01525"/>
     <xacro:include filename="$(find articubot_one)/robots/stingray/description/JP_camera.xacro" />
-    <xacro:property name="camera_rotation_y" value="-0.1571"/>    <!-- =9 degrees -->
+    <xacro:property name="camera_rotation_y" value="-0.1571"/>    =9 degrees
+    -->
     <!-- LIDAR -->
     <xacro:property name="lidar_support_offset_x" value="0.042"/>
@@ -38,4 +40,5 @@
     <xacro:include filename="$(find articubot_one)/robots/stingray/description/JP_lidar.xacro" />
     <!-- IMU -->
+    <!-- BNO055 IMU is placed at the center of the wheel axis = base_link -->
     <xacro:property name="imu_offset_x" value="0.0"/>
     <xacro:property name="imu_offset_y" value="0.0"/>
@@ -47,6 +50,10 @@
     <!-- BATTERY -->
     <xacro:include filename="$(find articubot_one)/robots/stingray/description/Zeee_LiPo_battery.xacro" />
-    <!-- OPTIONAL -->
-    <!-- xacro:include filename="../../../description/depth_camera.xacro" / -->
+    <!-- OAK-D Camera -->
+    <xacro:include filename="$(find articubot_one)/robots/stingray/description/oakd.xacro" />
+    <xacro:oakd_link mount_point="front_panel"/>
+   <xacro:oakd_joint x="0.023" y="0.01" z="0.030" roll="0" pitch="0" yaw="0" mount_point="front_panel"/>
+    <!-- RealSense Camera -->
+    <!-- <xacro:include filename="../../../description/RealSenseD455.xacro" /> -->
     <!-- ROS2 CONTROL -->
     <xacro:include filename="ros2_control.xacro" />

File: robots/stingray/description/robot_core.xacro (robot description, xacro)
@@ -15,5 +15,5 @@
     <xacro:property name="chassis_length" value="0.266"/>
     <xacro:property name="chassis_width" value="0.228"/>
-    <xacro:property name="chassis_height" value="0.081"/>
+    <xacro:property name="chassis_height" value="0.086"/>
     <xacro:property name="chassis_offset" value="0.0455"/>
     <xacro:property name="front_panel_offset" value="0.090"/>
@@ -26,4 +26,14 @@
     <!-- <xacro:property name="wheel_motor_assembly" value="0.375"/> -->
     <!-- WHEELS -->
+    <!--
+    https://www.pololu.com/product/4753
+    50:1 37Dx70L mm 12V 64 CPM Encoder 6mm D output shaft.
+    50 x 64 = 3200 counts/rev
+    Wheel 4 7/8" dia = 0.123825m dia x π = 0.3890m circ = m/rev
+    [= my tape measurement of 38.95mm circ]
+    Wheel radius = 0.123825m dia / 2 = 0.0619125 = 0.062m
+    1m / 0.39 m/R = 2.57 R/m
+    2.57 R/m x 3200 C/R = 8226 C/m
+    -->
     <xacro:property name="wheel_radius" value="0.062"/>
     <xacro:property name="wheel_thickness" value="0.02"/>
