Commit message: changed lidar SG to JP

File: robots/stingray/description/robot.urdf.xacro (robot description, xacro)
@@ -16,5 +16,5 @@
     <xacro:property name="laser_offset_x" value="${wheel_offset_x}"/>
     <xacro:property name="laser_offset_z" value="0.50"/>
-    <xacro:include filename="../../../description/lidar.xacro" />
+    <xacro:include filename="../../../description/JP_lidar.xacro" />
     <xacro:property name="gps_offset_x" value="${wheel_offset_x}"/>
     <xacro:property name="gps_offset_y" value="-0.16"/>

File: robots/stingray/description/robot_core.xacro (robot description, xacro)
@@ -11,5 +11,5 @@
     <xacro:property name="wheel_thickness" value="0.02"/>
     <xacro:property name="wheel_mass" value="0.058"/>
-    <xacro:property name="wheel_offset" value="0.13"/>
+    <xacro:property name="wheel_offset_x" value="0.13"/>
     <xacro:property name="wheel_separation" value="0.26"/>
     <xacro:property name="caster_radius" value="0.028"/>
@@ -17,4 +17,5 @@
     <xacro:property name="caster_z_offset" value="-0.035"/>
     <xacro:property name="caster_mass" value="0.022"/>
+<!--
     <xacro:property name="wheel_offset_x" value="0.13"/>
     <xacro:property name="wheel_offset_y" value="0.0"/>
@@ -26,4 +27,5 @@
     <xacro:property name="caster_wheel_offset_y" value="0.175"/>
     <xacro:property name="caster_wheel_offset_z" value="${wheel_offset_z - wheel_radius + caster_wheel_radius}"/>
+ -->
     <!-- we need the following because (unlike sim) real Dragger doesn't have a controller reporting caster's position -->
     <xacro:if value="$(arg sim_mode)">
@@ -109,5 +111,5 @@
         <parent link="base_link"/>
         <child link="left_wheel_link"/>
-        <origin xyz="0.0 ${wheel_offset} 0.0" rpy="-${pi/2} 0.0 0.0"/>
+        <origin xyz="0.0 ${wheel_offset_x} 0.0" rpy="-${pi/2} 0.0 0.0"/>
         <axis xyz="0 0 1"/>
     </joint>
@@ -140,5 +142,5 @@
         <parent link="chassis_link"/>
         <child link="right_wheel_link"/>
-        <origin xyz="0.0 ${-wheel_offset} 0.0" rpy="${pi/2} 0 0"/>
+        <origin xyz="0.0 ${-wheel_offset_x} 0.0" rpy="${pi/2} 0 0"/>
         <axis xyz="0 0 -1"/>
     </joint>

Commit message: camera SG>JP & reposition

File: robots/stingray/description/robot.urdf.xacro (robot description, xacro)
@@ -21,7 +21,7 @@
     <xacro:property name="gps_offset_z" value="0.45"/>
     <xacro:include filename="../../../description/gps.xacro" />
-    <xacro:property name="camera_offset_x" value="${wheel_offset_x + 0.05}"/>
-    <xacro:property name="camera_offset_z" value="0.45"/>
-    <xacro:include filename="../../../description/camera.xacro" />
+    <xacro:property name="camera_offset_x" value="${front_panel_offset}"/>
+    <xacro:property name="camera_offset_z" value="0.01525"/>
+    <xacro:include filename="../../../description/JP_camera.xacro" />
     <!-- xacro:include filename="../../../description/depth_camera.xacro" / -->
     <!-- xacro:include filename="../../../description/face.xacro" / -->

File: robots/stingray/description/robot_core.xacro (robot description, xacro)
@@ -8,4 +8,5 @@
     <xacro:property name="chassis_mass" value="0.98"/>
     <xacro:property name="chassis_offset" value="0.0455"/>
+    <xacro:property name="front_panel_offset" value="0.090"/>
     <xacro:property name="wheel_radius" value="0.0615"/>
     <xacro:property name="wheel_thickness" value="0.02"/>
@@ -17,15 +18,4 @@
     <xacro:property name="caster_z_offset" value="-0.035"/>
     <xacro:property name="caster_mass" value="0.022"/>
-<!--
-    <xacro:property name="wheel_offset_x" value="0.13"/>
-    <xacro:property name="wheel_offset_y" value="0.0"/>
-    <xacro:property name="wheel_offset_z" value="0.0"/>
-    <xacro:property name="caster_wheel_radius" value="0.05"/>
-    <xacro:property name="caster_wheel_thickness" value="0.02"/>
-    <xacro:property name="caster_wheel_mass" value="0.3"/>
-    <xacro:property name="caster_wheel_offset_x" value="${-chassis_length/2 - 0.08}"/>
-    <xacro:property name="caster_wheel_offset_y" value="0.175"/>
-    <xacro:property name="caster_wheel_offset_z" value="${wheel_offset_z - wheel_radius + caster_wheel_radius}"/>
- -->
     <!-- we need the following because (unlike sim) real Dragger doesn't have a controller reporting caster's position -->
     <xacro:if value="$(arg sim_mode)">

Commit message: lidar support mesh inserted

File: robots/stingray/description/robot.urdf.xacro (robot description, xacro)
@@ -17,4 +17,8 @@
     <xacro:property name="laser_offset_z" value="0.50"/>
     <xacro:include filename="../../../description/JP_lidar.xacro" />
+    <xacro:property name="lidar_support_offset_x" value="0.0"/>
+    <xacro:property name="lidar_support_offset_y" value="0.0"/>
+    <xacro:property name="lidar_support_offset_z" value="0.0"/>
+    <xacro:include filename="../../../description/lidar_support.xacro" />
     <xacro:property name="gps_offset_x" value="0.0"/>
     <xacro:property name="gps_offset_y" value="0.0"/>

File: robots/stingray/description/robot_core.xacro (robot description, xacro)
@@ -80,6 +80,5 @@
             <origin xyz="0.0 0.0 0.0" rpy="0.0 0.0 0.0"/>
             <geometry>
-                <!-- <mesh filename="model://meshes/Stingray.stl" scale="0.001 0.001 0.001"/> -->
-                <mesh filename="package://articubot_one/assets/meshes/Stingray.stl" scale="0.001 0.001 0.001"/>
+                <mesh filename="model://meshes/Stingray.stl" scale="0.001 0.001 0.001"/>
             </geometry>
             <material name="acrylic"/>

Commit message: lidar support raised to suface

File: robots/stingray/description/robot.urdf.xacro (robot description, xacro)
@@ -19,5 +19,6 @@
     <xacro:property name="lidar_support_offset_x" value="0.0"/>
     <xacro:property name="lidar_support_offset_y" value="0.0"/>
-    <xacro:property name="lidar_support_offset_z" value="0.0"/>
+    <!-- <xacro:property name="lidar_support_offset_z" value="0.0"/> -->
+    <xacro:property name="lidar_support_offset_z" value="${chassis_height/2 + 0.00375}"/>
     <xacro:include filename="../../../description/lidar_support.xacro" />
     <xacro:property name="gps_offset_x" value="0.0"/>

Commit message: organized robot.urdf.xacro

File: robots/stingray/description/robot.urdf.xacro (robot description, xacro)
@@ -8,26 +8,35 @@
           xacro install/articubot_one/share/articubot_one/robots/stingray/description/robot.urdf.xacro sim_mode:=false > src/articubot_one/robots/stingray/description/robot.urdf.generated.xml
     -->
+    <!-- COMMON -->
     <xacro:include filename="../../../description/common_properties.xacro" />
+    <!-- CORE -->
     <xacro:include filename="robot_core.xacro" />
-    <xacro:property name="imu_offset_x" value="0.0"/>
-    <xacro:property name="imu_offset_z" value="0.0"/>
-    <xacro:include filename="../../../description/imu.xacro" />
-    <xacro:include filename="../../../description/magnetometer.xacro" />
-    <xacro:property name="laser_offset_x" value="${wheel_offset_x}"/>
-    <xacro:property name="laser_offset_z" value="0.50"/>
-    <xacro:include filename="../../../description/JP_lidar.xacro" />
+    <!-- CAMERA -->
+    <xacro:property name="camera_offset_x" value="${front_panel_offset}"/>
+    <xacro:property name="camera_offset_z" value="0.01525"/>
+    <xacro:include filename="../../../description/JP_camera.xacro" />
+    <!-- LIDAR -->
     <xacro:property name="lidar_support_offset_x" value="0.0"/>
     <xacro:property name="lidar_support_offset_y" value="0.0"/>
     <xacro:property name="lidar_support_offset_z" value="${chassis_height/2 + 0.00375}"/>
     <xacro:include filename="../../../description/lidar_support.xacro" />
+    <xacro:property name="laser_offset_x" value="${wheel_offset_x}"/>
+    <xacro:property name="laser_offset_z" value="0.50"/>
+    <xacro:include filename="../../../description/JP_lidar.xacro" />
+    <!-- GPS -->
     <xacro:property name="gps_offset_x" value="0.0"/>
     <xacro:property name="gps_offset_y" value="0.0"/>
     <xacro:property name="gps_offset_z" value="0.02"/>
     <xacro:include filename="../../../description/JP_gps.xacro" />
-    <xacro:property name="camera_offset_x" value="${front_panel_offset}"/>
-    <xacro:property name="camera_offset_z" value="0.01525"/>
-    <xacro:include filename="../../../description/JP_camera.xacro" />
+    <!-- IMU -->
+    <xacro:property name="imu_offset_x" value="0.0"/>
+    <xacro:property name="imu_offset_z" value="0.0"/>
+    <xacro:include filename="../../../description/imu.xacro" />
+    <!-- MAG -->
+    <xacro:include filename="../../../description/magnetometer.xacro" />
+    <!-- OPTIONAL -->
     <!-- xacro:include filename="../../../description/depth_camera.xacro" / -->
     <!-- xacro:include filename="../../../description/face.xacro" / -->
+    <!-- ROS2 CONTROL -->
     <xacro:include filename="ros2_control.xacro" />
 </robot>

Commit message: battery.xacro

File: robots/stingray/description/robot.urdf.xacro (robot description, xacro)
@@ -35,4 +35,6 @@
     <!-- MAG -->
     <xacro:include filename="../../../description/magnetometer.xacro" />
+    <!-- BATTERY -->
+    <xacro:include filename="../../../description/battery.xacro" />
     <!-- OPTIONAL -->
     <!-- xacro:include filename="../../../description/depth_camera.xacro" / -->

File: robots/stingray/description/robot_core.xacro (robot description, xacro)
@@ -2,4 +2,6 @@
 <robot xmlns:xacro="http://www.ros.org/wiki/xacro" >
     <xacro:include filename="../../../description/inertial_macros.xacro"/>
+    <!-- TEMPLATE -->
+    <xacro:property name="TEMPLATE" value="0.0"/>
     <!-- CHASSIS -->
     <xacro:property name="chassis_length" value="0.266"/>

Commit message: new LD19 lidar, BNO055>BNO085

File: robots/stingray/description/robot.urdf.xacro (robot description, xacro)
@@ -6,7 +6,7 @@
         common_properties.xacro
         individual sensors - each with their positions
-            JP_lidar.xacro
+            ydlidar.xacro
             JP_imu.xacro
-            JP_camera.xacro
+            fisheye_camera.xacro
             OAK-D camera
             battery.xacro
@@ -28,15 +28,19 @@
     <xacro:property name="camera_offset_x" value="${front_panel_offset}"/>
     <xacro:property name="camera_offset_z" value="0.01525"/>
-    <xacro:include filename="$(find articubot_one)/robots/stingray/description/JP_camera.xacro" />
+    <xacro:include filename="$(find articubot_one)/robots/stingray/description/fisheye_camera.xacro" />
     <xacro:property name="camera_rotation_y" value="-0.1571"/>    =9 degrees
     -->
-    <!-- LIDAR -->
-    <xacro:property name="lidar_support_offset_x" value="0.042"/>
-    <xacro:property name="lidar_support_offset_y" value="-0.02"/>
-    <xacro:property name="lidar_support_offset_z" value="${chassis_height/2 + 0.00375}"/>
-    <xacro:include filename="$(find articubot_one)/robots/stingray/description/lidar_support.xacro"/>
-    <!-- <xacro:property name="laser_offset_x" value="${wheel_offset_x}"/> -->
-    <!-- <xacro:property name="laser_offset_z" value="0.50"/> -->
-    <xacro:include filename="$(find articubot_one)/robots/stingray/description/JP_lidar.xacro" />
+    <!-- YDLIDAR  -->
+    <!-- <xacro:property name="ydlidar_support_offset_x" value="0.042"/>
+    <xacro:property name="ydlidar_support_offset_y" value="-0.02"/>
+    <xacro:property name="ydlidar_support_offset_z" value="${chassis_height/2 + 0.00375}"/>
+    <xacro:include filename="$(find articubot_one)/robots/stingray/description/ydlidar_support.xacro"/>
+    <xacro:include filename="$(find articubot_one)/robots/stingray/description/ydlidar.xacro" /> -->
+    <!-- LDLIDAR LD19 -->
+    <xacro:property name="ldlidar_support_offset_x" value="0.04669"/>
+    <xacro:property name="ldlidar_support_offset_y" value="0.0"/>
+    <xacro:property name="ldlidar_support_offset_z" value="${chassis_height/2}"/>
+    <xacro:include filename="$(find articubot_one)/robots/stingray/description/ldlidar_support.xacro"/>
+    <xacro:include filename="$(find articubot_one)/robots/stingray/description/ldlidar.xacro"/>
     <!-- IMU -->
     <!-- BNO055 IMU is placed at the center of the wheel axis = base_link -->
@@ -47,5 +51,5 @@
     <xacro:property name="imu_rotation_y" value="0.0"/>
     <xacro:property name="imu_rotation_z" value="0.0"/>
-    <xacro:include filename="$(find articubot_one)/robots/stingray/description/JP_imu.xacro"/>
+    <xacro:include filename="$(find articubot_one)/robots/stingray/description/BNO055_imu.xacro"/>
     <!-- BATTERY -->
     <xacro:include filename="$(find articubot_one)/robots/stingray/description/Zeee_LiPo_battery.xacro" />
