Commit message: add OAK-D IMU frame

File: robots/stingray/description/oakd.xacro (robot description, xacro)
@@ -58,10 +58,21 @@
           </inertial>
   </link>
-  <!-- Corrected IMU frame for RViz visualization -->
-  <!-- The OAK-D driver publishes oak_imu_frame with non-standard orientation -->
-  <!-- This creates a corrected version aligned with base_link for display purposes -->
-  <!-- The actual IMU data at /oak/imu/data still uses oak_imu_frame (EKF doesn't care) -->
-  <!-- Note: This is a child of oak_imu_frame (published by driver), not oakd_front_panel -->
-  <!-- Waiting for driver to publish oak_imu_frame, then applying correction transform -->
+  <!-- OAK-D IMU frame -->
+  <!-- The depthai driver publishes oak_imu_frame with its own orientation -->
+  <!-- Add this link to the URDF so we can adjust its rotation to align with robot axes -->
+  <joint name="oak_imu_joint" type="fixed">
+    <!-- Rotation to align IMU axes with robot coordinate frame -->
+    <!-- Adjust these values to match your robot's coordinate system -->
+    <origin xyz="0 0 0" rpy="0 0 0" />
+    <parent link="oakd_${mount_point}" />
+    <child link="oak_imu_frame" />
+  </joint>
+  <link name="oak_imu_frame">
+    <inertial>
+      <mass value="0.001" />
+      <origin xyz="0 0 0" />
+      <inertia ixx="0.0001" ixy="0.0" ixz="0.0" iyy="0.0001" iyz="0.0" izz="0.0001" />
+    </inertial>
+  </link>
   <!-- Gazebo plugin for greyscale left/right stereo pairs -->
       <gazebo reference="oakd_${mount_point}">
