Commit message: further urdf tweaking

File: robots/stingray/description/ldlidar.xacro (robot description, xacro)
@@ -24,5 +24,5 @@
                 <box size="${ldlidar_chassis_width} ${ldlidar_chassis_width} ${ldlidar_chassis_height}"/>
             </geometry>
-            <material name="black"/>
+            <material name="blue"/>
         </visual>
         <visual>
@@ -31,13 +31,14 @@
                 <cylinder radius="${ldlidar_radius}" length="${ldlidar_height}"/>
             </geometry>
-            <material name="black"/>
+            <material name="blue"/>
         </visual>
         <collision>
+            <origin xyz="0 0 ${(ldlidar_chassis_height + ldlidar_height)/2}" rpy="0 0 0"/>
             <geometry>
-                <cylinder radius="${ldlidar_radius}" length="${ldlidar_height}"/>
+                <box size="${ldlidar_chassis_width} ${ldlidar_chassis_width} ${ldlidar_chassis_height + ldlidar_height}"/>
             </geometry>
         </collision>
         <xacro:inertial_cylinder mass="${ldlidar_mass}" length="${ldlidar_height}" radius="${ldlidar_radius}">
-            <origin xyz="0 0 0" rpy="0 0 0"/>
+            <origin xyz="0 0 ${ldlidar_chassis_height/2 + ldlidar_height/2}" rpy="0 0 0"/>
         </xacro:inertial_cylinder>
     </link>
@@ -50,6 +51,5 @@
     <link name="base_laser"/>
     <gazebo reference="ldlaser_frame">
-        <material><Gazebo/>
-        <Black></Black></material>
+        <material>Gazebo/Grey</material>
     	    <sensor name="ldlaser_frame" type="gpu_lidar">
             <pose> 0.0 0.0 0.0 0.0 0.0 0.0 </pose>

File: robots/stingray/description/oakd.xacro (robot description, xacro)
@@ -3,7 +3,7 @@
 <robot name="oakd" xmlns:xacro="http://ros.org/wiki/xacro">
       <xacro:macro name="oakd_link" params="mount_point">
-      <xacro:property name="oakd_length" value="0.0803" />
-      <xacro:property name="oakd_width" value="0.0957" />
-      <xacro:property name="oakd_depth" value="0.1267" />
+      <xacro:property name="oakd_x_length" value="0.033" />
+      <xacro:property name="oakd_y_width" value="0.110" />
+      <xacro:property name="oakd_z_height" value="0.0545" />
       <xacro:property name="oakd_mass" value="0.15" />
       <link name="oakd_${mount_point}">
@@ -17,7 +17,7 @@
           </visual>
           <collision>
-              <origin rpy="0 0 0" xyz="0 0 0" />
+              <origin rpy="0 0 0" xyz="${-oakd_x_length/2} 0 ${-oakd_z_height/4}" />
               <geometry>
-                  <box size="${oakd_length} ${oakd_width} ${oakd_depth}"/>
+                  <box size="${oakd_x_length} ${oakd_y_width} ${oakd_z_height}"/>
               </geometry>
           </collision>
@@ -25,6 +25,6 @@
           <xacro:inertial_box
               mass="${oakd_mass}"
-              x="${oakd_length}" y="${oakd_width}" z="${oakd_depth}" >
-            <origin xyz="0.0 0.0 0.0" rpy="0.0 0.0 0.0"/>
+              x="${oakd_x_length}" y="${oakd_y_width}" z="${oakd_z_height}" >
+            <origin xyz="${-oakd_x_length/2} 0.0 ${-oakd_z_height/4}" rpy="0.0 0.0 0.0"/>
           </xacro:inertial_box>
       </link>
@@ -60,5 +60,5 @@
   <!-- Gazebo plugin for greyscale left/right stereo pairs -->
       <gazebo reference="oakd_${mount_point}">
-    <material>Gazebo/DarkGrey</material>
+    <material>Gazebo/Grey</material>
     <sensor type="multicamera" name="stereo_camera">
       <update_rate>30.0</update_rate>

File: robots/stingray/description/robot.urdf.xacro (robot description, xacro)
@@ -57,5 +57,5 @@
     <xacro:include filename="$(find articubot_one)/robots/stingray/description/oakd.xacro" />
     <xacro:oakd_link mount_point="front_panel"/>
-   <xacro:oakd_joint x="0.023" y="0.01" z="0.030" roll="0" pitch="0" yaw="0" mount_point="front_panel"/>
+    <xacro:oakd_joint x="0.023" y="0.01" z="0.030" roll="0" pitch="0" yaw="0" mount_point="front_panel"/>
     <!-- RealSense Camera -->
     <!-- <xacro:include filename="../../../description/RealSenseD455.xacro" /> -->

Commit message: ldlidar rotation, oak-d TF

File: robots/stingray/description/ldlidar.xacro (robot description, xacro)
@@ -12,5 +12,5 @@
     <xacro:property name="ldlidar_rotation_x" value="0.0"/>
     <xacro:property name="ldlidar_rotation_y" value="0.0"/>
-    <xacro:property name="ldlidar_rotation_z" value="${pi}"/>
+    <xacro:property name="ldlidar_rotation_z" value="0.0"/>
     <joint name="ldlaser_joint" type="fixed">
         <parent link="ldlidar_support_link"/>

File: robots/stingray/description/oakd.xacro (robot description, xacro)
@@ -58,4 +58,10 @@
           </inertial>
   </link>
+  <!-- Corrected IMU frame for RViz visualization -->
+  <!-- The OAK-D driver publishes oak_imu_frame with non-standard orientation -->
+  <!-- This creates a corrected version aligned with base_link for display purposes -->
+  <!-- The actual IMU data at /oak/imu/data still uses oak_imu_frame (EKF doesn't care) -->
+  <!-- Note: This is a child of oak_imu_frame (published by driver), not oakd_front_panel -->
+  <!-- Waiting for driver to publish oak_imu_frame, then applying correction transform -->
   <!-- Gazebo plugin for greyscale left/right stereo pairs -->
       <gazebo reference="oakd_${mount_point}">

File: robots/stingray/description/robot.urdf.xacro (robot description, xacro)
@@ -43,6 +43,6 @@
     <xacro:include filename="$(find articubot_one)/robots/stingray/description/ldlidar_support.xacro"/>
     <xacro:include filename="$(find articubot_one)/robots/stingray/description/ldlidar.xacro"/>
-    <!-- IMU -->
-    <!-- BNO055 IMU is placed at the center of the wheel axis = base_link -->
+    <!-- IMU - BNO055 (commented out - using OAK-D IMU instead) -->
+    <!--
     <xacro:property name="imu_offset_x" value="0.0"/>
     <xacro:property name="imu_offset_y" value="0.0"/>
@@ -52,4 +52,5 @@
     <xacro:property name="imu_rotation_z" value="0.0"/>
     <xacro:include filename="$(find articubot_one)/robots/stingray/description/BNO055_imu.xacro"/>
+    -->
     <!-- BATTERY -->
     <xacro:include filename="$(find articubot_one)/robots/stingray/description/Zeee_LiPo_battery.xacro" />
@@ -58,4 +59,7 @@
     <xacro:oakd_link mount_point="front_panel"/>
     <xacro:oakd_joint x="0.023" y="0.01" z="0.030" roll="0" pitch="0" yaw="0" mount_point="front_panel"/>
+    <!-- Physical location: inside OAK-D camera body, approximately 15mm behind front face -->
+    <!-- Frame orientation: 90° pitch rotation relative to camera optical frame -->
+    <!-- EKF consumes angular velocity and linear acceleration (not orientation) from this IMU -->
     <!-- RealSense Camera -->
     <!-- <xacro:include filename="../../../description/RealSenseD455.xacro" /> -->

Commit message: minor tweaks

File: robots/stingray/description/ldlidar.xacro (robot description, xacro)
@@ -12,5 +12,5 @@
     <xacro:property name="ldlidar_rotation_x" value="0.0"/>
     <xacro:property name="ldlidar_rotation_y" value="0.0"/>
-    <xacro:property name="ldlidar_rotation_z" value="0.0"/>
+    <xacro:property name="ldlidar_rotation_z" value="${-pi/2}"/>
     <joint name="ldlaser_joint" type="fixed">
         <parent link="ldlidar_support_link"/>

File: robots/stingray/description/oakd.xacro (robot description, xacro)
@@ -57,21 +57,4 @@
 	  <inertia ixx="0.0001" ixy="0.0" ixz="0.0" iyy="0.0001" iyz="0.0" izz="0.0001" />
           </inertial>
-  </link>
-  <!-- OAK-D IMU frame -->
-  <!-- The depthai driver publishes oak_imu_frame with its own orientation -->
-  <!-- Add this link to the URDF so we can adjust its rotation to align with robot axes -->
-  <joint name="oak_imu_joint" type="fixed">
-    <!-- Rotation to align IMU axes with robot coordinate frame -->
-    <!-- Adjust these values to match your robot's coordinate system -->
-    <origin xyz="0 0 0" rpy="0 0 0" />
-    <parent link="oakd_${mount_point}" />
-    <child link="oak_imu_frame" />
-  </joint>
-  <link name="oak_imu_frame">
-    <inertial>
-      <mass value="0.001" />
-      <origin xyz="0 0 0" />
-      <inertia ixx="0.0001" ixy="0.0" ixz="0.0" iyy="0.0001" iyz="0.0" izz="0.0001" />
-    </inertial>
   </link>
   <!-- Gazebo plugin for greyscale left/right stereo pairs -->
