Commit message: WIP: Seggy URDF

File: robots/seggy/description/robot.urdf.xacro (robot description, xacro)
@@ -18,12 +18,4 @@
     <xacro:property name="laser_offset_z" value="0.50"/>
     <xacro:include filename="../../../description/lidar.xacro" />
-    <xacro:property name="sonars_offset_x" value="${chassis_length/2 + 0.005}"/>
-    <xacro:property name="sonars_offset_y" value="${chassis_width/2 - 0.02}"/>
-    <xacro:property name="sonars_offset_z" value="0.05"/>
-    <xacro:include filename="../../../description/sonars.xacro" />
-    <xacro:property name="gps_offset_x" value="${wheel_offset_x}"/>
-    <xacro:property name="gps_offset_y" value="-0.16"/>
-    <xacro:property name="gps_offset_z" value="0.45"/>
-    <xacro:include filename="../../../description/gps.xacro" />
     <xacro:property name="camera_offset_x" value="${wheel_offset_x + 0.05}"/>
     <xacro:property name="camera_offset_z" value="0.45"/>

File: robots/seggy/description/robot_core.xacro (robot description, xacro)
@@ -3,20 +3,20 @@
     <xacro:include filename="../../../description/inertial_macros.xacro"/>
 	<!-- Values corrected for Seggy robot -->
-    <xacro:property name="chassis_length" value="0.48"/>
-    <xacro:property name="chassis_width" value="0.42"/>
+    <xacro:property name="chassis_length" value="0.38"/>
+    <xacro:property name="chassis_width" value="0.37"/>
     <xacro:property name="chassis_height" value="0.45"/>
     <xacro:property name="chassis_mass" value="10.0"/>
     <xacro:property name="chassis_top_length" value="0.095"/>
-    <xacro:property name="wheel_radius" value="0.192"/>
-    <xacro:property name="wheel_thickness" value="0.045"/>
+    <xacro:property name="wheel_radius" value="0.12"/>
+    <xacro:property name="wheel_thickness" value="0.065"/>
     <xacro:property name="wheel_mass" value="1.0"/>
     <xacro:property name="wheel_offset_x" value="${chassis_length/2 - wheel_radius - 0.01}"/>
-    <xacro:property name="wheel_offset_y" value="0.280"/>
+    <xacro:property name="wheel_offset_y" value="0.23"/>
     <xacro:property name="wheel_offset_z" value="0.01"/>
     <xacro:property name="caster_wheel_radius" value="0.05"/>
-    <xacro:property name="caster_wheel_thickness" value="0.02"/>
+    <xacro:property name="caster_wheel_thickness" value="0.03"/>
     <xacro:property name="caster_wheel_mass" value="0.3"/>
-    <xacro:property name="caster_wheel_offset_x" value="${-chassis_length/2 - 0.08}"/>
-    <xacro:property name="caster_wheel_offset_y" value="0.175"/>
+    <xacro:property name="caster_wheel_offset_x" value="${-chassis_length/2 - 0.0}"/>
+    <xacro:property name="caster_wheel_offset_y" value="0.11"/>
     <xacro:property name="caster_wheel_offset_z" value="${wheel_offset_z - wheel_radius + caster_wheel_radius}"/>
     <!-- we need the following because (unlike sim) real Dragger doesn't have a controller reporting caster's position -->
@@ -103,14 +103,14 @@
         </visual>
         <visual name="chassis_front_axle_left">
-            <origin xyz="${wheel_offset_x} ${chassis_width*0.5} 0" rpy="-${pi/2} 0 0"/>
-            <geometry>
-                <cylinder radius="0.03" length="${chassis_width*0.5}"/>
+            <origin xyz="${wheel_offset_x} ${chassis_width*0.35} 0" rpy="-${pi/2} 0 0"/>
+            <geometry>
+                <cylinder radius="0.03" length="${chassis_width*0.6}"/>
             </geometry>
             <material name="body_color"/>
         </visual>
         <visual name="chassis_front_axle_right">
-            <origin xyz="${wheel_offset_x} ${-chassis_width*0.5} 0" rpy="${pi/2} 0 0"/>
-            <geometry>
-                <cylinder radius="0.03" length="${chassis_width*0.5}"/>
+            <origin xyz="${wheel_offset_x} ${-chassis_width*0.35} 0" rpy="${pi/2} 0 0"/>
+            <geometry>
+                <cylinder radius="0.03" length="${chassis_width*0.6}"/>
             </geometry>
             <material name="body_color"/>
@@ -158,5 +158,5 @@
         <parent link="chassis_link"/>
         <child link="left_wheel"/>
-        <origin xyz="${wheel_offset_x} ${wheel_offset_y} 0" rpy="-${pi/2 - 0.15} 0 0" />
+        <origin xyz="${wheel_offset_x} ${wheel_offset_y} 0" rpy="-${pi/2} 0 0" />
         <axis xyz="0 0 1">
           <limit>
@@ -229,5 +229,5 @@
         <parent link="chassis_link"/>
         <child link="right_wheel"/>
-        <origin xyz="${wheel_offset_x} ${-wheel_offset_y} 0" rpy="${pi/2 - 0.15} 0 0" />
+        <origin xyz="${wheel_offset_x} ${-wheel_offset_y} 0" rpy="${pi/2} 0 0" />
         <axis xyz="0 0 -1">
           <limit>

Commit message: WIP: Seggy URDF

File: robots/seggy/description/robot.urdf.xacro (robot description, xacro)
@@ -15,15 +15,12 @@
     <xacro:include filename="../../../description/imu.xacro" />
     <xacro:include filename="../../../description/magnetometer.xacro" />
-    <xacro:property name="laser_offset_x" value="${wheel_offset_x}"/>
-    <xacro:property name="laser_offset_z" value="0.50"/>
+    <xacro:property name="laser_offset_x" value="${wheel_offset_x + 0.05}"/>
+    <xacro:property name="laser_offset_z" value="0.27"/>
     <xacro:include filename="../../../description/lidar.xacro" />
-    <xacro:property name="camera_offset_x" value="${wheel_offset_x + 0.05}"/>
-    <xacro:property name="camera_offset_z" value="0.45"/>
-    <xacro:include filename="../../../description/camera.xacro" />
     <xacro:property name="open_circuit_voltage" value="12.592"/>
     <xacro:property name="battery_capacity" value="20.0"/>
     <xacro:include filename="../../../description/battery.xacro" />
     <xacro:property name="depth_camera_offset_x" value="${wheel_offset_x}"/>
-    <xacro:property name="depth_camera_offset_z" value="0.45"/>
+    <xacro:property name="depth_camera_offset_z" value="${chassis_top_offset + 0.12}"/>
     <xacro:include filename="../../../description/depth_camera.xacro"/>
     <xacro:unless value="$(arg sim_mode)">

File: robots/seggy/description/robot_core.xacro (robot description, xacro)
@@ -5,7 +5,9 @@
     <xacro:property name="chassis_length" value="0.38"/>
     <xacro:property name="chassis_width" value="0.37"/>
-    <xacro:property name="chassis_height" value="0.45"/>
-    <xacro:property name="chassis_mass" value="10.0"/>
-    <xacro:property name="chassis_top_length" value="0.095"/>
+    <xacro:property name="chassis_height" value="0.12"/>
+    <xacro:property name="chassis_mass" value="8.0"/>
+    <xacro:property name="chassis_top_length" value="0.37"/>
+    <xacro:property name="chassis_top_width" value="0.49"/>
+    <xacro:property name="chassis_top_offset" value="0.35"/>
     <xacro:property name="wheel_radius" value="0.12"/>
     <xacro:property name="wheel_thickness" value="0.065"/>
@@ -81,22 +83,15 @@
             <material name="body_color"/>
         </visual>
-        <visual name="chassis_visual_front">
-            <origin xyz="0.15 0 ${chassis_height/2-0.03}" rpy="0 ${pi/4} 0"/>
-            <geometry>
-                <box size="0.25 ${chassis_width} 0.01"/>
-            </geometry>
-            <material name="body_color"/>
-        </visual>
-        <visual name="chassis_visual_back">
-            <origin xyz="-0.07 0 ${chassis_height/2-0.03}" rpy="0 -${pi/4} 0"/>
-            <geometry>
-                <box size="0.25 ${chassis_width} 0.01"/>
+        <visual name="chassis_visual_support">
+            <origin xyz="0 0 ${chassis_top_offset/2}" rpy="${pi/2} 0 0"/>
+            <geometry>
+                <box size="0.15 ${chassis_top_offset} 0.02"/>
             </geometry>
             <material name="body_color"/>
         </visual>
         <visual name="chassis_top_visual">
-            <origin xyz="${wheel_offset_x} 0 ${chassis_height*3/4}"/>
-            <geometry>
-                <box size="${chassis_top_length} ${chassis_width} ${chassis_height/2}"/>
+            <origin xyz="${wheel_offset_x} 0 ${chassis_top_offset}"/>
+            <geometry>
+                <box size="${chassis_top_length} ${chassis_top_width} 0.02"/>
             </geometry>
             <material name="body_color"/>
@@ -117,7 +112,7 @@
         </visual>
         <visual name="chassis_caster_holder_left">
-            <origin xyz="${caster_wheel_offset_x+0.09} ${caster_wheel_offset_y*0.85} ${caster_wheel_offset_z*0.42}" rpy="0 ${pi/4} 0"/>
-            <geometry>
-                <cylinder radius="0.012" length="0.23"/>
+            <origin xyz="${caster_wheel_offset_x+0.05} ${caster_wheel_offset_y*0.77} ${caster_wheel_offset_z*0.42}" rpy="0 ${pi/4} 0"/>
+            <geometry>
+                <cylinder radius="0.009" length="0.12"/>
             </geometry>
             <material name="body_color"/>
@@ -131,7 +126,7 @@
         </visual>
         <visual name="chassis_caster_holder_right">
-            <origin xyz="${caster_wheel_offset_x+0.09} ${-caster_wheel_offset_y*0.85} ${caster_wheel_offset_z*0.42}" rpy="0 ${pi/4} 0"/>
-            <geometry>
-                <cylinder radius="0.012" length="0.23"/>
+            <origin xyz="${caster_wheel_offset_x+0.05} ${-caster_wheel_offset_y*0.77} ${caster_wheel_offset_z*0.42}" rpy="0 ${pi/4} 0"/>
+            <geometry>
+                <cylinder radius="0.009" length="0.12"/>
             </geometry>
             <material name="body_color"/>
