Commit message: Update robot_core.xacro

File: robots/fido/description/robot_core.xacro (robot description, xacro)
@@ -79,5 +79,6 @@
             <origin xyz="0 0 ${chassis_height/8}"/>
             <geometry>
-                <box size="${chassis_length} ${chassis_width} ${chassis_height/4}"/>
+                <cylinder radius="${chassis_length/2}" length="${chassis_height/4}"/>
+                <!-- box size="${chassis_length} ${chassis_width} ${chassis_height/4}"/ -->
             </geometry>
             <material name="body_color"/>
@@ -93,5 +94,6 @@
             <origin xyz="${wheel_offset_x} 0 ${chassis_top_offset}"/>
             <geometry>
-                <box size="${chassis_top_length} ${chassis_top_width} 0.02"/>
+                <cylinder radius="${chassis_top_length/2}" length="0.02"/>
+                <!-- box size="${chassis_top_length} ${chassis_top_width} 0.02"/ -->
             </geometry>
             <material name="body_color"/>
